File: SensingBoard/1.1/SensingBoard_rev1.1/SensingBoard_rev1.1.kicad_pcb (KiCad board)
At the start: 2 copper layers, 40 x 40 mm, 6 parts, among them J1 USB_C_Receptacle, J2 3221-10-0300-00, SW1 PTS815 SJM 250 SMTR LFS, U1 ESP32C3, U2 BNO055, U3 MIC5504-3.3YM5

Commit message: more component placement
Parts:
- added C1: 10uF, Capacitor_SMD:C_0603_1608Metric, F.Cu at (157.0, 73.5)
- added C2: 1uF, Capacitor_SMD:C_0201_0603Metric, F.Cu at (153.8, 67.9)
- added C3: 22pF, Capacitor_SMD:C_0201_0603Metric, F.Cu at (153.3, 61.2)
- added C4: 22pF, Capacitor_SMD:C_0201_0603Metric, F.Cu at (153.3, 62.9)
- added D1: LED, LED_SMD:LED_0603_1608Metric, F.Cu at (157.0, 68.3)
- added D2: LED, LED_SMD:LED_0603_1608Metric, F.Cu at (157.0, 70.9)
- added J3: F32R-1A7H1-11024, F32R-1A7H1-11024:AMPHENOL_F32R-1A7H1-11024, B.Cu at (127.8, 84.1)
- added J4: GRPB052VWQP-RC, GRPB052VWQP-RC:GRPB052VWQPRC, F.Cu at (135.3, 60.1)
- added R1: 100, Resistor_SMD:R_0201_0603Metric, F.Cu at (153.8, 69.7)
- added R2: 100, Resistor_SMD:R_0201_0603Metric, F.Cu at (153.8, 71.4)
- added R3: 6.1K, Resistor_SMD:R_0201_0603Metric, F.Cu at (153.8, 73.2)
- added R4: 5.1K, Resistor_SMD:R_0201_0603Metric, F.Cu at (153.8, 74.9)
- added R5: 10k, Resistor_SMD:R_0201_0603Metric, F.Cu at (153.3, 64.7)
- added XTAL1: ABS07-32.768KHZ-7-T, ABS07-32.768KHZ-7-T:XTAL_ABS07-32.768KHZ-7-T_ABR, F.Cu at (157.0, 61.9)
- U2, U3: moved to B.Cu
- moved SW1 12.7 mm to (116.0, 80.5)
- moved U3 2.59 mm to (117.3, 59.7), turned to 180 degrees
- moved U2 1.85 mm to (127.6, 59.9), turned to 180 degrees
- moved J1 1.73 mm to (112.1, 71.1)
- moved U1 0.05 mm to (127.9, 71.0)
Connections:
- net Net-(J1-VBUS-PadA4) renamed VBUS
- net Net-(U1-VDD3P3-Pad2) renamed +3.3V
- J1 pad A5: unconnected-(J1-CC1-PadA5) -> Net-(J1-CC1)
- J1 pad A6: unconnected-(J1-D+-PadA6) -> USB_DP
- J1 pad A7: unconnected-(J1-D--PadA7) -> USB_DN
- J1 pad B5: unconnected-(J1-CC2-PadB5) -> Net-(J1-CC2)
- J1 pad B6: unconnected-(J1-D+-PadB6) -> USB_DP
- J1 pad B7: unconnected-(J1-D--PadB7) -> USB_DN
- SW1 pad 2: unconnected-(SW1-Pad2) -> Net-(R5-Pad2)
- SW1 pad 4: unconnected-(SW1-Pad4) -> GND
- U1 pad 10: unconnected-(U1-MTDI-Pad10) -> D3
- U1 pad 12: unconnected-(U1-MTCK-Pad12) -> D4
- U1 pad 13: unconnected-(U1-MTDO-Pad13) -> D5
- U1 pad 14: unconnected-(U1-GPIO8-Pad14) -> D8
- U1 pad 15: unconnected-(U1-GPIO9-Pad15) -> D9
- U1 pad 16: unconnected-(U1-GPIO10-Pad16) -> D10
- U1 pad 25: unconnected-(U1-GPIO18-Pad25) -> USB_DN
- U1 pad 26: unconnected-(U1-GPIO19-Pad26) -> USB_DP
- U1 pad 27: unconnected-(U1-U0RXD-Pad27) -> RX_D7
- U1 pad 28: unconnected-(U1-U0TXD-Pad28) -> TX_D6
- U1 pad 33: unconnected-(U1-GND-Pad33) -> GND
- U1 pad 4: unconnected-(U1-XTAL_32K_P-Pad4) -> Net-(U1-XTAL_32K_P)
- U1 pad 5: unconnected-(U1-XTAL_32K_N-Pad5) -> Net-(U1-XTAL_32K_N)
- U1 pad 6: unconnected-(U1-GPIO2-Pad6) -> D0
- U1 pad 8: unconnected-(U1-GPIO3-Pad8) -> D1
- U1 pad 9: unconnected-(U1-MTMS-Pad9) -> D2
