File: SensingBoard/1.1/SensingBoard_rev1.1/SensingBoard_rev1.1.kicad_sch (KiCad schematic)
At the start: 6 parts, among them J1 USB_C_Receptacle, J7 3221-10-0300-00, SW1 PTS815 SJM 250 SMTR LFS, U1 ESP32C3, U2 BNO055, U3 MIC5504-3.3YM5

Commit message: more component placement
Parts:
- added C14, C15: 22pF, Capacitor_SMD:C_0201_0603Metric, symbol Device:C
- added C16: 10uF, Capacitor_SMD:C_0603_1608Metric, symbol Device:C
- added C17: 1uF, Capacitor_SMD:C_0201_0603Metric, symbol Device:C
- added D5, D6: LED, LED_SMD:LED_0603_1608Metric, symbol Device:LED
- added J3: F32R-1A7H1-11024, F32R-1A7H1-11024:AMPHENOL_F32R-1A7H1-11024, symbol F32R-1A7H1-11024:F32R-1A7H1-11024
- added J4: GRPB052VWQP-RC, GRPB052VWQP-RC:GRPB052VWQPRC, symbol GRPB052VWQP-RC:GRPB052VWQP-RC
- added R15: 10k, Resistor_SMD:R_0201_0603Metric, symbol Device:R_US
- added R16, R17: 100, Resistor_SMD:R_0201_0603Metric, symbol Device:R_US
- added R17: 5.1K, Resistor_SMD:R_0201_0603Metric, symbol Device:R_US
- added R17: 6.1K, Resistor_SMD:R_0201_0603Metric, symbol Device:R_US
- added XTAL1: ABS07-32.768KHZ-7-T, XTAL_ABS07-32.768KHZ-7-T_ABR, symbol ABS07-32.768KHZ-7-T:ABS07-32.768KHZ-7-T
Connections:
- net +3.3V: now also U1.2 (VDD3P3), U1.3 (VDD3P3), C16.2, C17.1, R15.1
- net GND: now also SW1.4, U1.33 (GND), C14.2, C15.2, J4.7, J4.9, R17.2, R17.2
- net VBUS: now also J1.A4 (VBUS), J1.A9 (VBUS), J1.B4 (VBUS), J1.B9 (VBUS)
- net at SW1.2: now also R15.2
- net D3: now reaches U1.10 (MTDI)
- net D3: now also J4.8
- net D4: now reaches U1.12 (MTCK)
- net D4: now also J4.10
- net D5: now reaches U1.13 (MTDO)
- net D5: now also J4.1
- net D8: now reaches U1.14 (GPIO8)
- net D8: now also J4.3
- net D9: now reaches U1.15 (GPIO9)
- net D9: now also J4.5
- net D10: now reaches U1.16 (GPIO10)
- net USB_DN: now reaches U1.25 (GPIO18)
- net USB_DN: now also J1.A7 (D-), J1.B7 (D-)
- net USB_DP: now reaches U1.26 (GPIO19)
- net USB_DP: now also J1.A6 (D+), J1.B6 (D+)
- net RX_D7: now reaches U1.27 (U0RXD)
- net TX_D6: now reaches U1.28 (U0TXD)
- net at U1.4 (XTAL_32K_P): now also C14.1, XTAL1.1
- net at U1.5 (XTAL_32K_N): now also C15.1, XTAL1.2
- net D0: now reaches U1.6 (GPIO2)
- net D0: now also J4.2
- net D1: now reaches U1.8 (GPIO3)
- net D1: now also J4.4
- net D2: now reaches U1.9 (MTMS)
- net D2: now also J4.6
- net at J1.A5 (CC1): now also R17.1
- net at J1.B5 (CC2): now also R17.1
- no-connect marks 0 -> 10
Other:
- note added: "CAMERA FLEX CONNECTOR"
- note added: "DEBUG + RESET"
- note added: "HEADERS"
- note added: "IMU"
- note added: "MICRO"
- note added: "POWER (switch between VUSB and VBATT)"
- note added: "USB-C RECPT"
- moved on the sheet: J1, J7, SW1, U2, U3
