File: Sensing_Board/1.1/SensingBoard_rev1.1/SensingBoard_rev1.1.kicad_pcb (KiCad board)
At the start: 2 copper layers, 40 x 40 mm, 20 parts, among them J1 USB_C_Receptacle, J2 3221-10-0300-00, J3 F32R-1A7H1-11024, J4 GRPB052VWQP-RC, SW1 PTS815 SJM 250 SMTR LFS, U1 ESP32C3, U2 BNO055, U3 MIC5504-3.3YM5

Commit message: motor driver
Parts:
- added U4: DRV8410PWPR, DRV8410PWPR:IC_DRV8410PWPR, F.Cu at (155.0, 83.1)
