File: Sensing_Board/1.1/SensingBoard_rev1.1/SensingBoard_rev1.1.kicad_sch (KiCad schematic)
At the start: 20 parts, among them J1 USB_C_Receptacle, J3 F32R-1A7H1-11024, J4 GRPB052VWQP-RC, J7 3221-10-0300-00, SW1 PTS815 SJM 250 SMTR LFS, U1 ESP32C3, U2 BNO055, U3 MIC5504-3.3YM5

Commit message: motor driver
Parts:
- added U4: DRV8410PWPR, DRV8410PWPR:IC_DRV8410PWPR, symbol DRV8410PWPR:DRV8410PWPR
Connections:
- new net: U4.11 (NC), U4.14 (NC)
Other:
- note added: "MOTOR DRIVER"
Changed lines of the file:
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@@
+    (fill (type none))
+  )
+  (rectangle (start 455.168 148.844) (end 561.848 267.208)
+    (stroke (width 0) (type default))
     (fill (type none))
   )
@@
   )
   (text "POWER\n(switch between VUSB and VBATT)" (at 62.992 42.418 0)
+    (effects (font (size 4 4)) (justify left bottom))
+  )
+  (text "MOTOR DRIVER\n" (at 486.918 145.796 0)
     (effects (font (size 4 4)) (justify left bottom))
   )
@@
         )
       )
+    )
+  )
+  (symbol (lib_id "DRV8410PWPR:DRV8410PWPR") (at 512.318 209.55 0) (unit 1)
+    (in_bom yes) (on_board yes) (dnp no) (fields_autoplaced)
+    (property "Reference" "U4" (at 512.318 184.15 0)
+      (effects (font (size 1.27 1.27)))
+    )
+    (property "Value" "DRV8410PWPR" (at 512.318 186.69 0)
+      (effects (font (size 1.27 1.27)))
+    )
+    (property "Footprint" "DRV8410PWPR:IC_DRV8410PWPR" (at 512.318 209.55 0)
+      (effects (font (size 1.27 1.27)) (justify bottom) hide)
+    )
+    (property "Datasheet" "" (at 512.318 209.55 0)
+      (effects (font (size 1.27 1.27)) hide)
+    )
+    (property "MF" "Texas Instruments" (at 512.318 209.55 0)
+      (effects (font (size 1.27 1.27)) (justify bottom) hide)
+    )
+    (property "MAXIMUM_PACKAGE_HEIGHT" "1.2mm" (at 512.318 209.55 0)
+      (effects (font (size 1.27 1.27)) (justify bottom) hide)
+    )
+    (property "Package" "PowerTSSOP-16 Texas Instruments" (at 512.318 209.55 0)
+      (effects (font (size 1.27 1.27)) (justify bottom) hide)
+    )
+    (property "Price" "None" (at 512.318 209.55 0)
+      (effects (font (size 1.27 1.27)) (justify bottom) hide)
+    )
+    (property "Check_prices" "https://www.snapeda.com/parts/DRV8410PWPR/Texas+Instruments/view-part/?ref=eda" (at 512.318 209.55 0)
+      (effects (font (size 1.27 1.27)) (justify bottom) hide)
+    )
+    (property "STANDARD" "Manufacturer Recommendations" (at 512.318 209.55 0)
+      (effects (font (size 1.27 1.27)) (justify bottom) hide)
+    )
+    (property "PARTREV" "B" (at 512.318 209.55 0)
+      (effects (font (size 1.27 1.27)) (justify bottom) hide)
+    )
+    (property "SnapEDA_Link" "https://www.snapeda.com/parts/DRV8410PWPR/Texas+Instruments/view-part/?ref=snap" (at 512.318 209.55 0)
+      (effects (font (size 1.27 1.27)) (justify bottom) hide)
+    )
+    (property "MP" "DRV8410PWPR" (at 512.318 209.55 0)
+      (effects (font (size 1.27 1.27)) (justify bottom) hide)
+    )
+    (property "Purchase-URL" "https://www.snapeda.com/api/url_track_click_mouser/?unipart_id=13462510&manufacturer=Texas Instruments&part_name=DRV8410PWPR&search_term=drv8410pwpr" (at 512.318 209.55 0)
+      (effects (font (size 1.27 1.27)) (justify bottom) hide)
+    )
+    (property "Description" "\n1.65-V to 11-V, 2.5-A, dual H-bridge motor driver with current regulation\n" (at 512.318 209.55 0)
+      (effects (font (size 1.27 1.27)) (justify bottom) hide)
+    )
+    (property "Availability" "In Stock" (at 512.318 209.55 0)
+      (effects (font (size 1.27 1.27)) (justify bottom) hide)
+    )
+    (property "MANUFACTURER" "Texas Instruments" (at 512.318 209.55 0)
+      (effects (font (size 1.27 1.27)) (justify bottom) hide)
+    )
+    (pin "1")
+    (pin "10")
+    (pin "11")
+    (pin "12")
+    (pin "13")
+    (pin "14")
+    (pin "15")
+    (pin "16")
+    (pin "17")
+    (pin "2")
+    (pin "3")
+    (pin "4")
+    (pin "5")
+    (pin "6")
+    (pin "7")
+    (pin "8")
+    (pin "9")
+    (instances
+      (project "SensingBoard_rev1.1"
+        (path "/b61d80ec-963d-4516-bd15-8e7f6f5207da"
+          (reference "U4") (unit 1)
+        )
+      )
