File: ESP32_POE_Board/1.2/ESP32_POE_rev1.2/ESP32-PoE_Rev_L1_v1.2.kicad_sch (KiCad schematic)
At the start: 146 parts, among them J1 USB_C_Receptacle, J2 SI-46020-F, Q1 Q12MHz/20pF/10ppm/4P/3.2x2.5mm, Q2 BC817-40(SOT23), Q3 BC817-40(SOT23), Q4 BC817, Q5 BC817, SW1 PTS815 SJM 250 SMTR LFS, T1 LMUN2211LT1G(SOT-23), U1 CH340T(SSOP20W), U10 ESP32-WROOM-32, U11 TPS2375D, U12 TX4138, U2 TPS2375D(SO-8), U3 MIC5504-3.3YM5, U4 FT232RQ, U4 LAN8710A-EZC(QFN32), U5 TX4138(ESOIC-8), U6 ESP32-WROVER-E, U7 ESDS314DBVR, U9 LAN8710A-EZC

Commit message: POE board partitioning
Parts:
- added D16: PMEG6010CEH, Diode_SMD:D_SOD-123F, symbol Diode:PMEG6010CEH
- added J4: Conn_02x05_Odd_Even, 3221-10-0300-00:CONN10_3221-10-0300-00_CNC, symbol Connector_Generic:Conn_02x05_Odd_Even
- added R14 (x2): 2.2k, Resistor_SMD:R_0402_1005Metric, symbol Device:R_US
- added R14 (x2): 10k, Resistor_SMD:R_0402_1005Metric, symbol Device:R_US
Connections:
- net +3.3V: now also J4.6 (Pin_6), R14.1, R14.1, R14.2, R14.2
- net GND: now also J4.1 (Pin_1)
- net GPI36\U1RXD: now also D16.2 (A), R14.1
- net GPIO13\I2C-SDA: now also J4.3 (Pin_3), R14.2
- net GPIO14\HS2_CLK: now also J4.10 (Pin_10)
- net GPIO15\HS2_CMD: now also J4.9 (Pin_9)
- net GPIO16\I2C-SCL: now also J4.8 (Pin_8), R14.2
- net GPIO4\U1TXD: now also J4.7 (Pin_7)
- net GPIO5\SPI_CS: now also J4.5 (Pin_5), R14.1
- new net: D16.1 (K), J4.2 (Pin_2)
Other:
- note added: "Debug"
- note added: "Weekend Schematic Review: - add NA resistors - wire debug correctly (change symbol)"
- note removed: "Extensions"
- moved on the sheet: C12, C20, C23, C24, C25, C26, C27, D4, D5, D8, L4, R14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
