File: ESP32_POE_Board/1.3/ESP32_POE_rev1.3a/ESP32-PoE_Rev_L1_1.3a.kicad_sch (KiCad schematic)
At the start: 154 parts, among them J1 RS1-02-G, J10 HMTSW-102-X-X-S-X, J11 HMTSW-102-X-X-S-X, J12 HMTSW-102-X-X-S-X, J13 RS1-02-G, J14 RS1-02-G, J15 RS1-02-G, J16 RS1-02-G, J17 RS1-02-G, J18 RS1-02-G, J19 RS1-02-G, J2 HMTSW-102-X-X-S-X, J20 HMTSW-102-X-X-S-X, J21 HMTSW-102-X-X-S-X, J22 HMTSW-102-X-X-S-X, J23 HMTSW-102-X-X-S-X, J24 HMTSW-102-X-X-S-X, J25 SI-46020-F, J26 USB_C_Receptacle, J3 RS1-02-G, J4 RS1-02-G, J5 RS1-02-G, J6 RS1-02-G, J7 HMTSW-102-X-X-S-X, J8 HMTSW-102-X-X-S-X, J9 HMTSW-102-X-X-S-X, Q1 Q12MHz/20pF/10ppm/4P/3.2x2.5mm, Q2 BC817-40(SOT23), Q3 BC817-40(SOT23), SW1 PTS815 SJM 250 SMTR LFS, SW2 PTS815 SJM 250 SMTR LFS, T1 LMUN2211LT1G(SOT-23), U1 CH340T(SSOP20W), U2 TPS2375D(SO-8), U3 BL4054B-42TPRN(SOT23-5), U4 LAN8710A-EZC(QFN32), U5 TX4138(ESOIC-8), U6 ESP32-WROVER-E, U7 SY8089AAAC(SOT23-5), U8 SN74LVC1G04DBVR(SOT23-5)

Commit message: updates
Parts:
- removed ACT1, CHRG1: LED/YELLOW/0603, OLIMEX_LEDs-FP:LED_0603_KA, symbol ESP32-PoE_Rev_L1-rescue:LED-ESP32-PoE_Rev_L1
- removed BAT1: DW02S, OLIMEX_Connectors-FP:LIPO_BAT_VERTICAL_DW02S, symbol ESP32-PoE_Rev_L1-rescue:BAT_CON-ESP32-PoE_Rev_L1
- removed BAT_SENS_E1: Opened, OLIMEX_Jumpers-FP:SJ_1_SMALLER, symbol ESP32-PoE_Rev_L1-rescue:SJ-ESP32-PoE_Rev_L1
- removed C1, C10, C13, C6, C9: 22uF/6.3V/20%/X5R/C0603, OLIMEX_RLC-FP:C_0603_5MIL_DWS, symbol ESP32-PoE_Rev_L1-rescue:C-ESP32-PoE_Rev_L1
- removed C11, C14, C15, C16, C18: 100nF/16V/10%/X7R/C0402, OLIMEX_RLC-FP:C_0402_5MIL_DWS, symbol ESP32-PoE_Rev_L1-rescue:C-ESP32-PoE_Rev_L1
- removed C12, C24: 100nF/100V/10%/X7R/C0603, OLIMEX_RLC-FP:C_0603_5MIL_DWS, symbol ESP32-PoE_Rev_L1-rescue:C-ESP32-PoE_Rev_L1
- removed C17: 2.2uF/6.3V/10%/X5R/C0603, OLIMEX_RLC-FP:C_0603_5MIL_DWS, symbol ESP32-PoE_Rev_L1-rescue:C-ESP32-PoE_Rev_L1
- removed C19: 1nF/50V/10%/X7R/C0402, OLIMEX_RLC-FP:C_0402_5MIL_DWS, symbol ESP32-PoE_Rev_L1-rescue:C-ESP32-PoE_Rev_L1
- removed C2: 1nF/2000V/10%/X7R/C1206, OLIMEX_RLC-FP:C_1206_5MIL_DWS_ISO, symbol ESP32-PoE_Rev_L1-rescue:C-ESP32-PoE_Rev_L1
- removed C21: NA(10uF/6.3V/20%/X5R/C0603), OLIMEX_RLC-FP:C_0603_5MIL_DWS, symbol ESP32-PoE_Rev_L1-rescue:C-ESP32-PoE_Rev_L1
- removed C22: 47uF/6.3V/20%/X5R/C0805, OLIMEX_RLC-FP:C_0805_5MIL_DWS, symbol ESP32-PoE_Rev_L1-rescue:C-ESP32-PoE_Rev_L1
- removed C23: 12pF/50V/5%/COG/C0402, OLIMEX_RLC-FP:C_0402_5MIL_DWS, symbol ESP32-PoE_Rev_L1-rescue:C-ESP32-PoE_Rev_L1
- removed C25: 470uF/10V/20%/Low_ESR/RM2.5/6.0x11mm, OLIMEX_RLC-FP:CPOL-RM2.5mm_6.3x11mm_PTH, symbol ESP32-PoE_Rev_L1-rescue:CP-ESP32-PoE_Rev_L1
- removed C26: NA(220pF/100V/C0603), OLIMEX_RLC-FP:C_0603_5MIL_DWS, symbol ESP32-PoE_Rev_L1-rescue:C-ESP32-PoE_Rev_L1
- removed C27: 15uF/100V/20%/RM2.5/6.3x11mm(Farnell:1281844), OLIMEX_RLC-FP:CPOL-RM2.5mm_6.3x11mm_PTH, symbol ESP32-PoE_Rev_L1-rescue:CP-ESP32-PoE_Rev_L1
- removed D1, D3: 1N5822/SS34/SMA, OLIMEX_Diodes-FP:SMA-KA, symbol ESP32-PoE_Rev_L1-rescue:D_Schottky-ESP32-PoE_Rev_L1
- removed D5: SS510/100V/5A/0.85V/DO214AB(SMC), OLIMEX_Diodes-FP:DO214AB(SMC)_1(K)-2(A), symbol ESP32-PoE_Rev_L1-rescue:D_Schottky_Small-ESP32-PoE_Rev_L1
- removed D8: SMAJ58A/SMA, OLIMEX_Diodes-FP:SMA-KA, symbol ESP32-PoE_Rev_L1-rescue:SMBJ6.0A-ESP32-PoE_Rev_L1
- removed FET1, FET2, FET3: WPM2015-3/TR, OLIMEX_Transistors-FP:SOT23, symbol ESP32-PoE_Rev_L1-rescue:P-MOS+DIOD-ESP32-PoE_Rev_L1
- removed J1, J13, J14, J15, J16, J17, J18, J19, J3, J4, J5, J6: RS1-02-G, CONN_RS1-02-G_ADM, symbol RS1-02-G:RS1-02-G
- removed J25: SI-46020-F, SI-46020-F:BEL_SI-46020-F, symbol SI-46020-F:SI-46020-F
- removed L1: FB0805/600R/2A, OLIMEX_RLC-FP:L_0805_5MIL_DWS, symbol ESP32-PoE_Rev_L1-rescue:L-ESP32-PoE_Rev_L1
- removed L2: 2.2uH/1.5A/DCR=72mR/20%/3.00x3.00x1.50mm/CD32(NR3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, OLIMEX_RLC-FP:CD32, symbol ESP32-PoE_Rev_L1-rescue:L-ESP32-PoE_Rev_L1
- removed L4: 33uH/2.1A/DCR=0.1R/20%/DBS135(PD3316MT330), OLIMEX_RLC-FP:DBS135, symbol ESP32-PoE_Rev_L1-rescue:L-ESP32-PoE_Rev_L1
- removed LNK1: LED/GREEN/0603, OLIMEX_LEDs-FP:LED_0603_KA, symbol ESP32-PoE_Rev_L1-rescue:LED-ESP32-PoE_Rev_L1
- removed PWR1: LED/RED/0603, OLIMEX_LEDs-FP:LED_0603_KA, symbol ESP32-PoE_Rev_L1-rescue:LED-ESP32-PoE_Rev_L1
- removed R1, R2, R25, R6: 10k/R0402, OLIMEX_RLC-FP:R_0402_5MIL_DWS, symbol ESP32-PoE_Rev_L1-rescue:R-ESP32-PoE_Rev_L1
- removed R10, R11, R12, R13: 49.9R/1%/R0402, OLIMEX_RLC-FP:R_0402_5MIL_DWS, symbol ESP32-PoE_Rev_L1-rescue:R-ESP32-PoE_Rev_L1
- removed R14, R15, R41, R5, R8: 2.2k/R0402, OLIMEX_RLC-FP:R_0402_5MIL_DWS, symbol ESP32-PoE_Rev_L1-rescue:R-ESP32-PoE_Rev_L1
- removed R17, R22: 470k/R0402, OLIMEX_RLC-FP:R_0402_5MIL_DWS, symbol ESP32-PoE_Rev_L1-rescue:R-ESP32-PoE_Rev_L1
- removed R23: 180k/1%/R0402, OLIMEX_RLC-FP:R_0402_5MIL_DWS, symbol ESP32-PoE_Rev_L1-rescue:R-ESP32-PoE_Rev_L1
- removed R26: 12.1k/1%/R0402, OLIMEX_RLC-FP:R_0402_5MIL_DWS, symbol ESP32-PoE_Rev_L1-rescue:R-ESP32-PoE_Rev_L1
- removed R27: 4.42k/1%/1/16W/R0402, OLIMEX_RLC-FP:R_0402_5MIL_DWS, symbol ESP32-PoE_Rev_L1-rescue:R-ESP32-PoE_Rev_L1
- removed R28: 0.03R/1%/R1206, OLIMEX_RLC-FP:R_1206_5MIL_DWS, symbol ESP32-PoE_Rev_L1-rescue:R-ESP32-PoE_Rev_L1
- removed R29: 220k/R0402, OLIMEX_RLC-FP:R_0402_5MIL_DWS, symbol ESP32-PoE_Rev_L1-rescue:R-ESP32-PoE_Rev_L1
- removed R3: 1k/R0402, OLIMEX_RLC-FP:R_0402_5MIL_DWS, symbol ESP32-PoE_Rev_L1-rescue:R-ESP32-PoE_Rev_L1
- removed R30: 49.9k/1%/R0402, OLIMEX_RLC-FP:R_0402_5MIL_DWS, symbol ESP32-PoE_Rev_L1-rescue:R-ESP32-PoE_Rev_L1
- removed R33: 4.7R/R0402, OLIMEX_RLC-FP:R_0402_5MIL_DWS, symbol ESP32-PoE_Rev_L1-rescue:R-ESP32-PoE_Rev_L1
- removed R34: 5.23k/1%/R0402, OLIMEX_RLC-FP:R_0402_5MIL_DWS, symbol ESP32-PoE_Rev_L1-rescue:R-ESP32-PoE_Rev_L1
- removed R38: 30.1k/1%/R0402, OLIMEX_RLC-FP:R_0402_5MIL_DWS, symbol ESP32-PoE_Rev_L1-rescue:R-ESP32-PoE_Rev_L1
- removed R4: 47k/R0402, OLIMEX_RLC-FP:R_0402_5MIL_DWS, symbol ESP32-PoE_Rev_L1-rescue:R-ESP32-PoE_Rev_L1
- removed R42: 4.7k/R2512, OLIMEX_RLC-FP:R_2512_MM_DWS, symbol ESP32-PoE_Rev_L1-rescue:R-ESP32-PoE_Rev_L1
- removed R43: NA(22R/R0603), OLIMEX_RLC-FP:R_0603_5MIL_DWS, symbol ESP32-PoE_Rev_L1-rescue:R-ESP32-PoE_Rev_L1
- removed R50: NA(130k/R0402), OLIMEX_RLC-FP:R_0402_5MIL_DWS, symbol ESP32-PoE_Rev_L1-rescue:R-ESP32-PoE_Rev_L1
- removed R51: NA(10k/R0402), OLIMEX_RLC-FP:R_0402_5MIL_DWS, symbol ESP32-PoE_Rev_L1-rescue:R-ESP32-PoE_Rev_L1
- removed R7: 24.9k/1%/R0402, OLIMEX_RLC-FP:R_0402_5MIL_DWS, symbol ESP32-PoE_Rev_L1-rescue:R-ESP32-PoE_Rev_L1
- removed R9: 100k/R0402, OLIMEX_RLC-FP:R_0402_5MIL_DWS, symbol ESP32-PoE_Rev_L1-rescue:R-ESP32-PoE_Rev_L1
- removed RM1, RM2: RA1206_(4X0603)_4B8_2.2k, OLIMEX_RLC-FP:R_MATRIX_4, symbol ESP32-PoE_Rev_L1-rescue:RA1206_(4x0603)_4B8_Smashed-ESP32-PoE_Rev_L1
- removed T1: LMUN2211LT1G(SOT-23), OLIMEX_Transistors-FP:SOT23, symbol ESP32-PoE_Rev_L1-rescue:LMUN2211LT1G(SOT-23)-ESP32-PoE_Rev_L1
- removed TVS1: ESDS314DBVR(SOT-23-5), OLIMEX_Diodes-FP:SOT-23-5, symbol ESP32-PoE_Rev_L1-rescue:ESDS314DBVR(SOT-23-5)-ESP32-PoE_Rev_L1
- removed TVS2, TVS3: NA(GG0402052R542P), OLIMEX_Diodes-FP:D_0402_5MIL_DWS, symbol ESP32-PoE_Rev_L1-rescue:GG0402052R542P-ESP32-PoE_Rev_L1
- removed U2: TPS2375D(SO-8), OLIMEX_IC-FP:SOIC-8_1.75mm, symbol ESP32-PoE_Rev_L1-rescue:TPS2375PW(TSSOP-8)-ESP32-PoE_Rev_L1
- removed U3: BL4054B-42TPRN(SOT23-5), OLIMEX_IC-FP:SOT-23-5, symbol ESP32-PoE_Rev_L1-rescue:BL4054B-42TPRN(SOT23-5)-ESP32-PoE_Rev_L1
- removed U4: LAN8710A-EZC(QFN32), OLIMEX_IC-FP:QFN32_EP(33)_5.00x5.00x0.90mm_Pitch_0.50mm, symbol ESP32-PoE_Rev_L1-rescue:LAN8710A-EZC(QFN32)-ESP32-PoE_Rev_L1
- removed U5: TX4138(ESOIC-8), OLIMEX_Regulators-FP:ESOIC-8, symbol ESP32-PoE_Rev_L1-rescue:TX4138(ESOIC-8)-ESP32-PoE_Rev_L1
- removed U7: SY8089AAAC(SOT23-5), OLIMEX_Regulators-FP:SOT-23-5, symbol ESP32-PoE_Rev_L1-rescue:SY8009AAAC(SOT23-5)-ESP32-PoE_Rev_L1
Connections:
- no-connect marks 22 -> 16
Other:
- note removed: "5V/2A"
- note removed: "Battery Measurement"
- note removed: "CDET"
- note removed: "CHARGING"
- note removed: "Class=0 (0.44 to 12.95W)"
- note removed: "Ethernet"
- note removed: "External Power Sense"
- note removed: "IBAT = 1000/Rprog = 100mA"
- note removed: "In RMII Mode"
- note removed: "LiPo Charger"
- note removed: "PoE Power Supply"
- note removed: "Power Supply"
- note removed: "RDET"
- note removed: "Ra"
- note removed: "Rb"
- note removed: "Rclass"
- note removed: "Rprog"
- note removed: "The PHY is setted up as follows: MODE: All capable(10/100Base) -Auto-negotiation enabled -RMII Configuration -SMI address: 0x00"
- note removed: "Vout=0.6*(1+Ra/Rb)"
- note removed: "Vout=0.8*(1+Ra/Rb)"
- moved on the sheet: C20, C28, C3, C4, C5, C7, C8, D2, D4, D6, D7, D9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

Commit message: board edges
Connections:
- no-connect marks 16 -> 14
Other:
- note added: "ESP32 Module"
- note added: "SD Card"
- note removed: "ESP32 MODULE"
- note removed: "SD/MMC Card"
- moved on the sheet: C4, C5, C7, C8, D2, D6, D7, D9, J10, J11, J12, J2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

Commit message: POE1 board
Parts:
- removed H3, H4: MountingHole, MountingHole:MountingHole_2.1mm, symbol Mechanical:MountingHole
Changed lines of the file:
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@@
     (fill (type none))
   )
-  (rectangle (start 466.852 345.948) (end 562.61 371.094)
+  (rectangle (start 466.852 345.948) (end 517.398 371.094)
     (stroke (width 0) (type default))
     (fill (type none))
@@
     )
   )
-  (symbol (lib_id "Mechanical:MountingHole") (at 538.734 356.87 0) (unit 1)
-    (in_bom yes) (on_board yes) (dnp no) (fields_autoplaced)
-    (property "Reference" "H4" (at 541.528 355.6 0)
-      (effects (font (size 1.27 1.27)) (justify left))
-    )
-    (property "Value" "MountingHole" (at 541.528 358.14 0)
-      (effects (font (size 1.27 1.27)) (justify left))
-    )
-    (property "Footprint" "MountingHole:MountingHole_2.1mm" (at 538.734 356.87 0)
-      (effects (font (size 1.27 1.27)) hide)
-    )
-    (property "Datasheet" "~" (at 538.734 356.87 0)
-      (effects (font (size 1.27 1.27)) hide)
-    )
-    (instances
-      (project "ESP32-PoE_Rev_L1_1.3a"
-        (path "/2ac5de54-6fdf-4ad0-b1b6-0eb3ccc9b17e"
-          (reference "H4") (unit 1)
-        )
-      )
-    )
-  )
   (symbol (lib_id "ESP32-PoE_Rev_L1-rescue:GND-ESP32-PoE_Rev_L1") (at 540.258 70.358 0) (unit 1)
     (in_bom yes) (on_board yes) (dnp no)
@@
         )
       )
-    )
-  )
-  (symbol (lib_id "Mechanical:MountingHole") (at 519.684 357.124 0) (unit 1)
-    (in_bom yes) (on_board yes) (dnp no) (fields_autoplaced)
-    (property "Reference" "H3" (at 522.478 355.854 0)
-      (effects (font (size 1.27 1.27)) (justify left))
-    )
-    (property "Value" "MountingHole" (at 522.478 358.394 0)
-      (effects (font (size 1.27 1.27)) (justify left))
-    )
-    (property "Footprint" "MountingHole:MountingHole_2.1mm" (at 519.684 357.124 0)
-      (effects (font (size 1.27 1.27)) hide)
-    )
-    (property "Datasheet" "~" (at 519.684 357.124 0)
-      (effects (font (size 1.27 1.27)) hide)
-    )
-    (instances
-      (project "ESP32-PoE_Rev_L1_1.3a"
-        (path "/2ac5de54-6fdf-4ad0-b1b6-0eb3ccc9b17e"
-          (reference "H3") (unit 1)
-        )
-      )
