File: ESP32_POE_Board/1.3/ESP32_POE_rev1.3b/ESP32_POE_rev1.3b/ESP32_POE_rev1.3b.kicad_sch (KiCad schematic)
At the start: 154 parts, among them J1 RS1-02-G, J10 HMTSW-102-X-X-S-X, J11 HMTSW-102-X-X-S-X, J12 HMTSW-102-X-X-S-X, J13 RS1-02-G, J14 RS1-02-G, J15 RS1-02-G, J16 RS1-02-G, J17 RS1-02-G, J18 RS1-02-G, J19 RS1-02-G, J2 HMTSW-102-X-X-S-X, J20 HMTSW-102-X-X-S-X, J21 HMTSW-102-X-X-S-X, J22 HMTSW-102-X-X-S-X, J23 HMTSW-102-X-X-S-X, J24 HMTSW-102-X-X-S-X, J25 SI-46020-F, J26 USB_C_Receptacle, J3 RS1-02-G, J4 RS1-02-G, J5 RS1-02-G, J6 RS1-02-G, J7 HMTSW-102-X-X-S-X, J8 HMTSW-102-X-X-S-X, J9 HMTSW-102-X-X-S-X, Q1 Q12MHz/20pF/10ppm/4P/3.2x2.5mm, Q2 BC817-40(SOT23), Q3 BC817-40(SOT23), SW1 PTS815 SJM 250 SMTR LFS, SW2 PTS815 SJM 250 SMTR LFS, T1 LMUN2211LT1G(SOT-23), U1 CH340T(SSOP20W), U2 TPS2375D(SO-8), U3 BL4054B-42TPRN(SOT23-5), U4 LAN8710A-EZC(QFN32), U5 TX4138(ESOIC-8), U6 ESP32-WROVER-E, U7 SY8089AAAC(SOT23-5), U8 SN74LVC1G04DBVR(SOT23-5)

Commit message: updates
Parts:
- removed C20: 1uF/10V/20%/X5R/C0603, OLIMEX_RLC-FP:C_0603_5MIL_DWS, symbol ESP32-PoE_Rev_L1-rescue:C-ESP32-PoE_Rev_L1
- removed C28, C8: 100nF/16V/10%/X7R/C0402, OLIMEX_RLC-FP:C_0402_5MIL_DWS, symbol ESP32-PoE_Rev_L1-rescue:C-ESP32-PoE_Rev_L1
- removed C3: 47uF/6.3V/20%/X5R/C0805, OLIMEX_RLC-FP:C_0805_5MIL_DWS, symbol ESP32-PoE_Rev_L1-rescue:C-ESP32-PoE_Rev_L1
- removed C4, C5: 27pF/50V/5%/C0G/C0402, OLIMEX_RLC-FP:C_0402_5MIL_DWS, symbol ESP32-PoE_Rev_L1-rescue:C-ESP32-PoE_Rev_L1
- removed C7: 22uF/6.3V/20%/X5R/C0603, OLIMEX_RLC-FP:C_0603_5MIL_DWS, symbol ESP32-PoE_Rev_L1-rescue:C-ESP32-PoE_Rev_L1
- removed D2: BAT54C(SOT23-3), OLIMEX_Diodes-FP:SOT23-3, symbol ESP32-PoE_Rev_L1-rescue:BAT54C(SOT23-3)-ESP32-PoE_Rev_L1
- removed D4, D6, D7, D9: 1N5819S4(SOD-123), OLIMEX_Diodes-FP:SOD-123_1C-2A_KA, symbol ESP32-PoE_Rev_L1-rescue:D_Schottky_Small-ESP32-PoE_Rev_L1
- removed H1, H2, H3, H4: MountingHole, MountingHole:MountingHole_2.1mm, symbol Mechanical:MountingHole
- removed J10, J11, J12, J2, J20, J21, J22, J23, J24, J7, J8, J9: HMTSW-102-X-X-S-X, HMTSW-102-X-X-S-X:SAMTEC_HMTSW-102-X-X-S-X, symbol HMTSW-102-X-X-S-X:HMTSW-102-X-X-S-X
- removed J26: USB_C_Receptacle, Connector_USB:USB_C_Receptacle_Molex_105450-0101-L, symbol Connector:USB_C_Receptacle
- removed L3, L5: FB0805/600R/2A, OLIMEX_RLC-FP:L_0805_5MIL_DWS, symbol ESP32-PoE_Rev_L1-rescue:L-ESP32-PoE_Rev_L1
- removed MICRO_SD1: TFC-9P-1.7H(ATFFS150A01BR016), OLIMEX_Connectors-FP:uSD(TFC-9P-1.xH(ATFFS150A01BR016)), symbol ESP32-PoE_Rev_L1-rescue:MICRO_SD(TFC-9P-1.xH(ATFFS150A01BR016))-ESP32-PoE_Rev_L1
- removed Q1: Q12MHz/20pF/10ppm/4P/3.2x2.5mm, OLIMEX_Crystal-FP:TSX-3.2x2.5mm_GND(3), symbol ESP32-PoE_Rev_L1-rescue:Crystal_GND-ESP32-PoE_Rev_L1
- removed Q2, Q3: BC817-40(SOT23), OLIMEX_Transistors-FP:SOT23, symbol ESP32-PoE_Rev_L1-rescue:Q_NPN_BEC-ESP32-PoE_Rev_L1
- removed R16: NA(10k/R0402), OLIMEX_RLC-FP:R_0402_5MIL_DWS, symbol ESP32-PoE_Rev_L1-rescue:R-ESP32-PoE_Rev_L1
- removed R18, R19, R32, R36, R37, R39, R48: 10k/R0402, OLIMEX_RLC-FP:R_0402_5MIL_DWS, symbol ESP32-PoE_Rev_L1-rescue:R-ESP32-PoE_Rev_L1
- removed R20, R21: 1k/R0402, OLIMEX_RLC-FP:R_0402_5MIL_DWS, symbol ESP32-PoE_Rev_L1-rescue:R-ESP32-PoE_Rev_L1
- removed R24, R46, R47: 220R/R0402, OLIMEX_RLC-FP:R_0402_5MIL_DWS, symbol ESP32-PoE_Rev_L1-rescue:R-ESP32-PoE_Rev_L1
- removed R31, R35: 2.2k/R0402, OLIMEX_RLC-FP:R_0402_5MIL_DWS, symbol ESP32-PoE_Rev_L1-rescue:R-ESP32-PoE_Rev_L1
- removed R40, R45: 10R/R0402, OLIMEX_RLC-FP:R_0402_5MIL_DWS, symbol ESP32-PoE_Rev_L1-rescue:R-ESP32-PoE_Rev_L1
- removed R44, R49: NA/R0402, OLIMEX_RLC-FP:R_0402_5MIL_DWS, symbol ESP32-PoE_Rev_L1-rescue:R-ESP32-PoE_Rev_L1
- removed RM3: RA1206_(4X0603)_4B8_2.2k, OLIMEX_RLC-FP:R_MATRIX_4, symbol ESP32-PoE_Rev_L1-rescue:RA1206_(4x0603)_4B8_Smashed-ESP32-PoE_Rev_L1
- removed SW1, SW2: PTS815 SJM 250 SMTR LFS, SW4_PTS815 SJM 250 SMTR LFS_CNK, symbol PTS815:PTS815_SJM_250_SMTR_LFS
- removed U1: CH340T(SSOP20W), OLIMEX_IC-FP:SSOP-20W, symbol ESP32-PoE_Rev_L1-rescue:CH340T(SSOP20W)-ESP32-PoE_Rev_L1
- removed U6: ESP32-WROVER-E, OLIMEX_Cases-FP:ESP32-WROVER(WROOM)-UNIVERSAL_MODULE, symbol ESP32-PoE_Rev_L1-rescue:ESP32-WROVER(WROOM)-UNIVERSAL-ESP32-PoE_Rev_L1
- removed U8: SN74LVC1G04DBVR(SOT23-5), OLIMEX_IC-FP:SOT-23-5, symbol ESP32-PoE_Rev_L1-rescue:SN74LVC1G04DBVR(SOT23-5)-ESP32-PoE_Rev_L1
- removed UEXT1: P-B-V-10-LF, OLIMEX_Connectors-FP:GBH-254-SMT-10, symbol ESP32-PoE_Rev_L1-rescue:BH10S-ESP32-PoE_Rev_L1
Connections:
- no-connect marks 22 -> 6
Other:
- note removed: "!!!WARNING!!! When the board is powered via PoE, don't include the USB cable for to programming it!!! In case this is required, USB-ISO must be used for to guarantee galvanic isolation! See: https://www.olimex.com/Products/USB-Modules/USB-ISO/"
- note removed: "0"
- note removed: "1"
- note removed: "1.8V"
- note removed: "3.3V"
- note removed: "Any GPIO"
- note removed: "Auto program"
- note removed: "Booting Mode"
- note removed: "Bootstrapping Pins Settings"
- note removed: "Buttons"
- note removed: "DTR RTS->EN IO0"
- note removed: "Debugging Log on U0TXD During Booting"
- note removed: "Default"
- note removed: "Don't-care"
- note removed: "Download Boot"
- note removed: "EMAC"
- note removed: "EMAC_COL_out"
- note removed: "EMAC_CRS_out"
- note removed: "EMAC_MDC_out"
- note removed: "EMAC_MDI_in"
- note removed: "EMAC_MDO_out"
- note removed: "ESP32 MODULE"
- note removed: "Falling-edge:Input"
- note removed: "Falling-edge:Output"
- note removed: "For more information refer to esp_wroom_32_datasheet_en.pdf."
- note removed: "GPIO0"
- note removed: "GPIO0:"
- note removed: "GPIO12/MTDI"
- note removed: "GPIO15/MTDO"
- note removed: "GPIO2"
- note removed: "GPIO2:"
- note removed: "GPIO4:"
- note removed: "GPIO5"
- note removed: "GPIO5:"
- note removed: "General Purpose SPI"
- note removed: "HSPICLK"
- note removed: "HSPICLK_in/_out"
- note removed: "HSPID"
- note removed: "HSPID_in/_out"
- note removed: "HSPIQ"
- note removed: "HSPIQ_in/_out"
- note removed: "HSPI_CS0_in/_out"
- note removed: "HSPI_CS1_out"
- note removed: "HSPI_CS2_out"
- note removed: "I2C"
- note removed: "I2CEXT0_SCL_in"
- note removed: "I2CEXT0_SCL_out"
- note removed: "I2CEXT0_SDA_in"
- note removed: "I2CEXT0_SDA_out"
- note removed: "I2CEXT1_SCL_in"
- note removed: "I2CEXT1_SCL_out"
- note removed: "I2CEXT1_SDA_in"
- note removed: "I2CEXT1_SDA_out"
- note removed: "Interface"
- note removed: "Internal Bootstrapping Resistors"
- note removed: "MTDI/GPIO12:"
- note removed: "MTDO/GPIO15:"
- note removed: "Mounting Holes"
- note removed: "Notes:"
- note removed: "Pin"
- note removed: "Pull-Down"
- note removed: "Pull-Up"
- note removed: "Rising-edge:Input"
- note removed: "Rising-edge:Output"
- note removed: "SD/MMC Card"
- note removed: "SPI Flash Boot"
- note removed: "Signal"
- note removed: "Software Selectable Pins"
- note removed: "Timing of SDIO Slave"
- note removed: "U0TXD Silent"
- note removed: "U0TXD Toggling"
- note removed: "U8, C28 and R45 have to be Populated -> when WROVER is used, U8, C28 and R45 have to be NA -> when WROOM is used."
- note removed: "UEXT"
- note removed: "USB to UART"
- note removed: "VSPICLK_in/_out"
- note removed: "VSPID_in/_out"
- note removed: "VSPIQ_in/_out"
- note removed: "VSPI_CS0_in/_out"
- note removed: "VSPI_CS1_out"
- note removed: "VSPI_CS2_out"
- note removed: "Voltage of Internal LDO(VDD_SDIO)"
- note removed: "or ESP32-WROOM-32E"
- moved on the sheet: ACT1, BAT1, BAT_SENS_E1, C1, C10, C11, C12, C13, C14, C15, C16, C17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

Commit message: POE 2 board
Parts:
- added J2: HMTSW-102-X-X-S-X, HMTSW-102-X-X-S-X:SAMTEC_HMTSW-102-X-X-S-X, symbol HMTSW-102-X-X-S-X:HMTSW-102-X-X-S-X
Other:
- note added: "POE Power Supply"
- note added: "Power Supply / LIPO Charger"
- note added: "Wireless Charger"
- note removed: "LiPo Charger"
- note removed: "PoE Power Supply"
- note removed: "Power Supply"
- moved on the sheet: J1, J13, J14, J15, J16, J17, J18, J19, J3, J4, J5, J6
