File: ESP32_POE_Board/1.4/ESP_POE_1.4_combined/ESP32-PoE-ISO_Rev_K.kicad_sch (KiCad schematic)
At the start: 139 parts, among them J2 HMTSW-102-X-X-S-X, J25 SI-46020-F, J26 USB_C_Receptacle, Q1 Q12MHz/20pF/10ppm/4P/3.2x2.5mm, Q2 BC817-40(SOT23), Q3 BC817-40(SOT23), SW1 PTS815 SJM 250 SMTR LFS, T1 LMUN2211LT1G(SOT-23), U1 CH340T(SSOP20W), U2 TPS2376PW(TSSOP-8), U3 BL4054B-42TPRN(SOT23-5), U4 LAN8710A-EZC(QFN32), U5 TX4138(ESOIC-8), U6 ESP32-WROVER-E, U7 SY8089AAAC(SOT23-5), U8 SN74LVC1G04DBVR(SOT23-5)

Commit message: updated combined POE schematic
Parts:
- removed BUT1, RST1: IT1185AU2, OLIMEX_Buttons-FP:IT1185AU2_V2, symbol ESP32-PoE-ISO_Rev_K:SIDE_WTCM-TR(3x4)
- removed LAN_CON1: RJP-003TC1(LPJ4112CNL), OLIMEX_Connectors-FP:RJP-003TC1(LPJ4112CNL), symbol ESP32-PoE-ISO_Rev_K:RJP-003TC1(LPJ4112CNL)
- removed R49: NA/R0402, OLIMEX_RLC-FP:R_0402_5MIL_DWS, symbol ESP32-PoE-ISO_Rev_K:R
- removed SW1: PTS815 SJM 250 SMTR LFS, SW4_PTS815 SJM 250 SMTR LFS_CNK, symbol PTS815:PTS815_SJM_250_SMTR_LFS
- removed USB-UART1: MISB-SWMM-5B-LF(USB_MICRO), OLIMEX_Connectors-FP:USB-MICRO_MISB-SWMM-5B_LF, symbol ESP32-PoE-ISO_Rev_K:USB-MINI
- added J4, J6: 20021111-00012T4LF, CONN_20021111-XX012XXLF_AMP, symbol 20021111-00012T4LF:20021111-00012T4LF
- added J5, J7: 20021311-00012T4LF, 20021311-00012T4LF:AMPHENOL_20021311-00012T4LF, symbol 20021311-00012T4LF:20021311-00012T4LF
- added R45: 220R/R0402, OLIMEX_RLC-FP:R_0402_5MIL_DWS, symbol ESP32-PoE-ISO_Rev_K:R
- added SW1 (x2): PTS815 SJM 250 SMTR LFS, SW4_PTS815 SJM 250 SMTR LFS_CNK, symbol PTS815:PTS815_SJM_250_SMTR_LFS
- R47: value 220R/R0402 -> 10k/R0402
- R48: value 10k/R0402 -> NA/R0402
- UEXT1: footprint OLIMEX_Connectors-FP:GBH-254-SMT-10 -> 3221-10-0300-00:CONN10_3221-10-0300-00_CNC
Connections:
- net +3V3: now also R47.1, J4.1, J5.1; no longer R48.1
- net +5VP: now also J4.3, J5.3
- net +5V_USB: now also J26.A1 (GND), J26.A12 (GND), J26.A4 (VBUS), J26.A9 (VBUS), J26.B1 (GND), J26.B12 (GND), J26.B4 (VBUS), J26.B9 (VBUS), J26.S1 (SHIELD), L3.1
- net D_Com: now also R48.2
- net ESP_EN: now also SW1.1
- net GND: now also J4.10, J4.12, J4.2, J4.4, J4.6, J4.8, J5.10, J5.12, J5.2, J5.4, J5.6, J5.8, J6.10, J6.12, J6.2, J6.4, J6.6, J6.8, J7.10, J7.12, J7.2, J7.4, J7.6, J7.8, R45.2, SW1.4; no longer R47.2
- net GPI34/BUT1: now also SW1.1; no longer R48.2
- net GPIO12/PHY_PWR: now also J6.5, J7.5
- net GPIO18/MDIO(RMII): now also J6.7, J7.7
- net GPIO19/EMAC_TXD0(RMII): now also J4.11, J5.11
- net GPIO21/EMAC_TX_EN(RMII): now also J4.7, J5.7
- net GPIO22/EMAC_TXD1(RMII): now also J4.9, J5.9
- net GPIO23/MDC(RMII): now also J6.9, J7.9
- net GPIO25/EMAC_RXD0(RMII): now also J4.5, J5.5
- net GPIO26/EMAC_RXD1(RMII): now also J6.11, J7.11
- net GPIO27/EMAC_RX_CRS_DV: now also J6.3, J7.3
- net RD+: now also J25.4 (RD+)
- net RD-: now also J25.6 (RD-)
- net Shield: now also J25.7 (P7), J25.S1 (SHIELD), J25.S2 (SHIELD)
- net Spare1: now also J25.9 (P9)
- net Spare2: now also J25.10 (P10)
- net TD+: now also J25.1 (TD+)
- net TD-: now also J25.3 (TD-)
- net USB_D+: now also J26.A6 (D+), J26.B6 (D+)
- net USB_D-: now also J26.A7 (D-), J26.B7 (D-)
- net at C11.1, C13.1, C15.1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: now also J25.2 (TCT), J25.5 (RCT)
- new net: R45.1, SW1.4
- new net: R47.2, R48.1, SW1.2
- no-connect marks 20 -> 19
Other:
- note added: "B2B Headers"
- moved on the sheet: C29, J25, J26, R42, U8
