File: ESP32_POE_Board/1.4/ESP_POE_1.4_combined/ESP32-PoE-ISO_Rev_K.kicad_pcb (KiCad board)
At the start: 4 copper layers, 28 x 98.2 mm, 145 parts, among them Q1 Q12MHz/20pF/10ppm/4P/3.2x2.5mm, Q2 BC817-40(SOT23), Q3 BC817-40(SOT23), T1 LMUN2211LT1G(SOT-23), U1 CH340T(SSOP20W), U2 TPS2376PW(TSSOP-8), U3 BL4054B-42TPRN(SOT23-5), U4 LAN8710A-EZC(QFN32), U5 TX4138(ESOIC-8), U6 ESP32-WROVER-E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

Commit message: updated combined POE schematic
Parts:
- removed BUT1, RST1: IT1185AU2, OLIMEX_Buttons-FP:IT1185AU2_V2
- removed EXT1, EXT2: NS(HN1x10), OLIMEX_Connectors-FP:HN1x10
- removed R49: NA/R0402, OLIMEX_RLC-FP:R_0402_5MIL_DWS
- removed USB-UART1: MISB-SWMM-5B-LF(USB_MICRO), OLIMEX_Connectors-FP:USB-MICRO_MISB-SWMM-5B_LF
- added J1: USB_C_Receptacle, Connector_USB:USB_C_Receptacle_Molex_105450-0101-L, F.Cu at (151.9, 123.8)
- added J2: SI-46020-F, SI-46020-F:BEL_SI-46020-F, F.Cu at (171.2, 153.3)
- added J3: HMTSW-102-X-X-S-X, HMTSW-102-X-X-S-X:SAMTEC_HMTSW-102-X-X-S-X, F.Cu at (169.3, 108.9)
- added J4: 20021111-00012T4LF, 20021111-00012T4LF:CONN_20021111-XX012XXLF_AMP, F.Cu at (163.7, 133.8)
- added J5: 20021311-00012T4LF, 20021311-00012T4LF:AMPHENOL_20021311-00012T4LF, B.Cu at (158.2, 151.5)
- added J6: 20021111-00012T4LF, 20021111-00012T4LF:CONN_20021111-XX012XXLF_AMP, F.Cu at (183.2, 133.5)
- added J7: 20021311-00012T4LF, 20021311-00012T4LF:AMPHENOL_20021311-00012T4LF, B.Cu at (184.6, 151.3)
- added SW1: PTS815 SJM 250 SMTR LFS, PTS815:SW4_PTS815 SJM 250 SMTR LFS_CNK, F.Cu at (171.2, 104.3)
- added SW2: PTS815 SJM 250 SMTR LFS, PTS815:SW4_PTS815 SJM 250 SMTR LFS_CNK, F.Cu at (159.3, 96.6)
- R47: value 220R/R0402 -> 10k/R0402
- R48: value 10k/R0402 -> NA/R0402
- UEXT1: footprint OLIMEX_Connectors-FP:GBH-254-SMT-10 -> 3221-10-0300-00:CONN10_3221-10-0300-00_CNC
- moved UEXT1 1.27 mm to (103.5, 125.4)
Connections:
- net /GPI36/U1RXD renamed /GPI36/U1RXD
- net /GPIO1/U0TXD renamed /GPIO1/U0TXD
- net /GPIO12/PHY_PWR renamed /GPIO12/PHY_PWR
- net /GPIO13/I2C-SDA renamed /GPIO13/I2C-SDA
- net /GPIO14/HS2_CLK renamed /GPIO14/HS2_CLK
- net /GPIO15/HS2_CMD renamed /GPIO15/HS2_CMD
- net /GPIO16/I2C-SCL renamed /GPIO16/I2C-SCL
- net /GPIO17/EMAC_CLK_OUT_180 renamed /GPIO17/EMAC_CLK_OUT_180
- net /GPIO18/MDIO(RMII) renamed /GPIO18/MDIO(RMII)
- net /GPIO19/EMAC_TXD0(RMII) renamed /GPIO19/EMAC_TXD0(RMII)
- net /GPIO2/HS2_DATA0 renamed /GPIO2/HS2_DATA0
- net /GPIO21/EMAC_TX_EN(RMII) renamed /GPIO21/EMAC_TX_EN(RMII)
- net /GPIO22/EMAC_TXD1(RMII) renamed /GPIO22/EMAC_TXD1(RMII)
- net /GPIO23/MDC(RMII) renamed /GPIO23/MDC(RMII)
- net /GPIO25/EMAC_RXD0(RMII) renamed /GPIO25/EMAC_RXD0(RMII)
- net /GPIO26/EMAC_RXD1(RMII) renamed /GPIO26/EMAC_RXD1(RMII)
- net /GPIO27/EMAC_RX_CRS_DV renamed /GPIO27/EMAC_RX_CRS_DV
- net /GPIO3/U0RXD renamed /GPIO3/U0RXD
- net /GPIO4/U1TXD renamed /GPIO4/U1TXD
- net /GPIO5/SPI_CS renamed /GPIO5/SPI_CS
- C11 pad 1: Net-(C11-Pad1) -> Net-(J2-RCT)
- C13 pad 1: Net-(C11-Pad1) -> Net-(J2-RCT)
- C15 pad 1: Net-(C11-Pad1) -> Net-(J2-RCT)
- C16 pad 1: Net-(C11-Pad1) -> Net-(J2-RCT)
- FID1 pad Fid1: Net-(FID1-PadFid1) -> unconnected-(FID1-FID*-PadFid1)
- FID2 pad Fid1: Net-(FID2-PadFid1) -> unconnected-(FID2-FID*-PadFid1)
- FID3 pad Fid1: Net-(FID3-PadFid1) -> unconnected-(FID3-FID*-PadFid1)
- FID4 pad Fid1: Net-(FID4-PadFid1) -> unconnected-(FID4-FID*-PadFid1)
- FID5 pad Fid1: Net-(FID5-PadFid1) -> unconnected-(FID5-FID*-PadFid1)
- FID6 pad Fid1: Net-(FID6-PadFid1) -> unconnected-(FID6-FID*-PadFid1)
- L1 pad 2: Net-(C11-Pad1) -> Net-(J2-RCT)
- L3 pad 1: Net-(L3-Pad1) -> /+5V_USB
- LAN_CON1 pad 4: Net-(C11-Pad1) -> Net-(LAN_CON1-RCT)
- LAN_CON1 pad 5: Net-(C11-Pad1) -> Net-(LAN_CON1-RCT)
- LNK1 pad 2: Net-(C11-Pad1) -> Net-(J2-RCT)
- MICRO_SD1 pad CD1: Net-(MICRO_SD1-PadCD1) -> unconnected-(MICRO_SD1-Card_Detect-PadCD1)
- R10 pad 1: Net-(C11-Pad1) -> Net-(J2-RCT)
- R11 pad 1: Net-(C11-Pad1) -> Net-(J2-RCT)
- R12 pad 1: Net-(C11-Pad1) -> Net-(J2-RCT)
- R13 pad 1: Net-(C11-Pad1) -> Net-(J2-RCT)
- R47 pad 1: Net-(BUT1-Pad2) -> +3V3
- R47 pad 2: GND -> Net-(R47-Pad2)
- R48 pad 1: +3V3 -> Net-(R47-Pad2)
- R48 pad 2: /GPI34/BUT1 -> /D_Com
- U1 pad 11: Net-(U1-Pad11) -> unconnected-(U1-CTS#-Pad11)
- U1 pad 12: Net-(U1-Pad12) -> unconnected-(U1-DSR#-Pad12)
- U1 pad 13: Net-(U1-Pad13) -> unconnected-(U1-RI#-Pad13)
- U1 pad 14: Net-(U1-Pad14) -> unconnected-(U1-DCD#-Pad14)
- U1 pad 17: Net-(U1-Pad17) -> unconnected-(U1-IR#-Pad17)
- U1 pad 20: Net-(U1-Pad20) -> unconnected-(U1-NOS#-Pad20)
- U4 pad 1: Net-(C11-Pad1) -> Net-(J2-RCT)
- U4 pad 14: Net-(U4-Pad14) -> unconnected-(U4-CRS-Pad14)
- U4 pad 18: Net-(U4-Pad18) -> unconnected-(U4-NINT/TXER/TXD4-Pad18)
- U4 pad 20: Net-(U4-Pad20) -> unconnected-(U4-TXCLK-Pad20)
- U4 pad 26: Net-(U4-Pad26) -> unconnected-(U4-RXDV-Pad26)
- U4 pad 27: Net-(C11-Pad1) -> Net-(J2-RCT)
- U4 pad 4: Net-(U4-Pad4) -> unconnected-(U4-XTAL2-Pad4)
- U5 pad 7: Net-(U5-Pad7) -> unconnected-(U5-POK-Pad7)
- U6 pad 17: Net-(U6-Pad17) -> unconnected-(U6-NC-Pad17)
- U6 pad 18: Net-(U6-Pad18) -> unconnected-(U6-NC-Pad18)
- U6 pad 19: Net-(U6-Pad19) -> unconnected-(U6-NC-Pad19)
- U6 pad 20: Net-(U6-Pad20) -> unconnected-(U6-NC-Pad20)
- U6 pad 21: Net-(U6-Pad21) -> unconnected-(U6-NC-Pad21)
- U6 pad 22: Net-(U6-Pad22) -> unconnected-(U6-NC-Pad22)
- U6 pad 32: Net-(U6-Pad32) -> unconnected-(U6-NC-Pad32)
- U6 pad 6: /GPI34/BUT1 -> /GPI34/BUT1
- U8 pad 1: Net-(U8-Pad1) -> unconnected-(U8-NC-Pad1)
Routing:
- net Net-(LAN_CON1-RCT): track 0.00 -> 96.2 mm, vias 0 -> 6
- net Net-(C11-Pad1): track 96.2 -> 0.00 mm, vias 6 -> 0
- net /GPI34/BUT1: track 0.00 -> 74.5 mm, vias 0 -> 5
- net /GPI34/BUT1: track 74.5 -> 0.00 mm, vias 5 -> 0
- net /+5V_USB: track 56.1 -> 77.7 mm
- net Net-(L3-Pad1): track 21.6 -> 0.00 mm
- net Net-(U6-Pad20): track 11.1 -> 0.00 mm
- net unconnected-(U6-NC-Pad20): track 0.00 -> 11.1 mm
- net Net-(U6-Pad19): track 11.0 -> 0.00 mm
- net unconnected-(U6-NC-Pad19): track 0.00 -> 11.0 mm
- net unconnected-(U6-NC-Pad21): track 0.00 -> 9.25 mm
- net Net-(U6-Pad21): track 9.25 -> 0.00 mm
- net unconnected-(U6-NC-Pad18): track 0.00 -> 9.21 mm
- net Net-(U6-Pad18): track 9.21 -> 0.00 mm
- net unconnected-(U6-NC-Pad22): track 0.00 -> 7.42 mm
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Other:
- board size 28 x 98.2 mm -> 101.8 x 98.2 mm
- net class Default removed
- net class Diff_Z=100 removed
- net class Diff_Z=90 removed
