File: ESP32_POE_Board/1.4/ESP_POE_1.4a/ESP_POE_1.4a/ESP_POE_1.4a.kicad_pcb (KiCad board)
At the start: 4 copper layers, 101.8 x 98.2 mm, 148 parts, among them J1 USB_C_Receptacle, J2 SI-46020-F, J3 HMTSW-102-X-X-S-X, J4 20021111-00012T4LF, J5 20021311-00012T4LF, J6 20021111-00012T4LF, J7 20021311-00012T4LF, Q1 Q12MHz/20pF/10ppm/4P/3.2x2.5mm, Q2 BC817-40(SOT23), Q3 BC817-40(SOT23)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

Commit message: updates
Parts:
- removed C1, C22, C6, C7: 22uF/6.3V/20%/X5R/C0603, OLIMEX_RLC-FP:C_0603_5MIL_DWS
- removed C28: 1nF/50V/10%/X7R/C0402, OLIMEX_RLC-FP:C_0402_5MIL_DWS
- removed C29, C8: 100nF/16V/10%/X7R/C0402, OLIMEX_RLC-FP:C_0402_5MIL_DWS
- removed C3: 47uF/6.3V/20%/X5R/C0805, OLIMEX_RLC-FP:C_0805_5MIL_DWS
- removed C31: 1uF/10V/20%/X5R/C0603, OLIMEX_RLC-FP:C_0603_5MIL_DWS
- removed C4, C5: 27pF/50V/5%/C0G/C0402, OLIMEX_RLC-FP:C_0402_5MIL_DWS
- removed CHRG1: LED/YELLOW/0603, OLIMEX_LEDs-FP:LED_0603_KA
- removed D1, D3, D4, D6, D7, D9: 1N5819S4/SOD123, OLIMEX_Diodes-FP:SOD-123_1C-2A_KA
- removed D2: BAT54C(SOT23-3), OLIMEX_Diodes-FP:SOT23-3
- removed FET1, FET2: WPM2015-3/TR, OLIMEX_Transistors-FP:SOT23
- removed FID2, FID3, FID5, FID6: Fiducial, OLIMEX_Other-FP:Fiducial1x3
- removed J1: USB_C_Receptacle, Connector_USB:USB_C_Receptacle_Molex_105450-0101-L
- removed J5, J7: 20021311-00012T4LF, 20021311-00012T4LF:AMPHENOL_20021311-00012T4LF
- removed L2: 2.2uH/1.5A/DCR=72mR/20%/3.00x3.00x1.50mm/CD32(NR3015T2R2M), OLIMEX_RLC-FP:CD32
- removed L3, L5: FB0805/600R/2A, OLIMEX_RLC-FP:L_0805_5MIL_DWS
- removed MH1, MH2, MH3: Mounting_Hole_NPTH, OLIMEX_Other-FP:NPTH_2.2mm
- removed PWR1: LED/RED/0603, OLIMEX_LEDs-FP:LED_0603_KA
- removed Q1: Q12MHz/20pF/10ppm/4P/3.2x2.5mm, OLIMEX_Crystal-FP:TSX-3.2x2.5mm_GND(3)
- removed Q2, Q3: BC817-40(SOT23), OLIMEX_Transistors-FP:SOT23
- removed R1, R18, R19, R32, R36, R37, R39, R47, R6: 10k/R0402, OLIMEX_RLC-FP:R_0402_5MIL_DWS
- removed R16, R7: 470k/R0402, OLIMEX_RLC-FP:R_0402_5MIL_DWS
- removed R17, R48: NA/R0402, OLIMEX_RLC-FP:R_0402_5MIL_DWS
- removed R20, R21: 1k/R0402, OLIMEX_RLC-FP:R_0402_5MIL_DWS
- removed R24, R46: 220R/R0402, OLIMEX_RLC-FP:R_0402_5MIL_DWS
- removed R29: 220k/R0402, OLIMEX_RLC-FP:R_0402_5MIL_DWS
- removed R30: 49.9k/1%/R0402, OLIMEX_RLC-FP:R_0402_5MIL_DWS
- removed R31, R35, R5, R8: 2.2k/R0402, OLIMEX_RLC-FP:R_0402_5MIL_DWS
- removed R4: 47k/R0402, OLIMEX_RLC-FP:R_0402_5MIL_DWS
- removed R40, R42: 10R/R0402, OLIMEX_RLC-FP:R_0402_5MIL_DWS
- removed R9: 100k/R0402, OLIMEX_RLC-FP:R_0402_5MIL_DWS
- removed RM3: RA1206_(4X0603)_4B8_2.2k, OLIMEX_RLC-FP:R_MATRIX_4
- removed SW1, SW2: PTS815 SJM 250 SMTR LFS, PTS815:SW4_PTS815 SJM 250 SMTR LFS_CNK
- removed U1: CH340T(SSOP20W), OLIMEX_IC-FP:SSOP-20W
- removed U3: BL4054B-42TPRN(SOT23-5), OLIMEX_IC-FP:SOT-23-5
- removed U7: SY8089AAAC(SOT23-5), OLIMEX_Regulators-FP:SOT-23-5
- removed U8: SN74LVC1G04DBVR(SOT23-5), OLIMEX_IC-FP:SOT-23-5
- added H1: MountingHole, MountingHole:MountingHole_2.1mm, F.Cu at (182.5, 110.9)
- added H2: MountingHole, MountingHole:MountingHole_2.1mm, F.Cu at (182.5, 116.6)
Routing:
- net (no net): track 0.00 -> 432.0 mm, vias 0 -> 19
- net +5V: track 116.1 -> 0.00 mm, vias 7 -> 0
- net /+5V_USB: track 77.7 -> 0.00 mm, vias 6 -> 0
- net Net-(Q3-E): track 53.8 -> 0.00 mm, vias 3 -> 0
- net /GPIO4/U1TXD: track 72.7 -> 125.3 mm, vias 6 -> 10
- net Net-(Q2-E): track 45.2 -> 0.00 mm, vias 3 -> 0
- net /USB_D-: track 27.6 -> 0.00 mm
- net /USB_D+: track 27.2 -> 0.00 mm
- net Net-(D9-K): track 21.5 -> 0.00 mm, vias 2 -> 0
- net Net-(D3-K): track 18.2 -> 0.00 mm
- net Net-(U1-XO): track 16.5 -> 0.00 mm
- net Net-(U7-LX): track 12.0 -> 0.00 mm
- net Net-(U1-V3): track 9.40 -> 0.00 mm
- net /D_Com: track 8.77 -> 0.00 mm
- net Net-(D6-K): track 8.57 -> 0.00 mm
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- removed copper zone on F.Cu, net GND

Commit message: starting POE1 route
Parts:
- removed BAT1: DW02S, OLIMEX_Connectors-FP:LIPO_BAT_VERTICAL_DW02S
- removed Drill_Slot1, Drill_Slot3: 2 mm, OLIMEX_Other-FP:Mounting_hole_2_mm
- removed FID4: Fiducial, OLIMEX_Other-FP:Fiducial1x3
- removed LAN_CON1: RJP-003TC1(LPJ4112CNL), OLIMEX_Connectors-FP:RJP-003TC1(LPJ4112CNL)
- removed Logo_OSHW: , OLIMEX_LOGOs-FP:LOGO_OPENHARDWARE_8x8
- removed Logo_Olimex: , OLIMEX_LOGOs-FP:OLIMEX_LOGO_TB
- removed MICRO_SD1: TFC-9P-1.7H(ATFFS150A01BR016), OLIMEX_Connectors-FP:uSD(TFC-9P-1.xH(ATFFS150A01BR016))
- removed Sign_Antistatic: Val**, OLIMEX_LOGOs-FP:LOGO_ANTISTATIC_1
- removed Sign_CE: CE_Sign, OLIMEX_LOGOs-FP:CE_Sign
- removed Sign_PB-Free: , OLIMEX_LOGOs-FP:LOGO_PBFREE
- removed Sign_RecycleBin: , OLIMEX_LOGOs-FP:LOGO_RECYCLEBIN_1
- removed U6: ESP32-WROVER-E, OLIMEX_Cases-FP:ESP32-WROVER(WROOM)-UNIVERSAL_MODULE
- removed UEXT1: P-B-V-10-LF, 3221-10-0300-00:CONN10_3221-10-0300-00_CNC
- added FID2: Fiducial, Fiducial:Fiducial_0.5mm_Mask1.5mm, B.Cu at (127.4, 154.1)
- added FID3: Fiducial, Fiducial:Fiducial_0.5mm_Mask1.5mm, F.Cu at (126.9, 154.1)
- added FID5: Fiducial, Fiducial:Fiducial_0.5mm_Mask1.5mm, F.Cu at (103.4, 126.4)
- FID1: footprint OLIMEX_Other-FP:Fiducial1x3 -> Fiducial:Fiducial_0.5mm_Mask1.5mm; moved to B.Cu
- moved H2 89.2 mm to (99.6, 149.6)
- moved J4 61.7 mm to (102.9, 144.0)
- moved J3 58.5 mm to (111.8, 98.4)
- moved J2 58.2 mm to (114.1, 142.0)
- moved H1 57.8 mm to (128.1, 130.4)
- moved J6 57.5 mm to (126.6, 144.0)
- moved C27 50.5 mm to (81.3, 124.7)
- moved C26 49.3 mm to (75.2, 128.7), turned to 90 degrees
- moved L4 47.1 mm to (127.0, 120.3), turned to 180 degrees
- moved R28 40.7 mm to (130.4, 135.8), turned to 90 degrees
- moved FID1 36.1 mm to (102.8, 126.4)
- moved D10 32.3 mm to (130.4, 141.9), turned to -90 degrees
- moved U2 30.4 mm to (130.4, 137.7), turned to -90 degrees
- moved U5 27.8 mm to (127.5, 148.4), turned to 90 degrees
- moved C2 27.0 mm to (121.0, 148.6), turned to 180 degrees
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Routing:
- net (no net): track 432.0 -> 0.00 mm, vias 19 -> 0
- net GND: track 358.2 -> 3.87 mm, vias 90 -> 0
- net /Shield: track 186.8 -> 0.00 mm, vias 17 -> 0
- net +3V3: track 148.9 -> 0.00 mm, vias 16 -> 0
- net Earth: track 148.2 -> 0.00 mm, vias 21 -> 0
- net /GPIO4/U1TXD: track 125.3 -> 0.00 mm, vias 10 -> 0
- net Spare1: track 120.8 -> 0.00 mm, vias 7 -> 0
- net Net-(D5-K): track 107.2 -> 0.00 mm, vias 8 -> 0
- net Net-(LAN_CON1-RCT): track 96.2 -> 0.00 mm, vias 6 -> 0
- net Net-(U3-VBAT): track 94.5 -> 0.00 mm, vias 2 -> 0
- net /GPIO3/U0RXD: track 89.5 -> 0.00 mm, vias 3 -> 0
- net /GPIO1/U0TXD: track 87.9 -> 0.00 mm, vias 3 -> 0
- net +5VP: track 80.7 -> 0.00 mm, vias 7 -> 0
- net Spare2: track 79.0 -> 0.00 mm, vias 8 -> 0
- net /GPIO16/I2C-SCL: track 76.4 -> 0.00 mm, vias 5 -> 0
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- removed copper zone on In2.Cu, net +3V3
- removed copper zone on In2.Cu, net /ILIM
- removed copper zone on B.Cu, net /Shield
- removed copper zone on F.Cu, net /Shield
- removed copper zone on In1.Cu, net /Shield
- removed copper zone on In2.Cu, net /Shield
- removed copper zone on B.Cu, net Earth
- removed copper zone on F.Cu, net Earth
- removed copper zone on In1.Cu, net Earth
- removed copper zone on B.Cu, net GND
- removed copper zone on In1.Cu, net GND
Other:
- board size 101.8 x 98.2 mm -> 40 x 40 mm
- board text removed: "(C) 2022"
- board text removed: "+"
- board text removed: "+3V3"
- board text removed: "+5V"
- board text removed: "-"
- board text removed: "0"
- board text removed: "1"
- board text removed: "13"
- board text removed: "14"
- board text removed: "15"
- board text removed: "16"
- board text removed: "2"
- board text removed: "3"
- board text removed: "32"
- board text removed: "33"
- board text removed: "34"
- board text removed: "35"
- board text removed: "36"
- board text removed: "39"
- board text removed: "4"
- board text removed: "4 Layer PCB Dimensions: 28x98mm"
- board text removed: "5"
- board text removed: "9"
- board text removed: "Compliant"
- board text removed: "ESP32-PoE-ISO"
- board text removed: "ESP_EN"
- board text removed: "GND"
- board text removed: "Rev.K"
- board text removed: "RoHS"
- board text removed: "https://www.olimex.com"

Commit message: updates
Parts:
- J4: moved to B.Cu
- R41: moved to F.Cu
- moved L4 36.4 mm to (114.2, 154.4)
- moved L1 36.3 mm to (121.8, 133.8), turned to 90 degrees
- moved C10 34.6 mm to (123.8, 132.8)
- moved R43 34.1 mm to (132.7, 141.7), turned to -90 degrees
- moved R44 32.6 mm to (132.7, 144.1), turned to -90 degrees
- moved FET3 32.2 mm to (117.7, 138.4)
- moved C13 31.8 mm to (114.6, 139.5)
- moved C19 20.0 mm to (98.0, 135.2), turned to 90 degrees
- moved C23 19.4 mm to (86.7, 137.6)
- moved C15 17.2 mm to (103.5, 128.3), turned to 180 degrees
- moved R41 13.3 mm to (127.4, 148.2), turned to 180 degrees
- moved D8 8.96 mm to (98.0, 140.6)
- moved C12 7.89 mm to (82.9, 145.7)
- moved DCDC1 5.24 mm to (114.5, 150.9), turned to 0 degrees
- moved J4 1.22 mm to (101.7, 144.0)
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Routing:
- net Earth: track 0.00 -> 51.5 mm, vias 0 -> 2
- net Spare1: track 0.00 -> 43.9 mm, vias 0 -> 2
- net Net-(J2-RCT): track 16.0 -> 57.6 mm
- net /Shield: track 0.00 -> 37.9 mm
- net /GPIO21/EMAC_TX_EN(RMII): track 0.00 -> 34.6 mm, vias 0 -> 1
- net /GPIO22/EMAC_TXD1(RMII): track 0.00 -> 32.5 mm, vias 0 -> 1
- net Net-(U4-LED2/NINTSEL): track 0.00 -> 31.9 mm, vias 0 -> 2
- net +3V3: track 0.00 -> 30.7 mm
- net /GPIO25/EMAC_RXD0(RMII): track 2.31 -> 32.7 mm
- net /GPIO19/EMAC_TXD0(RMII): track 0.00 -> 29.5 mm, vias 0 -> 1
- net Spare2: track 0.00 -> 29.1 mm, vias 0 -> 1
- net Net-(ACT1-A): track 0.00 -> 26.9 mm, vias 0 -> 2
- net /5V_DCDC: track 0.00 -> 21.3 mm
- net +3.3VLAN: track 18.8 -> 37.9 mm
- net /ILIM: track 0.00 -> 15.5 mm
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- added copper zone on In1.Cu, net GND
Other:
- copper layers 4 -> 6

Commit message: updates
Parts:
- moved C27 61.9 mm to (130.2, 162.5)
- moved R22 47.7 mm to (131.3, 133.0), turned to 180 degrees
- moved R27 45.4 mm to (132.8, 137.6)
- moved R33 45.0 mm to (128.7, 152.1)
- moved C26 43.3 mm to (101.8, 162.9), turned to 180 degrees
- moved C12 42.5 mm to (124.4, 155.1)
- moved TVS3 41.4 mm to (113.4, 138.0)
- moved TVS2 38.5 mm to (108.9, 138.8), turned to 180 degrees
- moved TVS1 35.7 mm to (101.8, 134.2)
- moved C23 34.5 mm to (114.0, 158.7)
- moved R23 32.8 mm to (123.0, 144.4)
- moved C24 31.2 mm to (127.3, 151.5), turned to 180 degrees
- moved C11 24.2 mm to (104.7, 153.3), turned to -90 degrees
- moved C25 17.3 mm to (110.1, 148.6), turned to -90 degrees
- moved R34 15.5 mm to (108.7, 148.6), turned to -90 degrees
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Routing:
- net Spare2: track 29.1 -> 61.0 mm, vias 1 -> 2
- net +5VP: track 15.4 -> 42.9 mm, vias 0 -> 2
- net Net-(U5-FB): track 0.00 -> 27.1 mm, vias 0 -> 2
- net /GPIO27/EMAC_RX_CRS_DV: track 19.4 -> 46.2 mm, vias 1 -> 2
- net Net-(D5-K): track 7.39 -> 33.1 mm, vias 1 -> 4
- net /RD-: track 22.6 -> 46.3 mm, vias 0 -> 1
- net Net-(J2-RCT): track 57.6 -> 80.2 mm, vias 0 -> 1
- net GND: track 12.7 -> 35.0 mm, vias 3 -> 10
- net /TD-: track 6.12 -> 25.5 mm, vias 1 -> 2
- net Earth: track 51.5 -> 69.6 mm
- net +3.3VLAN: track 37.9 -> 51.2 mm, vias 0 -> 2
- net /TD+: track 8.86 -> 22.1 mm, vias 0 -> 1
- net Net-(U2-ILIM): track 0.00 -> 13.2 mm
- net /GPIO18/MDIO(RMII): track 19.1 -> 30.5 mm, vias 1 -> 2
- net +3V3: track 30.7 -> 42.0 mm, vias 0 -> 2
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
Commit message: updates
Parts:
- moved J3 47.4 mm to (144.3, 132.8)

Commit message: updates
Parts:
- moved C27 44.6 mm to (99.6, 130.0), turned to -130 degrees
- moved C26 17.1 mm to (98.0, 146.1), turned to -55 degrees
- moved H2 0.16 mm to (99.4, 149.6)
Routing:
- net Earth: track 69.6 -> 100.4 mm
- net Spare1: track 53.0 -> 77.2 mm
- net Net-(U2-NC/UVLO): track 7.81 -> 30.4 mm
- net /5V_DCDC: track 30.0 -> 40.7 mm
- net /GPIO25/EMAC_RXD0(RMII): track 32.7 -> 33.3 mm
Other:
- copper layers 6 -> 4

Commit message: fixing DRC
Parts:
- moved J3 41.2 mm to (111.4, 157.6)
- moved C23 4.92 mm to (118.8, 157.5)
Connections:
- J3 pad 01: unconnected-(J3-Pad01) -> +5VP
- J3 pad 02: unconnected-(J3-Pad02) -> GND
Routing:
- net +5VP: track 42.9 -> 58.5 mm
- net Earth: track 100.4 -> 95.2 mm
- net GND: track 35.0 -> 33.5 mm
- net Spare1: track 77.2 -> 78.3 mm
- net Net-(J2-RCT): track 80.2 -> 80.9 mm
- net Spare2: track 61.0 -> 61.6 mm
Other:
- board text added: "- Wireless Charger Header is under Inductor (cut off through hole legs before soldering SMD)"

Commit message: POE 1 passes
Routing:
- net Spare2: track 61.6 -> 66.1 mm, vias 2 -> 3
- net /GPIO25/EMAC_RXD0(RMII): track 33.3 -> 31.6 mm, vias 0 -> 2
- net Net-(U2-DET): track 5.25 -> 5.46 mm, vias 0 -> 2
