File: ESP32_POE_Board/1.4/ESP_POE_1.4a/ESP_POE_1.4a/ESP_POE_1.4a.kicad_sch (KiCad schematic)
At the start: 70 parts, among them J2 HMTSW-102-X-X-S-X, J25 SI-46020-F, J4 20021111-00012T4LF, J6 20021111-00012T4LF, T1 LMUN2211LT1G(SOT-23), U2 TPS2376PW(TSSOP-8), U4 LAN8710A-EZC(QFN32), U5 TX4138(ESOIC-8)

Commit message: updates
Parts:
- removed FID2, FID3, FID5, FID6: Fiducial, OLIMEX_Other-FP:Fiducial1x3, symbol ESP32-PoE-ISO_Rev_K:Fiducial
- removed MH1, MH2, MH3: Mounting_Hole_NPTH, OLIMEX_Other-FP:NPTH_2.2mm, symbol ESP32-PoE-ISO_Rev_K:Mounting_Hole_NPTH
- added H1, H2: MountingHole, MountingHole:MountingHole_2.1mm, symbol Mechanical:MountingHole
Other:
- moved on the sheet: FID1, FID4

Commit message: starting POE1 route
Parts:
- removed FID1, FID4: Fiducial, OLIMEX_Other-FP:Fiducial1x3, symbol ESP32-PoE-ISO_Rev_K:Fiducial
- added FID1, FID2, FID3, FID5: Fiducial, Fiducial:Fiducial_0.5mm_Mask1.5mm, symbol Mechanical:Fiducial
Changed lines of the file:
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@@
-    )
-  )
-  (symbol (lib_id "ESP32-PoE-ISO_Rev_K:Fiducial") (at 518.668 314.706 0) (unit 1)
-    (in_bom yes) (on_board yes) (dnp no)
-    (property "Reference" "FID1" (at 521.9192 313.5376 0)
-      (effects (font (size 1.27 1.27)) (justify left))
-    )
-    (property "Value" "Fiducial" (at 521.9192 315.849 0)
-      (effects (font (size 1.27 1.27)) (justify left))
-    )
-    (property "Footprint" "OLIMEX_Other-FP:Fiducial1x3" (at 511.302 316.611 0)
-      (effects (font (size 0.508 0.508)) hide)
-    )
-    (property "Datasheet" "" (at 517.398 314.706 90)
-      (effects (font (size 1.524 1.524)))
-    )
-    (pin "Fid1")
-    (instances
-      (project "ESP_POE_1.4a"
-        (path "/e282cc28-a468-4b1a-8ebc-006ea330625e"
-          (reference "FID1") (unit 1)
-        )
-      )
     )
   )
@@
         (path "/e282cc28-a468-4b1a-8ebc-006ea330625e"
           (reference "#PWR023") (unit 1)
-        )
-      )
-    )
-  )
-  (symbol (lib_id "ESP32-PoE-ISO_Rev_K:Fiducial") (at 518.668 324.866 0) (unit 1)
-    (in_bom yes) (on_board yes) (dnp no)
-    (property "Reference" "FID4" (at 521.9192 323.6976 0)
-      (effects (font (size 1.27 1.27)) (justify left))
-    )
-    (property "Value" "Fiducial" (at 521.9192 326.009 0)
-      (effects (font (size 1.27 1.27)) (justify left))
-    )
-    (property "Footprint" "OLIMEX_Other-FP:Fiducial1x3" (at 511.302 326.771 0)
-      (effects (font (size 0.508 0.508)) hide)
-    )
-    (property "Datasheet" "" (at 517.398 324.866 90)
-      (effects (font (size 1.524 1.524)))
-    )
-    (pin "Fid1")
-    (instances
-      (project "ESP_POE_1.4a"
-        (path "/e282cc28-a468-4b1a-8ebc-006ea330625e"
-          (reference "FID4") (unit 1)
         )
       )
@@
     )
   )
+  (symbol (lib_id "Mechanical:Fiducial") (at 523.24 322.834 0) (unit 1)
+    (in_bom yes) (on_board yes) (dnp no) (fields_autoplaced)
+    (property "Reference" "FID2" (at 525.526 321.564 0)
+      (effects (font (size 1.27 1.27)) (justify left))
+    )
+    (property "Value" "Fiducial" (at 525.526 324.104 0)
+      (effects (font (size 1.27 1.27)) (justify left))
+    )
+    (property "Footprint" "Fiducial:Fiducial_0.5mm_Mask1.5mm" (at 523.24 322.834 0)
+      (effects (font (size 1.27 1.27)) hide)
+    )
+    (property "Datasheet" "~" (at 523.24 322.834 0)
+      (effects (font (size 1.27 1.27)) hide)
+    )
+    (instances
+      (project "ESP_POE_1.4a"
+        (path "/e282cc28-a468-4b1a-8ebc-006ea330625e"
+          (reference "FID2") (unit 1)
+        )
+      )
+    )
+  )
   (symbol (lib_id "HMTSW-102-X-X-S-X:HMTSW-102-X-X-S-X") (at 213.614 264.16 0) (unit 1)
     (in_bom yes) (on_board yes) (dnp no) (fields_autoplaced)
@@
     )
   )
+  (symbol (lib_id "Mechanical:Fiducial") (at 504.19 322.326 0) (unit 1)
+    (in_bom yes) (on_board yes) (dnp no) (fields_autoplaced)
+    (property "Reference" "FID1" (at 506.476 321.056 0)
+      (effects (font (size 1.27 1.27)) (justify left))
+    )
+    (property "Value" "Fiducial" (at 506.476 323.596 0)
+      (effects (font (size 1.27 1.27)) (justify left))
+    )
+    (property "Footprint" "Fiducial:Fiducial_0.5mm_Mask1.5mm" (at 504.19 322.326 0)
+      (effects (font (size 1.27 1.27)) hide)
+    )
+    (property "Datasheet" "~" (at 504.19 322.326 0)
+      (effects (font (size 1.27 1.27)) hide)
+    )
+    (instances
+      (project "ESP_POE_1.4a"
+        (path "/e282cc28-a468-4b1a-8ebc-006ea330625e"
+          (reference "FID1") (unit 1)
+        )
+      )
+    )
+  )
   (symbol (lib_id "Mechanical:MountingHole") (at 521.208 359.41 0) (unit 1)
     (in_bom yes) (on_board yes) (dnp no) (fields_autoplaced)
@@
         (path "/e282cc28-a468-4b1a-8ebc-006ea330625e"
           (reference "H2") (unit 1)
+        )
+      )
+    )
+  )
+  (symbol (lib_id "Mechanical:Fiducial") (at 523.748 314.198 0) (unit 1)
+    (in_bom yes) (on_board yes) (dnp no) (fields_autoplaced)
+    (property "Reference" "FID3" (at 526.034 312.928 0)
+      (effects (font (size 1.27 1.27)) (justify left))
+    )
+    (property "Value" "Fiducial" (at 526.034 315.468 0)
+      (effects (font (size 1.27 1.27)) (justify left))
+    )
+    (property "Footprint" "Fiducial:Fiducial_0.5mm_Mask1.5mm" (at 523.748 314.198 0)
+      (effects (font (size 1.27 1.27)) hide)
+    )
+    (property "Datasheet" "~" (at 523.748 314.198 0)
+      (effects (font (size 1.27 1.27)) hide)
+    )
+    (instances
+      (project "ESP_POE_1.4a"
+        (path "/e282cc28-a468-4b1a-8ebc-006ea330625e"
+          (reference "FID3") (unit 1)
         )
       )
@@
         )
       )
+    )
+  )
+  (symbol (lib_id "Mechanical:Fiducial") (at 504.698 313.69 0) (unit 1)
+    (in_bom yes) (on_board yes) (dnp no) (fields_autoplaced)
+    (property "Reference" "FID5" (at 506.984 312.42 0)
+      (effects (font (size 1.27 1.27)) (justify left))
+    )
+    (property "Value" "Fiducial" (at 506.984 314.96 0)
+      (effects (font (size 1.27 1.27)) (justify left))
+    )
+    (property "Footprint" "Fiducial:Fiducial_0.5mm_Mask1.5mm" (at 504.698 313.69 0)
+      (effects (font (size 1.27 1.27)) hide)
+    )
+    (property "Datasheet" "~" (at 504.698 313.69 0)
+      (effects (font (size 1.27 1.27)) hide)
+    )
+    (instances
+      (project "ESP_POE_1.4a"
+        (path "/e282cc28-a468-4b1a-8ebc-006ea330625e"
+          (reference "FID5") (unit 1)
+        )
+      )

Commit message: fixing DRC
Connections:
- net +5VP: now also J2.01
- net GND: now also J2.02
Changed lines of the file:
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@@
     (stroke (width 0) (type default))
   )
+  (wire (pts (xy 199.644 259.588) (xy 199.644 264.16))
+    (stroke (width 0) (type default))
+  )
   (wire (pts (xy 148.844 112.522) (xy 156.464 112.522))
     (stroke (width 0) (type default))
@@
     (stroke (width 0) (type default))
   )
+  (wire (pts (xy 199.644 266.7) (xy 203.454 266.7))
+    (stroke (width 0) (type default))
+  )
   (wire (pts (xy 194.564 143.002) (xy 199.644 143.002))
     (stroke (width 0) (type default))
@@
     (stroke (width 0) (type default))
   )
+  (wire (pts (xy 199.644 264.16) (xy 203.454 264.16))
+    (stroke (width 0) (type default))
+  )
   (wire (pts (xy 336.804 150.622) (xy 336.804 145.542))
     (stroke (width 0) (type default))
@@
     (stroke (width 0) (type default))
   )
+  (wire (pts (xy 199.644 271.78) (xy 199.644 266.7))
+    (stroke (width 0) (type default))
+  )
   (wire (pts (xy 291.084 145.542) (xy 291.084 137.922))
     (stroke (width 0) (type default))
@@
     (fill (type none))
   )
-  (rectangle (start 141.478 246.126) (end 253.492 289.052)
+  (rectangle (start 170.434 246.126) (end 253.492 289.052)
     (stroke (width 0) (type default))
     (fill (type none))
@@
     (effects (font (size 0.762 0.762)) (justify right bottom))
   )
-  (text "Wireless Charger" (at 141.478 243.586 0)
+  (text "Wireless Charger" (at 169.672 241.808 0)
     (effects (font (size 5.08 5.08) (thickness 1.016) bold italic) (justify left bottom))
   )
@@
     )
   )
-  (symbol (lib_id "ESP32-PoE_Rev_L1-rescue:GND-ESP32-PoE_Rev_L1") (at 149.352 275.59 0) (unit 1)
+  (symbol (lib_id "ESP32-PoE_Rev_L1-rescue:GND-ESP32-PoE_Rev_L1") (at 199.644 271.78 0) (unit 1)
     (in_bom yes) (on_board yes) (dnp no)
-    (property "Reference" "#PWR07" (at 149.352 281.94 0)
+    (property "Reference" "#PWR07" (at 199.644 278.13 0)
       (effects (font (size 1.27 1.27)) hide)
     )
-    (property "Value" "GND" (at 149.352 279.4 0)
+    (property "Value" "GND" (at 199.644 275.59 0)
       (effects (font (size 1.27 1.27)))
     )
-    (property "Footprint" "" (at 149.352 275.59 0)
+    (property "Footprint" "" (at 199.644 271.78 0)
       (effects (font (size 1.524 1.524)))
     )
-    (property "Datasheet" "" (at 149.352 275.59 0)
+    (property "Datasheet" "" (at 199.644 271.78 0)
       (effects (font (size 1.524 1.524)))
     )
@@
     )
   )
-  (symbol (lib_id "ESP32-PoE_Rev_L1-rescue:+5VP-ESP32-PoE_Rev_L1") (at 149.352 255.27 0) (unit 1)
+  (symbol (lib_id "ESP32-PoE_Rev_L1-rescue:+5VP-ESP32-PoE_Rev_L1") (at 199.644 259.588 0) (unit 1)
     (in_bom yes) (on_board yes) (dnp no)
-    (property "Reference" "#PWR05" (at 149.352 259.08 0)
+    (property "Reference" "#PWR05" (at 199.644 263.398 0)
       (effects (font (size 1.27 1.27)) hide)
     )
-    (property "Value" "+5VP" (at 149.733 250.8758 0)
+    (property "Value" "+5VP" (at 200.025 255.1938 0)
       (effects (font (size 1.27 1.27)))
     )
-    (property "Footprint" "" (at 149.352 255.27 0)
+    (property "Footprint" "" (at 199.644 259.588 0)
       (effects (font (size 1.524 1.524)))
     )
-    (property "Datasheet" "" (at 149.352 255.27 0)
+    (property "Datasheet" "" (at 199.644 259.588 0)
       (effects (font (size 1.524 1.524)))
     )

Commit message: POE 1 passes
Connections:
- no-connect marks 6 -> 11
Changed lines of the file:
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@@
   (no_connect (at 194.564 112.522))
   (no_connect (at 357.124 153.162))
+  (no_connect (at 297.18 335.026))
   (no_connect (at 194.564 115.062))
   (no_connect (at 194.564 130.302))
   (no_connect (at 194.564 150.622))
   (no_connect (at 164.084 137.922))
+  (no_connect (at 69.342 170.942))
+  (no_connect (at 69.342 168.402))
+  (no_connect (at 69.342 163.322))
+  (no_connect (at 69.342 165.862))
   (wire (pts (xy 352.044 145.542) (xy 352.044 143.002))
     (stroke (width 0) (type default))

Commit message: 1.4a half bom
Parts:
- ACT1: Mfr (none) -> Everlight Elec; Mfr P/N (none) -> 19-21/Y2C-CP1Q2B/4T; Price (none) -> 0.0328; Purchase-URL (none) -> https://www.lcsc.com/product-detail/span-style-background-c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; Supplier 1 (none) -> LCSC; Supplier 1 P/N (none) -> C2986008
- C10, C13, C19, C9: Mfr (none) -> Samsung Electro-Mechanics; Mfr P/N (none) -> CL10A226MP8NUNE; Price (none) -> 0.0123; Purchase-URL (none) -> https://www.lcsc.com/product-detail/Multilayer-Ceramic-Capa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; Supplier 1 (none) -> LCSC; Supplier 1 P/N (none) -> C86295
- C11, C14, C15, C16, C18: Mfr (none) -> YAGEO; Mfr P/N (none) -> CC0402KRX7R7BB104; Price (none) -> 0.0009; Purchase-URL (none) -> https://www.lcsc.com/product-detail/Multilayer-Ceramic-Capa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; Supplier 1 (none) -> LCSC; Supplier 1 P/N (none) -> C60474
- C12, C24: Mfr (none) -> YAGEO; Mfr P/N (none) -> CC0603KRX7R9BB104; Price (none) -> 0.0020; Purchase-URL (none) -> https://www.lcsc.com/product-detail/Multilayer-Ceramic-Capa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; Supplier 1 (none) -> LCSC; Supplier 1 P/N (none) -> C14663
- C17: Mfr (none) -> Samwha Capacitor; Mfr P/N (none) -> CS1608X5R225K100NRB; Price (none) -> 0.0047; Purchase-URL (none) -> https://www.lcsc.com/product-detail/Multilayer-Ceramic-Capa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; Supplier 1 (none) -> LCSC; Supplier 1 P/N (none) -> C5189830
- C2: Mfr (none) -> YAGEO; Mfr P/N (none) -> CC1206MKX7RDBB102; Price (none) -> 0.0142; Purchase-URL (none) -> https://www.lcsc.com/product-detail/Multilayer-Ceramic-Capa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; Supplier 1 (none) -> LCSC; Supplier 1 P/N (none) -> C527363
- C20: value NA(1.0nF/3kV/10%/X7R/SMD/1808(VISHAY-VJ1808Y102KBHAT4X_Farnell-2407291)) -> 1.0nF/3kV/10%/X7R/SMD/1808(VISHAY-VJ1808Y102KBHAT4X_Farnell-2407291); Mfr (none) -> IHHEC(HOLY STONE ENTERPRISE CO., LTD); Mfr P/N (none) -> SCC1808X102K502TS; Price (none) -> 0.1511; Purchase-URL (none) -> https://www.lcsc.com/product-detail/Safety-Capacitors_IHHEC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; Supplier 1 (none) -> LCSC; Supplier 1 P/N (none) -> C2939745
- C21: Mfr (none) -> Samsung Electro-Mechanics; Mfr P/N (none) -> CL10A106MA8NRNC; Price (none) -> 0.0166; Purchase-URL (none) -> https://www.lcsc.com/product-detail/Multilayer-Ceramic-Capa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; Supplier 1 (none) -> LCSC; Supplier 1 P/N (none) -> C96446
- C23: Mfr (none) -> IHHEC(HOLY STONE ENTERPRISE CO., LTD); Mfr P/N (none) -> SCC1808X102K502TS; Price (none) -> 0.1511; Purchase-URL (none) -> https://www.lcsc.com/product-detail/Safety-Capacitors_IHHEC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; Supplier 1 (none) -> LCSC; Supplier 1 P/N (none) -> C2939745
- C25: Mfr (none) -> Samsung Electro-Mechanics; Mfr P/N (none) -> CL05C120JB51PNC; Price (none) -> 0.0056; Purchase-URL (none) -> https://www.lcsc.com/product-detail/Multilayer-Ceramic-Capa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; Supplier 1 (none) -> LCSC; Supplier 1 P/N (none) -> C472446
- C26: Mfr (none) -> CX(Dongguan Chengxing Elec); Mfr P/N (none) -> GR477M016E12RR0EH4FP0; Price (none) -> 0.0285; Purchase-URL (none) -> https://www.lcsc.com/product-detail/Aluminum-Electrolytic-C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; Supplier 1 (none) -> LCSC; Supplier 1 P/N (none) -> C3039776
- C27: Mfr (none) -> Yunxing; Mfr P/N (none) -> EG22GM150F16OTMO; Price (none) -> 0.0995; Purchase-URL (none) -> https://www.lcsc.com/product-detail/Aluminum-Electrolytic-C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; Supplier 1 (none) -> LCSC; Supplier 1 P/N (none) -> C2841644
- D10: Mfr (none) -> STMicroelectronics; Mfr P/N (none) -> SMAJ58A-TR; Price (none) -> 0.1450; Purchase-URL (none) -> https://www.lcsc.com/product-detail/ESD-and-Surge-Protectio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; Supplier 1 (none) -> LCSC; Supplier 1 P/N (none) -> C132936
- D5: Mfr (none) -> Yangzhou Yangjie Elec Tech; Mfr P/N (none) -> SS510; Price (none) -> 0.0875; Purchase-URL (none) -> https://www.lcsc.com/product-detail/Schottky-Diodes_Yangzho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; Supplier 1 (none) -> LCSC; Supplier 1 P/N (none) -> C5339843
- DCDC1: Mfr (none) -> EVISUN; Mfr P/N (none) -> F0505S-2WR3; Price (none) -> 1.3296; Purchase-URL (none) -> https://www.lcsc.com/product-detail/Isolated-Power-Modules_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; Supplier 1 (none) -> LCSC; Supplier 1 P/N (none) -> C7465184
- FET3: Mfr (none) -> TECH PUBLIC; Mfr P/N (none) -> WPM2015-3/TR; Price (none) -> 0.0378; Purchase-URL (none) -> https://www.lcsc.com/product-detail/MOSFETs_TECH-PUBLIC-WPM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; Supplier 1 (none) -> LCSC; Supplier 1 P/N (none) -> C7472861
- J2: Mfr (none) -> Samtec; Mfr P/N (none) -> HTSW-102-23-G-S; Price None -> 0.2942; Purchase-URL (none) -> https://www.lcsc.com/product-detail/Pin-Headers_Samtec-HTSW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; Supplier 1 (none) -> LCSC; Supplier 1 P/N (none) -> C7204532
- J25: Mfr (none) -> Bel Fuse Inc.; Mfr P/N (none) -> SI-46020-F; Price None -> 6.40000; Purchase-URL https://www.snapeda.com/api/url_track_click_mouser/?unipart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 -> https://www.digikey.com/en/products/detail/bel-fuse-inc/SI-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; Supplier 1 (none) -> Digikey; Supplier 1 P/N (none) -> 507-SI-46020-F-ND
- J4, J6: Mfr (none) -> DEALON; Mfr P/N (none) -> DZ127R-11-09-25; Price (none) -> 0.0343; Purchase-URL (none) -> https://www.lcsc.com/product-detail/Pin-Headers_DEALON-DZ12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; Supplier 1 (none) -> LCSC; Supplier 1 P/N (none) -> C2935949
- L1: Mfr (none) -> BOURNS; Mfr P/N (none) -> MH2029-601Y; Price (none) -> 0.0451; Purchase-URL (none) -> https://www.lcsc.com/product-detail/Ferrite-Beads_BOURNS-MH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; Supplier 1 (none) -> LCSC; Supplier 1 P/N (none) -> C840592; note (none) -> the max current is 1A here
- L4: footprint OLIMEX_RLC-FP:DBS135 -> SRR1240-330M:IND_BOURNS_SRR1240; Mfr (none) -> Bourns Inc.; Mfr P/N (none) -> SRR1240-330M; Price (none) -> 1.15000; Purchase-URL (none) -> https://www.digikey.com/en/products/detail/bourns-inc/SRR12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; Supplier 1 (none) -> Digikey; Supplier 1 P/N (none) -> 118-SRR1240-330MCT-ND; note (none) -> i changed to a diff
- LNK1: Mfr (none) -> Everlight Elec; Mfr P/N (none) -> 18-225/R6G6C-A01/3T; Price (none) -> 0.0772; Purchase-URL (none) -> https://www.lcsc.com/product-detail/LED-Indication-Discrete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; Supplier 1 (none) -> LCSC; Supplier 1 P/N (none) -> C172883
