File: ESP32_POE_Board/1.4/ESP_POE_1.4a/ESP_POE_1.4a/ESP_POE_1.4a.kicad_sch (KiCad schematic)
At the start: 67 parts, among them J2 HMTSW-102-X-X-S-X, J25 SI-46020-F, J4 20021111-00012T4LF, J6 20021111-00012T4LF, T1 LMUN2211LT1G(SOT-23), U2 TPS2376PW(TSSOP-8), U4 LAN8710A-EZC(QFN32), U5 TX4138(ESOIC-8)

Commit message: some bom
Parts:
- R10, R11, R12, R13: Mfr (none) -> YAGEO; Mfr P/N (none) -> RC0402FR-0749R9P; Price (none) -> 0.0050; Purchase-URL (none) -> https://www.lcsc.com/product-detail/Chip-span-style-backgro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; Supplier 1 (none) -> LCSC; Supplier 1 P/N (none) -> C851839
- R14, R15: Mfr (none) -> YAGEO; Mfr P/N (none) -> AC0402JR-072K2L; Price (none) -> 0.0008; Purchase-URL (none) -> https://www.lcsc.com/product-detail/Chip-span-style-backgro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; Supplier 1 (none) -> LCSC; Supplier 1 P/N (none) -> C144718
- R2, R25, R44: Mfr (none) -> YAGEO; Mfr P/N (none) -> RC0402FR-0710KL; Price (none) -> 0.0005; Purchase-URL (none) -> https://www.lcsc.com/product-detail/Chip-span-style-backgro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; Supplier 1 (none) -> LCSC; Supplier 1 P/N (none) -> C60490
- R3: Mfr (none) -> YAGEO; Mfr P/N (none) -> RC0402FR-071KL; Price (none) -> 0.0006; Purchase-URL (none) -> https://www.lcsc.com/product-detail/Chip-span-style-backgro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; Supplier 1 (none) -> LCSC; Supplier 1 P/N (none) -> C106235
Changed lines of the file:
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@@
       (effects (font (size 1.27 1.27)) hide)
     )
+    (property "Mfr" "YAGEO" (at 145.034 150.622 0)
+      (effects (font (size 1.27 1.27)) hide)
+    )
+    (property "Mfr P/N" "AC0402JR-072K2L" (at 145.034 150.622 0)
+      (effects (font (size 1.27 1.27)) hide)
+    )
+    (property "Price" "0.0008" (at 145.034 150.622 0)
+      (effects (font (size 1.27 1.27)) hide)
+    )
+    (property "Purchase-URL" "https://www.lcsc.com/product-detail/Chip-span-style-background-color-ff0-Resistor-span-Surface-Mount_YAGEO-AC0402JR-072K2L_C144718.html" (at 145.034 150.622 0)
+      (effects (font (size 1.27 1.27)) hide)
+    )
+    (property "Supplier 1" "LCSC" (at 145.034 150.622 0)
+      (effects (font (size 1.27 1.27)) hide)
+    )
+    (property "Supplier 1 P/N" "C144718" (at 145.034 150.622 0)
+      (effects (font (size 1.27 1.27)) hide)
+    )
     (pin "1")
     (pin "2")
@@
       (effects (font (size 1.27 1.27)) hide)
     )
+    (property "Mfr" "YAGEO" (at 125.984 121.412 0)
+      (effects (font (size 1.27 1.27)) hide)
+    )
+    (property "Mfr P/N" "RC0402FR-0749R9P" (at 125.984 121.412 0)
+      (effects (font (size 1.27 1.27)) hide)
+    )
+    (property "Price" "0.0050" (at 125.984 121.412 0)
+      (effects (font (size 1.27 1.27)) hide)
+    )
+    (property "Purchase-URL" "https://www.lcsc.com/product-detail/Chip-span-style-background-color-ff0-Resistor-span-Surface-Mount_YAGEO-RC0402FR-0749R9P_C851839.html" (at 125.984 121.412 0)
+      (effects (font (size 1.27 1.27)) hide)
+    )
+    (property "Supplier 1" "LCSC" (at 125.984 121.412 0)
+      (effects (font (size 1.27 1.27)) hide)
+    )
+    (property "Supplier 1 P/N" "C851839" (at 125.984 121.412 0)
+      (effects (font (size 1.27 1.27)) hide)
+    )
     (pin "1")
     (pin "2")
@@
       (effects (font (size 1.27 1.27)) hide)
     )
+    (property "Mfr" "YAGEO" (at 128.524 121.412 0)
+      (effects (font (size 1.27 1.27)) hide)
+    )
+    (property "Mfr P/N" "RC0402FR-0749R9P" (at 128.524 121.412 0)
+      (effects (font (size 1.27 1.27)) hide)
+    )
+    (property "Price" "0.0050" (at 128.524 121.412 0)
+      (effects (font (size 1.27 1.27)) hide)
+    )
+    (property "Purchase-URL" "https://www.lcsc.com/product-detail/Chip-span-style-background-color-ff0-Resistor-span-Surface-Mount_YAGEO-RC0402FR-0749R9P_C851839.html" (at 128.524 121.412 0)
+      (effects (font (size 1.27 1.27)) hide)
+    )
+    (property "Supplier 1" "LCSC" (at 128.524 121.412 0)
+      (effects (font (size 1.27 1.27)) hide)
+    )
+    (property "Supplier 1 P/N" "C851839" (at 128.524 121.412 0)
+      (effects (font (size 1.27 1.27)) hide)
+    )
     (pin "1")
     (pin "2")
@@
       (effects (font (size 1.27 1.27)) hide)
     )
+    (property "Mfr" "YAGEO" (at 131.064 121.412 0)
+      (effects (font (size 1.27 1.27)) hide)
+    )
+    (property "Mfr P/N" "RC0402FR-0749R9P" (at 131.064 121.412 0)
+      (effects (font (size 1.27 1.27)) hide)
+    )
+    (property "Price" "0.0050" (at 131.064 121.412 0)
+      (effects (font (size 1.27 1.27)) hide)
+    )
+    (property "Purchase-URL" "https://www.lcsc.com/product-detail/Chip-span-style-background-color-ff0-Resistor-span-Surface-Mount_YAGEO-RC0402FR-0749R9P_C851839.html" (at 131.064 121.412 0)
+      (effects (font (size 1.27 1.27)) hide)
+    )
+    (property "Supplier 1" "LCSC" (at 131.064 121.412 0)
+      (effects (font (size 1.27 1.27)) hide)
+    )
+    (property "Supplier 1 P/N" "C851839" (at 131.064 121.412 0)
+      (effects (font (size 1.27 1.27)) hide)
+    )
     (pin "1")
     (pin "2")
@@
       (effects (font (size 1.27 1.27)) hide)
     )
+    (property "Mfr" "YAGEO" (at 133.604 121.412 0)
+      (effects (font (size 1.27 1.27)) hide)
+    )
+    (property "Mfr P/N" "RC0402FR-0749R9P" (at 133.604 121.412 0)
+      (effects (font (size 1.27 1.27)) hide)
+    )
+    (property "Price" "0.0050" (at 133.604 121.412 0)
+      (effects (font (size 1.27 1.27)) hide)
+    )
+    (property "Purchase-URL" "https://www.lcsc.com/product-detail/Chip-span-style-background-color-ff0-Resistor-span-Surface-Mount_YAGEO-RC0402FR-0749R9P_C851839.html" (at 133.604 121.412 0)
+      (effects (font (size 1.27 1.27)) hide)
+    )
+    (property "Supplier 1" "LCSC" (at 133.604 121.412 0)
+      (effects (font (size 1.27 1.27)) hide)
+    )
+    (property "Supplier 1 P/N" "C851839" (at 133.604 121.412 0)
+      (effects (font (size 1.27 1.27)) hide)
+    )
     (pin "1")
     (pin "2")
@@
       (effects (font (size 1.27 1.27)) hide)
     )
+    (property "Mfr" "YAGEO" (at 136.144 172.212 0)
+      (effects (font (size 1.27 1.27)) hide)
+    )
+    (property "Mfr P/N" "AC0402JR-072K2L" (at 136.144 172.212 0)
+      (effects (font (size 1.27 1.27)) hide)
+    )
+    (property "Price" "0.0008" (at 136.144 172.212 0)
+      (effects (font (size 1.27 1.27)) hide)
+    )
+    (property "Purchase-URL" "https://www.lcsc.com/product-detail/Chip-span-style-background-color-ff0-Resistor-span-Surface-Mount_YAGEO-AC0402JR-072K2L_C144718.html" (at 136.144 172.212 0)
+      (effects (font (size 1.27 1.27)) hide)
+    )
+    (property "Supplier 1" "LCSC" (at 136.144 172.212 0)
+      (effects (font (size 1.27 1.27)) hide)
+    )
+    (property "Supplier 1 P/N" "C144718" (at 136.144 172.212 0)
+      (effects (font (size 1.27 1.27)) hide)
+    )
     (pin "1")
     (pin "2")
@@
       (effects (font (size 1.27 1.27)) hide)
     )
+    (property "Mfr" "YAGEO" (at 213.614 160.782 0)
+      (effects (font (size 1.27 1.27)) hide)
+    )
+    (property "Mfr P/N" "RC0402FR-0710KL" (at 213.614 160.782 0)
+      (effects (font (size 1.27 1.27)) hide)
+    )
+    (property "Price" "0.0005" (at 213.614 160.782 0)
+      (effects (font (size 1.27 1.27)) hide)
+    )
+    (property "Purchase-URL" "https://www.lcsc.com/product-detail/Chip-span-style-background-color-ff0-Resistor-span-Surface-Mount_YAGEO-RC0402FR-0710KL_C60490.html" (at 213.614 160.782 0)
+      (effects (font (size 1.27 1.27)) hide)
+    )
+    (property "Supplier 1" "LCSC" (at 213.614 160.782 0)
+      (effects (font (size 1.27 1.27)) hide)
+    )
+    (property "Supplier 1 P/N" "C60490" (at 213.614 160.782 0)
+      (effects (font (size 1.27 1.27)) hide)
+    )
     (pin "1")
     (pin "2")
@@
       (effects (font (size 1.27 1.27)) hide)
     )
+    (property "Mfr" "YAGEO" (at 57.404 106.172 0)
+      (effects (font (size 1.27 1.27)) hide)
+    )
+    (property "Mfr P/N" "RC0402FR-071KL" (at 57.404 106.172 0)
+      (effects (font (size 1.27 1.27)) hide)
+    )
+    (property "Price" "0.0006" (at 57.404 106.172 0)
+      (effects (font (size 1.27 1.27)) hide)
+    )
+    (property "Purchase-URL" "https://www.lcsc.com/product-detail/Chip-span-style-background-color-ff0-Resistor-span-Surface-Mount_YAGEO-RC0402FR-071KL_C106235.html" (at 57.404 106.172 0)
+      (effects (font (size 1.27 1.27)) hide)
+    )
+    (property "Supplier 1" "LCSC" (at 57.404 106.172 0)
+      (effects (font (size 1.27 1.27)) hide)
+    )
+    (property "Supplier 1 P/N" "C106235" (at 57.404 106.172 0)
+      (effects (font (size 1.27 1.27)) hide)
+    )
     (pin "1")
     (pin "2")
@@
       (effects (font (size 1.27 1.27)) hide)
     )
+    (property "Mfr" "YAGEO" (at 49.784 88.392 0)
+      (effects (font (size 1.27 1.27)) hide)
+    )
+    (property "Mfr P/N" "RC0402FR-0710KL" (at 49.784 88.392 0)
+      (effects (font (size 1.27 1.27)) hide)
+    )
+    (property "Price" "0.0005" (at 49.784 88.392 0)
+      (effects (font (size 1.27 1.27)) hide)
+    )
+    (property "Purchase-URL" "https://www.lcsc.com/product-detail/Chip-span-style-background-color-ff0-Resistor-span-Surface-Mount_YAGEO-RC0402FR-0710KL_C60490.html" (at 49.784 88.392 0)
+      (effects (font (size 1.27 1.27)) hide)
+    )
+    (property "Supplier 1" "LCSC" (at 49.784 88.392 0)
+      (effects (font (size 1.27 1.27)) hide)
+    )
+    (property "Supplier 1 P/N" "C60490" (at 49.784 88.392 0)
+      (effects (font (size 1.27 1.27)) hide)
+    )
     (pin "1")
     (pin "2")
@@
       (effects (font (size 1.27 1.27)) hide)
     )
+    (property "Mfr" "YAGEO" (at 296.164 184.912 0)
+      (effects (font (size 1.27 1.27)) hide)
+    )
+    (property "Mfr P/N" "RC0402FR-0710KL" (at 296.164 184.912 0)
+      (effects (font (size 1.27 1.27)) hide)
+    )
+    (property "Price" "0.0005" (at 296.164 184.912 0)
+      (effects (font (size 1.27 1.27)) hide)
+    )
+    (property "Purchase-URL" "https://www.lcsc.com/product-detail/Chip-span-style-background-color-ff0-Resistor-span-Surface-Mount_YAGEO-RC0402FR-0710KL_C60490.html" (at 296.164 184.912 0)
+      (effects (font (size 1.27 1.27)) hide)
+    )
+    (property "Supplier 1" "LCSC" (at 296.164 184.912 0)
+      (effects (font (size 1.27 1.27)) hide)
+    )
+    (property "Supplier 1 P/N" "C60490" (at 296.164 184.912 0)
+      (effects (font (size 1.27 1.27)) hide)
+    )

Commit message: bom
Parts:
- DCDC1: Mfr P/N F0505S-2WR3 -> EVISUN F0505S-3WR2; Price 1.3296 -> 1.7214; Purchase-URL https://www.lcsc.com/product-detail/Isolated-Power-Modules_EVISUN-F0505S-2WR3_C7465184.html -> https://www.lcsc.com/product-detail/Isolated-Power-Modules_EVISUN-F0505S-3WR2_C7598643.html; Supplier 1 P/N C7465184 -> C7598643
- FET3: Mfr TECH PUBLIC -> KUU; Price 0.0378 -> 0.036; Purchase-URL https://www.lcsc.com/product-detail/MOSFETs_TECH-PUBLIC-WPM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 -> https://www.lcsc.com/product-detail/MOSFETs_span-style-back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; Supplier 1 P/N C7472861 -> C6562215
- J2: Mfr Samtec -> MOLEX; Mfr P/N HTSW-102-23-G-S -> 22284020; Price 0.2942 -> 0.0526; Purchase-URL https://www.lcsc.com/product-detail/Pin-Headers_Samtec-HTSW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 -> https://www.lcsc.com/product-detail/Pin-Headers_MOLEX-22284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; Supplier 1 P/N C7204532 -> C234182
- J4, J6: value 20021111-00012T4LF -> C3324132; Supplier 1 P/N C2935949 -> C3324132
- L1: Mfr BOURNS -> Murata Electronics; Mfr P/N MH2029-601Y -> BLM21SP601SZ1D; Price 0.0451 -> 0.2178; Purchase-URL https://www.lcsc.com/product-detail/Ferrite-Beads_BOURNS-MH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 -> https://www.lcsc.com/product-detail/span-style-background-c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; Supplier 1 P/N C840592 -> C2661781
- R22: Mfr (none) -> YAGEO; Mfr P/N (none) -> RT0402BRD0724K9L; Price (none) -> 0.0207; Purchase-URL (none) -> https://www.lcsc.com/product-detail/Chip-span-style-backgro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; Supplier 1 (none) -> LCSC; Supplier 1 P/N (none) -> C852664
- R23: Mfr (none) -> YAGEO; Mfr P/N (none) -> AC0402FR-07180KL; Price (none) -> 0.0010; Purchase-URL (none) -> https://www.lcsc.com/product-detail/Chip-span-style-backgro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; Supplier 1 (none) -> LCSC; Supplier 1 P/N (none) -> C144794
- R26: Mfr (none) -> YAGEO; Mfr P/N (none) -> RT0402BRD0712K1L; Price (none) -> 0.0204; Purchase-URL (none) -> https://www.lcsc.com/product-detail/Chip-span-style-backgro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; Supplier 1 (none) -> LCSC; Supplier 1 P/N (none) -> C281773
- R27: Mfr (none) -> YAGEO; Mfr P/N (none) -> RT0402BRD074K42L; Price (none) -> 0.0172; Purchase-URL (none) -> https://www.lcsc.com/product-detail/Chip-span-style-backgro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; Supplier 1 (none) -> LCSC; Supplier 1 P/N (none) -> C513571
- R28: Mfr (none) -> YAGEO; Mfr P/N (none) -> RL1206FR-070R03L; Price (none) -> 0.0121; Purchase-URL (none) -> https://www.lcsc.com/product-detail/Current-Sense-Resistors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; Supplier 1 (none) -> LCSC; Supplier 1 P/N (none) -> C375524
- R33: Mfr (none) -> YAGEO; Mfr P/N (none) -> RC0402FR-074R7L; Price (none) -> 0.0013; Purchase-URL (none) -> https://www.lcsc.com/product-detail/Chip-span-style-backgro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; Supplier 1 (none) -> LCSC; Supplier 1 P/N (none) -> C137962
- R34: Mfr (none) -> YAGEO; Mfr P/N (none) -> RC0402FR-0710K5L; Price (none) -> 0.0006; Purchase-URL (none) -> https://www.lcsc.com/product-detail/Chip-span-style-backgro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; Supplier 1 (none) -> LCSC; Supplier 1 P/N (none) -> C171695
- R38: Mfr (none) -> YAGEO; Mfr P/N (none) -> AC0402FR-0756K2L; Price (none) -> 0.0011; Purchase-URL (none) -> https://www.lcsc.com/product-detail/Chip-span-style-backgro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; Supplier 1 (none) -> LCSC; Supplier 1 P/N (none) -> C227142
- R41: Mfr (none) -> YAGEO; Mfr P/N (none) -> RC2512FK-074K7L; Price (none) -> 0.0362; Purchase-URL (none) -> https://www.lcsc.com/product-detail/Chip-span-style-backgro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; Supplier 1 (none) -> LCSC; Supplier 1 P/N (none) -> C163339
- R43: Mfr (none) -> YAGEO; Mfr P/N (none) -> RT0402BRD07130KL; Price (none) -> 0.0195; Purchase-URL (none) -> https://www.lcsc.com/product-detail/Chip-span-style-backgro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; Supplier 1 (none) -> LCSC; Supplier 1 P/N (none) -> C852515
- RM1, RM2: Mfr (none) -> UNI-ROYAL(Uniroyal Elec); Mfr P/N (none) -> 4D03WGJ0222T5E; Price (none) -> 0.0049; Purchase-URL (none) -> https://www.lcsc.com/product-detail/Resistor-Networks-Array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; Supplier 1 (none) -> LCSC; Supplier 1 P/N (none) -> C12001
- T1: Mfr (none) -> LRC; Mfr P/N (none) -> LMUN2211LT1G; Price (none) -> 0.0153; Purchase-URL (none) -> https://www.lcsc.com/product-detail/Digital-Transistors_LRC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; Supplier 1 (none) -> LCSC; Supplier 1 P/N (none) -> C12775
- TVS1: Mfr (none) -> Texas Instruments; Mfr P/N (none) -> ESDS314DBVR; Price (none) -> 0.2597; Purchase-URL (none) -> https://www.lcsc.com/product-detail/span-style-background-c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; Supplier 1 (none) -> LCSC; Supplier 1 P/N (none) -> C1847859
- U2: Mfr (none) -> Texas Instruments; Mfr P/N (none) -> TPS2376DDAR-H; Price (none) -> 0.6501; Purchase-URL (none) -> https://www.lcsc.com/product-detail/Power-Over-Ethernet-PoE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; Supplier 1 (none) -> LCSC; Supplier 1 P/N (none) -> C544899; note (none) -> we use the thermal pad version
- U4: Mfr (none) -> Microchip Tech; Mfr P/N (none) -> LAN8710A-EZC-TR; Price (none) -> 0.8993; Purchase-URL (none) -> https://www.lcsc.com/product-detail/Ethernet-Transceivers_M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; Supplier 1 (none) -> LCSC; Supplier 1 P/N (none) -> C46185
- U5: Mfr (none) -> XDS; Mfr P/N (none) -> TX4138; Price (none) -> 0.7668; Purchase-URL (none) -> https://www.lcsc.com/product-detail/DC-DC-Converters_XDS-TX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; Supplier 1 (none) -> LCSC; Supplier 1 P/N (none) -> C329267
