File: ESP32_POE_Board/1.4/ESP_POE_1.4a/ESP_POE_1.4a/ESP_POE_1.4a.kicad_sch (KiCad schematic)
At the start: 67 parts, among them J2 HMTSW-102-X-X-S-X, J25 SI-46020-F, J4 C3324132, J6 C3324132, T1 LMUN2211LT1G(SOT-23), U2 TPS2376PW(TSSOP-8), U4 LAN8710A-EZC(QFN32), U5 TX4138(ESOIC-8)

Commit message: s
Parts:
- T1: Mfr P/N LMUN2211LT1G -> S-LMUN2211LT1G; Price 0.0153 -> 0.0207; Purchase-URL https://www.lcsc.com/product-detail/Digital-Transistors_LRC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 -> https://cart.jlcpcb.com/smt-order/?pcbFileNo=f241306b48734e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; Supplier 1 P/N C12775 -> C5383045
Changed lines of the file:
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@@
       (effects (font (size 1.27 1.27)) hide)
     )
-    (property "Mfr P/N" "LMUN2211LT1G" (at 59.944 120.142 0)
+    (property "Mfr P/N" "S-LMUN2211LT1G" (at 59.944 120.142 0)
       (effects (font (size 1.27 1.27)) hide)
     )
-    (property "Price" "0.0153" (at 59.944 120.142 0)
+    (property "Price" "0.0207" (at 59.944 120.142 0)
       (effects (font (size 1.27 1.27)) hide)
     )
-    (property "Purchase-URL" "https://www.lcsc.com/product-detail/Digital-Transistors_LRC-LMUN2211LT1G_C12775.html" (at 59.944 120.142 0)
+    (property "Purchase-URL" "https://cart.jlcpcb.com/smt-order/?pcbFileNo=f241306b48734ea2ba9ef64a0df69072" (at 59.944 120.142 0)
       (effects (font (size 1.27 1.27)) hide)
     )
@@
       (effects (font (size 1.27 1.27)) hide)
     )
-    (property "Supplier 1 P/N" "C12775" (at 59.944 120.142 0)
+    (property "Supplier 1 P/N" "C5383045" (at 59.944 120.142 0)
       (effects (font (size 1.27 1.27)) hide)
     )

Commit message: all
Parts:
- C13: Supplier 1 LCSC -> Digikey; Supplier 1 P/N C86295 -> 1276-1274-1-ND; note (none) -> Solder later
- D5: Price 0.0875 -> 0.11000; Purchase-URL https://www.lcsc.com/product-detail/Schottky-Diodes_Yangzho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 -> https://www.digikey.com/en/products/detail/shenzhen-slkormi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; Supplier 1 LCSC -> Digikey; Supplier 1 P/N C5339843 -> 5399-SS510CT-ND; note (none) -> Solder later
- J4, J6: Mfr DEALON -> Amphenol ICC (FCI); Mfr P/N DZ127R-11-09-25 -> 20021111-00012T4LF; Price 0.0343 -> 1.16000; Purchase-URL https://www.lcsc.com/product-detail/Pin-Headers_DEALON-DZ12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 -> https://www.digikey.com/en/products/detail/amphenol-cs-fci/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; Supplier 1 LCSC -> Digikey; Supplier 1 P/N C3324132 -> 609-3713-ND
- LNK1: Mfr Everlight Elec -> Lite-On; Mfr P/N 18-225/R6G6C-A01/3T -> LTST-C190KGKT; Price 0.0772 -> 0.014; Purchase-URL https://www.lcsc.com/product-detail/LED-Indication-Discrete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 -> https://www.lcsc.com/product-detail/span-style-background-c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; Supplier 1 P/N C172883 -> C125094
- U2: Mfr P/N TPS2376DDAR-H -> TPS2376PWR; Price 0.6501 -> 2.87000; Purchase-URL https://www.lcsc.com/product-detail/Power-Over-Ethernet-PoE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 -> https://www.digikey.com/en/products/detail/texas-instrument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; Supplier 1 LCSC -> Digikey; Supplier 1 P/N C544899 -> 296-43734-1-ND; note we use the thermal pad version -> solder later
Changed lines of the file:
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@@
       (effects (font (size 1.27 1.27)) hide)
     )
-    (property "Supplier 1" "LCSC" (at 138.684 117.602 0)
+    (property "Supplier 1" "Digikey" (at 138.684 117.602 0)
       (effects (font (size 1.27 1.27)) hide)
     )
-    (property "Supplier 1 P/N" "C86295" (at 138.684 117.602 0)
+    (property "Supplier 1 P/N" "1276-1274-1-ND" (at 138.684 117.602 0)
       (effects (font (size 1.27 1.27)) hide)
     )
-    (property "note" "" (at 138.684 117.602 0)
+    (property "note" "Solder later" (at 138.684 117.602 0)
       (effects (font (size 1.27 1.27)) hide)
     )
@@
       (effects (font (size 1.27 1.27)) hide)
     )
-    (property "Mfr" "Everlight Elec" (at 136.144 137.922 0)
+    (property "Mfr" "Lite-On" (at 136.144 137.922 0)
       (effects (font (size 1.27 1.27)) hide)
     )
-    (property "Mfr P/N" "18-225/R6G6C-A01/3T" (at 136.144 137.922 0)
+    (property "Mfr P/N" "LTST-C190KGKT" (at 136.144 137.922 0)
       (effects (font (size 1.27 1.27)) hide)
     )
-    (property "Price" "0.0772" (at 136.144 137.922 0)
+    (property "Price" "0.014" (at 136.144 137.922 0)
       (effects (font (size 1.27 1.27)) hide)
     )
-    (property "Purchase-URL" "https://www.lcsc.com/product-detail/LED-Indication-Discrete_Everlight-Elec-18-225-R6G6C-A01-3T_C172883.html" (at 136.144 137.922 0)
+    (property "Purchase-URL" "https://www.lcsc.com/product-detail/span-style-background-color-ff0-LED-span-Indication-Discrete_Lite-On-LTST-C190KGKT_C125094.html" (at 136.144 137.922 0)
       (effects (font (size 1.27 1.27)) hide)
     )
@@
       (effects (font (size 1.27 1.27)) hide)
     )
-    (property "Supplier 1 P/N" "C172883" (at 136.144 137.922 0)
+    (property "Supplier 1 P/N" "C125094" (at 136.144 137.922 0)
       (effects (font (size 1.27 1.27)) hide)
     )
@@
       (effects (font (size 1.27 1.27)) hide)
     )
-    (property "note" "we use the thermal pad version" (at 319.024 150.622 0)
+    (property "note" "solder later" (at 319.024 150.622 0)
       (effects (font (size 1.27 1.27)) hide)
     )
@@
       (effects (font (size 1.27 1.27)) hide)
     )
-    (property "Mfr P/N" "TPS2376DDAR-H" (at 319.024 150.622 0)
+    (property "Mfr P/N" "TPS2376PWR" (at 319.024 150.622 0)
       (effects (font (size 1.27 1.27)) hide)
     )
-    (property "Price" "0.6501" (at 319.024 150.622 0)
+    (property "Price" "2.87000" (at 319.024 150.622 0)
       (effects (font (size 1.27 1.27)) hide)
     )
-    (property "Purchase-URL" "https://www.lcsc.com/product-detail/Power-Over-Ethernet-PoE-Controllers_Texas-Instruments-TPS2376DDAR-H_C544899.html" (at 319.024 150.622 0)
+    (property "Purchase-URL" "https://www.digikey.com/en/products/detail/texas-instruments/TPS2376PWR/1671144" (at 319.024 150.622 0)
       (effects (font (size 1.27 1.27)) hide)
     )
-    (property "Supplier 1" "LCSC" (at 319.024 150.622 0)
+    (property "Supplier 1" "Digikey" (at 319.024 150.622 0)
       (effects (font (size 1.27 1.27)) hide)
     )
-    (property "Supplier 1 P/N" "C544899" (at 319.024 150.622 0)
+    (property "Supplier 1 P/N" "296-43734-1-ND" (at 319.024 150.622 0)
+      (effects (font (size 1.27 1.27)) hide)
+    )
+    (property "Supplier 2" "" (at 319.024 150.622 0)
+      (effects (font (size 1.27 1.27)) hide)
+    )
+    (property "Supplier 2 P/N" "" (at 319.024 150.622 0)
+      (effects (font (size 1.27 1.27)) hide)
+    )
+    (property "Description" "" (at 319.024 150.622 0)
+      (effects (font (size 1.27 1.27)) hide)
+    )
+    (property "Untitled Field" "" (at 319.024 150.622 0)
       (effects (font (size 1.27 1.27)) hide)
     )
@@
       (effects (font (size 1.27 1.27)) hide)
     )
-    (property "Price" "0.0875" (at 390.144 150.622 0)
+    (property "Price" "0.11000" (at 390.144 150.622 0)
       (effects (font (size 1.27 1.27)) hide)
     )
-    (property "Purchase-URL" "https://www.lcsc.com/product-detail/Schottky-Diodes_Yangzhou-Yangjie-Elec-Tech-SS510_C5339843.html" (at 390.144 150.622 0)
+    (property "Purchase-URL" "https://www.digikey.com/en/products/detail/shenzhen-slkormicro-semicon-co-ltd/SS510/21853089" (at 390.144 150.622 0)
       (effects (font (size 1.27 1.27)) hide)
     )
-    (property "Supplier 1" "LCSC" (at 390.144 150.622 0)
+    (property "Supplier 1" "Digikey" (at 390.144 150.622 0)
       (effects (font (size 1.27 1.27)) hide)
     )
-    (property "Supplier 1 P/N" "C5339843" (at 390.144 150.622 0)
+    (property "Supplier 1 P/N" "5399-SS510CT-ND" (at 390.144 150.622 0)
       (effects (font (size 1.27 1.27)) hide)
     )
-    (property "note" "" (at 390.144 150.622 0)
+    (property "note" "Solder later" (at 390.144 150.622 0)
       (effects (font (size 1.27 1.27)) hide)
     )
@@
       (effects (font (size 1.27 1.27) italic) hide)
     )
-    (property "Mfr" "DEALON" (at 297.18 283.718 0)
+    (property "Mfr" "Amphenol ICC (FCI)" (at 297.18 283.718 0)
       (effects (font (size 1.27 1.27)) hide)
     )
-    (property "Mfr P/N" "DZ127R-11-09-25" (at 297.18 283.718 0)
+    (property "Mfr P/N" "20021111-00012T4LF" (at 297.18 283.718 0)
       (effects (font (size 1.27 1.27)) hide)
     )
-    (property "Price" "0.0343" (at 297.18 283.718 0)
+    (property "Price" "1.16000" (at 297.18 283.718 0)
       (effects (font (size 1.27 1.27)) hide)
     )
-    (property "Purchase-URL" "https://www.lcsc.com/product-detail/Pin-Headers_DEALON-DZ127R-11-09-25_C2935949.html" (at 297.18 283.718 0)
+    (property "Purchase-URL" "https://www.digikey.com/en/products/detail/amphenol-cs-fci/20021111-00012T4LF/2209074" (at 297.18 283.718 0)
       (effects (font (size 1.27 1.27)) hide)
     )
-    (property "Supplier 1" "LCSC" (at 297.18 283.718 0)
+    (property "Supplier 1" "Digikey" (at 297.18 283.718 0)
       (effects (font (size 1.27 1.27)) hide)
     )
-    (property "Supplier 1 P/N" "C3324132" (at 297.18 283.718 0)
+    (property "Supplier 1 P/N" "609-3713-ND" (at 297.18 283.718 0)
       (effects (font (size 1.27 1.27)) hide)
     )
@@
       (effects (font (size 1.27 1.27) italic) hide)
     )
-    (property "Mfr" "DEALON" (at 297.18 335.026 0)
+    (property "Mfr" "Amphenol ICC (FCI)" (at 297.18 335.026 0)
       (effects (font (size 1.27 1.27)) hide)
     )
-    (property "Mfr P/N" "DZ127R-11-09-25" (at 297.18 335.026 0)
+    (property "Mfr P/N" "20021111-00012T4LF" (at 297.18 335.026 0)
       (effects (font (size 1.27 1.27)) hide)
     )
-    (property "Price" "0.0343" (at 297.18 335.026 0)
+    (property "Price" "1.16000" (at 297.18 335.026 0)
       (effects (font (size 1.27 1.27)) hide)
     )
-    (property "Purchase-URL" "https://www.lcsc.com/product-detail/Pin-Headers_DEALON-DZ127R-11-09-25_C2935949.html" (at 297.18 335.026 0)
+    (property "Purchase-URL" "https://www.digikey.com/en/products/detail/amphenol-cs-fci/20021111-00012T4LF/2209074" (at 297.18 335.026 0)
       (effects (font (size 1.27 1.27)) hide)
     )
-    (property "Supplier 1" "LCSC" (at 297.18 335.026 0)
+    (property "Supplier 1" "Digikey" (at 297.18 335.026 0)
       (effects (font (size 1.27 1.27)) hide)
     )
-    (property "Supplier 1 P/N" "C3324132" (at 297.18 335.026 0)
+    (property "Supplier 1 P/N" "609-3713-ND" (at 297.18 335.026 0)
       (effects (font (size 1.27 1.27)) hide)
     )
