File: ESP32_POE_Board/1.4/ESP_POE_1.4b/ESP_POE_1.4b/ESP_POE_1.4b.kicad_sch (KiCad schematic)
At the start: 79 parts, among them J26 USB_C_Receptacle, J5 20021311-00012T4LF, J7 20021311-00012T4LF, Q1 Q12MHz/20pF/10ppm/4P/3.2x2.5mm, Q2 BC817-40(SOT23), Q3 BC817-40(SOT23), SW1 PTS815 SJM 250 SMTR LFS, U1 CH340T(SSOP20W), U3 BL4054B-42TPRN(SOT23-5), U6 ESP32-WROVER-E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

Commit message: POE2 layout
Parts:
- removed FID3, FID6: Fiducial, OLIMEX_Other-FP:Fiducial1x3, symbol ESP32-PoE-ISO_Rev_K:Fiducial
- removed MH1, MH2, MH3: Mounting_Hole_NPTH, OLIMEX_Other-FP:NPTH_2.2mm, symbol ESP32-PoE-ISO_Rev_K:Mounting_Hole_NPTH
Other:
- note removed: "Mounting Holes"
Changed lines of the file:
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@@
     (stroke (width 0) (type default))
   )
-  (polyline (pts (xy 459.74 340.36) (xy 576.58 340.36))
-    (stroke (width 0) (type default))
-  )
   (wire (pts (xy 26.416 37.592) (xy 26.416 55.372))
     (stroke (width 0) (type default))
@@
     (stroke (width 0) (type default))
   )
-  (polyline (pts (xy 459.74 368.3) (xy 576.58 368.3))
-    (stroke (width 0) (type default))
-  )
   (bus (pts (xy 464.82 193.04) (xy 464.82 195.58))
     (stroke (width 0) (type default))
@@
     (stroke (width 0) (type default))
   )
-  (polyline (pts (xy 576.58 340.36) (xy 576.58 368.3))
-    (stroke (width 0) (type default))
-  )
   (wire (pts (xy 43.18 161.544) (xy 48.514 161.544))
     (stroke (width 0) (type default))
@@
     (stroke (width 0) (type default))
   )
-  (polyline (pts (xy 459.74 340.36) (xy 459.74 368.3))
-    (stroke (width 0) (type default))
-  )
   (wire (pts (xy 386.08 91.44) (xy 424.18 91.44))
     (stroke (width 0) (type default))
@@
     (effects (font (size 1.8034 1.8034) (thickness 0.3607) bold) (justify left bottom))
   )
-  (text "Mounting Holes" (at 485.14 350.52 0)
-    (effects (font (size 5.08 5.08) (thickness 1.016) bold italic) (justify left bottom))
-  )
   (text "0" (at 417.957 206.248 0)
     (effects (font (size 1.524 1.524)) (justify left bottom))
@@
     )
   )
-  (symbol (lib_id "ESP32-PoE-ISO_Rev_K:Fiducial") (at 553.72 314.96 0) (unit 1)
-    (in_bom yes) (on_board yes) (dnp no)
-    (property "Reference" "FID3" (at 556.9712 313.7916 0)
-      (effects (font (size 1.27 1.27)) (justify left))
-    )
-    (property "Value" "Fiducial" (at 556.9712 316.103 0)
-      (effects (font (size 1.27 1.27)) (justify left))
-    )
-    (property "Footprint" "OLIMEX_Other-FP:Fiducial1x3" (at 546.354 316.865 0)
-      (effects (font (size 0.508 0.508)) hide)
-    )
-    (property "Datasheet" "" (at 552.45 314.96 90)
-      (effects (font (size 1.524 1.524)))
-    )
-    (pin "Fid1")
-    (instances
-      (project "ESP_POE_1.4b"
-        (path "/e282cc28-a468-4b1a-8ebc-006ea330625e"
-          (reference "FID3") (unit 1)
-        )
-      )
-    )
-  )
   (symbol (lib_id "ESP32-PoE-ISO_Rev_K:C") (at 178.816 96.012 0) (unit 1)
     (in_bom yes) (on_board yes) (dnp no)
@@
     )
   )
-  (symbol (lib_id "ESP32-PoE-ISO_Rev_K:Fiducial") (at 553.72 325.12 0) (unit 1)
-    (in_bom yes) (on_board yes) (dnp no)
-    (property "Reference" "FID6" (at 556.9712 323.9516 0)
-      (effects (font (size 1.27 1.27)) (justify left))
-    )
-    (property "Value" "Fiducial" (at 556.9712 326.263 0)
-      (effects (font (size 1.27 1.27)) (justify left))
-    )
-    (property "Footprint" "OLIMEX_Other-FP:Fiducial1x3" (at 546.354 327.025 0)
-      (effects (font (size 0.508 0.508)) hide)
-    )
-    (property "Datasheet" "" (at 552.45 325.12 90)
-      (effects (font (size 1.524 1.524)))
-    )
-    (pin "Fid1")
-    (instances
-      (project "ESP_POE_1.4b"
-        (path "/e282cc28-a468-4b1a-8ebc-006ea330625e"
-          (reference "FID6") (unit 1)
-        )
-      )
-    )
-  )
   (symbol (lib_id "ESP32-PoE-ISO_Rev_K:D_Schottky") (at 394.462 191.008 0) (unit 1)
     (in_bom yes) (on_board yes) (dnp no)
@@
         )
       )
-    )
-  )
-  (symbol (lib_id "ESP32-PoE-ISO_Rev_K:Mounting_Hole_NPTH") (at 482.6 360.68 0) (unit 1)
-    (in_bom yes) (on_board yes) (dnp no)
-    (property "Reference" "MH1" (at 480.695 355.6 0)
-      (effects (font (size 1.27 1.27)) (justify left))
-    )
-    (property "Value" "Mounting_Hole_NPTH" (at 473.075 365.125 0)
-      (effects (font (size 1.27 1.27)) (justify left))
-    )
-    (property "Footprint" "OLIMEX_Other-FP:NPTH_2.2mm" (at 481.33 360.68 0)
-      (effects (font (size 1.27 1.27)) hide)
-    )
-    (property "Datasheet" "" (at 481.33 360.68 0)
-      (effects (font (size 1.27 1.27)) hide)
-    )
-    (instances
-      (project "ESP_POE_1.4b"
-        (path "/e282cc28-a468-4b1a-8ebc-006ea330625e"
-          (reference "MH1") (unit 1)
-        )
-      )
-    )
-  )
-  (symbol (lib_id "ESP32-PoE-ISO_Rev_K:Mounting_Hole_NPTH") (at 518.16 360.68 0) (unit 1)
-    (in_bom yes) (on_board yes) (dnp no)
-    (property "Reference" "MH2" (at 516.255 355.6 0)
-      (effects (font (size 1.27 1.27)) (justify left))
-    )
-    (property "Value" "Mounting_Hole_NPTH" (at 508.635 365.125 0)
-      (effects (font (size 1.27 1.27)) (justify left))
-    )
-    (property "Footprint" "OLIMEX_Other-FP:NPTH_2.2mm" (at 516.89 360.68 0)
-      (effects (font (size 1.27 1.27)) hide)
-    )
-    (property "Datasheet" "" (at 516.89 360.68 0)
-      (effects (font (size 1.27 1.27)) hide)
-    )
-    (instances
-      (project "ESP_POE_1.4b"
-        (path "/e282cc28-a468-4b1a-8ebc-006ea330625e"
-          (reference "MH2") (unit 1)
-        )
-      )
-    )
-  )
-  (symbol (lib_id "ESP32-PoE-ISO_Rev_K:Mounting_Hole_NPTH") (at 553.72 360.68 0) (unit 1)
-    (in_bom yes) (on_board yes) (dnp no)
-    (property "Reference" "MH3" (at 551.815 355.6 0)
-      (effects (font (size 1.27 1.27)) (justify left))
-    )
-    (property "Value" "Mounting_Hole_NPTH" (at 544.195 365.125 0)
-      (effects (font (size 1.27 1.27)) (justify left))
-    )
-    (property "Footprint" "OLIMEX_Other-FP:NPTH_2.2mm" (at 552.45 360.68 0)
-      (effects (font (size 1.27 1.27)) hide)
-    )
-    (property "Datasheet" "" (at 552.45 360.68 0)
-      (effects (font (size 1.27 1.27)) hide)
-    )
-    (instances
-      (project "ESP_POE_1.4b"
-        (path "/e282cc28-a468-4b1a-8ebc-006ea330625e"
-          (reference "MH3") (unit 1)
-        )
-      )

Commit message: fixing DRC
Connections:
- no-connect marks 13 -> 29
Changed lines of the file:
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@@
   (no_connect (at 386.08 73.66))
   (no_connect (at 386.08 71.12))
+  (no_connect (at 233.934 200.66))
+  (no_connect (at 130.048 186.944))
+  (no_connect (at 48.514 174.244))
   (no_connect (at 342.392 208.788))
   (no_connect (at 556.26 121.92))
+  (no_connect (at 233.934 223.52))
+  (no_connect (at 233.934 228.6))
   (no_connect (at 386.08 68.58))
+  (no_connect (at 233.934 208.28))
   (no_connect (at 386.08 63.5))
+  (no_connect (at 48.768 199.644))
+  (no_connect (at 233.934 180.34))
   (no_connect (at 386.08 66.04))
+  (no_connect (at 233.934 198.12))
+  (no_connect (at 233.934 220.98))
   (no_connect (at 342.392 203.708))
+  (no_connect (at 92.456 314.452))
+  (no_connect (at 233.934 213.36))
   (no_connect (at 342.392 206.248))
   (no_connect (at 342.392 196.088))
+  (no_connect (at 233.934 215.9))
+  (no_connect (at 233.934 231.14))
   (no_connect (at 386.08 76.2))
   (no_connect (at 342.392 201.168))
+  (no_connect (at 233.934 177.8))
   (no_connect (at 342.392 211.328))
+  (no_connect (at 233.934 205.74))
   (bus_entry (at 439.42 86.36) (size -2.54 2.54)
     (stroke (width 0) (type default))

Commit message: fixed 1.4a
Parts:
- removed MICRO_SD1: TFC-9P-1.7H(ATFFS150A01BR016), OLIMEX_Connectors-FP:uSD(TFC-9P-1.xH(ATFFS150A01BR016)), symbol ESP32-PoE-ISO_Rev_K:MICRO_SD(TFC-9P-1.xH(ATFFS150A01BR016))
- added J2: 1051620001, 105162-0001_MOL, symbol 1051620001:1051620001
Connections:
- net GND: now also J2.G1 (GND), J2.G2 (GND), J2.G3 (GND), J2.G4 (GND), J2.P6 (VSS)
- net GPIO15/HS2_CMD: now also J2.P3 (CMD)
- net at R40.2: now also J2.P5 (CLK)
- net at C3.1, L5.2: now also J2.P4 (VDD)
- net at RM3.2.1: now also J2.P2 (CD/DAT3)
- net at RM3.3.1: now also J2.P1 (DAT2)
- net at RM3.1.1: now also J2.P8 (DAT1)
- net at R46.2: now also J2.P7 (DAT0)
