File: ESP32_POE_Board/1.4/ESP_POE_1.4b/ESP_POE_1.4b/ESP_POE_1.4b.kicad_sch (KiCad schematic)
At the start: 74 parts, among them J26 USB_C_Receptacle, J5 20021311-00012T4LF, J7 20021311-00012T4LF, Q1 Q12MHz/20pF/10ppm/4P/3.2x2.5mm, Q2 BC817-40(SOT23), Q3 BC817-40(SOT23), SW1 PTS815 SJM 250 SMTR LFS, U1 CH340T(SSOP20W), U3 BL4054B-42TPRN(SOT23-5), U6 ESP32-WROVER-E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

Commit message: fixed
Parts:
- removed MICRO_SD1: TFC-9P-1.7H(ATFFS150A01BR016), OLIMEX_Connectors-FP:uSD(TFC-9P-1.xH(ATFFS150A01BR016)), symbol ESP32-PoE-ISO_Rev_K:MICRO_SD(TFC-9P-1.xH(ATFFS150A01BR016))
- added J2: 1051620001, 105162-0001_MOL, symbol 1051620001:1051620001
- R45, R47, R48: footprint OLIMEX_RLC-FP:R_0402_5MIL_DWS -> Resistor_SMD:R_0402_1005Metric
Connections:
- net GND: now also J2.G1 (GND), J2.G2 (GND), J2.G3 (GND), J2.G4 (GND), J2.P6 (VSS)
- net GPIO15/HS2_CMD: now also J2.P3 (CMD)
- net at R40.2: now also J2.P5 (CLK)
- net at C3.1, L5.2: now also J2.P4 (VDD)
- net at RM3.2.1: now also J2.P2 (CD/DAT3)
- net at RM3.3.1: now also J2.P1 (DAT2)
- net at RM3.1.1: now also J2.P8 (DAT1)
- net at R46.2: now also J2.P7 (DAT0)

Commit message: all
Parts:
- BAT1: Mfr Diodes Incorporated -> JST; Mfr P/N DF02S -> B2B-XH-A; Supplier 1 P/N C151398 -> C158012; price 0.2519 -> 0.0342; purchase url https://www.lcsc.com/product-detail/Bridge-Rectifiers_Diode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 -> https://jlcpcb.com/smtReplace?orderNum=05f9fd6d17f9467f8ddf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
Changed lines of the file:
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@@
       (effects (font (size 1.524 1.524)) hide)
     )
-    (property "Mfr" "Diodes Incorporated" (at 163.576 97.282 0)
+    (property "Mfr" "JST" (at 163.576 97.282 0)
       (effects (font (size 1.27 1.27)) hide)
     )
-    (property "Mfr P/N" "DF02S" (at 163.576 97.282 0)
+    (property "Mfr P/N" "B2B-XH-A" (at 163.576 97.282 0)
       (effects (font (size 1.27 1.27)) hide)
     )
@@
       (effects (font (size 1.27 1.27)) hide)
     )
-    (property "Supplier 1 P/N" "C151398" (at 163.576 97.282 0)
+    (property "Supplier 1 P/N" "C158012" (at 163.576 97.282 0)
       (effects (font (size 1.27 1.27)) hide)
     )
-    (property "price" "0.2519" (at 163.576 97.282 0)
+    (property "price" "0.0342" (at 163.576 97.282 0)
       (effects (font (size 1.27 1.27)) hide)
     )
-    (property "purchase url" "https://www.lcsc.com/product-detail/Bridge-Rectifiers_Diodes-Incorporated-DF02S_C151398.html" (at 163.576 97.282 0)
+    (property "purchase url" "https://jlcpcb.com/smtReplace?orderNum=05f9fd6d17f9467f8ddf57472b9d52d7&stencilCountsSmt=2" (at 163.576 97.282 0)
       (effects (font (size 1.27 1.27)) hide)
     )
