File: ESP32_POE_Board/1.4/ESP_POE_1.4b/ESP_POE_1.4b/ESP_POE_1.4b.kicad_pcb (KiCad board)
At the start: 6 copper layers, 40 x 40 mm, 73 parts, among them J1 USB_C_Receptacle, J5 20021311-00012T4LF, J7 20021311-00012T4LF, Q1 Q12MHz/20pF/10ppm/4P/3.2x2.5mm, Q2 BC817-40(SOT23), Q3 BC817-40(SOT23), SW1 PTS815 SJM 250 SMTR LFS, SW2 PTS815 SJM 250 SMTR LFS, U1 CH340T(SSOP20W), U3 BL4054B-42TPRN(SOT23-5)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

Commit message: fixed 1.4a
Parts:
- removed MICRO_SD1: TFC-9P-1.7H(ATFFS150A01BR016), OLIMEX_Connectors-FP:uSD(TFC-9P-1.xH(ATFFS150A01BR016))
- added J2: 1051620001, 1051620001:105162-0001_MOL, F.Cu at (103.6, 144.1)
Routing:
- net GND: track 88.9 -> 101.3 mm
- net Net-(J2-CLK): track 10.5 -> 20.6 mm
- net Net-(J2-DAT0): track 25.5 -> 22.6 mm

Commit message: updates
Parts:
- moved R36 8.28 mm to (86.1, 142.5), turned to 90 degrees
- moved D9 0.61 mm to (102.8, 132.2)
Routing:
- net GND: track 101.3 -> 78.7 mm, vias 19 -> 21
- net Net-(D7-A): track 31.6 -> 44.5 mm, vias 2 -> 4
- net Net-(J2-DAT1): track 16.5 -> 5.03 mm, vias 0 -> 1
- net Net-(J2-CLK): track 20.6 -> 9.32 mm, vias 2 -> 1
- net /GPIO5/SPI_CS: track 17.9 -> 11.2 mm
- net Net-(J2-DAT2): track 6.05 -> 11.7 mm, vias 0 -> 1
- net /GPIO15/HS2_CMD: track 55.1 -> 60.0 mm
- net Net-(J2-DAT0): track 22.6 -> 18.5 mm
- net /GPIO13/I2C-SDA: track 34.2 -> 30.2 mm, vias 1 -> 2
- net Net-(J2-CD/DAT3): track 8.55 -> 12.1 mm, vias 0 -> 1
- net Net-(D9-K): track 20.3 -> 17.6 mm
- net +3V3: track 32.8 -> 30.4 mm, vias 8 -> 9
- net /GPIO12/PHY_PWR: track 13.8 -> 11.8 mm
- net Net-(U1-XI): track 16.9 -> 18.8 mm
- net Net-(J2-VDD): track 42.6 -> 40.8 mm
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
Commit message: 1.4b DRC check
Routing:
- net /+5V_USB: track 96.6 -> 94.4 mm
- net /GPIO25/EMAC_RXD0(RMII): track 34.0 -> 34.8 mm
- net /GPIO0: track 20.8 -> 21.4 mm
- net /USB_D+: track 13.7 -> 14.2 mm
- net /USB_D-: track 13.3 -> 13.5 mm, vias 3 -> 2

Commit message: jtag updates
Routing:
- net Net-(D4-K): track 18.0 -> 14.0 mm
- net /GPIO2/HS2_DATA0: track 64.0 -> 60.9 mm, vias 3 -> 4
- net /GPIO13/I2C-SDA: track 30.2 -> 28.5 mm
- net /GPIO5/SPI_CS: track 11.2 -> 12.2 mm
- net /GPIO16/I2C-SCL: track 21.2 -> 21.8 mm

Commit message: s
Parts:
- renumbered J2 to MICRO_SD1
Changed lines of the file:
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@@
     (property "ki_keywords" "1051620001")
     (attr smd)
-    (fp_text reference "J2" (at 0 3.517699 90 unlocked) (layer "F.SilkS")
+    (fp_text reference "MICRO_SD1" (at 0 3.517699 90 unlocked) (layer "F.SilkS")
         (effects (font (size 1 1) (thickness 0.15)))
     )
