File: Power_Board_out/1.1/PowerBoard_rev1.1/PowerBoard_rev1.1.kicad_pcb (KiCad board)
At the start: 4 copper layers, 40 x 40 mm, 31 parts, among them J1 HMTSW-102-X-X-S-X, J2 HMTSW-102-X-X-S-X, J3 HMTSW-102-X-X-S-X, J4 HMTSW-102-X-X-S-X, J5 HMTSW-102-X-X-S-X, J6 HMTSW-102-X-X-S-X, J7 530470210, J8 530470210, U1 DRV8410PWPR, U2 MCP73812T-420I-OT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

Commit message: POE 1 passes
Routing:
- net GND: track 28.4 -> 31.5 mm
- net MOTOR2_BIN1: track 31.3 -> 32.7 mm
- net Net-(U1-AOUT1): track 12.7 -> 13.3 mm

Commit message: board board edits
Routing:
- net GND: track 31.5 -> 33.0 mm
Changed lines of the file:
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@@
     (pad "17" smd roundrect (at 0 0) (size 3.4 5) (layers "F.Cu") (roundrect_rratio 0.015)
       (net 1 "GND") (pinfunction "EXP") (pintype "power_in"))
-    (pad "18_1" thru_hole circle (at -1 -1.8) (size 0.3 0.3) (drill 0.2) (layers "*.Cu"))
-    (pad "18_2" thru_hole circle (at -1 -0.6) (size 0.3 0.3) (drill 0.2) (layers "*.Cu"))
-    (pad "18_3" thru_hole circle (at -1 0.6) (size 0.3 0.3) (drill 0.2) (layers "*.Cu"))
-    (pad "18_4" thru_hole circle (at -1 1.8) (size 0.3 0.3) (drill 0.2) (layers "*.Cu"))
-    (pad "18_5" thru_hole circle (at 0 -1.8) (size 0.3 0.3) (drill 0.2) (layers "*.Cu"))
-    (pad "18_6" thru_hole circle (at 0 -0.6) (size 0.3 0.3) (drill 0.2) (layers "*.Cu"))
-    (pad "18_7" thru_hole circle (at 0 0.6) (size 0.3 0.3) (drill 0.2) (layers "*.Cu"))
-    (pad "18_8" thru_hole circle (at 0 1.8) (size 0.3 0.3) (drill 0.2) (layers "*.Cu"))
-    (pad "18_9" thru_hole circle (at 1 -1.8) (size 0.3 0.3) (drill 0.2) (layers "*.Cu"))
-    (pad "18_10" thru_hole circle (at 1 -0.6) (size 0.3 0.3) (drill 0.2) (layers "*.Cu"))
-    (pad "18_11" thru_hole circle (at 1 0.6) (size 0.3 0.3) (drill 0.2) (layers "*.Cu"))
-    (pad "18_12" thru_hole circle (at 1 1.8) (size 0.3 0.3) (drill 0.2) (layers "*.Cu"))
+    (pad "18_1" thru_hole circle (at -1 -1.8) (size 0.55 0.55) (drill 0.25) (layers "*.Cu"))
+    (pad "18_2" thru_hole circle (at -1 -0.6) (size 0.55 0.55) (drill 0.25) (layers "*.Cu"))
+    (pad "18_3" thru_hole circle (at -1 0.6) (size 0.55 0.55) (drill 0.25) (layers "*.Cu"))
+    (pad "18_4" thru_hole circle (at -1 1.8) (size 0.55 0.55) (drill 0.25) (layers "*.Cu"))
+    (pad "18_5" thru_hole circle (at 0 -1.8) (size 0.55 0.55) (drill 0.25) (layers "*.Cu"))
+    (pad "18_6" thru_hole circle (at 0 -0.6) (size 0.55 0.55) (drill 0.25) (layers "*.Cu"))
+    (pad "18_7" thru_hole circle (at 0 0.6) (size 0.55 0.55) (drill 0.25) (layers "*.Cu"))
+    (pad "18_8" thru_hole circle (at 0 1.8) (size 0.55 0.55) (drill 0.25) (layers "*.Cu"))
+    (pad "18_9" thru_hole circle (at 1 -1.8) (size 0.55 0.55) (drill 0.25) (layers "*.Cu"))
+    (pad "18_10" thru_hole circle (at 1 -0.6) (size 0.55 0.55) (drill 0.25) (layers "*.Cu"))
+    (pad "18_11" thru_hole circle (at 1 0.6) (size 0.55 0.55) (drill 0.25) (layers "*.Cu"))
+    (pad "18_12" thru_hole circle (at 1 1.8) (size 0.55 0.55) (drill 0.25) (layers "*.Cu"))
   )
   (footprint "Diode_SMD:D_SOD-323F" (layer "F.Cu")
@@
   (segment (start 155.448 82.55) (end 156.464 81.534) (width 0.508) (layer "F.Cu") (net 1))
   (segment (start 151.9936 72.0852) (end 151.2316 71.3232) (width 0.508) (layer "F.Cu") (net 1))
-  (segment (start 146.0196 75.5922) (end 144.516351 75.5922) (width 0.25) (layer "F.Cu") (net 1))
+  (segment (start 144.622418 75.5922) (end 144.297418 75.9172) (width 0.25) (layer "F.Cu") (net 1))
   (segment (start 148.1836 74.8792) (end 148.6916 74.3712) (width 0.25) (layer "F.Cu") (net 1))
   (segment (start 152.786 70.358) (end 152.1968 70.358) (width 0.508) (layer "F.Cu") (net 1))
@@
   (segment (start 135.7922 72.9018) (end 135.4328 72.5424) (width 0.25) (layer "F.Cu") (net 1))
   (segment (start 136.0443 78.9413) (end 135.5344 79.4512) (width 0.25) (layer "F.Cu") (net 1))
+  (segment (start 146.0196 75.5922) (end 144.622418 75.5922) (width 0.25) (layer "F.Cu") (net 1))
   (segment (start 141.986 89.3064) (end 141.8844 89.408) (width 0.25) (layer "F.Cu") (net 1))
   (segment (start 145.4662 86.6898) (end 145.5928 86.5632) (width 0.25) (layer "F.Cu") (net 1))
@@
   (segment (start 154.94 82.55) (end 155.448 82.55) (width 0.508) (layer "F.Cu") (net 1))
   (segment (start 131.3688 73.5076) (end 131.7832 73.5076) (width 0.25) (layer "F.Cu") (net 1))
+  (segment (start 144.297418 75.9172) (end 143.1196 75.9172) (width 0.25) (layer "F.Cu") (net 1))
   (segment (start 144.526 86.6898) (end 145.4662 86.6898) (width 0.25) (layer "F.Cu") (net 1))
   (via (at 148.6916 74.3712) (size 0.8) (drill 0.4) (layers "F.Cu" "B.Cu") (net 1))
@@
   (segment (start 146.0196 78.5164) (end 145.0848 79.4512) (width 0.25) (layer "F.Cu") (net 6))
   (via (at 145.0848 79.4512) (size 0.8) (drill 0.4) (layers "F.Cu" "B.Cu") (net 6))
+  (segment (start 136.8557 59.5879) (end 136.8557 60.6239) (width 0.25) (layer "B.Cu") (net 6))
+  (segment (start 145.0848 79.4512) (end 145.0848 78.486) (width 0.25) (layer "B.Cu") (net 6))
+  (segment (start 145.0848 78.486) (end 145.6436 77.9272) (width 0.25) (layer "B.Cu") (net 6))
+  (segment (start 144.9324 58.7756) (end 137.668 58.7756) (width 0.25) (layer "B.Cu") (net 6))
   (segment (start 145.6436 59.4868) (end 144.9324 58.7756) (width 0.25) (layer "B.Cu") (net 6))
-  (segment (start 136.8557 59.5879) (end 136.8557 60.6239) (width 0.25) (layer "B.Cu") (net 6))
+  (segment (start 145.6436 77.9272) (end 145.6436 59.4868) (width 0.25) (layer "B.Cu") (net 6))
   (segment (start 137.668 58.7756) (end 136.8557 59.5879) (width 0.25) (layer "B.Cu") (net 6))
-  (segment (start 145.0848 79.4512) (end 144.5768 78.9432) (width 0.25) (layer "B.Cu") (net 6))
-  (segment (start 145.6436 76.864952) (end 145.6436 59.4868) (width 0.25) (layer "B.Cu") (net 6))
-  (segment (start 144.5768 77.931752) (end 145.6436 76.864952) (width 0.25) (layer "B.Cu") (net 6))
-  (segment (start 144.5768 78.9432) (end 144.5768 77.931752) (width 0.25) (layer "B.Cu") (net 6))
-  (segment (start 144.9324 58.7756) (end 137.668 58.7756) (width 0.25) (layer "B.Cu") (net 6))
   (segment (start 151.13 67.9704) (end 151.7396 68.58) (width 0.508) (layer "F.Cu") (net 9))
   (segment (start 140.0357 87.3959) (end 141.036 87.3959) (width 0.508) (layer "F.Cu") (net 9))
@@
   (segment (start 140.8176 71.0692) (end 140.8176 76.0476) (width 0.25) (layer "B.Cu") (net 12))
   (segment (start 139.2936 77.5716) (end 138.7348 77.5716) (width 0.25) (layer "B.Cu") (net 12))
+  (segment (start 140.1838 76.2064) (end 140.2196 76.2422) (width 0.25) (layer "F.Cu") (net 13))
+  (segment (start 137.448504 76.2422) (end 137.484304 76.2064) (width 0.25) (layer "F.Cu") (net 13))
   (segment (start 136.1354 76.2422) (end 137.448504 76.2422) (width 0.25) (layer "F.Cu") (net 13))
   (segment (start 135.7376 75.8444) (end 136.1354 76.2422) (width 0.25) (layer "F.Cu") (net 13))
-  (segment (start 137.534304 76.1564) (end 139.361938 76.1564) (width 0.25) (layer "F.Cu") (net 13))
-  (segment (start 137.448504 76.2422) (end 137.534304 76.1564) (width 0.25) (layer "F.Cu") (net 13))
-  (segment (start 139.361938 76.1564) (end 139.447738 76.2422) (width 0.25) (layer "F.Cu") (net 13))
-  (segment (start 139.447738 76.2422) (end 140.2196 76.2422) (width 0.25) (layer "F.Cu") (net 13))
+  (segment (start 137.484304 76.2064) (end 140.1838 76.2064) (width 0.25) (layer "F.Cu") (net 13))
   (via (at 135.7376 75.8444) (size 0.8) (drill 0.4) (layers "F.Cu" "B.Cu") (net 13))
   (segment (start 134.7078 74.8146) (end 134.7078 72.242095) (width 0.25) (layer "B.Cu") (net 13))

Commit message: 1.4a and 1.4b ready to fab
Changed lines of the file:
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@@
       (outputformat 1)
       (mirror false)
-      (drillshape 1)
+      (drillshape 0)
       (scaleselection 1)
-      (outputdirectory "")
+      (outputdirectory "fab/Gerber/")
     )
   )
@@
     (fp_line (start 1 0.625) (end -1 0.625)
       (stroke (width 0.1) (type solid)) (layer "F.Fab"))
-    (pad "1" smd roundrect (at -0.9125 0 270) (size 1.025 1.4) (layers "F.Cu" "F.Paste" "F.Mask") (roundrect_rratio 0.243902)
+    (pad "1" smd roundrect (at -0.9125 0 270) (size 1.025 1.4) (layers "F.Cu" "F.Paste" "F.Mask") (roundrect_rratio 0.243902439)
       (net 22 "Net-(U1-BISEN)") (pintype "passive"))
-    (pad "2" smd roundrect (at 0.9125 0 270) (size 1.025 1.4) (layers "F.Cu" "F.Paste" "F.Mask") (roundrect_rratio 0.243902)
+    (pad "2" smd roundrect (at 0.9125 0 270) (size 1.025 1.4) (layers "F.Cu" "F.Paste" "F.Mask") (roundrect_rratio 0.243902439)
       (net 1 "GND") (pintype "passive"))
     (model "${KICAD6_3DMODEL_DIR}/Resistor_SMD.3dshapes/R_0805_2012Metric.wrl"
@@
     (fp_line (start 1 0.625) (end -1 0.625)
       (stroke (width 0.1) (type solid)) (layer "F.Fab"))
-    (pad "1" smd roundrect (at -0.9125 0 90) (size 1.025 1.4) (layers "F.Cu" "F.Paste" "F.Mask") (roundrect_rratio 0.243902)
+    (pad "1" smd roundrect (at -0.9125 0 90) (size 1.025 1.4) (layers "F.Cu" "F.Paste" "F.Mask") (roundrect_rratio 0.243902439)
       (net 21 "Net-(U1-AISEN)") (pintype "passive"))
-    (pad "2" smd roundrect (at 0.9125 0 90) (size 1.025 1.4) (layers "F.Cu" "F.Paste" "F.Mask") (roundrect_rratio 0.243902)
+    (pad "2" smd roundrect (at 0.9125 0 90) (size 1.025 1.4) (layers "F.Cu" "F.Paste" "F.Mask") (roundrect_rratio 0.243902439)
       (net 1 "GND") (pintype "passive"))
     (model "${KICAD6_3DMODEL_DIR}/Resistor_SMD.3dshapes/R_0805_2012Metric.wrl"
