File: Power_Board_out/1.1/PowerBoard_rev1.1/PowerBoard_rev1.1.kicad_sch (KiCad schematic)
At the start: 31 parts, among them J1 HMTSW-102-X-X-S-X, J2 HMTSW-102-X-X-S-X, J3 HMTSW-102-X-X-S-X, J4 HMTSW-102-X-X-S-X, J5 HMTSW-102-X-X-S-X, J6 HMTSW-102-X-X-S-X, J7 530470210, J8 530470210, U1 DRV8410PWPR, U2 MCP73812T-420I-OT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

Commit message: some bom on power out
Parts:
- C10: Mfr (none) -> YAGEO; Mfr P/N (none) -> CC0201MRX5R6BB105; Price (none) -> 0.0042; Purchase-URL (none) -> https://www.lcsc.com/product-detail/Multilayer-Ceramic-Capa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; Supplier 1 (none) -> LCSC; Supplier 1 P/N (none) -> C605210
- C9: Mfr (none) -> YAGEO; Mfr P/N (none) -> CC0402KRX7R7BB104; Price (none) -> 0.0009; Purchase-URL (none) -> https://www.lcsc.com/product-detail/Multilayer-Ceramic-Capa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; Supplier 1 (none) -> LCSC; Supplier 1 P/N (none) -> C60474
- C9: Mfr (none) -> SamYoung Electronics; Mfr P/N (none) -> NXB16V10M5*11 2.5TP; Price (none) -> 0.0613; Purchase-URL (none) -> https://www.lcsc.com/product-detail/Aluminum-Electrolytic-C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; Supplier 1 (none) -> LCSC; Supplier 1 P/N (none) -> C346926
- D11, D12, D13, D14, D5, D6: Mfr (none) -> DOWO; Mfr P/N (none) -> PMEG6010CEJ; Price (none) -> 0.0159; Purchase-URL (none) -> https://www.lcsc.com/product-detail/Schottky-Diodes_DOWO-PM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; Supplier 1 (none) -> LCSC; Supplier 1 P/N (none) -> C27636122
- J1, J2, J3, J4, J5, J6: Mfr (none) -> Samtec; Mfr P/N (none) -> HTSW-102-07-T-S; Price None -> 0.2216; Purchase-URL (none) -> https://www.lcsc.com/product-detail/Pin-Headers_Samtec-HTSW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; Supplier 1 (none) -> LCSC; Supplier 1 P/N (none) -> C6273326
- J7, J8: Mfr (none) -> MOLEX; Mfr P/N (none) -> 530470210; Price (none) -> 0.0844; Purchase-URL (none) -> https://www.lcsc.com/product-detail/Wire-To-Board-Connector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; Supplier 1 (none) -> LCSC; Supplier 1 P/N (none) -> C114130
- R21: Mfr LIZ Elec -> YAGEO; Mfr P/N CR0201JH0202G -> RC0201FR-072KL; Price (none) -> 0.00080; Purchase-URL (none) -> https://www.lcsc.com/product-detail/Chip-Resistor-Surface-M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; Supplier 1 P/N C100158 -> C327392
- R21: Mfr (none) -> YAGEO; Mfr P/N (none) -> AC0805FR-072RL; Price (none) -> 0.0080; Purchase-URL (none) -> https://www.lcsc.com/product-detail/Chip-span-style-backgro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; Supplier 1 (none) -> LCSC; Supplier 1 P/N (none) -> C228730
- R21: footprint Resistor_SMD:R_01005_0402Metric -> Resistor_SMD:R_0201_0603Metric; Mfr (none) -> YAGEO; Mfr P/N (none) -> RC0201FR-072KL; Price (none) -> 0.00080; Purchase-URL (none) -> https://www.lcsc.com/product-detail/Chip-Resistor-Surface-M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; Supplier 1 (none) -> LCSC; Supplier 1 P/N (none) -> C327392
- U1: Mfr (none) -> Texas Instruments; Mfr P/N (none) -> DRV8410PWPR; Price None -> 1.9877; Purchase-URL https://www.snapeda.com/api/url_track_click_mouser/?unipart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 -> https://www.lcsc.com/product-detail/New-Arrivals_Texas-Inst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; Supplier 1 (none) -> LCSC; Supplier 1 P/N (none) -> C7264874
- U2, U3: Mfr (none) -> Microchip Tech; Mfr P/N (none) -> MCP73812T-420I/OT; Price (none) -> 0.8619; Purchase-URL (none) -> https://www.lcsc.com/product-detail/Battery-Management_Micr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; Supplier 1 (none) -> LCSC; Supplier 1 P/N (none) -> C144308

Commit message: power board out BOM
Parts:
- C9: Mfr (none) -> Samsung Electro-Mechanics; Mfr P/N (none) -> CL21A106KAYNNNE; Price (none) -> 0.0102; Purchase-URL (none) -> https://www.lcsc.com/product-detail/Multilayer-Ceramic-Capa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; Supplier 1 (none) -> LCSC; Supplier 1 P/N (none) -> C15850
Changed lines of the file:
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@@
+      (effects (font (size 1.27 1.27)) hide)
+    )
+    (property "Mfr" "Samsung Electro-Mechanics" (at 105.41 58.928 0)
+      (effects (font (size 1.27 1.27)) hide)
+    )
+    (property "Mfr P/N" "CL21A106KAYNNNE" (at 105.41 58.928 0)
+      (effects (font (size 1.27 1.27)) hide)
+    )
+    (property "Price" "0.0102" (at 105.41 58.928 0)
+      (effects (font (size 1.27 1.27)) hide)
+    )
+    (property "Purchase-URL" "https://www.lcsc.com/product-detail/Multilayer-Ceramic-Capacitors-MLCC-SMD-SMT_Samsung-Electro-Mechanics-CL21A106KAYNNNE_C15850.html" (at 105.41 58.928 0)
+      (effects (font (size 1.27 1.27)) hide)
+    )
+    (property "Supplier 1" "LCSC" (at 105.41 58.928 0)
+      (effects (font (size 1.27 1.27)) hide)
+    )
+    (property "Supplier 1 P/N" "C15850" (at 105.41 58.928 0)
       (effects (font (size 1.27 1.27)) hide)
     )

Commit message: POE 1 passes
Parts:
- C9: footprint Capacitor_SMD:C_01005_0402Metric -> Capacitor_SMD:C_0603_1608Metric
Changed lines of the file:
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@@
       (effects (font (size 1.27 1.27)) (justify left))
     )
-    (property "Footprint" "Capacitor_SMD:C_01005_0402Metric" (at 228.8032 110.998 0)
+    (property "Footprint" "Capacitor_SMD:C_0603_1608Metric" (at 228.8032 110.998 0)
       (effects (font (size 1.27 1.27)) hide)
     )

Commit message: 1.4a half bom
Parts:
- C9: Mfr P/N CC0402KRX7R7BB104 -> CC0603KRX7R9BB104; Price 0.0009 -> 0.0020; Purchase-URL https://www.lcsc.com/product-detail/Multilayer-Ceramic-Capacitors-MLCC-SMD-SMT_YAGEO-CC0402KRX7R7BB104_C60474.html -> https://www.lcsc.com/product-detail/Multilayer-Ceramic-Capacitors-MLCC-SMD-SMT_YAGEO-CC0603KRX7R9BB104_C14663.html; Supplier 1 P/N C60474 -> C14663
Changed lines of the file:
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@@
       (effects (font (size 1.27 1.27)) hide)
     )
-    (property "Mfr P/N" "CC0402KRX7R7BB104" (at 227.838 107.188 0)
+    (property "Mfr P/N" "CC0603KRX7R9BB104" (at 227.838 107.188 0)
       (effects (font (size 1.27 1.27)) hide)
     )
-    (property "Price" "0.0009" (at 227.838 107.188 0)
+    (property "Price" "0.0020" (at 227.838 107.188 0)
       (effects (font (size 1.27 1.27)) hide)
     )
-    (property "Purchase-URL" "https://www.lcsc.com/product-detail/Multilayer-Ceramic-Capacitors-MLCC-SMD-SMT_YAGEO-CC0402KRX7R7BB104_C60474.html" (at 227.838 107.188 0)
+    (property "Purchase-URL" "https://www.lcsc.com/product-detail/Multilayer-Ceramic-Capacitors-MLCC-SMD-SMT_YAGEO-CC0603KRX7R9BB104_C14663.html" (at 227.838 107.188 0)
       (effects (font (size 1.27 1.27)) hide)
     )
@@
       (effects (font (size 1.27 1.27)) hide)
     )
-    (property "Supplier 1 P/N" "C60474" (at 227.838 107.188 0)
+    (property "Supplier 1 P/N" "C14663" (at 227.838 107.188 0)
       (effects (font (size 1.27 1.27)) hide)
     )
+    (property "Supplier 2" "" (at 227.838 107.188 0)
+      (effects (font (size 1.27 1.27)) hide)
+    )
+    (property "Supplier 2 P/N" "" (at 227.838 107.188 0)
+      (effects (font (size 1.27 1.27)) hide)
+    )
+    (property "Description" "" (at 227.838 107.188 0)
+      (effects (font (size 1.27 1.27)) hide)
+    )
+    (property "Untitled Field" "" (at 227.838 107.188 0)
+      (effects (font (size 1.27 1.27)) hide)
+    )

Commit message: 1.4a and 1.4b ready to fab
Parts:
- C10: footprint Capacitor_SMD:C_0201_0603Metric -> Capacitor_SMD:C_0805_2012Metric
- C9: Mfr (none) -> FH (Guangdong Fenghua Advanced Tech); Mfr P/N (none) -> 0805B502K500NT; Price (none) -> 0.0045; Purchase-URL (none) -> https://www.lcsc.com/product-detail/Multilayer-Ceramic-Capa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; Supplier 1 (none) -> LCSC; Supplier 1 P/N (none) -> C1748
- D11, D12, D13, D14, D5, D6: Mfr DOWO -> Nexperia; Mfr P/N PMEG6010CEJ -> PMEG6010CEJ,115; Supplier 1 P/N C27636122 -> C406049
- J1, J2, J3, J4, J5, J6: Mfr Samtec -> XFCN; Mfr P/N HTSW-102-07-T-S -> PZ254V-11-03P; Price 0.2216 -> 0.0145; Supplier 1 P/N C6273326 -> C2937625
- R21: footprint Resistor_SMD:R_0201_0603Metric -> Resistor_SMD:R_0805_2012Metric
- U1: Purchase-URL https://www.lcsc.com/product-detail/New-Arrivals_Texas-Inst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 -> https://www.digikey.com/en/products/detail/texas-instrument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; Supplier 1 LCSC -> Digikey; Supplier 1 P/N C7264874 -> 296-DRV8410PWPRCT-ND
