File: Sensing_Board_out/1.1/SensingBoard_rev1.1/SensingBoard_rev1.1.kicad_pcb (KiCad board)
At the start: 6 copper layers, 40 x 40 mm, 89 parts, among them J1 USB_C_Receptacle, J2 3221-10-0300-00, J3 F32R-1A7H1-11024, J5 RS1-02-G, J6 RS1-02-G, J7 RS1-02-G, J9 RS1-02-G, SW1 PTS815 SJM 250 SMTR LFS, SW2 PTS815 SJM 250 SMTR LFS, U2 BNO055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

Commit message: checking drc
Parts:
- moved C36 0.15 mm to (140.2, 63.5)
Connections:
- J2 pad 10: unconnected-(J2-Pad10) -> MTMS/IO42/PDM_CLK
- J2 pad 3: unconnected-(J2-Pad3) -> GND
- J2 pad 4: unconnected-(J2-Pad4) -> GND
- J2 pad 5: unconnected-(J2-Pad5) -> +3.3V
- J2 pad 6: unconnected-(J2-Pad6) -> CHIP_EN
- J2 pad 7: unconnected-(J2-Pad7) -> MTCK/IO39/CAM_SCL
- J2 pad 8: unconnected-(J2-Pad8) -> MTDO/IO40/CAM_SDA
- J2 pad 9: unconnected-(J2-Pad9) -> MTDI/IO41/PDM_DATA
Routing:
- net MTMS/IO42/PDM_CLK: track 0.00 -> 56.3 mm, vias 0 -> 2
- net MTDI/IO41/PDM_DATA: track 0.00 -> 50.0 mm, vias 0 -> 2
- net Net-(D4-K): track 7.83 -> 35.9 mm, vias 0 -> 2
- net MTDO/IO40/CAM_SDA: track 21.8 -> 46.2 mm, vias 2 -> 4
- net IO17/DVP_Y3: track 3.80 -> 27.5 mm, vias 1 -> 2
- net IO14/DVP_Y6: track 1.09 -> 23.4 mm, vias 1 -> 2
- net IO16/DVP_Y5: track 4.52 -> 25.9 mm, vias 0 -> 1
- net MTCK/IO39/CAM_SCL: track 21.3 -> 41.8 mm, vias 1 -> 3
- net IO15/DVP_Y2: track 0.92 -> 18.7 mm, vias 1 -> 2
- net IO12/DVP_Y7: track 3.00 -> 19.2 mm, vias 1 -> 2
- net IO13/DVP_PCLK: track 2.58 -> 17.5 mm, vias 1 -> 2
- net IO11/DVP_Y8: track 2.08 -> 16.5 mm
- net USB_DP: track 5.70 -> 18.7 mm, vias 0 -> 2
- net USB_DN: track 8.12 -> 19.9 mm, vias 2 -> 4
- net BNO_INT: track 0.00 -> 11.4 mm, vias 0 -> 2
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