File: Sensing_Board_out/1.1/SensingBoard_rev1.1/SensingBoard_rev1.1.kicad_sch (KiCad schematic)
At the start: 89 parts, among them J1 USB_C_Receptacle, J3 F32R-1A7H1-11024, J5 RS1-02-G, J6 RS1-02-G, J7 3221-10-0300-00, J7 RS1-02-G, J9 RS1-02-G, SW1 PTS815 SJM 250 SMTR LFS, SW2 PTS815 SJM 250 SMTR LFS, U2 BNO055, U3 MIC5504-3.3YM5, U4 FT232RQ, U5 MIC5504-1.8YM5, U6 MCP1700x-280xxTT, U7 ESP32-S3, U8 GD25D05CT, Y1 ABM8G-40.000MHZ-18-D2Y-T

Commit message: update sensing board bom
Parts:
- ANT1: Mfr (none) -> HRS(Hirose); Mfr P/N (none) -> U.FL-R-SMT-1(80); Price None -> 0.0805; Purchase-URL (none) -> https://www.lcsc.com/product-detail/Coaxial-Connectors-RF_H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; Supplier 1 (none) -> LCSC; Supplier 1 P/N (none) -> C88374
- C10: Mfr (none) -> YAGEO; Mfr P/N (none) -> CC0201MRX5R6BB105; Price (none) -> 0.0042; Purchase-URL (none) -> https://www.lcsc.com/product-detail/Multilayer-Ceramic-Capa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; Supplier 1 (none) -> LCSC; Supplier 1 P/N (none) -> C605210
- C14: Mfr (none) -> YAGEO; Mfr P/N (none) -> CC0201JRNPO9BN180; Price (none) -> 0.001; Purchase-URL (none) -> https://www.lcsc.com/product-detail/Multilayer-Ceramic-Capa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; Supplier 1 (none) -> LCSC; Supplier 1 P/N (none) -> C277474
- C14, C15: Mfr (none) -> YAGEO; Mfr P/N (none) -> CC0201JRNPO8BN220; Price (none) -> 0.001; Purchase-URL (none) -> https://www.lcsc.com/product-detail/Multilayer-Ceramic-Capa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; Supplier 1 (none) -> LCSC; Supplier 1 P/N (none) -> C526934
- C17: Mfr (none) -> YAGEO; Mfr P/N (none) -> CC0402KRX7R7BB104; Price (none) -> 0.0009; Purchase-URL (none) -> https://www.lcsc.com/product-detail/Multilayer-Ceramic-Capa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; Supplier 1 (none) -> LCSC; Supplier 1 P/N (none) -> C60474
- C17: Mfr (none) -> Murata Electronics; Mfr P/N (none) -> GJM1555C1H1R6WB01D; Price (none) -> 0.0417; Purchase-URL (none) -> https://www.lcsc.com/product-detail/Multilayer-Ceramic-Capa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; Supplier 1 (none) -> LCSC; Supplier 1 P/N (none) -> C88881
- C17: Mfr (none) -> YAGEO; Mfr P/N (none) -> CC0402KRX7R9BB103; Price (none) -> 0.0009; Purchase-URL (none) -> https://www.lcsc.com/product-detail/Multilayer-Ceramic-Capa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; Supplier 1 (none) -> LCSC; Supplier 1 P/N (none) -> C60133
- C17: Mfr (none) -> Samsung Electro-Mechanics; Mfr P/N (none) -> CL05A475MQ5NRNC; Price (none) -> 0.0028; Purchase-URL (none) -> https://www.lcsc.com/product-detail/Multilayer-Ceramic-Capa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; Supplier 1 (none) -> LCSC; Supplier 1 P/N (none) -> C307423
- C9: Mfr (none) -> YAGEO; Mfr P/N (none) -> CC0402KRX5R8BB225; Price (none) -> 0.0286; Purchase-URL (none) -> https://www.lcsc.com/product-detail/Multilayer-Ceramic-Capa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; Supplier 1 (none) -> LCSC; Supplier 1 P/N (none) -> C723363
- C9: Mfr (none) -> Samsung Electro-Mechanics; Mfr P/N (none) -> CL10A106KP8NNNC; Price (none) -> 0.005; Purchase-URL (none) -> https://www.lcsc.com/product-detail/Multilayer-Ceramic-Capa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; Supplier 1 (none) -> LCSC; Supplier 1 P/N (none) -> C19702
- D3: Mfr (none) -> Nexperia; Mfr P/N (none) -> PMEG6010CEJ,115; Price (none) -> 0.0382; Purchase-URL (none) -> https://www.lcsc.com/product-detail/Schottky-Diodes_Nexperi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; Supplier 1 (none) -> LCSC; Supplier 1 P/N (none) -> C406049
- D4: Mfr (none) -> Vishay Intertech; Mfr P/N (none) -> B140-E3/5AT; Price (none) -> 0.0667; Purchase-URL (none) -> https://www.lcsc.com/product-detail/Schottky-Diodes_Vishay-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; Supplier 1 (none) -> LCSC; Supplier 1 P/N (none) -> C2981056
- D6: Mfr (none) -> Everlight Elec; Mfr P/N (none) -> 19-21/GHC-YR1S2/4T; Price (none) -> 0.037; Purchase-URL (none) -> https://www.lcsc.com/product-detail/span-style-background-c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; Supplier 1 (none) -> LCSC; Supplier 1 P/N (none) -> C2986048
- FB1: Mfr (none) -> Murata Electronics; Mfr P/N (none) -> BLM21PG121SN1D; Price (none) -> 0.0171; Purchase-URL (none) -> https://www.lcsc.com/product-detail/span-style-background-c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; Supplier 1 (none) -> LCSC; Supplier 1 P/N (none) -> C79382
- J1: Mfr (none) -> GCT; Mfr P/N (none) -> 2073-USB4125-GF-ACT-ND; Price (none) -> 0.80000; Purchase-URL (none) -> https://www.digikey.com/en/products/detail/gct/USB4125-GF-A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; Supplier 1 (none) -> Digikey; Supplier 1 P/N (none) -> USB4125-GF-A
- J3: Mfr (none) -> CNC Tech; Mfr P/N (none) -> F32R-1A7H1-11024; Note (none) -> Solder later; Price None -> 0.93000; Purchase-URL (none) -> https://www.digikey.com/en/products/detail/amphenol-cs-fci/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; Supplier 1 (none) -> Digikey; Supplier 1 P/N (none) -> 609-F32R-1A7H1-11024CT-ND
- J5, J6, J7, J9: Mfr (none) -> Adam Tech; Mfr P/N (none) -> RS1-02-G; Price (none) -> 0.23000; Purchase-URL (none) -> https://www.digikey.com/en/products/detail/adam-tech/RS1-02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; Supplier 1 (none) -> Digikey; Supplier 1 P/N (none) -> 2057-RS1-02-G-ND
- J7: Mfr (none) -> CNC Tech; Mfr P/N (none) -> 3221-10-0300-00; Note (none) -> solder later; Price (none) -> 1.02000; Purchase-URL (none) -> https://www.digikey.com/en/products/detail/cnc-tech/3221-10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; Supplier 1 (none) -> Digikey; Supplier 1 P/N (none) -> 1175-1735-ND
- L1, L2: Mfr (none) -> Murata Electronics; Mfr P/N (none) -> LQP02TQ2N0B02D; Price (none) -> 0.014; Purchase-URL (none) -> https://www.lcsc.com/product-detail/Inductors-SMD_Murata-El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; Supplier 1 (none) -> LCSC; Supplier 1 P/N (none) -> C2048018
- R11, R12: Mfr (none) -> YAGEO; Mfr P/N (none) -> RC0201FR-070RL; Price (none) -> 0.0008; Purchase-URL (none) -> https://www.lcsc.com/product-detail/Chip-span-style-backgro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; Supplier 1 (none) -> LCSC; Supplier 1 P/N (none) -> C106227
- R14, R15, R2: Mfr (none) -> YAGEO; Mfr P/N (none) -> RC0201JR-0710KL; Price (none) -> 0.0008; Purchase-URL (none) -> https://www.lcsc.com/product-detail/Chip-span-style-backgro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; Supplier 1 (none) -> LCSC; Supplier 1 P/N (none) -> C138117
- R14: Mfr (none) -> YAGEO; Mfr P/N (none) -> RC0201JR-074K7L; Price (none) -> 0.0008; Purchase-URL (none) -> https://www.lcsc.com/product-detail/Chip-span-style-backgro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; Supplier 1 (none) -> LCSC; Supplier 1 P/N (none) -> C142008
- R14: Mfr (none) -> YAGEO; Mfr P/N (none) -> RC0201FR-07499RL; Price (none) -> 0.0009; Purchase-URL (none) -> https://www.lcsc.com/product-detail/Chip-span-style-backgro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; Supplier 1 (none) -> LCSC; Supplier 1 P/N (none) -> C138137
- R16: Mfr (none) -> YAGEO; Mfr P/N (none) -> AC0201FR-07100RL; Price (none) -> 0.0017; Purchase-URL (none) -> https://www.lcsc.com/product-detail/Chip-span-style-backgro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; Supplier 1 (none) -> LCSC; Supplier 1 P/N (none) -> C226395
- R17: Mfr (none) -> YAGEO; Mfr P/N (none) -> RC0201FR-075K1L; Price (none) -> 0.0009; Purchase-URL (none) -> https://www.lcsc.com/product-detail/Chip-span-style-backgro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; Supplier 1 (none) -> LCSC; Supplier 1 P/N (none) -> C274341
- R17: Mfr (none) -> YAGEO; Mfr P/N (none) -> RC0201DR-076K04L; Price (none) -> 0.0022; Purchase-URL (none) -> https://www.lcsc.com/product-detail/Chip-span-style-backgro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; Supplier 1 (none) -> LCSC; Supplier 1 P/N (none) -> C851784
- SW1, SW2: Mfr (none) -> C&K; Mfr P/N (none) -> PTS815SJG250SMTRLFS; Price (none) -> 0.085; Purchase-URL (none) -> https://www.lcsc.com/product-detail/Tactile-Switches_C-K-PT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; Supplier 1 (none) -> LCSC; Supplier 1 P/N (none) -> C411883
- U2: Mfr (none) -> Bosch Sensortec; Mfr P/N (none) -> BNO055; Price None -> 10.4432; Purchase-URL https://www.snapeda.com/api/url_track_click_mouser/?unipart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 -> https://www.lcsc.com/product-detail/Accelerometers_Bosch-Se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; Supplier 1 (none) -> LCSC; Supplier 1 P/N (none) -> C93216
- U3: Mfr (none) -> Microchip Tech; Mfr P/N (none) -> MIC5504-3.3YM5-TR; Price (none) -> 0.2143; Purchase-URL (none) -> https://www.lcsc.com/product-detail/Voltage-Regulators-Line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; Supplier 1 (none) -> LCSC; Supplier 1 P/N (none) -> C88419
- U4: Mfr (none) -> FTDI; Mfr P/N (none) -> FT232RQ-REEL; Price None -> 5.7103; Purchase-URL (none) -> https://www.lcsc.com/product-detail/USB-Converters_FTDI-FT2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; Supplier 1 (none) -> LCSC; Supplier 1 P/N (none) -> C14090
- U5: Mfr (none) -> Microchip Tech; Mfr P/N (none) -> MIC5504-1.8YM5-TR; Price (none) -> 0.2774; Purchase-URL (none) -> https://www.lcsc.com/product-detail/Voltage-Regulators-Line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; Supplier 1 (none) -> LCSC; Supplier 1 P/N (none) -> C626116
- U6: Mfr (none) -> Microchip Tech; Mfr P/N (none) -> MCP1700T-2802E/TT; Price (none) -> 0.4696; Purchase-URL (none) -> https://www.lcsc.com/product-detail/Voltage-Regulators-Line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; Supplier 1 (none) -> LCSC; Supplier 1 P/N (none) -> C625349
- U7: Mfr (none) -> Espressif Systems; Mfr P/N (none) -> ESP32-S3-WROOM-1-N8R2; Price (none) -> 4.3420; Purchase-URL (none) -> https://www.lcsc.com/product-detail/WiFi-Modules_Espressif-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; Supplier 1 (none) -> LCSC; Supplier 1 P/N (none) -> C2913204
- U8: Mfr (none) -> GigaDevice Semiconductor (HK) Limited; Mfr P/N (none) -> 1970-1000-1-ND; Note (none) -> solder later; Price (none) -> 0.33000; Purchase-URL (none) -> https://www.digikey.com/en/products/detail/gigadevice-semic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; Supplier 1 (none) -> Digikey; Supplier 1 P/N (none) -> GD25D05CTIGR
- XTAL1: Mfr (none) -> Abracon LLC; Mfr P/N (none) -> ABS07-32.768KHZ-7-T; Price (none) -> 0.5003; Purchase-URL (none) -> https://www.lcsc.com/product-detail/Crystals_Abracon-LLC-AB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; Supplier 1 (none) -> LCSC; Supplier 1 P/N (none) -> C276424
- Y1: Mfr (none) -> Abracon LLC; Mfr P/N (none) -> ABM8G-40.000MHZ-18-D2Y-T; Note (none) -> solder later; Price (none) -> 0.61000; Purchase-URL (none) -> https://www.digikey.com/en/products/detail/abracon-llc/ABM8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; Supplier 1 (none) -> Digikey; Supplier 1 P/N (none) -> 535-10281-1-ND
