File: Hardware/Gen1/ESP32_POE_Board/1.4/ESP_POE_1.4a/ESP_POE_1.4a/ESP_POE_1.4a.kicad_sch (KiCad schematic)
At the start: 67 parts, among them J2 HMTSW-102-X-X-S-X, J25 SI-46020-F, J4 C3324132, J6 C3324132, T1 LMUN2211LT1G(SOT-23), U2 TPS2376PW(TSSOP-8), U4 LAN8710A-EZC(QFN32), U5 TX4138(ESOIC-8)

Commit message: s
Parts:
- C13: note Solder later -> just in case (they should solder already)
Changed lines of the file:
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@@
       (effects (font (size 1.27 1.27)) hide)
     )
-    (property "note" "Solder later" (at 138.684 117.602 0)
+    (property "note" "just in case (they should solder already)" (at 138.684 117.602 0)
       (effects (font (size 1.27 1.27)) hide)
     )
