File: Hardware/Gen1/Sensing_Board_out/1.1/SensingBoard_rev1.1/SensingBoard_rev1.1.kicad_sch (KiCad schematic)
At the start: 89 parts, among them J1 USB_C_Receptacle, J3 F32R-1A7H1-11024, J5 RS1-02-G, J6 RS1-02-G, J7 3221-10-0300-00, J7 RS1-02-G, J9 RS1-02-G, SW1 PTS815 SJM 250 SMTR LFS, SW2 PTS815 SJM 250 SMTR LFS, U2 BNO055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

Commit message: s
Parts:
- U7: Mfr P/N ESP32-S3-WROOM-1-N8R2 -> ESP32-S3R8; Purchase-URL https://www.lcsc.com/product-detail/WiFi-Modules_Espressif-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 -> https://www.lcsc.com/product-detail/RF-Transceiver-ICs_Espr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; Supplier 1 P/N C2913204 -> C2913194
Changed lines of the file:
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@@
       (effects (font (size 1.27 1.27)) hide)
     )
-    (property "Mfr P/N" "ESP32-S3-WROOM-1-N8R2" (at 403.606 167.132 0)
+    (property "Mfr P/N" "ESP32-S3R8" (at 403.606 167.132 0)
       (effects (font (size 1.27 1.27)) hide)
     )
@@
       (effects (font (size 1.27 1.27)) hide)
     )
-    (property "Purchase-URL" "https://www.lcsc.com/product-detail/WiFi-Modules_Espressif-Systems-ESP32-S3-WROOM-1-N8R2_C2913204.html" (at 403.606 167.132 0)
+    (property "Purchase-URL" "https://www.lcsc.com/product-detail/RF-Transceiver-ICs_Espressif-Systems-ESP32-S3R8_C2913194.html" (at 403.606 167.132 0)
       (effects (font (size 1.27 1.27)) hide)
     )
@@
       (effects (font (size 1.27 1.27)) hide)
     )
-    (property "Supplier 1 P/N" "C2913204" (at 403.606 167.132 0)
+    (property "Supplier 1 P/N" "C2913194" (at 403.606 167.132 0)
       (effects (font (size 1.27 1.27)) hide)
     )

Commit message: s
Parts:
- C10: footprint Capacitor_SMD:C_01005_0402Metric -> Capacitor_SMD:C_0603_1608Metric
Changed lines of the file:
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@@
       (effects (font (size 1.27 1.27)) (justify left))
     )
-    (property "Footprint" "Capacitor_SMD:C_01005_0402Metric" (at 245.0592 62.23 0)
+    (property "Footprint" "Capacitor_SMD:C_0603_1608Metric" (at 245.0592 62.23 0)
       (effects (font (size 1.27 1.27)) hide)
     )
@@
       (effects (font (size 1.27 1.27)) (justify left))
     )
-    (property "Footprint" "Capacitor_SMD:C_01005_0402Metric" (at 306.2732 97.028 0)
-      (effects (font (size 1.27 1.27)) hide)
-    )
+    (property "Footprint" "Capacitor_SMD:C_0603_1608Metric" (at 306.2732 97.028 0)
+      (effects (font (size 1.27 1.27)) hide)
+    )
