File: Hardware/Gen1/Sensing_Board_out/1.1/SensingBoard_rev1.1/SensingBoard_rev1.1.kicad_sch (KiCad schematic)
At the start: 89 parts, among them J1 USB_C_Receptacle, J3 F32R-1A7H1-11024, J5 RS1-02-G, J6 RS1-02-G, J7 3221-10-0300-00, J7 RS1-02-G, J9 RS1-02-G, SW1 PTS815 SJM 250 SMTR LFS, SW2 PTS815 SJM 250 SMTR LFS, U2 BNO055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

Commit message: updates
Parts:
- L2: footprint Inductor_SMD:L_01005_0402Metric -> Inductor_SMD:L_0201_0603Metric
Changed lines of the file:
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@@
       (effects (font (size 1.27 1.27)))
     )
-    (property "Footprint" "Inductor_SMD:L_01005_0402Metric" (at 385.064 151.384 0)
+    (property "Footprint" "Inductor_SMD:L_0201_0603Metric" (at 385.064 151.384 0)
       (effects (font (size 1.27 1.27)) hide)
     )

Commit message: s
Parts:
- C10: Mfr (none) -> YAGEO; Mfr P/N (none) -> CC0603KRX7R9BB104; Supplier 1 P/N (none) -> C14663
- L1, L2: Mfr P/N LQP02TQ2N0B02D -> LQP03TG2N0B02D; Price 0.014 -> 0.0038; Purchase-URL https://www.lcsc.com/product-detail/Inductors-SMD_Murata-Electronics-LQP02TQ2N0B02D_C2048018.html -> https://www.lcsc.com/product-detail/Inductors-SMD_Murata-Electronics-LQP03TG2N0B02D_C86106.html; Supplier 1 P/N C2048018 -> C79382
Changed lines of the file:
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@@
       (effects (font (size 1.27 1.27)) hide)
     )
-    (property "Mfr P/N" "LQP02TQ2N0B02D" (at 385.064 151.384 0)
+    (property "Mfr P/N" "LQP03TG2N0B02D" (at 385.064 151.384 0)
       (effects (font (size 1.27 1.27)) hide)
     )
-    (property "Price" "0.014" (at 385.064 151.384 0)
+    (property "Price" "0.0038" (at 385.064 151.384 0)
       (effects (font (size 1.27 1.27)) hide)
     )
-    (property "Purchase-URL" "https://www.lcsc.com/product-detail/Inductors-SMD_Murata-Electronics-LQP02TQ2N0B02D_C2048018.html" (at 385.064 151.384 0)
+    (property "Purchase-URL" "https://www.lcsc.com/product-detail/Inductors-SMD_Murata-Electronics-LQP03TG2N0B02D_C86106.html" (at 385.064 151.384 0)
       (effects (font (size 1.27 1.27)) hide)
     )
@@
       (effects (font (size 1.27 1.27)) hide)
     )
-    (property "Supplier 1 P/N" "C2048018" (at 385.064 151.384 0)
+    (property "Supplier 1 P/N" "C79382" (at 385.064 151.384 0)
       (effects (font (size 1.27 1.27)) hide)
     )
@@
       (effects (font (size 1.27 1.27)) hide)
     )
+    (property "Mfr" "YAGEO" (at 244.094 58.42 0)
+      (effects (font (size 1.27 1.27)) hide)
+    )
+    (property "Mfr P/N" "CC0603KRX7R9BB104" (at 244.094 58.42 0)
+      (effects (font (size 1.27 1.27)) hide)
+    )
+    (property "Supplier 1 P/N" "C14663" (at 244.094 58.42 0)
+      (effects (font (size 1.27 1.27)) hide)
+    )
     (pin "1")
     (pin "2")
@@
       (effects (font (size 1.27 1.27)) hide)
     )
+    (property "Mfr" "YAGEO" (at 305.308 93.218 0)
+      (effects (font (size 1.27 1.27)) hide)
+    )
+    (property "Mfr P/N" "CC0603KRX7R9BB104" (at 305.308 93.218 0)
+      (effects (font (size 1.27 1.27)) hide)
+    )
+    (property "Supplier 1 P/N" "C14663" (at 305.308 93.218 0)
+      (effects (font (size 1.27 1.27)) hide)
+    )
     (pin "1")
     (pin "2")
@@
       (effects (font (size 1.27 1.27)) hide)
     )
-    (property "Mfr P/N" "LQP02TQ2N0B02D" (at 365.252 167.132 0)
+    (property "Mfr P/N" "LQP03TG2N0B02D" (at 365.252 167.132 0)
       (effects (font (size 1.27 1.27)) hide)
     )
-    (property "Price" "0.014" (at 365.252 167.132 0)
+    (property "Price" "0.0038" (at 365.252 167.132 0)
       (effects (font (size 1.27 1.27)) hide)
     )
-    (property "Purchase-URL" "https://www.lcsc.com/product-detail/Inductors-SMD_Murata-Electronics-LQP02TQ2N0B02D_C2048018.html" (at 365.252 167.132 0)
+    (property "Purchase-URL" "https://www.lcsc.com/product-detail/Inductors-SMD_Murata-Electronics-LQP03TG2N0B02D_C86106.html" (at 365.252 167.132 0)
       (effects (font (size 1.27 1.27)) hide)
     )
@@
       (effects (font (size 1.27 1.27)) hide)
     )
-    (property "Supplier 1 P/N" "C2048018" (at 365.252 167.132 0)
+    (property "Supplier 1 P/N" "C79382" (at 365.252 167.132 0)
       (effects (font (size 1.27 1.27)) hide)
     )
