File: Hardware/Gen1/ESP32_POE_Board/1.4/ESP_POE_1.4b/ESP_POE_1.4b/ESP_POE_1.4b.kicad_sch (KiCad schematic)
At the start: 74 parts, among them J2 1051620001, J26 USB_C_Receptacle, J5 20021311-00012T4LF, J7 20021311-00012T4LF, Q1 Q12MHz/20pF/10ppm/4P/3.2x2.5mm, Q2 BC817-40(SOT23), Q3 BC817-40(SOT23), SW1 PTS815 SJM 250 SMTR LFS, U1 CH340T(SSOP20W), U3 BL4054B-42TPRN(SOT23-5)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

Commit message: s
Parts:
- C29, C8: price (none) -> 0.0009
- J2: Mfr (none) -> Molex; Mfr P/N (none) -> 1051620001; Note (none) -> Solder Later; Supplier 1 (none) -> Digikey; Supplier 1 P/N (none) -> WM14405CT-ND; price (none) -> 0.99000; purchase url (none) -> https://www.digikey.com/en/products/detail/molex/1051620001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
- R1, R18, R19, R32, R36, R37, R39, R47, R6: price (none) -> 0.0005
- R9: price (none) -> 0.0006
Changed lines of the file:
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@@
       (effects (font (size 1.27 1.27)) hide)
     )
-    (property "price" "" (at 543.56 179.07 0)
+    (property "price" "0.0005" (at 543.56 179.07 0)
       (effects (font (size 1.27 1.27)) hide)
     )
@@
       (effects (font (size 1.27 1.27)) hide)
     )
-    (property "price" "" (at 494.03 96.52 0)
+    (property "price" "0.0005" (at 494.03 96.52 0)
       (effects (font (size 1.27 1.27)) hide)
     )
@@
       (effects (font (size 1.27 1.27)) hide)
     )
-    (property "price" "" (at 546.1 179.07 0)
+    (property "price" "0.0005" (at 546.1 179.07 0)
       (effects (font (size 1.27 1.27)) hide)
     )
@@
       (effects (font (size 1.27 1.27)) hide)
     )
-    (property "price" "" (at 275.59 68.58 0)
+    (property "price" "0.0005" (at 275.59 68.58 0)
       (effects (font (size 1.27 1.27)) hide)
     )
@@
       (effects (font (size 1.27 1.27)) hide)
     )
-    (property "price" "" (at 329.692 170.688 0)
+    (property "price" "0.0005" (at 329.692 170.688 0)
       (effects (font (size 1.27 1.27)) hide)
     )
@@
       (effects (font (size 1.27 1.27)) hide)
     )
-    (property "price" "" (at 329.692 175.768 0)
+    (property "price" "0.0005" (at 329.692 175.768 0)
       (effects (font (size 1.27 1.27)) hide)
     )
@@
       (effects (font (size 1.27 1.27)) hide)
     )
-    (property "price" "" (at 291.592 188.468 0)
+    (property "price" "0.0009" (at 291.592 188.468 0)
       (effects (font (size 1.27 1.27)) hide)
     )
@@
       (effects (font (size 1.27 1.27)) hide)
     )
-    (property "price" "" (at 26.416 94.742 0)
+    (property "price" "0.0005" (at 26.416 94.742 0)
       (effects (font (size 1.27 1.27)) hide)
     )
@@
       (effects (font (size 1.27 1.27)) hide)
     )
-    (property "price" "" (at 221.996 54.102 0)
+    (property "price" "0.0006" (at 221.996 54.102 0)
       (effects (font (size 1.27 1.27)) hide)
     )
@@
       (effects (font (size 1.27 1.27)) hide)
     )
-    (property "price" "" (at 136.906 103.632 0)
+    (property "price" "0.0005" (at 136.906 103.632 0)
       (effects (font (size 1.27 1.27)) hide)
     )
@@
       (effects (font (size 1.27 1.27)) hide)
     )
-    (property "price" "" (at 523.748 240.792 0)
+    (property "price" "0.0009" (at 523.748 240.792 0)
       (effects (font (size 1.27 1.27)) hide)
     )
@@
       (effects (font (size 1.27 1.27) italic) hide)
     )
+    (property "Mfr" "Molex" (at 608.838 116.84 0)
+      (effects (font (size 1.27 1.27)) hide)
+    )
+    (property "Mfr P/N" "1051620001" (at 608.838 116.84 0)
+      (effects (font (size 1.27 1.27)) hide)
+    )
+    (property "Note" "Solder Later" (at 608.838 116.84 0)
+      (effects (font (size 1.27 1.27)) hide)
+    )
+    (property "Supplier 1" "Digikey" (at 608.838 116.84 0)
+      (effects (font (size 1.27 1.27)) hide)
+    )
+    (property "Supplier 1 P/N" "WM14405CT-ND" (at 608.838 116.84 0)
+      (effects (font (size 1.27 1.27)) hide)
+    )
+    (property "price" "0.99000" (at 608.838 116.84 0)
+      (effects (font (size 1.27 1.27)) hide)
+    )
+    (property "purchase url" "https://www.digikey.com/en/products/detail/molex/1051620001/4555282?s=N4IgTCBcDaIIwAYCscBsYGbiAugXyA" (at 608.838 116.84 0)
+      (effects (font (size 1.27 1.27)) hide)
+    )
     (pin "G1")
     (pin "G2")
@@
       (effects (font (size 1.27 1.27)) hide)
     )
-    (property "price" "" (at 146.304 161.544 0)
+    (property "price" "0.0005" (at 146.304 161.544 0)
       (effects (font (size 1.27 1.27)) hide)
     )

Commit message: s
Parts:
- U6: Mfr P/N ESP32-WROVER-E-N8R8 -> ESP32-WROOM-32E-N8; Supplier 1 P/N C2973667 -> C701342; price 4.6460 -> 4.6453; purchase url https://www.lcsc.com/product-detail/WiFi-Modules_Espressif-Systems-ESP32-WROVER-E-N8R8_C2973667.html -> https://www.lcsc.com/product-detail/WiFi-Modules_Espressif-Systems-ESP32-WROOM-32E-N8_C701342.html
Changed lines of the file:
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@@
       (effects (font (size 1.27 1.27)) hide)
     )
-    (property "Mfr P/N" "ESP32-WROVER-E-N8R8" (at 337.82 86.36 0)
+    (property "Mfr P/N" "ESP32-WROOM-32E-N8" (at 337.82 86.36 0)
       (effects (font (size 1.27 1.27)) hide)
     )
@@
       (effects (font (size 1.27 1.27)) hide)
     )
-    (property "Supplier 1 P/N" "C2973667" (at 337.82 86.36 0)
+    (property "Supplier 1 P/N" "C701342" (at 337.82 86.36 0)
       (effects (font (size 1.27 1.27)) hide)
     )
-    (property "price" "4.6460" (at 337.82 86.36 0)
+    (property "price" "4.6453" (at 337.82 86.36 0)
       (effects (font (size 1.27 1.27)) hide)
     )
-    (property "purchase url" "https://www.lcsc.com/product-detail/WiFi-Modules_Espressif-Systems-ESP32-WROVER-E-N8R8_C2973667.html" (at 337.82 86.36 0)
+    (property "purchase url" "https://www.lcsc.com/product-detail/WiFi-Modules_Espressif-Systems-ESP32-WROOM-32E-N8_C701342.html" (at 337.82 86.36 0)
       (effects (font (size 1.27 1.27)) hide)
     )
