File: Hardware/Gen2Dev/OuterBoard/2.1/OuterBoard_rev2.1/_autosave-OuterBoard_rev2.1.kicad_pcb (KiCad board)
At the start: 4 copper layers, 101.6 x 76.2 mm, 206 parts, among them J1 HMTSW-102-X-X-S-X, J10 F32R-1A7H1-11024, J11 3221-10-0300-00, J12 HMTSW-102-X-X-S-X, J13 HMTSW-102-X-X-S-X, J14 HMTSW-102-X-X-S-X, J15 HMTSW-102-X-X-S-X, J16 HMTSW-102-X-X-S-X, J17 HMTSW-102-X-X-S-X, J18 HMTSW-102-X-X-S-X, J19 HMTSW-102-X-X-S-X, J2 HMTSW-102-X-X-S-X, J20 HMTSW-102-X-X-S-X, J21 HMTSW-102-X-X-S-X, J22 HMTSW-102-X-X-S-X, J23 HMTSW-102-X-X-S-X, J24 HMTSW-102-X-X-S-X, J25 HMTSW-102-X-X-S-X, J26 HMTSW-102-X-X-S-X, J27 HMTSW-102-X-X-S-X, J28 HMTSW-102-X-X-S-X, J29 HMTSW-102-X-X-S-X, J3 HMTSW-102-X-X-S-X, J30 HMTSW-102-X-X-S-X, J31 HMTSW-102-X-X-S-X, J32 HMTSW-102-X-X-S-X, J33 HMTSW-102-X-X-S-X, J34 HMTSW-102-X-X-S-X, J35 HMTSW-102-X-X-S-X, J36 HMTSW-102-X-X-S-X, J37 HMTSW-102-X-X-S-X, J38 HMTSW-102-X-X-S-X, J39 HMTSW-102-X-X-S-X, J4 HMTSW-102-X-X-S-X, J40 HMTSW-102-X-X-S-X, J41 HMTSW-102-X-X-S-X, J42 UJ31-CH-G2-SMT-TR, J5 HMTSW-102-X-X-S-X, J6 HMTSW-102-X-X-S-X, J7 530470210, J8 530470210, SW1 PTS815 SJM 250 SMTR LFS, SW2 PTS815 SJM 250 SMTR LFS, U1 MCP73812T-420I-OT, U10 GD25D05CT, U2 DRV8410PWPR, U3 MCP73812T-420I-OT, U4 MIC5504-3.3YM5, U5 MIC5504-1.8YM5, U6 MCP1700x-280xxTT, U7 FT232RQ, U8 BNO055, U9 ESP32-S3, Y1 ABM8G-40.000MHZ-18-D2Y-T

Commit message: updates
Parts:
- moved TP40 23.0 mm to (179.0, 133.6)
- moved TP44 18.5 mm to (169.6, 127.5)
- moved TP39 11.5 mm to (178.5, 108.9)
Changed lines of the file:
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@@
   )
   (footprint "TestPoint:TestPoint_Pad_D2.0mm" (layer "F.Cu")
-    (at 187.0456 121.158)
+    (at 169.6212 127.508)
     (descr "SMD pad as test Point, diameter 2.0mm")
     (tags "test point SMD pad")
@@
   )
   (footprint "TestPoint:TestPoint_Pad_D2.0mm" (layer "F.Cu")
-    (at 194.31 116.4844)
+    (at 178.9684 133.604)
     (descr "SMD pad as test Point, diameter 2.0mm")
     (tags "test point SMD pad")
@@
   )
   (footprint "TestPoint:TestPoint_Pad_D2.0mm" (layer "F.Cu")
-    (at 187.452 116.1796)
+    (at 178.5112 108.9152)
     (descr "SMD pad as test Point, diameter 2.0mm")
     (tags "test point SMD pad")
