File: Hardware/Gen2Dev/OuterBoard/2.1/OuterBoard_rev2.1/OuterBoard_rev2.1.kicad_sch (KiCad schematic)
At the start: 112 parts, among them J1 HMTSW-102-X-X-S-X, J1 USB_C_Receptacle, J2 HMTSW-102-X-X-S-X, J3 F32R-1A7H1-11024, J7 3221-10-0300-00, J7 530470210, J8 530470210, SW1 PTS815 SJM 250 SMTR LFS, SW2 PTS815 SJM 250 SMTR LFS, U1 DRV8410PWPR, U2 BNO055, U2 MCP73812T-420I-OT, U3 MCP73812T-420I-OT, U3 MIC5504-3.3YM5, U4 FT232RQ, U5 MIC5504-1.8YM5, U6 MCP1700x-280xxTT, U7 ESP32-S3, U8 GD25D05CT, Y1 ABM8G-40.000MHZ-18-D2Y-T

Commit message: dev board
Other:
- note added: "Updates: Battery Status LED Light DCDC for Wireless Charger Wireless Charging IC"
- note removed: "Updates: Battery Status"
- moved on the sheet: ANT1, C10, C14, C15, C17, C9, D3, D4, D6, FB1, J1, J2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

Commit message: update
Parts:
- removed R11 (x5), R12 (x4): 0k, Resistor_SMD:R_0201_0603Metric, symbol Device:R_US
- added J1, J12, J13, J14, J15, J16, J17, J18, J19, J2, J20, J21, J22, J3, J4: HMTSW-102-X-X-S-X, HMTSW-102-X-X-S-X:SAMTEC_HMTSW-102-X-X-S-X, symbol HMTSW-102-X-X-S-X:HMTSW-102-X-X-S-X
- added TP10, TP3, TP4, TP5, TP6, TP7: TestPoint, TestPoint:TestPoint_Pad_D2.0mm, symbol Connector:TestPoint
Connections:
- net +1V8: now also J22.02; no longer U5.5 (VOUT)
- net +2V8: now also J21.02; no longer U6.2 (VO)
- net +3.3V: now also J20.02; no longer U3.5 (VOUT)
- net +BATT: now also J12.01, J13.01, TP3.1; no longer J7.1, J8.1
- net DRV_FAULT: now also J16.01
- net GND: now also J4.01; no longer D11.2 (A), D12.2 (A)
- net GPIO37: now also J16.02
- net VCC: now also J14.01, J15.01, J3.02, TP5.1; no longer D13.1 (K), D14.1 (K), U2.4 (V_{DD}), U3.4 (V_{DD})
- net VDC: now also J17.01, J18.01, J19.01, TP4.1, TP6.1; no longer U3.1 (VIN), U3.3 (EN), U5.1 (VIN), U5.3 (EN), U6.3 (VI)
- net at D11.1 (K), D13.2 (A): now also J1.02; no longer TP5.1
- net at R21.1, U2.5 (PROG): now also TP7.1
- net at R21.1, U3.5 (PROG): now also TP10.1
- net at D12.1 (K), D14.2 (A): now also J2.01; no longer TP6.1
- new net: D11.2 (A), D12.2 (A), J4.02
- new net: J13.02, J7.1
- new net: J14.02, U2.4 (V_{DD})
- new net: J17.02, U3.1 (VIN), U3.3 (EN)
- new net: J12.02, J8.1
- new net: J21.01, U6.2 (VO)
- new net: J20.01, U3.5 (VOUT)
- new net: J1.01, TP5.1
- new net: D13.1 (K), D14.1 (K), J3.01
- new net: J19.02, U6.3 (VI)
- new net: J2.02, TP6.1
- new net: J22.01, U5.5 (VOUT)
- new net: J18.02, U5.1 (VIN), U5.3 (EN)
- new net: J15.02, U3.4 (V_{DD})
Other:
- moved on the sheet: C10, C9, D5, D6, U3, U5, U6

Commit message: dev board
Parts:
- removed J1: USB_C_Receptacle, Connector_USB:USB_C_Receptacle_Molex_105450-0101-L, symbol Connector:USB_C_Receptacle
- removed R17: 5.1K, Resistor_SMD:R_0201_0603Metric, symbol Device:R_US
- removed R17: 6.1K, Resistor_SMD:R_0201_0603Metric, symbol Device:R_US
- added D6 (x4): LED, LED_SMD:LED_0603_1608Metric, symbol Device:LED
- added J2, J24, J25, J26, J27, J28, J29, J30, J31, J32, J33, J34, J35, J36, J37, J38, J39, J40, J41: HMTSW-102-X-X-S-X, HMTSW-102-X-X-S-X:SAMTEC_HMTSW-102-X-X-S-X, symbol HMTSW-102-X-X-S-X:HMTSW-102-X-X-S-X
- added J42: UJ31-CH-G2-SMT-TR, UJ31-CH-G2-SMT-TR:CUI_UJ31-CH-G2-SMT-TR, symbol UJ31_CH_G2_SMT_TR:UJ31-CH-G2-SMT-TR
- added R16 (x3): 100, Resistor_SMD:R_0201_0603Metric, symbol Device:R_US
- added R16: 100, Resistor_SMD:R_0805_2012Metric, symbol Device:R_US
- added R17: 6.1K, Resistor_SMD:R_0201_0603Metric, symbol Device:R_US
- added R17: 5.1K, Resistor_SMD:R_0201_0603Metric, symbol Device:R_US
- added TP11, TP12, TP13, TP14, TP15, TP16, TP17, TP18, TP19, TP20, TP21, TP22, TP23, TP24, TP25, TP26, TP29, TP30, TP31, TP32, TP33, TP34, TP35, TP36, TP37, TP38, TP39, TP40, TP41, TP42, TP43, TP44, TP45, TP46, TP47, TP48, TP49, TP50, TP51, TP52, TP53, TP54, TP55, TP56, TP57, TP58, TP59, TP60, TP61, TP62, TP63, TP64, TP65, TP8, TP9: TestPoint, TestPoint:TestPoint_Pad_D2.0mm, symbol Connector:TestPoint
- C10, C9: footprint Capacitor_SMD:C_0603_1608Metric -> Capacitor_SMD:C_0805_2012Metric
- C10: footprint Capacitor_SMD:C_0201_0603Metric -> Capacitor_SMD:C_0805_2012Metric
- R11: BOM DNP -> NOSTUFF
Connections:
- net +1V8: now also R16.2, TP48.1
- net +2V8: now also TP42.1, TP49.1, TP63.1; no longer C9.1, J21.02
- net +3.3V: now also J33.02, J34.01, J35.01, J38.01, R16.2, TP12.1, TP38.1; no longer C17.1, U2.28 (VDDIO), U2.3 (VDD), U4.1 (VCCIO), U4.19 (VCC), U7.55 (VDDA), U7.56 (VDDA)
- net +5V: now also J36.01, J42.A4 (VBUS), J42.A9 (VBUS__1), J42.B4 (VBUS__2), J42.B9 (VBUS__3), R16.2; no longer D3.2 (A)
- net +BATT: now also J2.02; no longer U1.12 (VM)
- net BNO_INT: now also J25.01
- net BNO_SCL: now also J26.01
- net BNO_SDA: now also J27.01
- net CAM_RESET: now also TP44.1
- net CHIP_EN: now also TP20.1
- net D0/A0: now also J31.01
- net D1/A1: now also J30.01
- net D2/A2: now also J29.01
- net D3/A3: now also J28.01
- net DRV_FAULT: now also TP11.1
- net DRV_SLEEP: now also J24.01
- net GND: now also D6.1 (K), D6.1 (K), D6.1 (K), D6.1 (K), J39.01, J40.01, J41.01, J42.A1 (GND), J42.A12 (GND__1), J42.B1 (GND__2), J42.B12 (GND__3), J42.SH1 (SHIELD), J42.SH2 (SHIELD__1), J42.SH3 (SHIELD__2), J42.SH4 (SHIELD__3), R17.2, R17.2, TP37.1, TP39.1, TP53.1, TP61.1; no longer U2.10 (PIN10), U2.15 (PIN15), U2.16 (PIN16)
- net GPIO33: now also J27.02
- net GPIO34: now also J26.02
- net GPIO35: now also J25.02
- net GPIO36: now also J24.02
- net IO10/XMCLK: now also TP51.1
- net IO11/DVP_Y8: now also TP52.1
- net IO12/DVP_Y7: now also TP54.1
- net IO13/DVP_PCLK: now also TP55.1
- net IO14/DVP_Y6: now also TP56.1
- net IO15/DVP_Y2: now also TP57.1
- net IO16/DVP_Y5: now also TP58.1
- net IO17/DVP_Y3: now also TP59.1
- net IO18/DVP_Y4: now also TP60.1
- net IO38/DVP_VSYNC: now also TP45.1
- net IO47/DVP_HREF: now also TP47.1
- net IO48/DVP_Y9: now also TP50.1
- net MOTOR1_AIN1: now also J28.02
- net MOTOR1_AIN2: now also J29.02
- net MOTOR2_BIN1: now also J30.02
- net MOTOR2_BIN2: now also J31.02
- net MTCK/IO39/CAM_SCL: now also TP21.1, TP43.1
- net MTDI/IO41/PDM_DATA: now also TP23.1
- net MTDO/IO40/CAM_SDA: now also TP22.1, TP40.1
- net MTMS/IO42/PDM_CLK: now also TP24.1
- net RX_D7: now also TP29.1
- net SPICLK: now also TP16.1
- net SPICS0: now also TP15.1
- net SPID: now also TP17.1
- net SPIQ: now also TP18.1
- net SPIWP: now also TP19.1
- net TX_D6: now also TP30.1
- net USB_DN: now also J42.A6 (DP1), J42.A7 (DN1), TP25.1
- net USB_DP: now also J42.B6 (DP2), J42.B7 (DN2), TP26.1
- net VDC: now also J37.02; no longer D3.1 (K)
- net at R2.1, U2.6 (PS0): now also TP33.1
- net at U7.2 (VDD3P3), U7.3 (VDD3P3): now also J32.02; no longer C17.1, L2.2
- net at C14.1, U7.53 (XTAL_N), Y1.1: now also TP14.1
- net at C14.1, U7.54 (XTAL_P), Y1.3: now also TP13.1
- net at C14.1, U2.26 (XOUT32), XTAL1.1: now also TP32.1
- net at C17.1, C9.1, D4.1 (K)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: now also TP62.1
- net at R21.1, U1.3 (AISEN): now also TP9.1
- net at C15.1, U2.27 (XIN32), XTAL1.2: now also TP31.1
- net at R21.1, U1.6 (BISEN): now also TP8.1
- net at C10.1, U2.9 (CAP): now also TP36.1
- net at R2.1, U2.17 (COM3): now also TP35.1
- net at R2.1, U2.5 (PS1): now also TP34.1
- net at FB1.2, J3.4: now also TP41.1
- net at J3.8, R14.1: now also TP46.1
- new net: J42.A5 (CC1), R17.1, TP64.1
- new net: D6.2 (A), R16.1 (x4)
- new net: J33.01, U7.55 (VDDA), U7.56 (VDDA)
- new net: C17.1, J32.01, L2.2
- new net: J42.B5 (CC2), R17.1, TP65.1
- new net: J2.01, U1.12 (VM)
- new net: J40.02, U2.15 (PIN15)
- new net: C9.1, J21.02, R16.2
- new net: D3.1 (K), J37.01
- new net: D3.2 (A), J36.02
- new net: J35.02, U4.1 (VCCIO), U4.19 (VCC)
- new net: J39.02, U2.10 (PIN10)
- new net: J41.02, U2.16 (PIN16)
- new net: J38.02, U2.28 (VDDIO), U2.3 (VDD)
- new net: C17.1, J34.02
- no-connect marks 12 -> 2
Other:
- note added: "check forward voltage"
- moved on the sheet: ANT1, C10, C14, C15, C17, C9, D3, D4, D6, FB1, J1, J16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

Commit message: updates
Parts:
- C10: footprint Capacitor_SMD:C_0201_0603Metric -> Capacitor_SMD:C_0805_2012Metric
- C10: footprint Capacitor_SMD:C_01005_0402Metric -> Capacitor_SMD:C_0805_2012Metric
- C17, C9: footprint Capacitor_SMD:C_0402_1005Metric -> Capacitor_SMD:C_0805_2012Metric
- C9: footprint Capacitor_SMD:C_0603_1608Metric -> Capacitor_SMD:C_0805_2012Metric
- R11, R14, R15, R16, R17, R2: footprint Resistor_SMD:R_0201_0603Metric -> Resistor_SMD:R_0805_2012Metric
Other:
- moved on the sheet: C10, C9, D6, R14, R16, TP37, TP64

Commit message: stuff
Parts:
- removed R14 (x2): 10k, Resistor_SMD:R_0201_0603Metric, symbol Device:R_US
- added R14 (x2): 10k, Resistor_SMD:R_0805_2012Metric, symbol Device:R_US
- L1, L2: footprint Inductor_SMD:L_01005_0402Metric -> Inductor_SMD:L_0402_1005Metric
- R14, R16: footprint Resistor_SMD:R_0201_0603Metric -> Resistor_SMD:R_0805_2012Metric
Connections:
- net +3.3V: now also C17.1, J34.02, R14.1, R14.1; no longer J34.01, U8.8 (VCC)
- net BNO_SCL: now also R14.2
- net BNO_SDA: now also R14.2
- new net: J34.01, U8.8 (VCC)
Other:
- moved on the sheet: C10, J34, TP36

Commit message: stuff
Other:
- note added: "Updates: Battery Status Mounting Holes"
- note removed: "Updates: Battery Status LED Light DCDC for Wireless Charger Wireless Charging IC"
Changed lines of the file:
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@@
     (effects (font (size 4 4)) (justify left bottom))
   )
-  (text "Updates:\nBattery Status\nLED Light\nDCDC for Wireless Charger\nWireless Charging IC"
-    (at 862.838 110.744 0)
+  (text "Updates:\nBattery Status\nMounting Holes" (at 862.838 110.744 0)
     (effects (font (size 1.27 1.27)) (justify left bottom))
   )

Commit message: stuff
Other:
- note added: "Updates: Battery Status Mounting Holes needs 5V to 9V boost for charging rail"
- note removed: "Updates: Battery Status Mounting Holes"
Changed lines of the file:
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@@
     (effects (font (size 4 4)) (justify left bottom))
   )
-  (text "Updates:\nBattery Status\nMounting Holes" (at 862.838 110.744 0)
+  (text "Updates:\nBattery Status\nMounting Holes\nneeds 5V to 9V boost for charging rail"
+    (at 862.838 110.744 0)
     (effects (font (size 1.27 1.27)) (justify left bottom))
   )

Commit message: stuff
Parts:
- added H1, H2, H3, H4: MountingHole, MountingHole:MountingHole_2.1mm, symbol Mechanical:MountingHole
- added TP27: TestPoint, TestPoint:TestPoint_Pad_D2.0mm, symbol Connector:TestPoint
Connections:
- net IO21/USER_LED: now also TP27.1
Other:
- note added: "Mounting Holes"
- note removed: "Updates: Battery Status Mounting Holes needs 5V to 9V boost for charging rail"
Changed lines of the file:
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@@
   (junction (at 47.498 68.58) (diameter 0) (color 0 0 0 0)
   )
+  (junction (at 543.306 284.988) (diameter 0) (color 0 0 0 0)
+  )
   (junction (at 671.83 529.844) (diameter 0) (color 0 0 0 0)
   )
@@
     (stroke (width 0) (type default))
   )
+  (polyline (pts (xy 68.072 503.174) (xy 184.912 503.174))
+    (stroke (width 0) (type default))
+  )
   (wire (pts (xy 577.596 117.602) (xy 601.472 117.602))
     (stroke (width 0) (type default))
@@
     (stroke (width 0) (type default))
   )
+  (polyline (pts (xy 184.912 503.174) (xy 184.912 547.116))
+    (stroke (width 0) (type default))
+  )
   (wire (pts (xy 695.96 255.778) (xy 690.372 255.778))
     (stroke (width 0) (type default))
@@
     (stroke (width 0) (type default))
   )
+  (wire (pts (xy 556.768 284.988) (xy 556.768 284.226))
+    (stroke (width 0) (type default))
+  )
   (wire (pts (xy 684.784 381.254) (xy 690.88 381.254))
     (stroke (width 0) (type default))
@@
     (stroke (width 0) (type default))
   )
+  (wire (pts (xy 543.306 284.988) (xy 556.768 284.988))
+    (stroke (width 0) (type default))
+  )
   (wire (pts (xy 281.178 148.59) (xy 281.178 148.336))
     (stroke (width 0) (type default))
@@
     (stroke (width 0) (type default))
   )
+  (polyline (pts (xy 68.072 547.116) (xy 184.912 547.116))
+    (stroke (width 0) (type default))
+  )
   (wire (pts (xy 545.846 224.028) (xy 545.846 222.25))
     (stroke (width 0) (type default))
@@
     (stroke (width 0) (type default))
   )
+  (polyline (pts (xy 68.072 503.174) (xy 68.072 547.116))
+    (stroke (width 0) (type default))
+  )
   (wire (pts (xy 79.502 285.496) (xy 79.502 288.036))
     (stroke (width 0) (type default))
@@
     (effects (font (size 4 4)) (justify left bottom))
   )
+  (text "Mounting Holes" (at 99.568 510.794 0)
+    (effects (font (size 4 4)) (justify left bottom))
+  )
   (text "BOOT" (at 586.486 408.686 0)
     (effects (font (size 1.27 1.27)) (justify left bottom))
@@
     (effects (font (size 4 4)) (justify left bottom))
   )
-  (text "Updates:\nBattery Status\nMounting Holes\nneeds 5V to 9V boost for charging rail"
-    (at 862.838 110.744 0)
-    (effects (font (size 1.27 1.27)) (justify left bottom))
-  )
   (text "2v8 LDO" (at 143.256 162.052 0)
     (effects (font (size 4 4)) (justify left bottom))
@@
     )
   )
+  (symbol (lib_id "Mechanical:MountingHole") (at 128.524 534.67 0) (unit 1)
+    (in_bom yes) (on_board yes) (dnp no) (fields_autoplaced)
+    (property "Reference" "H4" (at 131.572 533.4 0)
+      (effects (font (size 1.27 1.27)) (justify left))
+    )
+    (property "Value" "MountingHole" (at 131.572 535.94 0)
+      (effects (font (size 1.27 1.27)) (justify left))
+    )
+    (property "Footprint" "MountingHole:MountingHole_2.1mm" (at 128.524 534.67 0)
+      (effects (font (size 1.27 1.27)) hide)
+    )
+    (property "Datasheet" "~" (at 128.524 534.67 0)
+      (effects (font (size 1.27 1.27)) hide)
+    )
+    (property "note" "" (at 128.524 534.67 0)
+      (effects (font (size 1.27 1.27)) hide)
+    )
+    (instances
+      (project "InnerBoard_rev2.1"
+        (path "/5675e374-4d13-4550-a947-518e8da4d5de"
+          (reference "H4") (unit 1)
+        )
+      )
+      (project "OuterBoard_rev2.1"
+        (path "/e0487af4-02df-420a-a23b-b16cb445dead"
+          (reference "H3") (unit 1)
+        )
+      )
+      (project "ESP_POE_1.4a"
+        (path "/e282cc28-a468-4b1a-8ebc-006ea330625e"
+          (reference "H2") (unit 1)
+        )
+      )
+    )
+  )
   (symbol (lib_id "ESP32S3:ESP32-S3") (at 624.332 202.438 0) (unit 1)
     (in_bom yes) (on_board yes) (dnp no) (fields_autoplaced)
@@
     )
   )
+  (symbol (lib_id "Mechanical:MountingHole") (at 99.314 521.716 0) (unit 1)
+    (in_bom yes) (on_board yes) (dnp no) (fields_autoplaced)
+    (property "Reference" "H1" (at 102.362 520.446 0)
+      (effects (font (size 1.27 1.27)) (justify left))
+    )
+    (property "Value" "MountingHole" (at 102.362 522.986 0)
+      (effects (font (size 1.27 1.27)) (justify left))
+    )
+    (property "Footprint" "MountingHole:MountingHole_2.1mm" (at 99.314 521.716 0)
+      (effects (font (size 1.27 1.27)) hide)
+    )
+    (property "Datasheet" "~" (at 99.314 521.716 0)
+      (effects (font (size 1.27 1.27)) hide)
+    )
+    (property "note" "" (at 99.314 521.716 0)
+      (effects (font (size 1.27 1.27)) hide)
+    )
+    (instances
+      (project "InnerBoard_rev2.1"
+        (path "/5675e374-4d13-4550-a947-518e8da4d5de"
+          (reference "H1") (unit 1)
+        )
+      )
+      (project "OuterBoard_rev2.1"
+        (path "/e0487af4-02df-420a-a23b-b16cb445dead"
+          (reference "H2") (unit 1)
+        )
+      )
+      (project "ESP_POE_1.4a"
+        (path "/e282cc28-a468-4b1a-8ebc-006ea330625e"
+          (reference "H1") (unit 1)
+        )
+      )
+    )
+  )
   (symbol (lib_id "power:VCC") (at 101.6 35.814 0) (unit 1)
     (in_bom yes) (on_board yes) (dnp no) (fields_autoplaced)
@@
     )
   )
+  (symbol (lib_id "Mechanical:MountingHole") (at 98.298 534.162 0) (unit 1)
+    (in_bom yes) (on_board yes) (dnp no) (fields_autoplaced)
+    (property "Reference" "H3" (at 101.346 532.892 0)
+      (effects (font (size 1.27 1.27)) (justify left))
+    )
+    (property "Value" "MountingHole" (at 101.346 535.432 0)
+      (effects (font (size 1.27 1.27)) (justify left))
+    )
+    (property "Footprint" "MountingHole:MountingHole_2.1mm" (at 98.298 534.162 0)
+      (effects (font (size 1.27 1.27)) hide)
+    )
+    (property "Datasheet" "~" (at 98.298 534.162 0)
+      (effects (font (size 1.27 1.27)) hide)
+    )
+    (property "note" "" (at 98.298 534.162 0)
+      (effects (font (size 1.27 1.27)) hide)
+    )
+    (instances
+      (project "InnerBoard_rev2.1"
+        (path "/5675e374-4d13-4550-a947-518e8da4d5de"
+          (reference "H3") (unit 1)
+        )
+      )
+      (project "OuterBoard_rev2.1"
+        (path "/e0487af4-02df-420a-a23b-b16cb445dead"
+          (reference "H1") (unit 1)
+        )
+      )
+      (project "ESP_POE_1.4a"
+        (path "/e282cc28-a468-4b1a-8ebc-006ea330625e"
+          (reference "H1") (unit 1)
+        )
+      )
+    )
+  )
   (symbol (lib_id "HMTSW-102-X-X-S-X:HMTSW-102-X-X-S-X") (at 656.59 140.462 270) (unit 1)
     (in_bom yes) (on_board yes) (dnp no)
@@
     )
   )
+  (symbol (lib_id "Connector:TestPoint") (at 556.768 284.226 0) (unit 1)
+    (in_bom yes) (on_board yes) (dnp no)
+    (property "Reference" "TP27" (at 554.736 278.892 0)
+      (effects (font (size 1.27 1.27)) (justify left))
+    )
+    (property "Value" "TestPoint" (at 552.704 278.892 0)
+      (effects (font (size 1.27 1.27)) (justify left) hide)
+    )
+    (property "Footprint" "TestPoint:TestPoint_Pad_D2.0mm" (at 561.848 284.226 0)
+      (effects (font (size 1.27 1.27)) hide)
+    )
+    (property "Datasheet" "~" (at 561.848 284.226 0)
+      (effects (font (size 1.27 1.27)) hide)
+    )
+    (pin "1")
+    (instances
+      (project "OuterBoard_rev2.1"
+        (path "/e0487af4-02df-420a-a23b-b16cb445dead"
+          (reference "TP27") (unit 1)
+        )
+      )
+    )
+  )
   (symbol (lib_id "Connector:TestPoint") (at 86.106 295.656 180) (unit 1)
     (in_bom yes) (on_board yes) (dnp no)
@@
         )
       )
+    )
+  )
+  (symbol (lib_id "Mechanical:MountingHole") (at 129.54 522.224 0) (unit 1)
+    (in_bom yes) (on_board yes) (dnp no) (fields_autoplaced)
+    (property "Reference" "H2" (at 132.588 520.954 0)
+      (effects (font (size 1.27 1.27)) (justify left))
+    )
+    (property "Value" "MountingHole" (at 132.588 523.494 0)
+      (effects (font (size 1.27 1.27)) (justify left))
+    )
+    (property "Footprint" "MountingHole:MountingHole_2.1mm" (at 129.54 522.224 0)
+      (effects (font (size 1.27 1.27)) hide)
+    )
+    (property "Datasheet" "~" (at 129.54 522.224 0)
+      (effects (font (size 1.27 1.27)) hide)
+    )
+    (property "note" "" (at 129.54 522.224 0)
+      (effects (font (size 1.27 1.27)) hide)
+    )
+    (instances
+      (project "InnerBoard_rev2.1"
+        (path "/5675e374-4d13-4550-a947-518e8da4d5de"
+          (reference "H2") (unit 1)
+        )
+      )
+      (project "OuterBoard_rev2.1"
+        (path "/e0487af4-02df-420a-a23b-b16cb445dead"
+          (reference "H4") (unit 1)
+        )
+      )
+      (project "ESP_POE_1.4a"
+        (path "/e282cc28-a468-4b1a-8ebc-006ea330625e"
+          (reference "H2") (unit 1)
+        )
+      )
