File: Hardware/Gen2Dev/OuterBoard/2.1/OuterBoard_rev2.1/OuterBoard_rev2.1.kicad_sch (KiCad schematic)
At the start: 211 parts, among them J1 HMTSW-102-X-X-S-X, J12 HMTSW-102-X-X-S-X, J13 HMTSW-102-X-X-S-X, J14 HMTSW-102-X-X-S-X, J15 HMTSW-102-X-X-S-X, J16 HMTSW-102-X-X-S-X, J17 HMTSW-102-X-X-S-X, J18 HMTSW-102-X-X-S-X, J19 HMTSW-102-X-X-S-X, J2 HMTSW-102-X-X-S-X, J20 HMTSW-102-X-X-S-X, J21 HMTSW-102-X-X-S-X, J22 HMTSW-102-X-X-S-X, J24 HMTSW-102-X-X-S-X, J25 HMTSW-102-X-X-S-X, J26 HMTSW-102-X-X-S-X, J27 HMTSW-102-X-X-S-X, J28 HMTSW-102-X-X-S-X, J29 HMTSW-102-X-X-S-X, J3 F32R-1A7H1-11024, J3 HMTSW-102-X-X-S-X, J30 HMTSW-102-X-X-S-X, J31 HMTSW-102-X-X-S-X, J32 HMTSW-102-X-X-S-X, J33 HMTSW-102-X-X-S-X, J34 HMTSW-102-X-X-S-X, J35 HMTSW-102-X-X-S-X, J36 HMTSW-102-X-X-S-X, J37 HMTSW-102-X-X-S-X, J38 HMTSW-102-X-X-S-X, J39 HMTSW-102-X-X-S-X, J4 HMTSW-102-X-X-S-X, J40 HMTSW-102-X-X-S-X, J41 HMTSW-102-X-X-S-X, J42 UJ31-CH-G2-SMT-TR, J7 3221-10-0300-00, J7 530470210, J8 530470210, SW1 PTS815 SJM 250 SMTR LFS, SW2 PTS815 SJM 250 SMTR LFS, U1 DRV8410PWPR, U2 BNO055, U2 MCP73812T-420I-OT, U3 MCP73812T-420I-OT, U3 MIC5504-3.3YM5, U4 FT232RQ, U5 MIC5504-1.8YM5, U6 MCP1700x-280xxTT, U7 ESP32-S3, U8 GD25D05CT, Y1 ABM8G-40.000MHZ-18-D2Y-T

Commit message: stuff
Other:
- moved on the sheet: ANT1, C10, C14, C15, C17, C9, D4, D6, FB1, H1, H2, H3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

Commit message: poe
Parts:
- U8: value GD25D05CT -> GD25WQ80ETIGR; Mfr GigaDevice Semiconductor (HK) Limited -> (none); Mfr P/N 1970-1000-1-ND -> (none); Note solder later -> (none); Price 0.33000 -> (none); Purchase-URL https://www.digikey.com/en/products/detail/gigadevice-semic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 -> (none); Supplier 1 Digikey -> (none); Supplier 1 P/N GD25D05CTIGR -> GD25WQ80ETIGR
Other:
- note added: "Notes on things to fix based on Gen 1 Boards: Get rid of FTDI Make sure we have 8MB of Flash"
Changed lines of the file:
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@@
     (effects (font (size 4 4)) (justify left bottom))
   )
+  (text "Notes on things to fix based on Gen 1 Boards:\n\nGet rid of FTDI\nMake sure we have 8MB of Flash"
+    (at 849.376 37.846 0)
+    (effects (font (size 1.27 1.27)) (justify left bottom))
+  )
   (text "BATTERY CHARGER 2" (at 257.302 24.892 0)
     (effects (font (size 3 3)) (justify left bottom))
@@
       (effects (font (size 1.27 1.27)) (justify left))
     )
-    (property "Value" "GD25D05CT" (at 564.134 180.34 0)
+    (property "Value" "GD25WQ80ETIGR" (at 564.134 180.34 0)
       (effects (font (size 1.27 1.27)) (justify left))
     )
@@
       (effects (font (size 1.27 1.27)) hide)
     )
-    (property "Datasheet" "http://www.elm-tech.com/en/products/spi-flash-memory/gd25d10/gd25d10.pdf" (at 555.244 172.212 0)
+    (property "Datasheet" "" (at 555.244 172.212 0)
       (effects (font (size 1.27 1.27)) hide)
     )
-    (property "Mfr" "GigaDevice Semiconductor (HK) Limited" (at 555.244 172.212 0)
+    (property "Mfr" "" (at 555.244 172.212 0)
       (effects (font (size 1.27 1.27)) hide)
     )
-    (property "Mfr P/N" "1970-1000-1-ND" (at 555.244 172.212 0)
+    (property "Mfr P/N" "" (at 555.244 172.212 0)
       (effects (font (size 1.27 1.27)) hide)
     )
-    (property "Note" "solder later" (at 555.244 172.212 0)
+    (property "Note" "" (at 555.244 172.212 0)
       (effects (font (size 1.27 1.27)) hide)
     )
-    (property "Price" "0.33000" (at 555.244 172.212 0)
+    (property "Price" "" (at 555.244 172.212 0)
       (effects (font (size 1.27 1.27)) hide)
     )
-    (property "Purchase-URL" "https://www.digikey.com/en/products/detail/gigadevice-semiconductor-hk-limited/GD25D05CTIGR/9484665" (at 555.244 172.212 0)
+    (property "Purchase-URL" "" (at 555.244 172.212 0)
       (effects (font (size 1.27 1.27)) hide)
     )
-    (property "Supplier 1" "Digikey" (at 555.244 172.212 0)
+    (property "Supplier 1" "" (at 555.244 172.212 0)
       (effects (font (size 1.27 1.27)) hide)
     )
-    (property "Supplier 1 P/N" "GD25D05CTIGR" (at 555.244 172.212 0)
+    (property "Supplier 1 P/N" "GD25WQ80ETIGR" (at 555.244 172.212 0)
       (effects (font (size 1.27 1.27)) hide)
     )

Commit message: stuff
Parts:
- removed TP29, TP30: TestPoint, TestPoint:TestPoint_Pad_D2.0mm, symbol Connector:TestPoint
- added D3: PMEG6010CEJ, Diode_SMD:D_SOD-323F, symbol Diode:PMEG6010CEJ
- added D6: LED, LED_SMD:LED_0603_1608Metric, symbol Device:LED
- added J43, J45, J46, J47, J48, J49, J50, J51, J52, J9: HMTSW-102-X-X-S-X, HMTSW-102-X-X-S-X:SAMTEC_HMTSW-102-X-X-S-X, symbol HMTSW-102-X-X-S-X:HMTSW-102-X-X-S-X
- added J44: 87520-0010BLF, 87520-0010BLF:AMPHENOL_87520-0010BLF, symbol 87520-0010BLF:87520-0010BLF
- added R16: 100, Resistor_SMD:R_0805_2012Metric, symbol Device:R_US
- U8: value GD25WQ80ETIGR -> GD25Q64CSIGR
Connections:
- net +5V: now also J44.1 (VCC), J45.01, R16.2
- net GND: now also D6.1 (K), J44.4 (GND), J44.SH1 (SHIELD), J44.SH2 (SHIELD__1)
- net RX_D7: now also J51.02; no longer U4.30 (TXD)
- net TX_D6: now also J52.01; no longer U4.2 (RXD)
- net USB_DN: now also J43.02, J47.02, J49.02; no longer J42.A6 (DP1), J42.A7 (DN1), TP25.1, U4.15 (USBDM)
- net USB_DP: now also J48.01, J50.01, J9.01; no longer J42.B6 (DP2), J42.B7 (DN2), TP26.1, U4.14 (USBDP)
- net VDC: now also J46.02
- new net: J9.02, U4.14 (USBDP)
- new net: J44.2 (D-), J47.01
- new net: J44.3 (D+), J48.02
- new net: D3.1 (K), J46.01
- new net: J43.01, U4.15 (USBDM)
- new net: J52.02, U4.2 (RXD)
- new net: D6.2 (A), R16.1
- new net: D3.2 (A), J45.02
- new net: J42.A6 (DP1), J42.A7 (DN1), J49.01, TP25.1
- new net: J42.B6 (DP2), J42.B7 (DN2), J50.02, TP26.1
- new net: J51.01, U4.30 (TXD)
Other:
- note added: "FIX FLASH FOOTPRINT"
- note added: "USB 2.0"
- note removed: "Notes on things to fix based on Gen 1 Boards: Get rid of FTDI Make sure we have 8MB of Flash"
- moved on the sheet: J7, R15, SW1, SW2, TP20, TP21, TP22, TP23, TP24, TP25, TP26

Commit message: stuff
Parts:
- removed TP15, TP18, TP19: TestPoint, TestPoint:TestPoint_Pad_D2.0mm, symbol Connector:TestPoint
- removed U8: GD25Q64CSIGR, Package_SO:SOP-8_3.9x4.9mm_P1.27mm, symbol Memory_Flash:GD25D05CT
- added TP28, TP29, TP30: TestPoint, TestPoint:TestPoint_Pad_D2.0mm, symbol Connector:TestPoint
- added U11: GD25Q64CSIGR, SOP8_208MIL_GDV, symbol GD25Q64CSIGR:GD25Q64CSIGR
Connections:
- net GND: now also U11.4 (VSS)
- net SPICLK: now also U11.6 (SCLK)
- net SPICS0: now also TP17.1, U11.1 (CS#)
- net SPID: now also TP30.1, U11.5 (SI(IO0)); no longer TP17.1
- net SPIQ: now also TP28.1, U11.2 (SO(IO1))
- net SPIWP: now also TP29.1, U11.3 (WP#(IO2))
- net at J34.01: now also U11.8 (VCC)
- no-connect marks 2 -> 3
Other:
- note removed: "FIX FLASH FOOTPRINT"

Commit message: stuff
Parts:
- added TP15: TestPoint, TestPoint:TestPoint_Pad_D2.0mm, symbol Connector:TestPoint
Connections:
- net +3.3V: no longer C17.1, J34.02
- net SPIHD: now also U11.7 (HOLD#(IO3)), TP15.1
- net VDD_SPI: now also C17.1, J34.02
- no-connect marks 3 -> 2
Other:
- moved on the sheet: TP16, TP30

Commit message: a
Parts:
- ANT1, C9: Note (none) -> 1
- C9: Mfr P/N CL21A106KAYNNNE -> CL10A106KP8NNNC; Note (none) -> 1
Changed lines of the file:
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@@
       (effects (font (size 1.27 1.27)) hide)
     )
-    (property "Mfr P/N" "CL21A106KAYNNNE" (at 101.6 56.896 0)
+    (property "Mfr P/N" "CL10A106KP8NNNC" (at 101.6 56.896 0)
       (effects (font (size 1.27 1.27)) hide)
     )
@@
       (effects (font (size 1.27 1.27)) hide)
     )
+    (property "Note" "1" (at 101.6 56.896 0)
+      (effects (font (size 1.27 1.27)) hide)
+    )
     (pin "1")
     (pin "2")
@@
       (effects (font (size 1.27 1.27)) hide)
     )
-    (property "Note" "" (at 202.692 276.86 0)
+    (property "Note" "1" (at 202.692 276.86 0)
       (effects (font (size 1.27 1.27)) hide)
     )
@@
       (effects (font (size 1.27 1.27)) hide)
     )
-    (property "Note" "" (at 199.39 182.372 0)
+    (property "Note" "1" (at 199.39 182.372 0)
       (effects (font (size 1.27 1.27)) hide)
     )
@@
       (effects (font (size 1.27 1.27)) hide)
     )
-    (property "Note" "" (at 137.16 181.61 0)
+    (property "Note" "1" (at 137.16 181.61 0)
       (effects (font (size 1.27 1.27)) hide)
     )
@@
       (effects (font (size 1.27 1.27)) hide)
     )
-    (property "Note" "" (at 241.3 114.3 0)
+    (property "Note" "1" (at 241.3 114.3 0)
       (effects (font (size 1.27 1.27)) hide)
     )
@@
       (effects (font (size 1.27 1.27)) hide)
     )
+    (property "Note" "1" (at 90.424 56.896 0)
+      (effects (font (size 1.27 1.27)) hide)
+    )
     (pin "1")
     (pin "2")
@@
       (effects (font (size 1.27 1.27)) hide)
     )
-    (property "Note" "" (at 136.906 111.252 0)
+    (property "Note" "1" (at 136.906 111.252 0)
       (effects (font (size 1.27 1.27)) hide)
     )
@@
       (effects (font (size 1.27 1.27)) hide)
     )
-    (property "Note" "" (at 298.958 114.554 0)
+    (property "Note" "1" (at 298.958 114.554 0)
       (effects (font (size 1.27 1.27)) hide)
     )
@@
       (effects (font (size 1.27 1.27)) (justify bottom) hide)
     )
-    (property "Note" "" (at 592.074 145.034 0)
+    (property "Note" "1" (at 592.074 145.034 0)
       (effects (font (size 1.27 1.27)) hide)
     )
@@
       (effects (font (size 1.27 1.27)) hide)
     )
-    (property "Note" "" (at 192.532 114.808 0)
+    (property "Note" "1" (at 192.532 114.808 0)
       (effects (font (size 1.27 1.27)) hide)
     )

Commit message: stuff
Parts:
- C14, C15: footprint Capacitor_SMD:C_0201_0603Metric -> Capacitor_SMD:C_0402_1005Metric
Changed lines of the file:
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@@
       (effects (font (size 1.27 1.27)))
     )
-    (property "Footprint" "Capacitor_SMD:C_0201_0603Metric" (at 736.092 277.6728 0)
+    (property "Footprint" "Capacitor_SMD:C_0402_1005Metric" (at 736.092 277.6728 0)
       (effects (font (size 1.27 1.27)) hide)
     )
@@
       (effects (font (size 1.27 1.27)))
     )
-    (property "Footprint" "Capacitor_SMD:C_0201_0603Metric" (at 736.092 267.0048 0)
+    (property "Footprint" "Capacitor_SMD:C_0402_1005Metric" (at 736.092 267.0048 0)
       (effects (font (size 1.27 1.27)) hide)
     )
