File: Hardware/Gen2Dev/OuterBoard/2.1/OuterBoard_rev2.1/OuterBoard_rev2.1.kicad_pcb (KiCad board)
At the start: 4 copper layers, 101.6 x 76.2 mm, 206 parts, among them J1 HMTSW-102-X-X-S-X, J10 F32R-1A7H1-11024, J11 3221-10-0300-00, J12 HMTSW-102-X-X-S-X, J13 HMTSW-102-X-X-S-X, J14 HMTSW-102-X-X-S-X, J15 HMTSW-102-X-X-S-X, J16 HMTSW-102-X-X-S-X, J17 HMTSW-102-X-X-S-X, J18 HMTSW-102-X-X-S-X, J19 HMTSW-102-X-X-S-X, J2 HMTSW-102-X-X-S-X, J20 HMTSW-102-X-X-S-X, J21 HMTSW-102-X-X-S-X, J22 HMTSW-102-X-X-S-X, J23 HMTSW-102-X-X-S-X, J24 HMTSW-102-X-X-S-X, J25 HMTSW-102-X-X-S-X, J26 HMTSW-102-X-X-S-X, J27 HMTSW-102-X-X-S-X, J28 HMTSW-102-X-X-S-X, J29 HMTSW-102-X-X-S-X, J3 HMTSW-102-X-X-S-X, J30 HMTSW-102-X-X-S-X, J31 HMTSW-102-X-X-S-X, J32 HMTSW-102-X-X-S-X, J33 HMTSW-102-X-X-S-X, J34 HMTSW-102-X-X-S-X, J35 HMTSW-102-X-X-S-X, J36 HMTSW-102-X-X-S-X, J37 HMTSW-102-X-X-S-X, J38 HMTSW-102-X-X-S-X, J39 HMTSW-102-X-X-S-X, J4 HMTSW-102-X-X-S-X, J40 HMTSW-102-X-X-S-X, J41 HMTSW-102-X-X-S-X, J42 UJ31-CH-G2-SMT-TR, J5 HMTSW-102-X-X-S-X, J6 HMTSW-102-X-X-S-X, J7 530470210, J8 530470210, SW1 PTS815 SJM 250 SMTR LFS, SW2 PTS815 SJM 250 SMTR LFS, U1 MCP73812T-420I-OT, U10 GD25D05CT, U2 DRV8410PWPR, U3 MCP73812T-420I-OT, U4 MIC5504-3.3YM5, U5 MIC5504-1.8YM5, U6 MCP1700x-280xxTT, U7 FT232RQ, U8 BNO055, U9 ESP32-S3, Y1 ABM8G-40.000MHZ-18-D2Y-T

Commit message: stuff
Parts:
- removed R20, R21: 10k, Resistor_SMD:R_0201_0603Metric
- added R11: 10k, Resistor_SMD:R_0805_2012Metric, F.Cu at (128.5, 128.7)
- added R12: 10k, Resistor_SMD:R_0805_2012Metric, F.Cu at (117.9, 124.3)
- L1, L2: footprint Inductor_SMD:L_01005_0402Metric -> Inductor_SMD:L_0402_1005Metric
- R19, R25: footprint Resistor_SMD:R_0201_0603Metric -> Resistor_SMD:R_0805_2012Metric
- moved C40 195.6 mm to (112.6, 109.9), turned to -90 degrees
- moved C39 195.3 mm to (108.0, 109.9), turned to -90 degrees
- moved C41 190.8 mm to (117.1, 109.9), turned to -90 degrees
- moved C42 179.8 mm to (132.8, 128.7)
- moved TP7 178.1 mm to (102.3, 89.6)
- moved R13 178.0 mm to (103.0, 114.4)
- moved R14 172.4 mm to (108.4, 114.4)
- moved C32 171.2 mm to (132.8, 125.2)
- moved D9 166.4 mm to (114.1, 134.2)
- moved L2 166.3 mm to (121.1, 105.1)
- moved R31 162.9 mm to (124.5, 128.0), turned to 180 degrees
- moved TP25 161.2 mm to (93.3, 126.5)
- moved C29 161.0 mm to (124.3, 95.5), turned to -90 degrees
- moved TP26 159.8 mm to (93.2, 122.9)
- moved C44 159.2 mm to (145.7, 90.6), turned to 180 degrees
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Connections:
- C44 pad 1: Net-(C44-Pad1) -> +3.3V
- J34 pad 01: +3.3V -> Net-(U10-VCC)
- J34 pad 02: Net-(C44-Pad1) -> +3.3V
- U10 pad 8: +3.3V -> Net-(U10-VCC)
Routing:
- net Net-(D3-K): track 0.00 -> 20.5 mm
- net Net-(D1-A): track 0.00 -> 16.4 mm
- net Net-(D1-K): track 0.00 -> 11.8 mm
- net Net-(D2-K): track 0.00 -> 10.0 mm
- net VCC: track 0.00 -> 9.77 mm
- net Net-(J1-Pad01): track 0.00 -> 3.69 mm
- net Net-(J2-Pad02): track 0.00 -> 3.68 mm
- net GND: track 0.00 -> 3.37 mm, vias 0 -> 2
Other:
- outline, holes or cut-outs redrawn
- board text added: "Camera Connector"
- board text added: "ESP32"
- board text added: "JTAG"

Commit message: stuff
Parts:
- added H1: MountingHole, MountingHole:MountingHole_2.1mm, F.Cu at (84.8, 132.6)
- added H2: MountingHole, MountingHole:MountingHole_2.1mm, F.Cu at (178.7, 64.2)
- added H3: MountingHole, MountingHole:MountingHole_2.1mm, F.Cu at (105.6, 81.5)
- added H4: MountingHole, MountingHole:MountingHole_2.1mm, F.Cu at (144.1, 80.8)
- added TP27: TestPoint, TestPoint:TestPoint_Pad_D2.0mm, F.Cu at (110.4, 130.1)
- moved TP21 25.0 mm to (155.3, 103.8)
- moved TP24 22.0 mm to (178.8, 94.9)
- moved J31 12.8 mm to (124.8, 114.2), turned to 0 degrees
- moved TP34 12.0 mm to (116.7, 87.4)
- moved TP14 11.0 mm to (137.2, 115.0)
- moved R22 10.8 mm to (170.0, 71.4), turned to 180 degrees
- moved R17 4.75 mm to (111.5, 93.6)
- moved D10 4.48 mm to (174.2, 70.4), turned to 0 degrees
- moved R16 3.88 mm to (111.4, 88.7)
- moved TP20 2.94 mm to (155.3, 99.2)
- moved C11 2.87 mm to (145.6, 66.9)
- moved C13 2.87 mm to (166.9, 66.8)
- moved C16 2.87 mm to (170.4, 66.8)
- moved J17 2.87 mm to (153.2, 66.8)
- moved J20 2.87 mm to (163.2, 66.8)
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Routing:
- net IO14/DVP_Y6: track 0.00 -> 224.6 mm, vias 0 -> 5
- net VDC: track 0.00 -> 214.6 mm
- net GND: track 3.37 -> 176.1 mm, vias 2 -> 75
- net DRV_FAULT: track 0.00 -> 166.9 mm, vias 0 -> 1
- net CHIP_EN: track 0.00 -> 140.3 mm, vias 0 -> 2
- net DRV_SLEEP: track 0.00 -> 139.9 mm, vias 0 -> 1
- net MTCK/IO39/CAM_SCL: track 0.00 -> 139.6 mm, vias 0 -> 4
- net +BATT: track 0.00 -> 136.3 mm
- net BNO_SCL: track 0.00 -> 130.3 mm, vias 0 -> 1
- net +3.3V: track 0.00 -> 123.3 mm, vias 0 -> 13
- net IO10/XMCLK: track 0.00 -> 114.5 mm, vias 0 -> 4
- net MTDO/IO40/CAM_SDA: track 0.00 -> 113.9 mm, vias 0 -> 5
- net +2V8: track 0.00 -> 105.3 mm
- net Net-(R6-Pad1): track 0.00 -> 100.6 mm, vias 0 -> 2
- net VCC: track 9.77 -> 110.0 mm
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- added copper zone on In2.Cu, net +3.3V
- added copper zone on In1.Cu, net GND

Commit message: stuff
Parts:
- removed TP29, TP30: TestPoint, TestPoint:TestPoint_Pad_D2.0mm
- added D14: LED, LED_SMD:LED_0603_1608Metric, F.Cu at (115.7, 101.4)
- added D15: PMEG6010CEJ, Diode_SMD:D_SOD-323F, F.Cu at (111.4, 100.8)
- added J43: HMTSW-102-X-X-S-X, HMTSW-102-X-X-S-X:SAMTEC_HMTSW-102-X-X-S-X, F.Cu at (103.2, 119.6)
- added J44: 87520-0010BLF, 87520-0010BLF:AMPHENOL_87520-0010BLF, F.Cu at (89.0, 107.7)
- added J45: HMTSW-102-X-X-S-X, HMTSW-102-X-X-S-X:SAMTEC_HMTSW-102-X-X-S-X, F.Cu at (106.5, 101.3)
- added J46: HMTSW-102-X-X-S-X, HMTSW-102-X-X-S-X:SAMTEC_HMTSW-102-X-X-S-X, F.Cu at (106.5, 98.1)
- added J47: HMTSW-102-X-X-S-X, HMTSW-102-X-X-S-X:SAMTEC_HMTSW-102-X-X-S-X, F.Cu at (94.2, 129.9)
- added J48: HMTSW-102-X-X-S-X, HMTSW-102-X-X-S-X:SAMTEC_HMTSW-102-X-X-S-X, F.Cu at (103.2, 113.1)
- added J49: HMTSW-102-X-X-S-X, HMTSW-102-X-X-S-X:SAMTEC_HMTSW-102-X-X-S-X, F.Cu at (96.2, 114.0)
- added J50: HMTSW-102-X-X-S-X, HMTSW-102-X-X-S-X:SAMTEC_HMTSW-102-X-X-S-X, F.Cu at (96.2, 117.4)
- added J51: HMTSW-102-X-X-S-X, HMTSW-102-X-X-S-X:SAMTEC_HMTSW-102-X-X-S-X, F.Cu at (105.4, 127.7)
- added J52: HMTSW-102-X-X-S-X, HMTSW-102-X-X-S-X:SAMTEC_HMTSW-102-X-X-S-X, F.Cu at (110.8, 126.6)
- added J9: HMTSW-102-X-X-S-X, HMTSW-102-X-X-S-X:SAMTEC_HMTSW-102-X-X-S-X, F.Cu at (103.2, 116.4)
- added R20: 100, Resistor_SMD:R_0805_2012Metric, F.Cu at (111.4, 97.2)
- U10: value GD25D05CT -> GD25Q64CSIGR
- moved J37 28.9 mm to (106.8, 91.9), turned to -90 degrees
- moved D13 15.0 mm to (95.5, 105.2)
- moved R25 14.9 mm to (95.5, 102.2), turned to 180 degrees
- moved D8 14.6 mm to (108.5, 105.4), turned to -90 degrees
- moved C8 11.5 mm to (95.4, 98.1)
- moved J8 10.9 mm to (84.8, 93.9)
- moved TP6 10.5 mm to (103.3, 75.7)
- moved J12 9.00 mm to (100.5, 98.1)
- moved TP10 7.83 mm to (108.1, 110.2)
- moved J13 6.97 mm to (96.6, 109.0), turned to -90 degrees
- moved C7 6.28 mm to (90.8, 97.5), turned to 0 degrees
- moved R14 6.14 mm to (104.3, 109.8)
- moved R13 5.21 mm to (100.5, 109.8)
- moved C23 5.10 mm to (111.7, 122.1)
- moved TP4 5.07 mm to (99.8, 75.8)
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Connections:
- J42 pad A6: USB_DN -> Net-(J42-DN1)
- J42 pad A7: USB_DN -> Net-(J42-DN1)
- J42 pad B6: USB_DP -> Net-(J42-DN2)
- J42 pad B7: USB_DP -> Net-(J42-DN2)
- TP25 pad 1: USB_DN -> Net-(J42-DN1)
- TP26 pad 1: USB_DP -> Net-(J42-DN2)
- U7 pad 14: USB_DP -> Net-(U7-USBDP)
- U7 pad 15: USB_DN -> Net-(U7-USBDM)
- U7 pad 2: TX_D6 -> Net-(U7-RXD)
- U7 pad 30: RX_D7 -> Net-(U7-TXD)
Routing:
- net VDC: track 214.6 -> 145.3 mm, vias 0 -> 2
- net +5V: track 28.0 -> 69.1 mm, vias 0 -> 1
- net VCC: track 110.0 -> 145.0 mm
- net Net-(J42-DN2): track 0.00 -> 31.9 mm, vias 0 -> 1
- net Net-(J44-D-): track 0.00 -> 26.8 mm
- net Net-(D8-K): track 0.00 -> 23.7 mm
- net Net-(J42-DN1): track 0.00 -> 23.5 mm
- net Net-(U7-RXD): track 0.00 -> 19.7 mm
- net TX_D6: track 32.5 -> 13.8 mm
- net Net-(U7-USBDM): track 0.00 -> 18.4 mm, vias 0 -> 1
- net Net-(U7-USBDP): track 0.00 -> 13.5 mm, vias 0 -> 1
- net GND: track 176.1 -> 189.4 mm, vias 75 -> 71
- net USB_DN: track 46.1 -> 58.7 mm, vias 2 -> 1
- net Net-(J44-D+): track 0.00 -> 12.1 mm
- net +3.3V: track 123.3 -> 111.3 mm
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
Commit message: stuff
Parts:
- removed TP15, TP18, TP19: TestPoint, TestPoint:TestPoint_Pad_D2.0mm
- removed U10: GD25Q64CSIGR, Package_SO:SOP-8_3.9x4.9mm_P1.27mm
- added G***: LOGO, CharmLabLogo:Charm, B.Cu at (167.7, 131.2)
- added TP28: TestPoint, TestPoint:TestPoint_Pad_D2.0mm, F.Cu at (141.1, 90.1)
- added TP29: TestPoint, TestPoint:TestPoint_Pad_D2.0mm, F.Cu at (136.0, 103.2)
- added TP30: TestPoint, TestPoint:TestPoint_Pad_D2.0mm, F.Cu at (148.2, 104.7)
- added U11: GD25Q64CSIGR, GD25Q64CSIGR:SOP8_208MIL_GDV, F.Cu at (142.1, 99.1)
- moved TP17 16.6 mm to (135.5, 96.3)
- moved TP21 3.89 mm to (159.0, 105.1)
- moved H3 3.71 mm to (101.9, 81.6)
- moved H4 1.35 mm to (144.9, 81.9)
- moved C32 1.00 mm to (134.7, 125.8)
Connections:
- TP17 pad 1: SPID -> SPICS0
Routing:
- net SPIQ: track 45.2 -> 53.0 mm, vias 2 -> 4
- net MTCK/IO39/CAM_SCL: track 139.6 -> 136.3 mm
- net SPIWP: track 37.3 -> 34.5 mm
- net +3.3V: track 111.3 -> 108.8 mm
- net SPICS0: track 56.6 -> 55.1 mm
- net SPID: track 48.5 -> 47.2 mm
- net D2/A2: track 25.7 -> 26.5 mm
- net RX_D7: track 42.9 -> 43.7 mm
- net Net-(U11-VCC): track 6.09 -> 6.82 mm
- net MTMS/IO42/PDM_CLK: track 74.7 -> 74.0 mm
- net IO16/DVP_Y5: track 87.0 -> 87.7 mm
- net MTDI/IO41/PDM_DATA: track 76.4 -> 77.1 mm
- net MTDO/IO40/CAM_SDA: track 113.9 -> 114.6 mm
- net IO12/DVP_Y7: track 80.3 -> 80.9 mm
- net GND: vias 71 -> 72
Other:
- board text added: "SenseDev Board Version 2.1 Designed in Stanford, CA"
