File: Hardware/Gen2Dev/OuterBoard/2.1/OuterBoard_rev2.1/OuterBoard_rev2.1.kicad_pcb (KiCad board)
At the start: 4 copper layers, 101.6 x 76.2 mm, 224 parts, among them J1 HMTSW-102-X-X-S-X, J10 F32R-1A7H1-11024, J11 3221-10-0300-00, J12 HMTSW-102-X-X-S-X, J13 HMTSW-102-X-X-S-X, J14 HMTSW-102-X-X-S-X, J15 HMTSW-102-X-X-S-X, J16 HMTSW-102-X-X-S-X, J17 HMTSW-102-X-X-S-X, J18 HMTSW-102-X-X-S-X, J19 HMTSW-102-X-X-S-X, J2 HMTSW-102-X-X-S-X, J20 HMTSW-102-X-X-S-X, J21 HMTSW-102-X-X-S-X, J22 HMTSW-102-X-X-S-X, J23 HMTSW-102-X-X-S-X, J24 HMTSW-102-X-X-S-X, J25 HMTSW-102-X-X-S-X, J26 HMTSW-102-X-X-S-X, J27 HMTSW-102-X-X-S-X, J28 HMTSW-102-X-X-S-X, J29 HMTSW-102-X-X-S-X, J3 HMTSW-102-X-X-S-X, J30 HMTSW-102-X-X-S-X, J31 HMTSW-102-X-X-S-X, J32 HMTSW-102-X-X-S-X, J33 HMTSW-102-X-X-S-X, J34 HMTSW-102-X-X-S-X, J35 HMTSW-102-X-X-S-X, J36 HMTSW-102-X-X-S-X, J37 HMTSW-102-X-X-S-X, J38 HMTSW-102-X-X-S-X, J39 HMTSW-102-X-X-S-X, J4 HMTSW-102-X-X-S-X, J40 HMTSW-102-X-X-S-X, J41 HMTSW-102-X-X-S-X, J42 UJ31-CH-G2-SMT-TR, J43 HMTSW-102-X-X-S-X, J44 87520-0010BLF, J45 HMTSW-102-X-X-S-X, J46 HMTSW-102-X-X-S-X, J47 HMTSW-102-X-X-S-X, J48 HMTSW-102-X-X-S-X, J49 HMTSW-102-X-X-S-X, J5 HMTSW-102-X-X-S-X, J50 HMTSW-102-X-X-S-X, J51 HMTSW-102-X-X-S-X, J52 HMTSW-102-X-X-S-X, J6 HMTSW-102-X-X-S-X, J7 530470210, J8 530470210, J9 HMTSW-102-X-X-S-X, SW1 PTS815 SJM 250 SMTR LFS, SW2 PTS815 SJM 250 SMTR LFS, U1 MCP73812T-420I-OT, U11 GD25Q64CSIGR, U2 DRV8410PWPR, U3 MCP73812T-420I-OT, U4 MIC5504-3.3YM5, U5 MIC5504-1.8YM5, U6 MCP1700x-280xxTT, U7 FT232RQ, U8 BNO055, U9 ESP32-S3, Y1 ABM8G-40.000MHZ-18-D2Y-T

Commit message: stuff
Parts:
- added TP15: TestPoint, TestPoint:TestPoint_Pad_D2.0mm, F.Cu at (150.3, 98.8)
- moved TP16 3.06 mm to (150.8, 102.2)
Connections:
- C44 pad 1: +3.3V -> VDD_SPI
- J34 pad 02: +3.3V -> VDD_SPI
- U11 pad 7: unconnected-(U11-HOLD#(IO3)-Pad7) -> SPIHD
Routing:
- net VDD_SPI: track 0.00 -> 84.3 mm, vias 0 -> 6
- net SPIHD: track 0.00 -> 55.2 mm, vias 0 -> 2
- net +3.3V: track 108.8 -> 105.1 mm
- net SPICLK: track 55.6 -> 58.1 mm
- net IO10/XMCLK: track 114.4 -> 116.4 mm
- net CHIP_EN: track 140.3 -> 142.1 mm
- net IO12/DVP_Y7: track 80.9 -> 82.7 mm
- net USB_DP: track 47.1 -> 48.3 mm
- net MOTOR2_BIN2: track 51.6 -> 52.8 mm
- net IO16/DVP_Y5: track 87.7 -> 88.9 mm
- net USB_DN: track 59.1 -> 60.0 mm
- net GND: track 189.4 -> 188.7 mm
- net IO11/DVP_Y8: track 89.8 -> 90.4 mm

Commit message: stuff
Parts:
- moved TP41 11.1 mm to (179.4, 125.6)
- moved TP48 11.1 mm to (179.7, 118.9)
- moved TP45 5.45 mm to (170.5, 129.8)
- moved D7 5.22 mm to (169.5, 109.7), turned to 0 degrees
- moved TP42 3.67 mm to (167.7, 106.3)
- moved TP63 2.25 mm to (174.5, 107.7)
- moved R31 0.78 mm to (124.3, 129.9)
Routing:
- net IO38/DVP_VSYNC: track 47.7 -> 66.9 mm, vias 2 -> 3
- net DRV_FAULT: track 174.9 -> 169.4 mm
- net +2V8: track 105.3 -> 99.7 mm
- net IO48/DVP_Y9: track 59.5 -> 54.6 mm
- net IO10/XMCLK: track 116.4 -> 111.8 mm
- net IO14/DVP_Y6: track 224.5 -> 228.0 mm
- net MTCK/IO39/CAM_SCL: track 136.3 -> 139.6 mm
- net Net-(J42-CC1): track 24.9 -> 27.9 mm
- net Net-(D7-K): track 85.3 -> 87.9 mm
- net Net-(FB1-Pad2): track 49.1 -> 51.3 mm
- net SPIHD: track 55.2 -> 57.4 mm
- net SPIQ: track 53.0 -> 55.2 mm
- net D2/A2: track 26.5 -> 28.5 mm
- net SPID: track 47.2 -> 49.1 mm
- net +1V8: track 70.3 -> 68.4 mm
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