File: Hardware/Gen2Dev/InnerBoard/2.1/InnerBoard_rev2.1/InnerBoard_rev2.1.kicad_sch (KiCad schematic)
At the start: 135 parts, among them J2 HMTSW-102-X-X-S-X, J25 SI-46020-F, J26 USB_C_Receptacle, J8 1051620001, Q1 Q12MHz/20pF/10ppm/4P/3.2x2.5mm, Q2 BC817-40(SOT23), Q3 BC817-40(SOT23), SW1 PTS815 SJM 250 SMTR LFS, T1 LMUN2211LT1G(SOT-23), U1 LAN8710A-EZC(QFN32)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

Commit message: dev board
Parts:
- removed R24: 220R/R0402, Resistor_SMD:R_0402_1005Metric, symbol ESP32-PoE-ISO_Rev_K:R
- removed R26: 10k/R0402, Resistor_SMD:R_0402_1005Metric, symbol ESP32-PoE-ISO_Rev_K:R
- removed R27: NA/R0402, Resistor_SMD:R_0402_1005Metric, symbol ESP32-PoE-ISO_Rev_K:R
- added R24: 0, Resistor_SMD:R_0805_2012Metric, symbol Device:R_US
- added R26: 10k, Resistor_SMD:R_0805_2012Metric, symbol Device:R_US
- added R49: 220, Resistor_SMD:R_0805_2012Metric, symbol Device:R_US
Connections:
- net +3V3: now also R26.1
- net D_Com: now also R24.1
- net GND: now also R49.2
- net at SW1.2: now also R24.2, R26.2
- net at SW1.4: now also R49.1

Commit message: stuff
Parts:
- removed J26: USB_C_Receptacle, Connector_USB:USB_C_Receptacle_Molex_105450-0101-L, symbol Connector:USB_C_Receptacle
- added C31: 10uF, Capacitor_SMD:C_0805_2012Metric, symbol Device:C
- added D11: LED, LED_SMD:LED_0603_1608Metric, symbol Device:LED
- added D12: PMEG6010CEJ, Diode_SMD:D_SOD-323F, symbol Diode:PMEG6010CEJ
- added D13, D14: 1N5819WS, Diode_SMD:D_SOD-323, symbol Diode:1N5819WS
- added J3, J5: UJ31-CH-G2-SMT-TR, UJ31-CH-G2-SMT-TR:CUI_UJ31-CH-G2-SMT-TR, symbol UJ31_CH_G2_SMT_TR:UJ31-CH-G2-SMT-TR
- added J4, J6, J7: HMTSW-102-X-X-S-X, HMTSW-102-X-X-S-X:SAMTEC_HMTSW-102-X-X-S-X, symbol HMTSW-102-X-X-S-X:HMTSW-102-X-X-S-X
- added L6: FB0805/600R/2A, Inductor_SMD:L_0805_2012Metric, symbol Device:L
- added R27: 5.1K, Resistor_SMD:R_0805_2012Metric, symbol Device:R_US
- added R50: 6.1K, Resistor_SMD:R_0805_2012Metric, symbol Device:R_US
- added R51: 100, Resistor_SMD:R_0805_2012Metric, symbol Device:R_US
- added TP1, TP2, TP3, TP4, TP5, TP6: TestPoint, TestPoint:TestPoint_Pad_D2.0mm, symbol Connector:TestPoint
- added U9: FT232RQ, FT232RQ:QFN50P500X500X90-33N, symbol FT232RQ:FT232RQ
Connections:
- net +5V_USB: now also J3.A1 (GND), J3.A12 (GND__1), J3.A4 (VBUS), J3.A9 (VBUS__1), J3.B1 (GND__2), J3.B12 (GND__3), J3.B4 (VBUS__2), J3.B9 (VBUS__3), J3.SH1 (SHIELD), J3.SH2 (SHIELD__1), J3.SH3 (SHIELD__2), J3.SH4 (SHIELD__3)
- net GND: now also C31.2, D11.1 (K), L6.2, R27.2, R50.2, U9.17 (GND), U9.20 (GND), U9.24 (AGND), U9.4 (GND)
- new net: D12.1 (K), J7.01
- new net: D13.1 (K), TP1.1, U9.30 (TXD)
- new net: J5.B5 (CC2), R50.1, TP4.1
- new net: J5.A1 (GND), J5.A12 (GND__1), J5.B1 (GND__2), J5.B12 (GND__3), J5.SH1 (SHIELD), J5.SH2 (SHIELD__1), J5.SH3 (SHIELD__2), J5.SH4 (SHIELD__3), L6.1
- new net: J5.A5 (CC1), R27.1, TP3.1
- new net: J4.02, U9.1 (VCCIO), U9.19 (VCC)
- new net: D14.2 (A), TP2.1, U9.2 (RXD)
- new net: D11.2 (A), R51.1
- new net: D12.2 (A), J6.02
- new net +3.3V: C31.1, J4.01
- new net GPIO1/U0TXD: D14.1 (K)
- new net GPIO3/U0RXD: D13.2 (A)
- new net USB_DN: J3.A7 (DN1), J3.B7 (DN2), J5.A6 (DP1), J5.A7 (DN1), TP5.1, U9.15 (USBDM)
- new net USB_DP: J3.A6 (DP1), J3.B6 (DP2), J5.B6 (DP2), J5.B7 (DN2), TP6.1, U9.14 (USBDP)
- new net VBUS: J5.A4 (VBUS), J5.A9 (VBUS__1), J5.B4 (VBUS__2), J5.B9 (VBUS__3), J6.01, R51.2
- new net VDC: J7.02
- no-connect marks 38 -> 26
Other:
- note added: "ESP32-WROOM"
- note added: "FTDI"
- note added: "JTAG"
- note added: "LIPO Charger"
- note added: "Notes: DCDC for Wireless Charger (45V -> 9V Isolated) Wireless Charging IC for charging coil"
- note added: "POE Supply"
- note added: "SD Card"
- note added: "USB-C RECPT"
- note removed: "ESP32-WROOM-32E MODULE"
- note removed: "LiPo Charger"
- note removed: "PoE Power Supply"
- note removed: "SD/MMC Card"
- note removed: "UEXT"
- moved on the sheet: J2, R24, R26, R49, SW1

Commit message: stuff
Parts:
- added U10: ESP32-WROOM-32E-N8, symbol ESP32_WROOM_32E_N8:ESP32-WROOM-32E-N8
- added U11: LAN8710A-EZC, QFN32_5X5MC_MCH, symbol LAN8710A_EZC:LAN8710A-EZC
- added U12: TPS2376PW, PW8, symbol TPS2376PW:TPS2376PW
- added U13: RFM-0505S, SIP4_RFM_RCP, symbol RFM_0505S:RFM-0505S
- added U14, U15: TPS54561DPRR, WSON10_DPR_TEX, symbol TPS54561DPRR:TPS54561DPRR
- added U16: ROE-0512S, ROE_RCP, symbol ROE-0512S:ROE-0512S
