File: Hardware/Gen2Dev/InnerBoard/2.1/InnerBoard_rev2.1/InnerBoard_rev2.1.kicad_sch (KiCad schematic)
At the start: 144 parts, among them J2 HMTSW-102-X-X-S-X, J25 SI-46020-F, J4 HMTSW-102-X-X-S-X, J5 UJ31-CH-G2-SMT-TR, J6 HMTSW-102-X-X-S-X, J7 HMTSW-102-X-X-S-X, J8 3221-10-0300-00, Q4 BC817, Q5 BC817, SW1 PTS815 SJM 250 SMTR LFS, T1 LMUN2211LT1G(SOT-23), U1 LAN8710A-EZC(QFN32), U10 ESP32-WROOM-32E-N8, U11 LAN8710A-EZC, U12 TPS2376PW, U13 RFM-0505S, U14 TPS54561DPRR, U15 TPS54561DPRR, U16 ROE-0512S, U2 TPS2376PW(TSSOP-8), U3 TX4138(ESOIC-8), U4 BL4054B-42TPRN(SOT23-5), U5 SY8089AAAC(SOT23-5), U6 74LVC1G04, U9 FT232RQ, Y1 ABLS2-12.000MHZ-D4Y-T

Commit message: stuff
Parts:
- removed BAT1: DW02S, OLIMEX_Connectors-FP:LIPO_BAT_VERTICAL_DW02S, symbol ESP32-PoE-ISO_Rev_K:BAT_CON
- removed C20, C21, C23: 22uF/6.3V/20%/X5R/C0603, OLIMEX_RLC-FP:C_0603_5MIL_DWS, symbol ESP32-PoE-ISO_Rev_K:C
- removed C22: 1nF/50V/10%/X7R/C0402, OLIMEX_RLC-FP:C_0402_5MIL_DWS, symbol ESP32-PoE-ISO_Rev_K:C
- removed CHRG1: LED/YELLOW/0603, OLIMEX_LEDs-FP:LED_0603_KA, symbol ESP32-PoE-ISO_Rev_K:LED
- removed D12: PMEG6010CEJ, Diode_SMD:D_SOD-323F, symbol Diode:PMEG6010CEJ
- removed D4, D5: 1N5819S4/SOD123, OLIMEX_Diodes-FP:SOD-123_1C-2A_KA, symbol ESP32-PoE-ISO_Rev_K:D_Schottky
- removed FET2, FET3: WPM2015-3/TR, OLIMEX_Transistors-FP:SOT23, symbol ESP32-PoE-ISO_Rev_K:P-MOS+DIOD
- removed J6, J7: HMTSW-102-X-X-S-X, HMTSW-102-X-X-S-X:SAMTEC_HMTSW-102-X-X-S-X, symbol HMTSW-102-X-X-S-X:HMTSW-102-X-X-S-X
- removed L3: 2.2uH/1.5A/DCR=72mR/20%/3.00x3.00x1.50mm/CD32(NR3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, OLIMEX_RLC-FP:CD32, symbol ESP32-PoE-ISO_Rev_K:L
- removed PWR1: LED/RED/0603, OLIMEX_LEDs-FP:LED_0603_KA, symbol ESP32-PoE-ISO_Rev_K:LED
- removed R21, R25: 10k/R0402, OLIMEX_RLC-FP:R_0402_5MIL_DWS, symbol ESP32-PoE-ISO_Rev_K:R
- removed R22, R23: 2.2k/R0402, OLIMEX_RLC-FP:R_0402_5MIL_DWS, symbol ESP32-PoE-ISO_Rev_K:R
- removed R28, R29: 470k/R0402, OLIMEX_RLC-FP:R_0402_5MIL_DWS, symbol ESP32-PoE-ISO_Rev_K:R
- removed R30: 220k/R0402, OLIMEX_RLC-FP:R_0402_5MIL_DWS, symbol ESP32-PoE-ISO_Rev_K:R
- removed R31: 49.9k/1%/R0402, OLIMEX_RLC-FP:R_0402_5MIL_DWS, symbol ESP32-PoE-ISO_Rev_K:R
- removed R32: 47k/R0402, OLIMEX_RLC-FP:R_0402_5MIL_DWS, symbol ESP32-PoE-ISO_Rev_K:R
- removed R33: 100k/R0402, OLIMEX_RLC-FP:R_0402_5MIL_DWS, symbol ESP32-PoE-ISO_Rev_K:R
- removed U4: BL4054B-42TPRN(SOT23-5), OLIMEX_IC-FP:SOT-23-5, symbol ESP32-PoE-ISO_Rev_K:BL4054B-42TPRN(SOT23-5)
- removed U5: SY8089AAAC(SOT23-5), OLIMEX_Regulators-FP:SOT-23-5, symbol ESP32-PoE-ISO_Rev_K:SY8009AAAC(SOT23-5)
- added BAT/BUT1: Opened(2-3)/Soldered(1-2), OLIMEX_Jumpers-FP:SJ_2_SMALL, symbol ESP32-EVB_Rev_K1-rescue:SJ2W_Closed(1-2)-ESP32-EVB_Rev_K1
- added BAT1: DW02R, OLIMEX_Connectors-FP:LIPO_BAT-CON2DW02R, symbol ESP32-EVB_Rev_K1-rescue:BAT_CON-ESP32-EVB_Rev_K1
- added BUT1, RST1: T1107A(6x3,8x2,5MM), OLIMEX_Buttons-FP:T1107A(6x3,8x2,5MM), symbol ESP32-EVB_Rev_K1-rescue:SIDE_WTCM-TR(3x4)-ESP32-EVB_Rev_K1
- added C1, C3: NA(47uF/6.3V/20%/X5R/C0805), OLIMEX_RLC-FP:C_0805_5MIL_DWS, symbol ESP32-EVB_Rev_K1-rescue:C-ESP32-EVB_Rev_K1
- added C11, C13, C14, C15, C17, C24, C30: 100nF/50V/20%/Y5V/C0603, OLIMEX_RLC-FP:C_0603_5MIL_DWS, symbol ESP32-EVB_Rev_K1-rescue:C-ESP32-EVB_Rev_K1
- added C12, C23, C29, C5, C6, C7, C8, C9: 22uF/6.3V/20%/X5R/C0603, OLIMEX_RLC-FP:C_0603_5MIL_DWS, symbol ESP32-EVB_Rev_K1-rescue:C-ESP32-EVB_Rev_K1
- added C16: 2.2uF/6.3V/10%/X5R/C0603, OLIMEX_RLC-FP:C_0603_5MIL_DWS, symbol ESP32-EVB_Rev_K1-rescue:C-ESP32-EVB_Rev_K1
- added C18: 1nF/50V/5%/NPO(COG)/C0603, OLIMEX_RLC-FP:C_0603_5MIL_DWS, symbol ESP32-EVB_Rev_K1-rescue:C-ESP32-EVB_Rev_K1
- added C19: 1nF/2000V/10%/X7R/C1206, OLIMEX_RLC-FP:C_1206_5MIL_DWS_ISO, symbol ESP32-EVB_Rev_K1-rescue:C-ESP32-EVB_Rev_K1
- added C2, C4: 47uF/6.3V/20%/X5R/C0805, OLIMEX_RLC-FP:C_0805_5MIL_DWS, symbol ESP32-EVB_Rev_K1-rescue:C-ESP32-EVB_Rev_K1
- added C20: NA(1nF/2000V/10%/X7R/C1206), OLIMEX_RLC-FP:C_1206_5MIL_DWS_ISO, symbol ESP32-EVB_Rev_K1-rescue:C-ESP32-EVB_Rev_K1
- added C20, C22: 10uF, Capacitor_SMD:C_0805_2012Metric, symbol Device:C
- added C21, C23: 1uF, Capacitor_SMD:C_0805_2012Metric, symbol Device:C
- added C21, C22: 27pF/50V/5%/C0G/C0603, OLIMEX_RLC-FP:C_0603_5MIL_DWS, symbol ESP32-EVB_Rev_K1-rescue:C-ESP32-EVB_Rev_K1
- added C26: 100nF, symbol Device:C
- added C27: 10uF, symbol Device:C
- added C28: NA(470nF/16V/10%/X7R/C0603), OLIMEX_RLC-FP:C_0603_5MIL_DWS, symbol ESP32-EVB_Rev_K1-rescue:C-ESP32-EVB_Rev_K1
- added C31, C32: 1uF/10V/10%/X5R/C0603, OLIMEX_RLC-FP:C_0603_5MIL_DWS, symbol ESP32-EVB_Rev_K1-rescue:C-ESP32-EVB_Rev_K1
- added CHARGE?: LED/Yellow/0603, OLIMEX_LEDs-FP:LED_0603_KA, symbol ESP32-EVB_Rev_K1-rescue:LED-ESP32-EVB_Rev_K1
- added CON1, CON2: TB3-DG306-5.0-3P, OLIMEX_Connectors-FP:TB3-DG306-5.0_3P, symbol ESP32-EVB_Rev_K1-rescue:CON3-ESP32-EVB_Rev_K1
- added CR1: Q50MHz/25ppm/3V/4P/5x3.2mm, OLIMEX_Crystal-FP:5032-4P_HCX-3S, symbol ESP32-EVB_Rev_K1-rescue:Oscillator-100MHZ_TXC-7W-ESP32-EVB_Rev_K1
- added D1, D3: 1N5819S4(SOD-123), OLIMEX_Diodes-FP:SOD-123_1C-2A_KA, symbol ESP32-EVB_Rev_K1-rescue:D_Schottky-ESP32-EVB_Rev_K1
- added D10: BAT54A(SOT23-3), OLIMEX_Diodes-FP:SOT23-3, symbol ESP32-EVB_Rev_K1-rescue:BAT54A(SOT23-3)-ESP32-EVB_Rev_K1
- added D2: SMBJ6.0A(DO-214AA), OLIMEX_Diodes-FP:DO214AA_1(K)-2(A), symbol ESP32-EVB_Rev_K1-rescue:SMBJ6.0A-ESP32-EVB_Rev_K1
- added D4, D5, D7: LED, LED_SMD:LED_0603_1608Metric, symbol Device:LED
- added D4, D6: 1N5822/SS34/SMA, OLIMEX_Diodes-FP:SMA-KA, symbol ESP32-EVB_Rev_K1-rescue:D_Schottky-ESP32-EVB_Rev_K1
- added D5, D7, D8, D9: 1N5819S4(SOD-123), OLIMEX_Diodes-FP:SOD-123_1C-2A_KA, symbol ESP32-EVB_Rev_K1-rescue:D_Schottky_Small-ESP32-EVB_Rev_K1
- added D6: 1N5819, Diode_THT:D_DO-41_SOD81_P10.16mm_Horizontal, symbol Diode:1N5819
- added FET1, FET2, FET3: WPM2015-3/TR, OLIMEX_Transistors-FP:SOT23, symbol ESP32-EVB_Rev_K1-rescue:P-MOS+DIOD-ESP32-EVB_Rev_K1
- added FET4: BSS138, OLIMEX_Transistors-FP:SOT23, symbol ESP32-EVB_Rev_K1-rescue:N-MOS+DIOD-ESP32-EVB_Rev_K1
- added GND1: TESTPAD, OLIMEX_Other-FP:TESTPAD_40-ROUND, symbol ESP32-EVB_Rev_K1-rescue:TESTPAD-ESP32-EVB_Rev_K1
- added J3, J9: HMTSW-102-X-X-S-X, HMTSW-102-X-X-S-X:SAMTEC_HMTSW-102-X-X-S-X, symbol HMTSW-102-X-X-S-X:HMTSW-102-X-X-S-X
- added L1, L3: FB0805/600R/2A, OLIMEX_RLC-FP:L_0805_5MIL_DWS, symbol ESP32-EVB_Rev_K1-rescue:L-ESP32-EVB_Rev_K1
- added L2: 2.2uH/1.5A/DCR=72mR/20%/3.00x3.00x1.50mm/CD32(NR3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, OLIMEX_RLC-FP:CD32, symbol ESP32-EVB_Rev_K1-rescue:L-ESP32-EVB_Rev_K1
- added L5: NA(FB0805/600R/2A), OLIMEX_RLC-FP:L_0805_5MIL_DWS, symbol ESP32-EVB_Rev_K1-rescue:L-ESP32-EVB_Rev_K1
- added LAN1: RJLD-060TC1(LPJ4013EDNL), OLIMEX_Connectors-FP:RJLBC-060TC1, symbol ESP32-EVB_Rev_K1-rescue:RJLBC-060TC1_GND-ESP32-EVB_Rev_K1
- added LED1, LED2: LED/GREEN/0603, OLIMEX_LEDs-FP:LED_0603_KA, symbol ESP32-EVB_Rev_K1-rescue:LED-ESP32-EVB_Rev_K1
- added MH2, MH3: Mounting_hole_Shield_3.3mm, OLIMEX_Other-FP:Mounting_hole_Shield_3.3mm, symbol ESP32-EVB_Rev_K1-rescue:Mounting_hole_Shield_3.3mm-ESP32-EVB_Rev_K1
- added PHY_RST1: Opened, OLIMEX_Jumpers-FP:SJ, symbol ESP32-EVB_Rev_K1-rescue:SJ-ESP32-EVB_Rev_K1
- added PWR1: PWRJ-2mm(YDJ-1134), OLIMEX_Connectors-FP:PWRJ-2mm(YDJ-1136), symbol ESP32-EVB_Rev_K1-rescue:PWR-JAKPWR_JACK_UNI_MILLING-ESP32-EVB_Rev_K1
- added PWR2: NA(TB2 DG306-5.0-2P), OLIMEX_Connectors-FP:TB2-DG306-5.0_2P, symbol ESP32-EVB_Rev_K1-rescue:CON2-ESP32-EVB_Rev_K1
- added PWRLED1: LED/RED/0603, OLIMEX_LEDs-FP:LED_0603_KA, symbol ESP32-EVB_Rev_K1-rescue:LED-ESP32-EVB_Rev_K1
- added Q1, Q2, Q4, Q5: BC817-40(SOT23), OLIMEX_Transistors-FP:SOT23, symbol ESP32-EVB_Rev_K1-rescue:Q_NPN_BEC-ESP32-EVB_Rev_K1
- added Q1: SI2323DS-T1-GE3, SI2323DS-T1-GE3:SOT23, symbol SI2323DS-T1-GE3:SI2323DS-T1-GE3
- added Q3: Q12MHz/20pF/30ppm/2P/HC-49SM(SMD), OLIMEX_Crystal-FP:Q_49U3HMS, symbol ESP32-EVB_Rev_K1-rescue:Crystal-ESP32-EVB_Rev_K1
- added R1, R41, R42, R5, R50: 1k/R0603, OLIMEX_RLC-FP:R_0603_5MIL_DWS, symbol ESP32-EVB_Rev_K1-rescue:R-ESP32-EVB_Rev_K1
- added R10, R9: 470k/R0603, OLIMEX_RLC-FP:R_0603_5MIL_DWS, symbol ESP32-EVB_Rev_K1-rescue:R-ESP32-EVB_Rev_K1
- added R11, R18, R21, R3, R4, R?: 2.2k/R0603, OLIMEX_RLC-FP:R_0603_5MIL_DWS, symbol ESP32-EVB_Rev_K1-rescue:R-ESP32-EVB_Rev_K1
- added R14, R26, R27, R37: 220R/R0603, OLIMEX_RLC-FP:R_0603_5MIL_DWS, symbol ESP32-EVB_Rev_K1-rescue:R-ESP32-EVB_Rev_K1
- added R17, R44, R46, R54: NA/R0603, OLIMEX_RLC-FP:R_0603_5MIL_DWS, symbol ESP32-EVB_Rev_K1-rescue:R-ESP32-EVB_Rev_K1
- added R19: 220k/R0603, OLIMEX_RLC-FP:R_0603_5MIL_DWS, symbol ESP32-EVB_Rev_K1-rescue:R-ESP32-EVB_Rev_K1
- added R2, R22, R23, R24, R30, R34, R35, R38, R40, R45, R51, R6: 10k/R0603, OLIMEX_RLC-FP:R_0603_5MIL_DWS, symbol ESP32-EVB_Rev_K1-rescue:R-ESP32-EVB_Rev_K1
- added R20: 49.9k/1%/R0603, OLIMEX_RLC-FP:R_0603_5MIL_DWS, symbol ESP32-EVB_Rev_K1-rescue:R-ESP32-EVB_Rev_K1
- added R21, R30: 10k, Resistor_SMD:R_0805_2012Metric, symbol Device:R_US
- added R22, R29: 2.2k, Resistor_SMD:R_0805_2012Metric, symbol Device:R_US
- added R23, R25, R28: 100, Resistor_SMD:R_0805_2012Metric, symbol Device:R_US
- added R25: 0R(board_mounted), OLIMEX_RLC-FP:0R_0603, symbol ESP32-EVB_Rev_K1-rescue:R-ESP32-EVB_Rev_K1
- added R28, R31, R32, R33, R58: 49.9R/1%/R0402, OLIMEX_RLC-FP:R_0402_5MIL_DWS, symbol ESP32-EVB_Rev_K1-rescue:R-ESP32-EVB_Rev_K1
- added R36: 10R/R0603, OLIMEX_RLC-FP:R_0603_5MIL_DWS, symbol ESP32-EVB_Rev_K1-rescue:R-ESP32-EVB_Rev_K1
- added R39: 12.1k/1%/R0603, OLIMEX_RLC-FP:R_0603_5MIL_DWS, symbol ESP32-EVB_Rev_K1-rescue:R-ESP32-EVB_Rev_K1
- added R52: 100k/R0603, OLIMEX_RLC-FP:R_0603_5MIL_DWS, symbol ESP32-EVB_Rev_K1-rescue:R-ESP32-EVB_Rev_K1
- added R57: NA(1k/R0603), OLIMEX_RLC-FP:R_0603_5MIL_DWS, symbol ESP32-EVB_Rev_K1-rescue:R-ESP32-EVB_Rev_K1
- added R?: 2k/1%/R0603, OLIMEX_RLC-FP:R_0603_5MIL_DWS, symbol ESP32-EVB_Rev_K1-rescue:R-ESP32-EVB_Rev_K1
- added REL1, REL2: RAS-0515, OLIMEX_Relays-FP:Relay_RAS-05-15, symbol ESP32-EVB_Rev_K1-rescue:Relay-ESP32-EVB_Rev_K1
- added RM2, RM3: RA1206_(4X0603)_4B8_2.2k, OLIMEX_RLC-FP:R_MATRIX_4, symbol ESP32-EVB_Rev_K1-rescue:RA1206_(4x0603)_4B8_Smashed-ESP32-EVB_Rev_K1
- added TVS1: ESDS314DBVR(SOT-23-5), OLIMEX_Diodes-FP:SOT-23-5, symbol ESP32-EVB_Rev_K1-rescue:ESDS314DBVR(SOT-23-5)-ESP32-EVB_Rev_K1
- added U10, U9: BAT54C(SOT23-3), OLIMEX_Diodes-FP:SOT23-3, symbol ESP32-EVB_Rev_K1-rescue:BAT54C(SOT23-3)-ESP32-EVB_Rev_K1
- added U11: HX7027(SOT-23), OLIMEX_IC-FP:SOT-23, symbol ESP32-EVB_Rev_K1-rescue:VDA2710NTA(SOT-23)-ESP32-EVB_Rev_K1
- added U2: SY8089AAAC(SOT23-5), OLIMEX_Regulators-FP:SOT-23-5, symbol ESP32-EVB_Rev_K1-rescue:SY8009AAAC(SOT23-5)-ESP32-EVB_Rev_K1
- added U3: ESP-WROOM-32, OLIMEX_Cases-FP:ESP-WROOM-32_MODULE, symbol ESP32-EVB_Rev_K1-rescue:ESP-WROOM-32-ESP32-EVB_Rev_K1
- added U4: LAN8710A-EZC(QFN32), OLIMEX_IC-FP:QFN32_EP(33)_5.00x5.00x0.90mm_Pitch_0.50mm, symbol ESP32-EVB_Rev_K1-rescue:LAN8710A-EZC(QFN32)-ESP32-EVB_Rev_K1
- added U4: MIC5504-3.3YM5, Package_TO_SOT_SMD:SOT-23-5, symbol Regulator_Linear:MIC5504-3.3YM5
- added U5: CH340T(SSOP20W), OLIMEX_IC-FP:SSOP-20W, symbol ESP32-EVB_Rev_K1-rescue:CH340T(SSOP20W)-ESP32-EVB_Rev_K1
- added U7: LD1117S50TR_SOT223, Package_TO_SOT_SMD:SOT-223-3_TabPin2, symbol Regulator_Linear:LD1117S50TR_SOT223
- added U8: NA(NCP303LSN27T1G(SOT-23-5)), OLIMEX_IC-FP:SOT-23-5, symbol ESP32-EVB_Rev_K1-rescue:BD5230G-TR(SSOP5_SOT-23-5)-ESP32-EVB_Rev_K1
- added U?: BL4054B-42TPRN(SOT23-5), OLIMEX_IC-FP:SOT-23-5, symbol ESP32-EVB_Rev_K1-rescue:BL4054B-42TPRN(SOT23-5)-ESP32-EVB_Rev_K1
- added UEXT1: BH10S, OLIMEX_Connectors-FP:UEXT_ML10, symbol ESP32-EVB_Rev_K1-rescue:BH10S-ESP32-EVB_Rev_K1
- added USB-UART1: MISB-SWMM-5B-LF(USB_MICRO), OLIMEX_Connectors-FP:USB-MICRO_MISB-SWMM-5B_LF, symbol ESP32-EVB_Rev_K1-rescue:USB-MINI-ESP32-EVB_Rev_K1
- added Y2: 402F2501XIAR, 402F2501XIAR:XTAL_402F2501XIAR, symbol 402F2501XIAR:402F2501XIAR
Connections:
- net +3.3V: now also C22.1, C23.1, C29.1, C6.1, C7.1, CR1.4 (VDD), D10.1 (C1), FET3.2, J9.02, L1.1, L2.2, L5.1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
- net +3.3VLAN: now also C13.1, C8.1, C9.1, FET3.3, L3.1, L5.2, R38.2, RM2.3.1, RM2.4.1, RM3.1.2, RM3.2.2, RM3.3.2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
- net +5V: now also C1.1, C2.1, C20.1, C21.1, C27.1, CHARGE?.2 (A), D1.1 (K), D2.1 (K), D3.1 (K), D4.2 (A), D6.1 (K), D6.1 (K)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
- net +5VP: now also D6.2 (A), Q1.1, R21.2
- net +5V_USB: now also C23.1, FET2.3, R35.1, U5.19 (VCC), USB-UART1.1 (VBUS)
- net D_Com: now also R37.2, R46.2, U10.3 (CC), U9.3 (CC)
- net ESP_EN: now also C31.2, D10.2 (C2), D9.2 (A), R24.2, R52.2, RST1.1, U3.3 (EN), U8.2 (VDD)
- net GND: now also U11.24 (TXD2), U11.25 (TXD3), BAT1.2, C1.2, C11.2, C12.2, C13.2, C14.2, C15.2, C16.2, C17.2, C18.1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
- net GPI34/BUT1: now also BAT/BUT1.2, U3.6 (GPI34/ADC1_CH6/RTC_GPIO4)
- net GPIO18/MDIO(RMII): now also RM3.1.1, U3.30 (GPIO18/VSPICLK/HS1_DATA7), U4.16 (MDIO)
- net GPIO18/MDIO(RMII): now also U11.16 (MDIO), R22.1
- net GPIO19/EMAC_TXD0(RMII): now also U3.31 (GPIO19/VSPIQ/U0CTS/EMAC_TXD0), U4.22 (TXD0)
- net GPIO19/EMAC_TXD0(RMII): now also U11.22 (TXD0)
- net GPIO21/EMAC_TX_EN(RMII): now also U3.33 (GPIO21/VSPIHD/EMAC_TX_EN), U4.21 (TXEN)
- net GPIO21/EMAC_TX_EN(RMII): now also U11.21 (TXEN)
- net GPIO22/EMAC_TXD1(RMII): now also U3.36 (GPIO22/VSPIWP/U0RTS/EMAC_TXD1), U4.23 (TXD1)
- net GPIO22/EMAC_TXD1(RMII): now also U11.23 (TXD1)
- net GPIO23/MDC(RMII): now also U3.37 (GPIO23/VSPID/HS1_STROBE), U4.17 (MDC)
- net GPIO23/MDC(RMII): now also U11.17 (MDC)
- net GPIO25/EMAC_RXD0(RMII): now also RM3.3.1, U3.10 (GPIO25/DAC_1/ADC2_CH8/RTC_GPIO6/EMAC_RXD0), U4.11 (RXD0/MODE0)
- net GPIO25/EMAC_RXD0(RMII): now also U11.11 (RXD0/*MODE0)
- net GPIO26/EMAC_RXD1(RMII): now also RM2.4.2, U3.11 (GPIO26/DAC_2/ADC2_CH9/RTC_GPIO7/EMAC_RXD1), U4.10 (RXD1/MODE1)
- net GPIO26/EMAC_RXD1(RMII): now also U11.10 (RXD1/*MODE1)
- net GPIO27/EMAC_RX_CRS_DV: now also RM3.2.1, U3.12 (GPIO27/ADC2_CH7/TOUCH7/RTC_GPIO17/EMAC_RX_DV), U4.15 (COL/CRS_DV/MODE2)
- net GPIO27/EMAC_RX_CRS_DV: now also U11.15 (COL/CRS_DV/*MODE2), R29.1
- net VBUS: now also Q1.3
- net PHYAD0: now reaches U11.13 (RXER/RXD4/*PHYAD0)
- net PHYAD0: now also RM3.4.1, U4.13 (RXER/RXD4/PHYAD0)
- net at U11.19 (NRST): now also R30.1
- net PHYAD1: now reaches U11.7 (RXCLK/*PHYAD1)
- net PHYAD1: now also RM2.1.2, U4.7 (RXCLK/PHYAD1)
- net PHYAD2: now reaches U11.8 (RXD3/*PHYAD2)
- net PHYAD2: now also RM2.2.2, U4.8 (RXD3/PHYAD2)
- new net: C3.1, C4.1, D4.1 (K), FET1.2, R17.2, U2.1 (EN), U2.4 (IN)
- new net: BAT/BUT1.3, C30.1, R10.1, R9.2
- new net: D3.2 (A), LED2.1 (K), Q2.3 (C), REL2.2
- new net: LED2.2 (A), R11.2
- new net: D1.2 (A), LED1.1 (K), Q1.3 (C), REL1.2
- new net: D8.2 (A), R35.2, U5.4 (RXD)
- new net: PWRLED1.1 (K), R4.1
- new net: C24.1, R40.1, U5.5 (V3)
- new net: C19.1, C20.1, LAN1.GND1, LAN1.GND2
- new net: BAT1.1, FET1.3, R17.1, R9.1, U?.3 (VBAT)
- new net: C5.2, L1.2, R18.1, R21.1, R22.1, R23.1, UEXT1.1
- new net: D5.1 (K), UEXT1.4
- new net: Q1.1 (B), R1.2, R2.2
- new net: D5.2 (A), R23.1
- new net: C29.2, FET3.1, R50.2, R51.2
- new net: U5.7 (UD-), USB-UART1.2 (D-)
- new net: U5.6 (UD+), USB-UART1.3 (D+)
- new net: C28.1, U8.5 (CT)
- new net: Q4.1 (B), R41.2
- new net: Q4.2 (E), R42.1, U5.16 (RTS#)
- new net: D9.1 (K), Q4.3 (C)
- new net: C18.2, PHY_RST1.2, R38.1, R57.1, U4.19 (NRST)
- new net: LAN1.KG1 (KG), U4.2 (LED2/NINTSEL)
- new net: LAN1.AY1 (AY), U4.3 (LED1/REGOFF)
- new net: R39.1, U4.32 (RBIAS)
- new net: J9.01, U4.5 (VOUT)
- new net: Q2.1 (B), R5.2, R6.2
- new net: BUT1.2, R14.1
- new net: LED1.2 (A), R3.2
- new net: CR1.3 (OUT), R36.1
- new net: R44.2, U9.1 (A1)
- new net: C21.1, Q3.1, U5.9 (XI)
- new net: C22.1, Q3.2, U5.10 (XO)
- new net: C11.1, LAN1.3 (COM), LAN1.6 (NC), R25.2
- new net: LAN1.AG1 (AG), R26.2
- new net: LAN1.KY1 (KY), R27.1
- new net: Q5.3 (C), R37.1
- new net: J3.02, U4.1 (VIN), U4.3 (EN)
- new net: R?.2, U?.5 (PROG)
- new net: CHARGE?.1 (K), R?.2
- new net: CON1.2, REL1.COM0
- new net: CON1.3, REL1.NC0
- new net: CON1.1, REL1.NO0
- new net: Q5.2 (E), R41.1, U5.15 (DTR#)
- new net: D7.1 (K), U5.3 (TXD)
- new net: CON2.2, REL2.COM0
- new net: CON2.3, REL2.NC0
- new net: CON2.1, REL2.NO0
- new net: L2.1, U2.3 (LX)
- new net: Q5.1 (B), R42.2
- new net: R19.1, R20.1, U2.5 (FB)
- new net: D4.2 (A), R25.1
- new net: C32.2, R52.1, R58.2, U11.3 (VIn)
- new net: D7.2 (A), R28.1
- new net: FET4.3 (D), R50.1
- new net: D10.3 (CA), R58.1
- new net: R?.1, U?.1 (CHRGb)
- new net +5V_EXT: D6.2 (A), FET2.1, PWR1.+, PWR2.1, R30.1
- new net +9V: C26.1, U7.3 (VI)
- new net BUT1: BAT/BUT1.1, BUT1.1, R45.2, R46.1
- new net GPI35/CAN-RX: U3.7 (GPI35/ADC1_CH7/RTC_GPIO5)
- new net GPI36/U1RXD: D5.2 (A), R23.2, U3.4 (GPI36/SENSOR_VP/ADC_H/ADC1_CH0/RTC_GPIO0)
- new net GPI39/IR_RECEIVE: U3.5 (GPI39/SENSOR_VN/ADC1_CH3/ADC_H/RTC_GPIO3)
- new net GPIO0/XTAL1/CLKIN: R36.2, R54.1, U3.25 (GPIO0/ADC2_CH1/TOUCH1/RTC_GPIO11/CLK_OUT1/EMAC_TX_CLK), U4.5 (XTAL1/CLKIN), U9.2 (A2)
- new net GPIO1/U0TXD: D8.1 (K), U3.35 (GPIO1/U0TXD/CLK_OUT3/EMAC_RXD2)
- new net GPIO10/SD_DATA3: U3.18 (GPIO10/SD_DATA3/SPIWP/HS1_DATA3/U1TXD)
- new net GPIO11/SD_CMD: U3.19 (GPIO11/SD_CMD/SPICS0/HS1_CMD/U1RTS)
- new net GPIO12/IR_Transmit: U3.14 (GPIO12/ADC2_CH5/TOUCH5/RTC_GPIO15/MTDI/HSPIQ/HS2_DATA2/SD_DATA2/EMAC_TXD3)
- new net GPIO13/I2C-SDA: R21.2, U3.16 (GPIO13/ADC2_CH4/TOUCH4/RTC_GPIO14/MTCK/HSPID/HS2_DATA3/SD_DATA3/EMAC_RX_ER), UEXT1.6
- new net GPIO14/HS2_CLK: U3.13 (GPIO14/ADC2_CH6/TOUCH6/RTC_GPIO16/MTMS/HSPICLK/HS2_CLK/SD_CLK/EMAC_TXD2), UEXT1.9
- new net GPIO15/HS2_CMD: U3.23 (GPIO15/ADC2_CH3/TOUCH3/MTDO/HSPICS0/RTC_GPIO13/HS2_CMD/SD_CMD/EMAC_RXD3), UEXT1.7
- new net GPIO16/I2C-SCL: R18.2, U3.27 (GPIO16/HS1_DATA4/U2RXD/EMAC_CLK_OUT), UEXT1.5
- new net GPIO17/SPI_CS: R22.2, U3.28 (GPIO17/HS1_DATA5/U2TXD/EMAC_CLK_OUT_180), UEXT1.10
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Other:
- note added: "+"
- note added: "+5V_Only!!!"
- note added: "-"
- note added: "3v3 LDO"
- note added: "9V->5V LDO"
- note added: "=================== Desired Tdelay=500ms =================== 1. 49.9k/1%/R0603; 10uF/6.3V/20%/X5R/C0603; ===> Tdelay=750ms(Measured) 2. 220k/R0603; 1uF/10V/10%/X5R/C0603; =======> Tdelay=500ms(Measured) = OK!!!"
- note added: "Auto program"
- note added: "CD"
- note added: "DTR RTS->EN IO0"
- note added: "ESP-WROOM-32 MODULE"
- note added: "HSPICLK"
- note added: "HSPID"
- note added: "HSPIQ"
- note added: "IBAT = 1000/Rprog = 500mA"
- note added: "LiPo Charger"
- note added: "NCP303LSN18T1G is OK too!"
- note added: "Relays"
- note added: "UEXT"
- note added: "USB to UART"
- note added: "USB/POE Power Switch"
- note added: "tD2 ≈ RD * CD RD = 1M Ohm -> typiclally CD = 470nF -> selected then: tD2 approx. 470ms"
- note removed: "CHARGING"
- note removed: "External Power Sense"
- note removed: "Galvanic Isolated Part"
- note removed: "IBAT = 1000/Rprog = 100mA"
- note removed: "LIPO Charger"

Commit message: poe
Parts:
- removed ACT1: LED/YELLOW/0603, OLIMEX_LEDs-FP:LED_0603_KA, symbol ESP32-PoE-ISO_Rev_K:LED
- removed C1, C2, C6: 22uF/6.3V/20%/X5R/C0603, OLIMEX_RLC-FP:C_0603_5MIL_DWS, symbol ESP32-PoE-ISO_Rev_K:C
- removed C10, C4, C5, C7, C8: 100nF/16V/10%/X7R/C0402, OLIMEX_RLC-FP:C_0402_5MIL_DWS, symbol ESP32-PoE-ISO_Rev_K:C
- removed C11: NA(10uF/6.3V/20%/X5R/C0603), OLIMEX_RLC-FP:C_0603_5MIL_DWS, symbol ESP32-PoE-ISO_Rev_K:C
- removed C11, C13, C14, C15, C17: 100nF/50V/20%/Y5V/C0603, OLIMEX_RLC-FP:C_0603_5MIL_DWS, symbol ESP32-EVB_Rev_K1-rescue:C-ESP32-EVB_Rev_K1
- removed C12, C29, C8, C9: 22uF/6.3V/20%/X5R/C0603, OLIMEX_RLC-FP:C_0603_5MIL_DWS, symbol ESP32-EVB_Rev_K1-rescue:C-ESP32-EVB_Rev_K1
- removed C16: 2.2uF/6.3V/10%/X5R/C0603, OLIMEX_RLC-FP:C_0603_5MIL_DWS, symbol ESP32-EVB_Rev_K1-rescue:C-ESP32-EVB_Rev_K1
- removed C18: 1nF/50V/5%/NPO(COG)/C0603, OLIMEX_RLC-FP:C_0603_5MIL_DWS, symbol ESP32-EVB_Rev_K1-rescue:C-ESP32-EVB_Rev_K1
- removed C19: 1nF/2000V/10%/X7R/C1206, OLIMEX_RLC-FP:C_1206_5MIL_DWS_ISO, symbol ESP32-EVB_Rev_K1-rescue:C-ESP32-EVB_Rev_K1
- removed C20: NA(1nF/2000V/10%/X7R/C1206), OLIMEX_RLC-FP:C_1206_5MIL_DWS_ISO, symbol ESP32-EVB_Rev_K1-rescue:C-ESP32-EVB_Rev_K1
- removed C28: NA(470nF/16V/10%/X7R/C0603), OLIMEX_RLC-FP:C_0603_5MIL_DWS, symbol ESP32-EVB_Rev_K1-rescue:C-ESP32-EVB_Rev_K1
- removed C3: 1nF/2000V/10%/X7R/C1206, OLIMEX_RLC-FP:C_1206_5MIL_DWS_ISO, symbol ESP32-PoE-ISO_Rev_K:C
- removed C32: 1uF/10V/10%/X5R/C0603, OLIMEX_RLC-FP:C_0603_5MIL_DWS, symbol ESP32-EVB_Rev_K1-rescue:C-ESP32-EVB_Rev_K1
- removed C9: 2.2uF/6.3V/10%/X5R/C0603, OLIMEX_RLC-FP:C_0603_5MIL_DWS, symbol ESP32-PoE-ISO_Rev_K:C
- removed CR1: Q50MHz/25ppm/3V/4P/5x3.2mm, OLIMEX_Crystal-FP:5032-4P_HCX-3S, symbol ESP32-EVB_Rev_K1-rescue:Oscillator-100MHZ_TXC-7W-ESP32-EVB_Rev_K1
- removed D10: BAT54A(SOT23-3), OLIMEX_Diodes-FP:SOT23-3, symbol ESP32-EVB_Rev_K1-rescue:BAT54A(SOT23-3)-ESP32-EVB_Rev_K1
- removed FET1: WPM2015-3/TR, OLIMEX_Transistors-FP:SOT23, symbol ESP32-PoE-ISO_Rev_K:P-MOS+DIOD
- removed FET3: WPM2015-3/TR, OLIMEX_Transistors-FP:SOT23, symbol ESP32-EVB_Rev_K1-rescue:P-MOS+DIOD-ESP32-EVB_Rev_K1
- removed FET4: BSS138, OLIMEX_Transistors-FP:SOT23, symbol ESP32-EVB_Rev_K1-rescue:N-MOS+DIOD-ESP32-EVB_Rev_K1
- removed L1: FB0805/600R/2A, OLIMEX_RLC-FP:L_0805_5MIL_DWS, symbol ESP32-PoE-ISO_Rev_K:L
- removed L3: FB0805/600R/2A, OLIMEX_RLC-FP:L_0805_5MIL_DWS, symbol ESP32-EVB_Rev_K1-rescue:L-ESP32-EVB_Rev_K1
- removed L5: NA(FB0805/600R/2A), OLIMEX_RLC-FP:L_0805_5MIL_DWS, symbol ESP32-EVB_Rev_K1-rescue:L-ESP32-EVB_Rev_K1
- removed LAN1: RJLD-060TC1(LPJ4013EDNL), OLIMEX_Connectors-FP:RJLBC-060TC1, symbol ESP32-EVB_Rev_K1-rescue:RJLBC-060TC1_GND-ESP32-EVB_Rev_K1
- removed LNK1: LED/GREEN/0603, OLIMEX_LEDs-FP:LED_0603_KA, symbol ESP32-PoE-ISO_Rev_K:LED
- removed PHY_RST1: Opened, OLIMEX_Jumpers-FP:SJ, symbol ESP32-EVB_Rev_K1-rescue:SJ-ESP32-EVB_Rev_K1
- removed R1, R9: 10k/R0402, OLIMEX_RLC-FP:R_0402_5MIL_DWS, symbol ESP32-PoE-ISO_Rev_K:R
- removed R10: 12.1k/1%/R0402, OLIMEX_RLC-FP:R_0402_5MIL_DWS, symbol ESP32-PoE-ISO_Rev_K:R
- removed R2: 1k/R0402, OLIMEX_RLC-FP:R_0402_5MIL_DWS, symbol ESP32-PoE-ISO_Rev_K:R
- removed R25: 0R(board_mounted), OLIMEX_RLC-FP:0R_0603, symbol ESP32-EVB_Rev_K1-rescue:R-ESP32-EVB_Rev_K1
- removed R26, R27: 220R/R0603, OLIMEX_RLC-FP:R_0603_5MIL_DWS, symbol ESP32-EVB_Rev_K1-rescue:R-ESP32-EVB_Rev_K1
- removed R28, R31, R32, R33, R58: 49.9R/1%/R0402, OLIMEX_RLC-FP:R_0402_5MIL_DWS, symbol ESP32-EVB_Rev_K1-rescue:R-ESP32-EVB_Rev_K1
- removed R3, R4, R5, R6: 49.9R/1%/R0402, OLIMEX_RLC-FP:R_0402_5MIL_DWS, symbol ESP32-PoE-ISO_Rev_K:R
- removed R34, R38, R51: 10k/R0603, OLIMEX_RLC-FP:R_0603_5MIL_DWS, symbol ESP32-EVB_Rev_K1-rescue:R-ESP32-EVB_Rev_K1
- removed R36: 10R/R0603, OLIMEX_RLC-FP:R_0603_5MIL_DWS, symbol ESP32-EVB_Rev_K1-rescue:R-ESP32-EVB_Rev_K1
- removed R39: 12.1k/1%/R0603, OLIMEX_RLC-FP:R_0603_5MIL_DWS, symbol ESP32-EVB_Rev_K1-rescue:R-ESP32-EVB_Rev_K1
- removed R50: 1k/R0603, OLIMEX_RLC-FP:R_0603_5MIL_DWS, symbol ESP32-EVB_Rev_K1-rescue:R-ESP32-EVB_Rev_K1
- removed R52: 100k/R0603, OLIMEX_RLC-FP:R_0603_5MIL_DWS, symbol ESP32-EVB_Rev_K1-rescue:R-ESP32-EVB_Rev_K1
- removed R57: NA(1k/R0603), OLIMEX_RLC-FP:R_0603_5MIL_DWS, symbol ESP32-EVB_Rev_K1-rescue:R-ESP32-EVB_Rev_K1
- removed R7, R8: 2.2k/R0402, OLIMEX_RLC-FP:R_0402_5MIL_DWS, symbol ESP32-PoE-ISO_Rev_K:R
- removed RM1, RM2: RA1206_(4X0603)_4B8_2.2k, OLIMEX_RLC-FP:R_MATRIX_4, symbol ESP32-PoE-ISO_Rev_K:RA1206_(4x0603)_4B8_Smashed
- removed RM2, RM3: RA1206_(4X0603)_4B8_2.2k, OLIMEX_RLC-FP:R_MATRIX_4, symbol ESP32-EVB_Rev_K1-rescue:RA1206_(4x0603)_4B8_Smashed-ESP32-EVB_Rev_K1
- removed T1: LMUN2211LT1G(SOT-23), OLIMEX_Transistors-FP:SOT23, symbol ESP32-PoE-ISO_Rev_K:LMUN2211LT1G(SOT-23)
- removed TVS1: ESDS314DBVR(SOT-23-5), OLIMEX_Diodes-FP:SOT-23-5, symbol ESP32-EVB_Rev_K1-rescue:ESDS314DBVR(SOT-23-5)-ESP32-EVB_Rev_K1
- removed TVS1: ESDS314DBVR(SOT-23-5), OLIMEX_Diodes-FP:SOT-23-5, symbol ESP32-PoE-ISO_Rev_K:ESDS314DBVR(SOT-23-5)
- removed TVS2, TVS3: NA(GG0402052R542P), OLIMEX_Diodes-FP:D_0402_5MIL_DWS, symbol ESP32-PoE-ISO_Rev_K:GG0402052R542P
- removed U1: LAN8710A-EZC(QFN32), OLIMEX_IC-FP:QFN32_EP(33)_5.00x5.00x0.90mm_Pitch_0.50mm, symbol ESP32-PoE-ISO_Rev_K:LAN8710A-EZC(QFN32)
- removed U11: HX7027(SOT-23), OLIMEX_IC-FP:SOT-23, symbol ESP32-EVB_Rev_K1-rescue:VDA2710NTA(SOT-23)-ESP32-EVB_Rev_K1
- removed U4: LAN8710A-EZC(QFN32), OLIMEX_IC-FP:QFN32_EP(33)_5.00x5.00x0.90mm_Pitch_0.50mm, symbol ESP32-EVB_Rev_K1-rescue:LAN8710A-EZC(QFN32)-ESP32-EVB_Rev_K1
- removed U8: NA(NCP303LSN27T1G(SOT-23-5)), OLIMEX_IC-FP:SOT-23-5, symbol ESP32-EVB_Rev_K1-rescue:BD5230G-TR(SSOP5_SOT-23-5)-ESP32-EVB_Rev_K1
- removed Y2: 402F2501XIAR, 402F2501XIAR:XTAL_402F2501XIAR, symbol 402F2501XIAR:402F2501XIAR
- added C59, C69: 1nF, Capacitor_SMD:C_0805_2012Metric, symbol Device:C
- added C60, C66, C67, C71: 22uF, Capacitor_SMD:C_0805_2012Metric, symbol Device:C
- added C61, C62, C64, C65, C68, C70: 100nF, Capacitor_SMD:C_0805_2012Metric, symbol Device:C
- added C63: 2.2uF, Capacitor_SMD:C_0805_2012Metric, symbol Device:C
- added C72: 1uF, Capacitor_SMD:C_0805_2012Metric, symbol Device:C
- added D23: SMAJ58A, Diode_SMD:D_SMA, symbol Diode:SMAJ58A
- added D24: BAT54A, Package_TO_SOT_SMD:SOT-23, symbol Diode:BAT54A
- added JP1: SolderJumper_2_Open, symbol Jumper:SolderJumper_2_Open
- added L8, L9: 600R/2A, Inductor_SMD:L_0805_2012Metric, symbol Device:L
- added Q10: BSS138, Package_TO_SOT_SMD:SOT-23, symbol Transistor_FET:BSS138
- added Q9: SI2323DS-T1-GE3, SI2323DS-T1-GE3:SOT23, symbol SI2323DS-T1-GE3:SI2323DS-T1-GE3
- added R100, R101, R97: 10k, Resistor_SMD:R_0805_2012Metric, symbol Device:R_US
- added R104, R105, R106, R107: 2.2k, Resistor_SMD:R_0805_2012Metric, symbol Device:R_US
- added R108: 49.9k, Resistor_SMD:R_0805_2012Metric, symbol Device:R_US
- added R109: 100k, Resistor_SMD:R_0805_2012Metric, symbol Device:R_US
- added R31: 12.1k, Resistor_SMD:R_0805_2012Metric, symbol Device:R_US
- added R32, R99: 1k, Resistor_SMD:R_0805_2012Metric, symbol Device:R_US
- added R33, R81, R82, R83: 49.9, Resistor_SMD:R_0805_2012Metric, symbol Device:R_US
- added R84, R89: 220, Resistor_SMD:R_0805_2012Metric, symbol Device:R_US
- added R90: 24.9k, Resistor_SMD:R_0805_2012Metric, symbol Device:R_US
- added R93: 180k, Resistor_SMD:R_0805_2012Metric, symbol Device:R_US
- added R94: 4.42k, Resistor_SMD:R_0805_2012Metric, symbol Device:R_US
- added U23: ESDS314DBVR, DBV0005A_N, symbol ESDS314DBVR:ESDS314DBVR
- added U25: MCP100-270D, symbol Power_Supervisor:MCP100-270D
- added Y3: ASV-50.000MHZ-LCS-T, ASV-50.000MHZ-LCS-T:XTAL_ASV-50.000MHZ-LCS-T, symbol ASV-50.000MHZ-LCS-T:ASV-50.000MHZ-LCS-T
Connections:
- net RD+ is gone; now on an unnamed net: J25.4 (RD+)
- net RD- is gone; now on an unnamed net: J25.6 (RD-)
- net TD+ is gone; now on an unnamed net: J25.1 (TD+)
- net TD- is gone; now on an unnamed net: J25.3 (TD-)
- net +3.3V: now also C71.1, D24.1, L9.1, Q9.2, R100.1, R97.2, Y3.4 (VDD); no longer R22.2, R29.2, R30.2
- net +3.3VLAN: now also R22.2, R29.2, R30.2, U11.12 (VDDIO), C65.1, C66.1, C67.1, L8.2, L9.2, Q9.3, R107.1
- net ESP_EN: now also D24.2, R109.1
- net GND: now also C59.2, C63.2, C64.2, C65.2, C66.2, C67.2, C68.2, C69.2, C72.2, JP1.1 (A), Q10.2 (S), R104.2, R105.2, R106.2, R31.1, R89.1, U23.2 (GND), U25.3 (VSS), Y3.2 (GND)
- net OSC_DIS: now also Q10.1 (G), R100.2, R32.1, U25.1 (~{RST}), Y3.1 (TRI_STATE)
- net PHYAD0: now also R104.1
- net PHYAD1: now also R105.1
- net PHYAD2: now also R106.1
- net RMIISEL: now also R107.2
- net Spare1: now also U12.8 (VDD), C70.1, D23.1 (A1), R90.2
- net Spare2: now also U12.4 (VSS), C70.2, D23.2 (A2), R93.1, R94.1
- net VDDA1/2: now reaches J25.2 (TCT), J25.5 (RCT)
- net VDDA1/2: now also U11.1 (VDD2A), U11.27 (VDD1A), C60.2, C61.2, C62.1, C68.1, L8.1, R33.2, R81.2, R82.2, R83.2, R84.2
- net at R30.1, U11.19 (NRST): now also C59.1, JP1.2 (B), R32.2
- net LED2: now reaches U11.2 (LED2/*NINTSEL)
- net LED2: now also J25.GK2
- net at U11.28 (TXN): now also R82.1, U23.3 (I_O2)
- net at U11.29 (TXP): now also R83.1, U23.1 (I_O1)
- net LED1: now reaches U11.3 (LED1/*REGOFF)
- net LED1: now also J25.GA1
- net at U11.30 (RXN): now also R33.1, U23.5 (I_O4)
- net at U11.31 (RXP): now also R81.1, U23.4 (I_O3)
- net at U11.32 (RBIAS): now also R31.2
- net at U11.33 (EPAD): now also C60.1, C61.1, C62.2
- net GPIO0/XTAL1/CLKIN: now reaches U11.5 (XTAL1/CLKIN)
- net GPIO0/XTAL1/CLKIN: now also R101.1
- net at U11.6 (VDDCR): now also C63.1, C64.1
- net at U12.1 (ILIM): now also R93.2
- net at U12.2 (CLASS): now also R94.2
- net at U12.3 (DET): now also R90.1
- net at J25.GA2: now also R84.1
- net at J25.GK1: now also R89.2
- net Shield: no longer names the net of J25.7 (P7), J25.S1 (SHIELD), J25.S2 (SHIELD)
- net Shield: now also C69.1
- new net: C71.2, Q9.1, R97.1, R99.2
- new net: D24.3, R108.1
- new net: C72.1, R108.2, R109.2, U25.2 (VDD)
- new net: Q10.3 (D), R99.1
- new net: R101.2, Y3.3 (OUTPUT)
- no-connect marks 26 -> 12
Other:
- note added: "ETHERNET"
- note removed: "=================== Desired Tdelay=500ms =================== 1. 49.9k/1%/R0603; 10uF/6.3V/20%/X5R/C0603; ===> Tdelay=750ms(Measured) 2. 220k/R0603; 1uF/10V/10%/X5R/C0603; =======> Tdelay=500ms(Measured) = OK!!!"
- note removed: "CD"
- note removed: "Ethernet"
- note removed: "GPIO4:"
- note removed: "In RMII Mode"
- note removed: "NCP303LSN18T1G is OK too!"
- note removed: "Notes:"
- note removed: "The PHY is setted up as follows: MODE: All capable(10/100Base) -Auto-negotiation enabled -RMII Configuration -SMI address: 0x00"
- note removed: "tD2 ≈ RD * CD RD = 1M Ohm -> typiclally CD = 470nF -> selected then: tD2 approx. 470ms"
- moved on the sheet: C31, R22, R24, R29, R30, R54, U11, U12, U3

Commit message: stuff
Parts:
- removed BUT1, RST1: T1107A(6x3,8x2,5MM), OLIMEX_Buttons-FP:T1107A(6x3,8x2,5MM), symbol ESP32-EVB_Rev_K1-rescue:SIDE_WTCM-TR(3x4)-ESP32-EVB_Rev_K1
- removed C12, C14: 100nF/100V/10%/X7R/C0603, OLIMEX_RLC-FP:C_0603_5MIL_DWS, symbol ESP32-PoE-ISO_Rev_K:C
- removed C13: 15uF/100V/20%/RM2.5/6.3x11mm(Farnell:1281844), OLIMEX_RLC-FP:CPOL-RM2.5mm_6.3x11mm_PTH, symbol ESP32-PoE-ISO_Rev_K:CP
- removed C15: 12pF/50V/5%/COG/C0402, OLIMEX_RLC-FP:C_0402_5MIL_DWS, symbol ESP32-PoE-ISO_Rev_K:C
- removed C16: 470uF/10V/20%/Low_ESR/RM2.5/6.0x11mm, OLIMEX_RLC-FP:CPOL-RM2.5mm_6.3x11mm_PTH, symbol ESP32-PoE-ISO_Rev_K:CP
- removed C17, C18: 1.0nF/3kV/10%/X7R/SMD/1808(VISHAY-VJ1808Y102KBHAT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, OLIMEX_RLC-FP:C_1808(4520)_5MIL_DWS_ISO, symbol ESP32-PoE-ISO_Rev_K:C
- removed C19: 22uF/6.3V/20%/X5R/C0603, OLIMEX_RLC-FP:C_0603_5MIL_DWS, symbol ESP32-PoE-ISO_Rev_K:C
- removed C31: 1uF/10V/10%/X5R/C0603, OLIMEX_RLC-FP:C_0603_5MIL_DWS, symbol ESP32-EVB_Rev_K1-rescue:C-ESP32-EVB_Rev_K1
- removed C5: 22uF/6.3V/20%/X5R/C0603, OLIMEX_RLC-FP:C_0603_5MIL_DWS, symbol ESP32-EVB_Rev_K1-rescue:C-ESP32-EVB_Rev_K1
- removed CON1, CON2: TB3-DG306-5.0-3P, OLIMEX_Connectors-FP:TB3-DG306-5.0_3P, symbol ESP32-EVB_Rev_K1-rescue:CON3-ESP32-EVB_Rev_K1
- removed D1: SMAJ58A/SMA, OLIMEX_Diodes-FP:SMA-KA, symbol ESP32-PoE-ISO_Rev_K:SMBJ6.0A
- removed D1, D3: 1N5819S4(SOD-123), OLIMEX_Diodes-FP:SOD-123_1C-2A_KA, symbol ESP32-EVB_Rev_K1-rescue:D_Schottky-ESP32-EVB_Rev_K1
- removed D2: SS510/100V/5A/0.85V/DO214AB(SMC), OLIMEX_Diodes-FP:DO214AB(SMC)_1(K)-2(A), symbol ESP32-PoE-ISO_Rev_K:D_Schottky_Small
- removed D3: NA(SMBJ6.0A), OLIMEX_Diodes-FP:DO214AA_1(K)-2(A), symbol ESP32-PoE-ISO_Rev_K:SMBJ6.0A
- removed D5: 1N5819S4(SOD-123), OLIMEX_Diodes-FP:SOD-123_1C-2A_KA, symbol ESP32-EVB_Rev_K1-rescue:D_Schottky_Small-ESP32-EVB_Rev_K1
- removed DCDC1: F0505S-2WR2(SIP-7), OLIMEX_Regulators-FP:SIP-7_Universal, symbol ESP32-PoE-ISO_Rev_K:F0505S-2WR2_AM1D-0505S-NZ(SIP-7_Universal)
- removed L1: FB0805/600R/2A, OLIMEX_RLC-FP:L_0805_5MIL_DWS, symbol ESP32-EVB_Rev_K1-rescue:L-ESP32-EVB_Rev_K1
- removed L2: 33uH/2.1A/DCR=0.1R/20%/DBS135(PD3316MT330), SRR1240-330M:IND_BOURNS_SRR1240, symbol ESP32-PoE-ISO_Rev_K:L
- removed LED1, LED2: LED/GREEN/0603, OLIMEX_LEDs-FP:LED_0603_KA, symbol ESP32-EVB_Rev_K1-rescue:LED-ESP32-EVB_Rev_K1
- removed Q1, Q2: BC817-40(SOT23), OLIMEX_Transistors-FP:SOT23, symbol ESP32-EVB_Rev_K1-rescue:Q_NPN_BEC-ESP32-EVB_Rev_K1
- removed R1, R5: 1k/R0603, OLIMEX_RLC-FP:R_0603_5MIL_DWS, symbol ESP32-EVB_Rev_K1-rescue:R-ESP32-EVB_Rev_K1
- removed R11: 130k/R0402, OLIMEX_RLC-FP:R_0402_5MIL_DWS, symbol ESP32-PoE-ISO_Rev_K:R
- removed R11, R18, R21, R3: 2.2k/R0603, OLIMEX_RLC-FP:R_0603_5MIL_DWS, symbol ESP32-EVB_Rev_K1-rescue:R-ESP32-EVB_Rev_K1
- removed R12: 10k/R0402, OLIMEX_RLC-FP:R_0402_5MIL_DWS, symbol ESP32-PoE-ISO_Rev_K:R
- removed R13: 24.9k/1%/R0402, OLIMEX_RLC-FP:R_0402_5MIL_DWS, symbol ESP32-PoE-ISO_Rev_K:R
- removed R14: 180k/1%/R0402, OLIMEX_RLC-FP:R_0402_5MIL_DWS, symbol ESP32-PoE-ISO_Rev_K:R
- removed R14: 220R/R0603, OLIMEX_RLC-FP:R_0603_5MIL_DWS, symbol ESP32-EVB_Rev_K1-rescue:R-ESP32-EVB_Rev_K1
- removed R15: 4.42k/1%/1/16W/R0402, OLIMEX_RLC-FP:R_0402_5MIL_DWS, symbol ESP32-PoE-ISO_Rev_K:R
- removed R16: 4.7k/R2512, OLIMEX_RLC-FP:R_2512_MM_DWS, symbol ESP32-PoE-ISO_Rev_K:R
- removed R17: 0.03R/1%/R1206, OLIMEX_RLC-FP:R_1206_5MIL_DWS, symbol ESP32-PoE-ISO_Rev_K:R
- removed R18: 4.7R/R0402, OLIMEX_RLC-FP:R_0402_5MIL_DWS, symbol ESP32-PoE-ISO_Rev_K:R
- removed R19: 10.5k/1%/R0402, OLIMEX_RLC-FP:R_0402_5MIL_DWS, symbol ESP32-PoE-ISO_Rev_K:R
- removed R2, R22, R23, R24, R45, R6: 10k/R0603, OLIMEX_RLC-FP:R_0603_5MIL_DWS, symbol ESP32-EVB_Rev_K1-rescue:R-ESP32-EVB_Rev_K1
- removed R20: 56.2k/1%/R0402, OLIMEX_RLC-FP:R_0402_5MIL_DWS, symbol ESP32-PoE-ISO_Rev_K:R
- removed R46, R54: NA/R0603, OLIMEX_RLC-FP:R_0603_5MIL_DWS, symbol ESP32-EVB_Rev_K1-rescue:R-ESP32-EVB_Rev_K1
- removed REL1, REL2: RAS-0515, OLIMEX_Relays-FP:Relay_RAS-05-15, symbol ESP32-EVB_Rev_K1-rescue:Relay-ESP32-EVB_Rev_K1
- removed U14, U15: TPS54561DPRR, WSON10_DPR_TEX, symbol TPS54561DPRR:TPS54561DPRR
- removed U2: TPS2376PW(TSSOP-8), OLIMEX_IC-FP:TSSOP-8_Pitch-0.65mm_Dimensions-4.40x3.00x1.20mm, symbol ESP32-PoE-ISO_Rev_K:TPS2375PW(TSSOP-8)
- removed U3: ESP-WROOM-32, OLIMEX_Cases-FP:ESP-WROOM-32_MODULE, symbol ESP32-EVB_Rev_K1-rescue:ESP-WROOM-32-ESP32-EVB_Rev_K1
- removed U3: TX4138(ESOIC-8), OLIMEX_Regulators-FP:ESOIC-8, symbol ESP32-PoE-ISO_Rev_K:TX4138(ESOIC-8)
- removed UEXT1: BH10S, OLIMEX_Connectors-FP:UEXT_ML10, symbol ESP32-EVB_Rev_K1-rescue:BH10S-ESP32-EVB_Rev_K1
- added C1: 15uF, Capacitor_SMD:C_0805_2012Metric, symbol Device:C
- added C2, C8: 100pF, Capacitor_SMD:C_0805_2012Metric, symbol Device:C
- added C3: 220nF, Capacitor_SMD:C_0805_2012Metric, symbol Device:C
- added C4: 470pF, Capacitor_SMD:C_0805_2012Metric, symbol Device:C
- added C5: 12nF, Capacitor_SMD:C_0805_2012Metric, symbol Device:C
- added C6: 100nF, Capacitor_SMD:C_0805_2012Metric, symbol Device:C
- added C7: 1uF, Capacitor_SMD:C_0805_2012Metric, symbol Device:C
- added R1: 130k, Resistor_SMD:R_0805_2012Metric, symbol Device:R_US
- added R2: 10k, Resistor_SMD:R_0805_2012Metric, symbol Device:R_US
- added R3: 18k, Resistor_SMD:R_0805_2012Metric, symbol Device:R_US
- added R4: 8.25k, Resistor_SMD:R_0805_2012Metric, symbol Device:R_US
- added R5: 9.3k, Resistor_SMD:R_0805_2012Metric, symbol Device:R_US
- added R6: 6k, Resistor_SMD:R_0805_2012Metric, symbol Device:R_US
- added R7: 100, Resistor_SMD:R_0805_2012Metric, symbol Device:R_US
- added R8: 5.24M, Resistor_SMD:R_0805_2012Metric, symbol Device:R_US
- added U1: LM5156DSSR, DSS0012B, symbol LM5156DSSR:LM5156DSSR
Connections:
- net GND: now also C70.2, D23.2 (A2), J25.9 (P9), R93.1, R94.1, U12.4 (VSS), U12.5 (RTN), C1.2, C2.2, C3.2, C6.2, C7.2, C8.2, R2.1, R4.1, R5.1, R6.1, R8.1, U1.4 (GND)
- net Spare1: now also J25.10 (P10), C1.1, C6.1, R1.2, R3.2, U1.1 (BIAS); no longer J25.9 (P9)
- net at U12.7 (UVLO): now also R1.1, R2.2
- removed net Spare2: C70.2, D23.2 (A2), J25.10 (P10), R93.1, R94.1, U12.4 (VSS)
- new net: C4.1, C5.1, U1.6 (COMP)
- new net: C4.2, C5.2, R6.2
- new net: C2.1, R3.1, R4.2, U1.12 (UVLO_SYNC)
- new net: R7.1, R8.2
- new net: C8.1, R7.2, U1.5 (CS)
- new net: R5.2, U1.10 (RT)
- new net: C7.1, U1.2 (VCC), U1.7 (DITHOFF)
- new net: C3.1, U1.9 (SS)
- no-connect marks 12 -> 11
Other:
- note added: "Ethernet"
- note removed: "5V/2A"
- note removed: "CDET"
- note removed: "Class=0 (0.44 to 12.95W)"
- note removed: "ESP-WROOM-32 MODULE"
- note removed: "ETHERNET"
- note removed: "HSPICLK"
- note removed: "HSPID"
- note removed: "HSPIQ"
- note removed: "POE Supply"
- note removed: "RDET"
- note removed: "Rclass"
- note removed: "Relays"
- note removed: "UEXT"
- note removed: "Vout=0.8*(1+Ra/Rb)"
- moved on the sheet: C20, C21, C22, C23, C24, C25, C26, C27, C32, C59, C60, C61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

Commit message: stuff
Parts:
- removed BAT/BUT1: Opened(2-3)/Soldered(1-2), OLIMEX_Jumpers-FP:SJ_2_SMALL, symbol ESP32-EVB_Rev_K1-rescue:SJ2W_Closed(1-2)-ESP32-EVB_Rev_K1
- removed BAT1: DW02R, OLIMEX_Connectors-FP:LIPO_BAT-CON2DW02R, symbol ESP32-EVB_Rev_K1-rescue:BAT_CON-ESP32-EVB_Rev_K1
- removed C1, C3: NA(47uF/6.3V/20%/X5R/C0805), OLIMEX_RLC-FP:C_0805_5MIL_DWS, symbol ESP32-EVB_Rev_K1-rescue:C-ESP32-EVB_Rev_K1
- removed C2, C4: 47uF/6.3V/20%/X5R/C0805, OLIMEX_RLC-FP:C_0805_5MIL_DWS, symbol ESP32-EVB_Rev_K1-rescue:C-ESP32-EVB_Rev_K1
- removed C21, C22: 27pF/50V/5%/C0G/C0603, OLIMEX_RLC-FP:C_0603_5MIL_DWS, symbol ESP32-EVB_Rev_K1-rescue:C-ESP32-EVB_Rev_K1
- removed C23, C6, C7: 22uF/6.3V/20%/X5R/C0603, OLIMEX_RLC-FP:C_0603_5MIL_DWS, symbol ESP32-EVB_Rev_K1-rescue:C-ESP32-EVB_Rev_K1
- removed C24, C30: 100nF/50V/20%/Y5V/C0603, OLIMEX_RLC-FP:C_0603_5MIL_DWS, symbol ESP32-EVB_Rev_K1-rescue:C-ESP32-EVB_Rev_K1
- removed CHARGE?: LED/Yellow/0603, OLIMEX_LEDs-FP:LED_0603_KA, symbol ESP32-EVB_Rev_K1-rescue:LED-ESP32-EVB_Rev_K1
- removed D2: SMBJ6.0A(DO-214AA), OLIMEX_Diodes-FP:DO214AA_1(K)-2(A), symbol ESP32-EVB_Rev_K1-rescue:SMBJ6.0A-ESP32-EVB_Rev_K1
- removed D4, D6: 1N5822/SS34/SMA, OLIMEX_Diodes-FP:SMA-KA, symbol ESP32-EVB_Rev_K1-rescue:D_Schottky-ESP32-EVB_Rev_K1
- removed D7, D8, D9: 1N5819S4(SOD-123), OLIMEX_Diodes-FP:SOD-123_1C-2A_KA, symbol ESP32-EVB_Rev_K1-rescue:D_Schottky_Small-ESP32-EVB_Rev_K1
- removed FET1, FET2: WPM2015-3/TR, OLIMEX_Transistors-FP:SOT23, symbol ESP32-EVB_Rev_K1-rescue:P-MOS+DIOD-ESP32-EVB_Rev_K1
- removed GND1: TESTPAD, OLIMEX_Other-FP:TESTPAD_40-ROUND, symbol ESP32-EVB_Rev_K1-rescue:TESTPAD-ESP32-EVB_Rev_K1
- removed L2: 2.2uH/1.5A/DCR=72mR/20%/3.00x3.00x1.50mm/CD32(NR3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, OLIMEX_RLC-FP:CD32, symbol ESP32-EVB_Rev_K1-rescue:L-ESP32-EVB_Rev_K1
- removed PWR1: PWRJ-2mm(YDJ-1134), OLIMEX_Connectors-FP:PWRJ-2mm(YDJ-1136), symbol ESP32-EVB_Rev_K1-rescue:PWR-JAKPWR_JACK_UNI_MILLING-ESP32-EVB_Rev_K1
- removed PWR2: NA(TB2 DG306-5.0-2P), OLIMEX_Connectors-FP:TB2-DG306-5.0_2P, symbol ESP32-EVB_Rev_K1-rescue:CON2-ESP32-EVB_Rev_K1
- removed PWRLED1: LED/RED/0603, OLIMEX_LEDs-FP:LED_0603_KA, symbol ESP32-EVB_Rev_K1-rescue:LED-ESP32-EVB_Rev_K1
- removed Q3: Q12MHz/20pF/30ppm/2P/HC-49SM(SMD), OLIMEX_Crystal-FP:Q_49U3HMS, symbol ESP32-EVB_Rev_K1-rescue:Crystal-ESP32-EVB_Rev_K1
- removed Q4, Q5: BC817-40(SOT23), OLIMEX_Transistors-FP:SOT23, symbol ESP32-EVB_Rev_K1-rescue:Q_NPN_BEC-ESP32-EVB_Rev_K1
- removed R10, R9: 470k/R0603, OLIMEX_RLC-FP:R_0603_5MIL_DWS, symbol ESP32-EVB_Rev_K1-rescue:R-ESP32-EVB_Rev_K1
- removed R17, R44: NA/R0603, OLIMEX_RLC-FP:R_0603_5MIL_DWS, symbol ESP32-EVB_Rev_K1-rescue:R-ESP32-EVB_Rev_K1
- removed R19: 220k/R0603, OLIMEX_RLC-FP:R_0603_5MIL_DWS, symbol ESP32-EVB_Rev_K1-rescue:R-ESP32-EVB_Rev_K1
- removed R20: 49.9k/1%/R0603, OLIMEX_RLC-FP:R_0603_5MIL_DWS, symbol ESP32-EVB_Rev_K1-rescue:R-ESP32-EVB_Rev_K1
- removed R30, R35, R40: 10k/R0603, OLIMEX_RLC-FP:R_0603_5MIL_DWS, symbol ESP32-EVB_Rev_K1-rescue:R-ESP32-EVB_Rev_K1
- removed R37: 220R/R0603, OLIMEX_RLC-FP:R_0603_5MIL_DWS, symbol ESP32-EVB_Rev_K1-rescue:R-ESP32-EVB_Rev_K1
- removed R4, R?: 2.2k/R0603, OLIMEX_RLC-FP:R_0603_5MIL_DWS, symbol ESP32-EVB_Rev_K1-rescue:R-ESP32-EVB_Rev_K1
- removed R41, R42: 1k/R0603, OLIMEX_RLC-FP:R_0603_5MIL_DWS, symbol ESP32-EVB_Rev_K1-rescue:R-ESP32-EVB_Rev_K1
- removed R?: 2k/1%/R0603, OLIMEX_RLC-FP:R_0603_5MIL_DWS, symbol ESP32-EVB_Rev_K1-rescue:R-ESP32-EVB_Rev_K1
- removed U10, U9: BAT54C(SOT23-3), OLIMEX_Diodes-FP:SOT23-3, symbol ESP32-EVB_Rev_K1-rescue:BAT54C(SOT23-3)-ESP32-EVB_Rev_K1
- removed U13: RFM-0505S, SIP4_RFM_RCP, symbol RFM_0505S:RFM-0505S
- removed U16: ROE-0512S, ROE_RCP, symbol ROE-0512S:ROE-0512S
- removed U2: SY8089AAAC(SOT23-5), OLIMEX_Regulators-FP:SOT-23-5, symbol ESP32-EVB_Rev_K1-rescue:SY8009AAAC(SOT23-5)-ESP32-EVB_Rev_K1
- removed U5: CH340T(SSOP20W), OLIMEX_IC-FP:SSOP-20W, symbol ESP32-EVB_Rev_K1-rescue:CH340T(SSOP20W)-ESP32-EVB_Rev_K1
- removed U?: BL4054B-42TPRN(SOT23-5), OLIMEX_IC-FP:SOT-23-5, symbol ESP32-EVB_Rev_K1-rescue:BL4054B-42TPRN(SOT23-5)-ESP32-EVB_Rev_K1
- removed USB-UART1: MISB-SWMM-5B-LF(USB_MICRO), OLIMEX_Connectors-FP:USB-MICRO_MISB-SWMM-5B_LF, symbol ESP32-EVB_Rev_K1-rescue:USB-MINI-ESP32-EVB_Rev_K1
Connections:
- no-connect marks 11 -> 4
Other:
- note removed: "+"
- note removed: "+5V_Only!!!"
- note removed: "-"
- note removed: "Auto program"
- note removed: "Battery Measurement"
- note removed: "DTR RTS->EN IO0"
- note removed: "IBAT = 1000/Rprog = 500mA"
- note removed: "LiPo Charger"
- note removed: "Ra"
- note removed: "Rb"
- note removed: "Rprog"
- note removed: "USB to UART"
- note removed: "Vout=0.6*(1+Ra/Rb)"
