File: Hardware/Gen2Dev/InnerBoard/2.1/InnerBoard_rev2.1/InnerBoard_rev2.1.kicad_sch (KiCad schematic)
At the start: 142 parts, among them J2 HMTSW-102-X-X-S-X, J25 SI-46020-F, J3 HMTSW-102-X-X-S-X, J4 HMTSW-102-X-X-S-X, J5 UJ31-CH-G2-SMT-TR, J8 3221-10-0300-00, J9 HMTSW-102-X-X-S-X, Q1 SI2323DS-T1-GE3, Q10 BSS138, Q4 BC817, Q5 BC817, Q9 SI2323DS-T1-GE3, SW1 PTS815 SJM 250 SMTR LFS, U1 LM5156DSSR, U10 ESP32-WROOM-32E-N8, U11 LAN8710A-EZC, U12 TPS2376PW, U23 ESDS314DBVR, U25 MCP100-270D, U4 MIC5504-3.3YM5, U6 74LVC1G04, U7 LD1117S50TR_SOT223, U9 FT232RQ, Y1 ABLS2-12.000MHZ-D4Y-T, Y3 ASV-50.000MHZ-LCS-T

Commit message: schematic for v2.1 dev board done. Footprints update progress. Layout will roll when footprints finalize
Parts:
- removed L6: FB0805/600R/2A, Inductor_SMD:L_0805_2012Metric, symbol Device:L
- removed TP7: TestPoint, TestPoint:TestPoint_Pad_D2.0mm, symbol Connector:TestPoint
- added J1, J10, J11, J12, J13, J14, J15, J16, J17, J18, J19, J7: HMTSW-102-X-X-S-X, Connector_PinHeader_2.54mm:PinHeader_1x02_P2.54mm_Vertical, symbol HMTSW-102-X-X-S-X:HMTSW-102-X-X-S-X
- added TP10, TP11, TP12, TP13, TP14, TP15, TP16, TP17, TP18, TP19, TP20, TP21, TP22, TP23, TP24, TP25, TP26, TP27, TP28, TP29, TP30, TP8, TP9: TestPoint, TestPoint:TestPoint_Pad_D2.0mm, symbol Connector:TestPoint
- C26, C27: footprint (none) -> Capacitor_SMD:C_0805_2012Metric
- J2, J3, J4, J9: footprint HMTSW-102-X-X-S-X:SAMTEC_HMTSW-102-X-X-S-X -> Connector_PinHeader_2.54mm:PinHeader_1x02_P2.54mm_Vertical
- JP1: footprint (none) -> Jumper:SolderJumper-2_P1.3mm_Open_Pad1.0x1.5mm
- R50: value 6.1K -> 5.1K
- U1: footprint DSS0012B -> 5156:DSS0012B
Connections:
- net +3.3V: now also TP23.1
- net +3.3VLAN: now also J10.01, TP16.1; no longer U11.12 (VDDIO)
- net +5V: now also TP21.1
- net +5VP: now also TP19.1
- net +9V: now also TP22.1
- net D_Com: now also TP13.1
- net ESP_EN: now also TP15.1
- net GND: now also J5.A1 (GND), J5.A12 (GND__1), J5.B1 (GND__2), J5.B12 (GND__3), J5.SH1 (SHIELD), J5.SH2 (SHIELD__1), J5.SH3 (SHIELD__2), J5.SH4 (SHIELD__3), TP10.1, TP17.1
- net GPIO0: now also TP29.1
- net GPIO12/PHY_PWR: now also TP26.1
- net GPIO15/HS2_CMD: now also TP27.1
- net GPIO2/HS2_DATA0: now also TP28.1
- net GPIO5/SPI_CS: now also TP30.1
- net OSC_DIS: now also TP8.1
- net PHYAD0: now also J13.01; no longer R104.1
- net PHYAD1: now also J14.01; no longer R105.1
- net PHYAD2: now also J15.01; no longer R106.1
- net RMIISEL: now also TP24.1
- net Spare1: now also TP11.1
- net USB_DN: now also J5.B7 (DN2), J11.01; no longer J5.A6 (DP1), U9.15 (USBDM)
- net USB_DP: now also J5.A6 (DP1), J12.01; no longer J5.B7 (DN2), U9.14 (USBDP)
- net VBUS: now also TP20.1
- net VDDA1/2: now also J1.01, J7.02, TP14.1; no longer U11.1 (VDD2A), U11.27 (VDD1A)
- net at C71.2, Q9.1, R97.1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: now also TP9.1
- net at C72.1, R108.2, R109.2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: now also TP25.1
- net at J25.1 (TD+), R83.1, U23.1 (I_O1): now also J19.01; no longer U11.29 (TXP)
- net at J25.6 (RD-), R33.1, U23.5 (I_O4): now also J16.02; no longer U11.30 (RXN)
- net at J25.4 (RD+), R81.1, U23.4 (I_O3): now also J17.02; no longer U11.31 (RXP)
- net at C60.1, C61.1, C62.2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: now also TP12.1
- net at R1.1, R2.2, U12.7 (UVLO): now also TP18.1
- new net: J1.02, U11.1 (VDD2A)
- new net: J10.02, U11.12 (VDDIO)
- new net: J7.01, U11.27 (VDD1A)
- new net: J18.02, U11.29 (TXP)
- new net: J16.01, U11.30 (RXN)
- new net: J17.01, U11.31 (RXP)
- new net: J15.02, R106.1
- new net: J12.02, U9.14 (USBDP)
- new net: J11.02, U9.15 (USBDM)
- new net: J14.02, R105.1
- new net: J13.02, R104.1
- new net: J18.01, J19.02
Other:
- moved on the sheet: D11, J5, R27, R50, R51, TP3, TP4, TP5, TP6

Commit message: Inner board 2.1 footprint links fixed (for future work) and more included. Layout will roll when footprints finalize
Parts:
- J1, J10, J11, J12, J13, J14, J15, J16, J17, J18, J19, J2, J3, J4, J7, J9: footprint Connector_PinHeader_2.54mm:PinHeader_1x02_P2.54mm_Vertical -> HMTSW-102-X-X-S-X:SAMTEC_HMTSW-102-X-X-S-X
- J8: footprint CONN10_3221-10-0300-00_CNC -> CONN10_3221-10-0300-00_CNC:CONN10_3221-10-0300-00_CNC
- SW1: footprint SW4_PTS815 SJM 250 SMTR LFS_CNK -> PTS815:SW4_PTS815 SJM 250 SMTR LFS_CNK
- U12: footprint PW8 -> TPS2376PW:PW8
- U23: footprint DBV0005A_N -> ESDS314DBVR:DBV0005A_N
Changed lines of the file:
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@@
 			)
 		)
-		(property "Footprint" "Connector_PinHeader_2.54mm:PinHeader_1x02_P2.54mm_Vertical"
+		(property "Footprint" "HMTSW-102-X-X-S-X:SAMTEC_HMTSW-102-X-X-S-X"
 			(at 349.25 120.65 0)
 			(effects
@@
 			)
 		)
-		(property "Footprint" "DBV0005A_N"
+		(property "Footprint" "ESDS314DBVR:DBV0005A_N"
 			(at 292.608 82.042 0)
 			(effects
@@
 			)
 		)
-		(property "Footprint" "Connector_PinHeader_2.54mm:PinHeader_1x02_P2.54mm_Vertical"
+		(property "Footprint" "HMTSW-102-X-X-S-X:SAMTEC_HMTSW-102-X-X-S-X"
 			(at 699.516 223.52 0)
 			(effects
@@
 			)
 		)
-		(property "Footprint" "Connector_PinHeader_2.54mm:PinHeader_1x02_P2.54mm_Vertical"
+		(property "Footprint" "HMTSW-102-X-X-S-X:SAMTEC_HMTSW-102-X-X-S-X"
 			(at 60.96 86.36 0)
 			(effects
@@
 			)
 		)
-		(property "Footprint" "SW4_PTS815 SJM 250 SMTR LFS_CNK"
+		(property "Footprint" "PTS815:SW4_PTS815 SJM 250 SMTR LFS_CNK"
 			(at 38.862 550.418 0)
 			(effects
@@
 			)
 		)
-		(property "Footprint" "PW8"
+		(property "Footprint" "TPS2376PW:PW8"
 			(at 545.084 98.806 0)
 			(effects
@@
 			)
 		)
-		(property "Footprint" "Connector_PinHeader_2.54mm:PinHeader_1x02_P2.54mm_Vertical"
+		(property "Footprint" "HMTSW-102-X-X-S-X:SAMTEC_HMTSW-102-X-X-S-X"
 			(at 187.96 105.41 0)
 			(effects
@@
 			)
 		)
-		(property "Footprint" "Connector_PinHeader_2.54mm:PinHeader_1x02_P2.54mm_Vertical"
+		(property "Footprint" "HMTSW-102-X-X-S-X:SAMTEC_HMTSW-102-X-X-S-X"
 			(at 668.782 220.726 0)
 			(effects
@@
 			)
 		)
-		(property "Footprint" "Connector_PinHeader_2.54mm:PinHeader_1x02_P2.54mm_Vertical"
+		(property "Footprint" "HMTSW-102-X-X-S-X:SAMTEC_HMTSW-102-X-X-S-X"
 			(at 106.68 133.35 0)
 			(effects
@@
 			)
 		)
-		(property "Footprint" "Connector_PinHeader_2.54mm:PinHeader_1x02_P2.54mm_Vertical"
+		(property "Footprint" "HMTSW-102-X-X-S-X:SAMTEC_HMTSW-102-X-X-S-X"
 			(at 265.43 427.99 0)
 			(effects
@@
 			)
 		)
-		(property "Footprint" "Connector_PinHeader_2.54mm:PinHeader_1x02_P2.54mm_Vertical"
+		(property "Footprint" "HMTSW-102-X-X-S-X:SAMTEC_HMTSW-102-X-X-S-X"
 			(at 341.63 102.87 0)
 			(effects
@@
 			)
 		)
-		(property "Footprint" "Connector_PinHeader_2.54mm:PinHeader_1x02_P2.54mm_Vertical"
+		(property "Footprint" "HMTSW-102-X-X-S-X:SAMTEC_HMTSW-102-X-X-S-X"
 			(at 311.15 113.03 0)
 			(effects
@@
 			)
 		)
-		(property "Footprint" "Connector_PinHeader_2.54mm:PinHeader_1x02_P2.54mm_Vertical"
+		(property "Footprint" "HMTSW-102-X-X-S-X:SAMTEC_HMTSW-102-X-X-S-X"
 			(at 77.47 236.982 0)
 			(effects
@@
 			)
 		)
-		(property "Footprint" "Connector_PinHeader_2.54mm:PinHeader_1x02_P2.54mm_Vertical"
+		(property "Footprint" "HMTSW-102-X-X-S-X:SAMTEC_HMTSW-102-X-X-S-X"
 			(at 322.58 110.49 0)
 			(effects
@@
 			)
 		)
-		(property "Footprint" "Connector_PinHeader_2.54mm:PinHeader_1x02_P2.54mm_Vertical"
+		(property "Footprint" "HMTSW-102-X-X-S-X:SAMTEC_HMTSW-102-X-X-S-X"
 			(at 270.51 414.02 0)
 			(effects
@@
 			)
 		)
-		(property "Footprint" "Connector_PinHeader_2.54mm:PinHeader_1x02_P2.54mm_Vertical"
+		(property "Footprint" "HMTSW-102-X-X-S-X:SAMTEC_HMTSW-102-X-X-S-X"
 			(at 322.58 135.89 0)
 			(effects
@@
 			)
 		)
-		(property "Footprint" "CONN10_3221-10-0300-00_CNC"
+		(property "Footprint" "CONN10_3221-10-0300-00_CNC:CONN10_3221-10-0300-00_CNC"
 			(at 257.556 552.704 0)
 			(effects
@@
 			)
 		)
-		(property "Footprint" "SW4_PTS815 SJM 250 SMTR LFS_CNK"
+		(property "Footprint" "PTS815:SW4_PTS815 SJM 250 SMTR LFS_CNK"
 			(at 38.608 525.018 0)
 			(effects
@@
 			)
 		)
-		(property "Footprint" "Connector_PinHeader_2.54mm:PinHeader_1x02_P2.54mm_Vertical"
+		(property "Footprint" "HMTSW-102-X-X-S-X:SAMTEC_HMTSW-102-X-X-S-X"
 			(at 69.85 80.01 0)
 			(effects
@@
 			)
 		)
-		(property "Footprint" "Connector_PinHeader_2.54mm:PinHeader_1x02_P2.54mm_Vertical"
+		(property "Footprint" "HMTSW-102-X-X-S-X:SAMTEC_HMTSW-102-X-X-S-X"
 			(at 78.74 73.66 0)
 			(effects
@@
 			)
 		)
-		(property "Footprint" "Connector_PinHeader_2.54mm:PinHeader_1x02_P2.54mm_Vertical"
+		(property "Footprint" "HMTSW-102-X-X-S-X:SAMTEC_HMTSW-102-X-X-S-X"
 			(at 277.114 393.7 0)
 			(effects

Commit message: Inner board 2.1 footprint links refactored (for future work) and more included. Layout will roll when footprints finalize
Parts:
- U11: footprint QFN32_5X5MC_MCH -> LAN8710A-EZC:QFN32_5X5MC_MCH
Changed lines of the file:
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@@
 			)
 		)
-		(property "Footprint" "QFN32_5X5MC_MCH"
+		(property "Footprint" "LAN8710A-EZC:QFN32_5X5MC_MCH"
 			(at 195.58 115.57 0)
 			(effects

Commit message: Inner board 2.1 footprint links refactored (for future work) and added all links. Routing progress
Parts:
- removed TP17: TestPoint, TestPoint:TestPoint_Pad_D2.0mm, symbol Connector:TestPoint
- MH2, MH3: footprint OLIMEX_Other-FP:Mounting_hole_Shield_3.3mm -> MountingHole:MountingHole_3.2mm_M3_Pad_Via; now not fitted
- R24: now not fitted
- U25: footprint (none) -> MCP100-270D:TO127P254X495-3
