File: Hardware/Gen2Dev/InnerBoard/2.2/ESP_POE_combined/ESP32-PoE-ISO_Rev_K.kicad_pcb (KiCad board)
At the start: 4 copper layers, 101.8 x 98.2 mm, 148 parts, among them J1 USB_C_Receptacle, J2 SI-46020-F, J3 HMTSW-102-X-X-S-X, J4 20021111-00012T4LF, J5 20021311-00012T4LF, J6 20021111-00012T4LF, J7 20021311-00012T4LF, Q1 Q12MHz/20pF/10ppm/4P/3.2x2.5mm, Q2 BC817-40(SOT23), Q3 BC817-40(SOT23), SW1 PTS815 SJM 250 SMTR LFS, SW2 PTS815 SJM 250 SMTR LFS, T1 LMUN2211LT1G(SOT-23), U1 CH340T(SSOP20W), U2 TPS2376PW(TSSOP-8), U3 BL4054B-42TPRN(SOT23-5), U4 LAN8710A-EZC(QFN32), U5 TX4138(ESOIC-8), U6 ESP32-WROVER-E, U7 SY8089AAAC(SOT23-5), U8 SN74LVC1G04DBVR(SOT23-5)

Commit message: fix lib
Parts:
- removed C29: 100nF/16V/10%/X7R/C0402, OLIMEX_RLC-FP:C_0402_5MIL_DWS
- removed C3: 47uF/6.3V/20%/X5R/C0805, OLIMEX_RLC-FP:C_0805_5MIL_DWS
- removed D4: 1N5819S4/SOD123, OLIMEX_Diodes-FP:SOD-123_1C-2A_KA
- removed Drill_Slot1, Drill_Slot3: 2 mm, OLIMEX_Other-FP:Mounting_hole_2_mm
- removed J2: SI-46020-F, SI-46020-F:BEL_SI-46020-F
- removed L3, L5: FB0805/600R/2A, OLIMEX_RLC-FP:L_0805_5MIL_DWS
- removed LAN_CON1: RJP-003TC1(LPJ4112CNL), OLIMEX_Connectors-FP:RJP-003TC1(LPJ4112CNL)
- removed Logo_OSHW: , OLIMEX_LOGOs-FP:LOGO_OPENHARDWARE_8x8
- removed Logo_Olimex: , OLIMEX_LOGOs-FP:OLIMEX_LOGO_TB
- removed MICRO_SD1: TFC-9P-1.7H(ATFFS150A01BR016), OLIMEX_Connectors-FP:uSD(TFC-9P-1.xH(ATFFS150A01BR016))
- removed Q1: Q12MHz/20pF/10ppm/4P/3.2x2.5mm, OLIMEX_Crystal-FP:TSX-3.2x2.5mm_GND(3)
- removed R31, R35: 2.2k/R0402, OLIMEX_RLC-FP:R_0402_5MIL_DWS
- removed R36, R37, R39: 10k/R0402, OLIMEX_RLC-FP:R_0402_5MIL_DWS
- removed R40, R42: 10R/R0402, OLIMEX_RLC-FP:R_0402_5MIL_DWS
- removed R46: 220R/R0402, OLIMEX_RLC-FP:R_0402_5MIL_DWS
- removed RM3: RA1206_(4X0603)_4B8_2.2k, OLIMEX_RLC-FP:R_MATRIX_4
- removed Sign_Antistatic: Val**, OLIMEX_LOGOs-FP:LOGO_ANTISTATIC_1
- removed Sign_CE: CE_Sign, OLIMEX_LOGOs-FP:CE_Sign
- removed Sign_PB-Free: , OLIMEX_LOGOs-FP:LOGO_PBFREE
- removed Sign_RecycleBin: , OLIMEX_LOGOs-FP:LOGO_RECYCLEBIN_1
- removed U8: SN74LVC1G04DBVR(SOT23-5), OLIMEX_IC-FP:SOT-23-5
- removed UEXT1: P-B-V-10-LF, 3221-10-0300-00:CONN10_3221-10-0300-00_CNC
- added J10: HMTSW-102-X-X-S-X, HMTSW-102:SAMTEC_HMTSW-102-X-X-S-X, F.Cu at (57.2, 106.6)
- added J11: HMTSW-102-X-X-S-X, HMTSW-102:SAMTEC_HMTSW-102-X-X-S-X, F.Cu at (57.2, 110.6)
- added J12: HMTSW-102-X-X-S-X, HMTSW-102:SAMTEC_HMTSW-102-X-X-S-X, F.Cu at (57.2, 114.6)
- added J13: HMTSW-102-X-X-S-X, HMTSW-102:SAMTEC_HMTSW-102-X-X-S-X, F.Cu at (57.2, 118.7)
- added J14: HMTSW-102-X-X-S-X, HMTSW-102:SAMTEC_HMTSW-102-X-X-S-X, F.Cu at (57.2, 122.7)
- added J15: HMTSW-102-X-X-S-X, HMTSW-102:SAMTEC_HMTSW-102-X-X-S-X, F.Cu at (57.2, 126.7)
- added J16: HMTSW-102-X-X-S-X, HMTSW-102:SAMTEC_HMTSW-102-X-X-S-X, F.Cu at (57.2, 130.8)
- added J8: HMTSW-102-X-X-S-X, HMTSW-102:SAMTEC_HMTSW-102-X-X-S-X, F.Cu at (57.2, 98.5)
- added J9: HMTSW-102-X-X-S-X, HMTSW-102:SAMTEC_HMTSW-102-X-X-S-X, F.Cu at (57.2, 102.5)
- added R45: 220R/R0402, Resistor_SMD:R_0402_1005Metric, F.Cu at (62.5, 102.0)
- added Y1: ECS-120-20-33-CKM-TR3, ECS_120_20_33_CKM_TR3:XTAL_ECS-120-20-33-CKM-TR3, F.Cu at (64.0, 98.7)
- ACT1, CHRG1, PWR1: footprint OLIMEX_LEDs-FP:LED_0603_KA -> LED_SMD:LED_0603_1608Metric
- C10, C12, C13, C17, C19, C21, C22, C24, C31, C7, C9: footprint OLIMEX_RLC-FP:C_0603_5MIL_DWS -> Capacitor_SMD:C_0603_1608Metric
- C11, C14, C15, C16, C18, C25, C28, C4, C5, C8: footprint OLIMEX_RLC-FP:C_0402_5MIL_DWS -> Capacitor_SMD:C_0402_1005Metric
- C2: footprint OLIMEX_RLC-FP:C_1206_5MIL_DWS_ISO -> Capacitor_SMD:C_1206_3216Metric
- C26: footprint OLIMEX_RLC-FP:CPOL-RM2.5mm_6.3x11mm_PTH -> Capacitor_THT:CP_Radial_Tantal_D6.0mm_P2.50mm
- C27: footprint OLIMEX_RLC-FP:CPOL-RM2.5mm_6.3x11mm_PTH -> Capacitor_THT:CP_Radial_D6.3mm_P2.50mm
- D1, D3, D6, D7, D9: footprint OLIMEX_Diodes-FP:SOD-123_1C-2A_KA -> Diode_SMD:D_SOD-123
- D10: footprint OLIMEX_Diodes-FP:SMA-KA -> Diode_SMD:D_SMA
- D2: footprint OLIMEX_Diodes-FP:SOT23-3 -> Package_TO_SOT_SMD:SOT-23-3
- D5: footprint OLIMEX_Diodes-FP:DO214AB(SMC)_1(K)-2(A) -> DO-214AB:CDBC-G
- FET1, FET2, FET3, Q2, Q3, T1: footprint OLIMEX_Transistors-FP:SOT23 -> Package_TO_SOT_SMD:SOT-23
- J1: value USB_C_Receptacle -> HMTSW-102-X-X-S-X; footprint Connector_USB:USB_C_Receptacle_Molex_105450-0101-L -> HMTSW-102:SAMTEC_HMTSW-102-X-X-S-X
- J3: footprint HMTSW-102-X-X-S-X:SAMTEC_HMTSW-102-X-X-S-X -> HMTSW-102:SAMTEC_HMTSW-102-X-X-S-X
- J4: value 20021111-00012T4LF -> ARJP11B-MASA-B-A-EMU2; footprint 20021111-00012T4LF:CONN_20021111-XX012XXLF_AMP -> ARJP11B-MASA-B-A-EMU2_ABR:ARJP11B-MASA-B-A-EMU2_ABR
- J5: value 20021311-00012T4LF -> 87520-0010BLF; footprint 20021311-00012T4LF:AMPHENOL_20021311-00012T4LF -> 87520-0010BLF:CONN4_87520-0010_FCI
- J6: value 20021111-00012T4LF -> HMTSW-102-X-X-S-X; footprint 20021111-00012T4LF:CONN_20021111-XX012XXLF_AMP -> HMTSW-102:SAMTEC_HMTSW-102-X-X-S-X
- J7: value 20021311-00012T4LF -> HMTSW-102-X-X-S-X; footprint 20021311-00012T4LF:AMPHENOL_20021311-00012T4LF -> HMTSW-102:SAMTEC_HMTSW-102-X-X-S-X
- L1: footprint OLIMEX_RLC-FP:L_0805_5MIL_DWS -> Inductor_SMD:L_0805_2012Metric
- R1, R10, R11, R12, R13, R14, R15, R16, R17, R18, R19, R2, R20, R21, R22, R23, R24, R25, R26, R27, R29, R3, R30, R32, R33, R34, R38, R4, R43, R44, R47, R48, R5, R6, R7, R8, R9: footprint OLIMEX_RLC-FP:R_0402_5MIL_DWS -> Resistor_SMD:R_0402_1005Metric
- R28: footprint OLIMEX_RLC-FP:R_1206_5MIL_DWS -> Resistor_SMD:R_1206_3216Metric
- R41: footprint OLIMEX_RLC-FP:R_2512_MM_DWS -> Resistor_SMD:R_2512_6332Metric
- RM1, RM2: footprint OLIMEX_RLC-FP:R_MATRIX_4 -> Resistor_SMD:R_Array_Concave_4x0603
- SW1, SW2: footprint PTS815:SW4_PTS815 SJM 250 SMTR LFS_CNK -> PTS815 SJM 250 SMTR LFS:SW4_PTS815 SJM 250 SMTR LFS_CNK
- TVS1: footprint OLIMEX_Diodes-FP:SOT-23-5 -> Package_TO_SOT_SMD:SOT-23-5
- TVS2, TVS3: footprint OLIMEX_Diodes-FP:D_0402_5MIL_DWS -> Diode_SMD:D_0402_1005Metric
- U2: footprint OLIMEX_IC-FP:TSSOP-8_Pitch-0.65mm_Dimensions-4.40x3.00x1.20mm -> TPS2376PW(TSSOP-8):PW8
- U3: footprint OLIMEX_IC-FP:SOT-23-5 -> Package_TO_SOT_SMD:SOT-23-5
- U4: footprint OLIMEX_IC-FP:QFN32_EP(33)_5.00x5.00x0.90mm_Pitch_0.50mm -> LAN8710A-EZC(QFN32):QFN32_5X5MC_MCH-L
- U5: footprint OLIMEX_Regulators-FP:ESOIC-8 -> TX4138(ESOIC-8):ESOIC8_XDS
- U6: footprint OLIMEX_Cases-FP:ESP32-WROVER(WROOM)-UNIVERSAL_MODULE -> ESP32-WROOM-32E-N8:ESP32­WROOM­32E_EXP
- U7: footprint OLIMEX_Regulators-FP:SOT-23-5 -> Package_TO_SOT_SMD:SOT-23-5
Connections:
- net /5V_DCDC renamed 5V_DCDC
- net /D_Com renamed D_Com
- net /ESP_EN renamed ESP_EN
- net /GPI34/BUT1 renamed GPI34/BUT1
- net /GPIO17/EMAC_CLK_OUT_180 renamed GPIO17/EMAC_CLK_OUT_180
- net /GPIO2/HS2_DATA0 renamed GPIO2/HS2_DATA0
- net /GPIO32 renamed GPIO32
- C11 pad 1: Net-(J2-RCT) -> Net-(LNK1-A)
- C13 pad 1: Net-(J2-RCT) -> Net-(LNK1-A)
- C14 pad 1: +3.3VLAN -> Net-(U4-VDDIO)
- C15 pad 1: Net-(J2-RCT) -> Net-(LNK1-A)
- C16 pad 1: Net-(J2-RCT) -> Net-(LNK1-A)
- C24 pad 1: Spare1 -> Net-(C27-+)
- C24 pad 2: Spare2 -> Net-(D10-A)
- C27 pad 1: Spare1 -> Net-(C27-+)
- C28 pad 1: /GPI35 -> GPI35
- C7 pad 1: /+5V_USB -> Net-(U1-VCC)
- D10 pad 1: Spare1 -> Net-(C27-+)
- D10 pad 2: Spare2 -> Net-(D10-A)
- D2 pad 2: /GPIO0 -> GPIO0
- D6 pad 2: /GPIO3/U0RXD -> Net-(D6-A)
- D7 pad 1: /GPIO1/U0TXD -> Net-(D7-K)
- FET1 pad 3: /+5V_USB -> +5V_USB
- J3 pad 01: unconnected-(J3-Pad01) -> Spare2
- J3 pad 02: unconnected-(J3-Pad02) -> Net-(J4-V-)
- J4 pad 1: +3V3 -> /TD+
- J4 pad 10: GND -> Net-(J4-V-)
- J4 pad 11: /GPIO19/EMAC_TXD0(RMII) -> unconnected-(J4-ANODE-Pad11)
- J4 pad 12: GND -> unconnected-(J4-CATHODE-Pad12)
- J4 pad 2: GND -> /TD-
- J4 pad 3: +5VP -> /RD+
- J4 pad 4: GND -> Net-(LNK1-A)
- J4 pad 5: /GPIO25/EMAC_RXD0(RMII) -> Net-(LNK1-A)
- J4 pad 6: GND -> /RD-
- J4 pad 7: /GPIO21/EMAC_TX_EN(RMII) -> /Shield
- J4 pad 9: /GPIO22/EMAC_TXD1(RMII) -> Net-(J4-V+)
- J5 pad 1: +3V3 -> +5V_USB
- J5 pad 2: GND -> Net-(J5-D-)
- J5 pad 3: +5VP -> Net-(J5-D+)
- J5 pad 5: /GPIO25/EMAC_RXD0(RMII) -> (no net)
- J5 pad 6: GND -> (no net)
- L1 pad 2: Net-(J2-RCT) -> Net-(LNK1-A)
- LNK1 pad 2: Net-(J2-RCT) -> Net-(LNK1-A)
- R10 pad 1: Net-(J2-RCT) -> Net-(LNK1-A)
- R11 pad 1: Net-(J2-RCT) -> Net-(LNK1-A)
- R12 pad 1: Net-(J2-RCT) -> Net-(LNK1-A)
- R13 pad 1: Net-(J2-RCT) -> Net-(LNK1-A)
- R16 pad 1: /GPI35 -> GPI35
- R17 pad 2: /GPIO3/U0RXD -> Net-(D6-A)
- R18 pad 1: /+5V_USB -> Net-(U1-VCC)
- R19 pad 2: /GPIO3/U0RXD -> Net-(D6-A)
- R22 pad 1: Spare1 -> Net-(C27-+)
- R23 pad 2: Spare2 -> Net-(D10-A)
- R27 pad 1: Spare2 -> Net-(D10-A)
- R28 pad 2: Spare1 -> Net-(C27-+)
- R4 pad 2: /GPI39 -> GPI35
- R41 pad 1: Spare1 -> Net-(C27-+)
- R7 pad 2: /GPI35 -> GPI35
- R9 pad 1: /GPI39 -> GPI35
- T1 pad 1: /GPIO12/PHY_PWR -> GPIO12/PHY_PWR
- U1 pad 19: /+5V_USB -> Net-(U1-VCC)
- U2 pad 4: Spare2 -> Net-(D10-A)
- U2 pad 8: Spare1 -> Net-(C27-+)
- U4 pad 1: Net-(J2-RCT) -> Net-(LNK1-A)
- U4 pad 10: /GPIO26/EMAC_RXD1(RMII) -> GPIO26/EMAC_RXD1(RMII)
- U4 pad 11: /GPIO25/EMAC_RXD0(RMII) -> GPIO25/EMAC_RXD0(RMII)
- U4 pad 12: +3.3VLAN -> Net-(U4-VDDIO)
- U4 pad 15: /GPIO27/EMAC_RX_CRS_DV -> GPIO27/EMAC_RX_CRS_DV
- U4 pad 16: /GPIO18/MDIO(RMII) -> GPIO18/MDIO(RMII)
- U4 pad 17: /GPIO23/MDC(RMII) -> GPIO23/MDC(RMII)
- U4 pad 21: /GPIO21/EMAC_TX_EN(RMII) -> GPIO21/EMAC_TX_EN(RMII)
- U4 pad 22: /GPIO19/EMAC_TXD0(RMII) -> GPIO19/EMAC_TXD0(RMII)
- U4 pad 23: /GPIO22/EMAC_TXD1(RMII) -> GPIO22/EMAC_TXD1(RMII)
- U4 pad 27: Net-(J2-RCT) -> Net-(LNK1-A)
- U5 pad 3: Spare1 -> Net-(U5-Vin)
- U5 pad 6: Net-(U2-PG) -> Net-(U5-EN)
- U6 pad 10: /GPIO25/EMAC_RXD0(RMII) -> GPIO25/EMAC_RXD0(RMII)
- U6 pad 11: /GPIO26/EMAC_RXD1(RMII) -> GPIO26/EMAC_RXD1(RMII)
- U6 pad 12: /GPIO27/EMAC_RX_CRS_DV -> GPIO27/EMAC_RX_CRS_DV
- U6 pad 13: /GPIO14/HS2_CLK -> GPIO14/HS2_CLK
- U6 pad 14: /GPIO12/PHY_PWR -> GPIO12/PHY_PWR
- U6 pad 16: /GPIO13/I2C-SDA -> GPIO13/I2C-SDA
- U6 pad 2: +3V3 -> Net-(U6-VDD33(3V3))
- U6 pad 23: /GPIO15/HS2_CMD -> GPIO15/HS2_CMD
- U6 pad 25: /GPIO0 -> GPI0
- U6 pad 26: /GPIO4/U1TXD -> GPIO4/U1TXD
- U6 pad 27: /GPIO16/I2C-SCL -> GPIO16/I2C-SCL
- U6 pad 29: /GPIO5/SPI_CS -> GPIO5/SPI_CS
- U6 pad 30: /GPIO18/MDIO(RMII) -> GPIO18/MDIO(RMII)
- U6 pad 31: /GPIO19/EMAC_TXD0(RMII) -> GPIO19/EMAC_TXD0(RMII)
- U6 pad 33: /GPIO21/EMAC_TX_EN(RMII) -> GPIO21/EMAC_TX_EN(RMII)
- U6 pad 34: /GPIO3/U0RXD -> GPIO3/U0RXD
- U6 pad 35: /GPIO1/U0TXD -> GPIO1/U0TXD
- U6 pad 36: /GPIO22/EMAC_TXD1(RMII) -> GPIO22/EMAC_TXD1(RMII)
- U6 pad 37: /GPIO23/MDC(RMII) -> GPIO23/MDC(RMII)
- U6 pad 4: /GPI36/U1RXD -> GPI36/U1RXD
- U6 pad 5: /GPI39 -> GPI39
- U6 pad 7: /GPI35 -> GPI35
- U6 pad 9: /GPIO33 -> GPIO33
Routing:
- net (no net): track 0.00 -> 177.7 mm, vias 0 -> 11
- net Net-(LAN_CON1-RCT): track 96.2 -> 0.00 mm, vias 6 -> 0
- net GPI34/BUT1: track 74.5 -> 0.00 mm
- net /GPI34/BUT1: track 0.00 -> 74.5 mm
- net GPIO2/HS2_DATA0: track 73.4 -> 0.00 mm
- net /GPIO2/HS2_DATA0: track 0.00 -> 73.4 mm
- net GND: track 356.8 -> 423.6 mm, vias 89 -> 91
- net /GPIO23/MDC(RMII): track 66.8 -> 0.00 mm, vias 2 -> 0
- net GPIO32: track 57.7 -> 0.00 mm, vias 2 -> 0
- net /GPIO32: track 0.00 -> 57.7 mm, vias 0 -> 2
- net GPIO17/EMAC_CLK_OUT_180: track 56.2 -> 0.00 mm, vias 5 -> 0
- net /GPIO17/EMAC_CLK_OUT_180: track 0.00 -> 56.2 mm, vias 0 -> 5
- net 5V_DCDC: track 55.7 -> 0.00 mm, vias 1 -> 0
- net /5V_DCDC: track 0.00 -> 55.7 mm, vias 0 -> 1
- net ESP_EN: track 50.3 -> 0.00 mm, vias 3 -> 0
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
Commit message: wait for testing result
Parts:
- removed BAT1: DW02S, OLIMEX_Connectors-FP:LIPO_BAT_VERTICAL_DW02S
- removed C1, C6: 22uF/6.3V/20%/X5R/C0603, OLIMEX_RLC-FP:C_0603_5MIL_DWS
- removed C22: 22uF/6.3V/20%/X5R/C0603, Capacitor_SMD:C_0603_1608Metric
- removed C28: 1nF/50V/10%/X7R/C0402, Capacitor_SMD:C_0402_1005Metric
- removed CHRG1: LED/YELLOW/0603, LED_SMD:LED_0603_1608Metric
- removed D1, D3: 1N5819S4/SOD123, Diode_SMD:D_SOD-123
- removed FET1, FET2: WPM2015-3/TR, Package_TO_SOT_SMD:SOT-23
- removed FID1, FID2, FID3, FID4, FID5, FID6: Fiducial, OLIMEX_Other-FP:Fiducial1x3
- removed L2: 2.2uH/1.5A/DCR=72mR/20%/3.00x3.00x1.50mm/CD32(NR3015T2R2M), OLIMEX_RLC-FP:CD32
- removed MH1, MH2, MH3: Mounting_Hole_NPTH, OLIMEX_Other-FP:NPTH_2.2mm
- removed PWR1: LED/RED/0603, LED_SMD:LED_0603_1608Metric
- removed R1, R6: 10k/R0402, Resistor_SMD:R_0402_1005Metric
- removed R16, R7: 470k/R0402, Resistor_SMD:R_0402_1005Metric
- removed R29: 220k/R0402, Resistor_SMD:R_0402_1005Metric
- removed R30: 49.9k/1%/R0402, Resistor_SMD:R_0402_1005Metric
- removed R4: 47k/R0402, Resistor_SMD:R_0402_1005Metric
- removed R5, R8: 2.2k/R0402, Resistor_SMD:R_0402_1005Metric
- removed R9: 100k/R0402, Resistor_SMD:R_0402_1005Metric
- removed RM1, RM2: RA1206_(4X0603)_4B8_2.2k, Resistor_SMD:R_Array_Concave_4x0603
- removed U3: BL4054B-42TPRN(SOT23-5), Package_TO_SOT_SMD:SOT-23-5
- removed U7: SY8089AAAC(SOT23-5), Package_TO_SOT_SMD:SOT-23-5
- added R31: TC164-JR-072K2L, TC164_JR_072K2L:YAG_TC164_YAG, F.Cu at (161.9, 116.4)
- added R35: TC164-JR-072K2L, TC164_JR_072K2L:YAG_TC164_YAG, F.Cu at (161.9, 122.2)
- DCDC1, R32, R47, R48: moved to B.Cu
- moved U5 132.1 mm to (239.3, 159.6)
- moved J1 127.6 mm to (28.4, 156.0)
- moved J3 127.6 mm to (45.8, 141.1)
- moved J6 127.6 mm to (59.7, 165.7)
- moved J7 127.6 mm to (61.2, 183.5)
- moved Y1 115.8 mm to (176.4, 126.4)
- moved C23 103.3 mm to (201.6, 155.8)
- moved C12 103.3 mm to (206.4, 155.5)
- moved R33 103.3 mm to (206.4, 157.8)
- moved C26 101.0 mm to (215.9, 158.6)
- moved R17 96.4 mm to (191.4, 145.8)
- moved C27 92.3 mm to (194.6, 177.7)
- moved D8 90.3 mm to (187.4, 141.0)
- moved C21 90.0 mm to (199.7, 125.6)
- moved C9 90.0 mm to (200.2, 132.0)
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Routing:
- net (no net): track 177.7 -> 476.8 mm, vias 11 -> 20
- net +5V: track 116.1 -> 0.00 mm, vias 7 -> 0
- net Net-(U3-VBAT): track 94.5 -> 0.00 mm, vias 2 -> 0
- net /+5V_USB: track 77.7 -> 0.00 mm, vias 6 -> 0
- net GPIO16/I2C-SCL: track 0.00 -> 76.4 mm
- net /GPIO16/I2C-SCL: track 76.4 -> 0.00 mm
- net GPI34/BUT1: track 0.00 -> 74.5 mm
- net /GPI34/BUT1: track 74.5 -> 0.00 mm
- net GPIO2/HS2_DATA0: track 0.00 -> 73.4 mm
- net /GPIO2/HS2_DATA0: track 73.4 -> 0.00 mm
- net GPIO15/HS2_CMD: track 0.00 -> 73.3 mm
- net /GPIO15/HS2_CMD: track 73.3 -> 0.00 mm
- net GPIO4/U1TXD: track 0.00 -> 72.7 mm
- net /GPIO4/U1TXD: track 72.7 -> 0.00 mm
- net GPIO13/I2C-SDA: track 0.00 -> 72.2 mm, vias 0 -> 3
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Other:
- board size 101.8 x 98.2 mm -> 28 x 98.2 mm
