File: Hardware/Gen2Dev/InnerBoard/2.2/ESP_POE_combined/ESP32-PoE-ISO_Rev_K.kicad_sch (KiCad schematic)
At the start: 137 parts, among them J1 HMTSW-102-X-X-S-X, J10 HMTSW-102-X-X-S-X, J11 HMTSW-102-X-X-S-X, J12 HMTSW-102-X-X-S-X, J13 HMTSW-102-X-X-S-X, J14 HMTSW-102-X-X-S-X, J15 HMTSW-102-X-X-S-X, J16 HMTSW-102-X-X-S-X, J3 HMTSW-102-X-X-S-X, J4 ARJP11B-MASA-B-A-EMU2, J5 87520-0010BLF, J6 HMTSW-102-X-X-S-X, J7 HMTSW-102-X-X-S-X, J8 HMTSW-102-X-X-S-X, J9 HMTSW-102-X-X-S-X, Q1 Q12MHz/20pF/10ppm/4P/3.2x2.5mm, Q2 BC817-40(SOT23), Q3 BC817-40(SOT23), SW1 PTS815 SJM 250 SMTR LFS, T1 LMUN2211LT1G(SOT-23), U1 CH340T(SSOP20W), U2 TPS2376PW(TSSOP-8), U3 BL4054B-42TPRN(SOT23-5), U4 LAN8710A-EZC(QFN32), U5 TX4138(ESOIC-8), U6 ESP32-WROVER-E, U7 SY8089AAAC(SOT23-5)

Commit message: footprints on buttons
stuff
Parts:
- R45, R47, R48: footprint OLIMEX_RLC-FP:R_0402_5MIL_DWS -> Resistor_SMD:R_0402_1005Metric
Changed lines of the file:
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@@
       (effects (font (size 0.9906 0.9906)) (justify left))
     )
-    (property "Footprint" "OLIMEX_RLC-FP:R_0402_5MIL_DWS" (at 351.79 401.828 0)
+    (property "Footprint" "Resistor_SMD:R_0402_1005Metric" (at 351.79 401.828 0)
       (effects (font (size 0.762 0.762)) hide)
     )
@@
       (effects (font (size 1.27 1.27)))
     )
-    (property "Footprint" "OLIMEX_RLC-FP:R_0402_5MIL_DWS" (at 364.49 394.208 0)
+    (property "Footprint" "Resistor_SMD:R_0402_1005Metric" (at 364.49 394.208 0)
       (effects (font (size 0.762 0.762)) hide)
     )
@@
       (effects (font (size 1.27 1.27)))
     )
-    (property "Footprint" "OLIMEX_RLC-FP:R_0402_5MIL_DWS" (at 364.49 389.128 0)
+    (property "Footprint" "Resistor_SMD:R_0402_1005Metric" (at 364.49 389.128 0)
       (effects (font (size 0.762 0.762)) hide)
     )

Commit message: stuff
Parts:
- ACT1, CHRG1, PWR1: footprint OLIMEX_LEDs-FP:LED_0603_KA -> LED_SMD:LED_0603_1608Metric
- C13, C17, C19, C22, C24, C31, C9: footprint OLIMEX_RLC-FP:C_0603_5MIL_DWS -> Capacitor_SMD:C_0603_1608Metric
- C14, C15, C16, C18, C28: footprint OLIMEX_RLC-FP:C_0402_5MIL_DWS -> Capacitor_SMD:C_0402_1005Metric
- C2: footprint OLIMEX_RLC-FP:C_1206_5MIL_DWS_ISO -> Capacitor_SMD:C_1206_3216Metric
- D1, D3, D6, D7, D9: footprint OLIMEX_Diodes-FP:SOD-123_1C-2A_KA -> Diode_SMD:D_SOD-123
- D2: footprint OLIMEX_Diodes-FP:SOT23-3 -> Package_TO_SOT_SMD:SOT-23-3
- FET1, FET2, FET3, Q2, Q3, T1: footprint OLIMEX_Transistors-FP:SOT23 -> Package_TO_SOT_SMD:SOT-23
- L1: footprint OLIMEX_RLC-FP:L_0805_5MIL_DWS -> Inductor_SMD:L_0805_2012Metric
- R1, R10, R11, R12, R13, R14, R15, R16, R2, R20, R21, R22, R24, R25, R26, R29, R3, R30, R31, R32, R33, R34, R35, R36, R37, R38, R4, R5, R6, R7, R8, R9: footprint OLIMEX_RLC-FP:R_0402_5MIL_DWS -> Resistor_SMD:R_0402_1005Metric
- R28: footprint OLIMEX_RLC-FP:R_1206_5MIL_DWS -> Resistor_SMD:R_1206_3216Metric
- TVS1: footprint OLIMEX_Diodes-FP:SOT-23-5 -> Package_TO_SOT_SMD:SOT-23-5
- U3: footprint OLIMEX_IC-FP:SOT-23-5 -> Package_TO_SOT_SMD:SOT-23-5

Commit message: updates
Parts:
- removed D4: 1N5819S4/SOD123, OLIMEX_Diodes-FP:SOD-123_1C-2A_KA, symbol ESP32-PoE-ISO_Rev_K:D_Schottky_Small
- removed R31, R35: 2.2k/R0402, Resistor_SMD:R_0402_1005Metric, symbol ESP32-PoE-ISO_Rev_K:R
- removed R36, R37: 10k/R0402, Resistor_SMD:R_0402_1005Metric, symbol ESP32-PoE-ISO_Rev_K:R
- removed UEXT1: P-B-V-10-LF, 3221-10-0300-00:CONN10_3221-10-0300-00_CNC, symbol ESP32-PoE-ISO_Rev_K:BH10S
- C10, C12, C21, C7: footprint OLIMEX_RLC-FP:C_0603_5MIL_DWS -> Capacitor_SMD:C_0603_1608Metric
- C11, C25, C4, C5, C8: footprint OLIMEX_RLC-FP:C_0402_5MIL_DWS -> Capacitor_SMD:C_0402_1005Metric
- D10: footprint OLIMEX_Diodes-FP:SMA-KA -> Diode_SMD:D_SMA
- R17, R18, R19, R23, R27, R43, R44: footprint OLIMEX_RLC-FP:R_0402_5MIL_DWS -> Resistor_SMD:R_0402_1005Metric
- R41: footprint OLIMEX_RLC-FP:R_2512_MM_DWS -> Resistor_SMD:R_2512_6332Metric
- RM1, RM2: footprint OLIMEX_RLC-FP:R_MATRIX_4 -> Resistor_SMD:R_Array_Concave_4x0603
- RM1: footprint OLIMEX_RLC-FP:R_MATRIX_4 -> Resistor_SMD:R_Array_Concave_4x0603; Fieldname 1 Value 1 -> (none); Fieldname2 Value2 -> (none); Fieldname3 Value3 -> (none)
- TVS2, TVS3: footprint OLIMEX_Diodes-FP:D_0402_5MIL_DWS -> Diode_SMD:D_0402_1005Metric
- U7: footprint OLIMEX_Regulators-FP:SOT-23-5 -> Package_TO_SOT_SMD:SOT-23-5
Other:
- note removed: "HSPICLK"
- note removed: "HSPID"
- note removed: "HSPIQ"
- note removed: "UEXT"
- moved on the sheet: ACT1, C10, C11, C12, C13, C14, C15, C16, C17, C18, C19, C2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

Commit message: fix lib
Parts:
- removed Q1: Q12MHz/20pF/10ppm/4P/3.2x2.5mm, OLIMEX_Crystal-FP:TSX-3.2x2.5mm_GND(3), symbol ESP32-PoE-ISO_Rev_K:Crystal_GND
- added Y1: ECS-120-20-33-CKM-TR3, ECS_120_20_33_CKM_TR3:XTAL_ECS-120-20-33-CKM-TR3, symbol ECS_120_20_33_CKM_TR3:ECS-120-20-33-CKM-TR3
- C26: footprint OLIMEX_RLC-FP:CPOL-RM2.5mm_6.3x11mm_PTH -> Capacitor_THT:CP_Radial_Tantal_D6.0mm_P2.50mm
- C27: footprint OLIMEX_RLC-FP:CPOL-RM2.5mm_6.3x11mm_PTH -> Capacitor_THT:CP_Radial_D6.3mm_P2.50mm
- D5: footprint OLIMEX_Diodes-FP:DO214AB(SMC)_1(K)-2(A) -> DO-214AB:CDBC-G
- J1, J10, J11, J12, J13, J14, J15, J16, J3, J6, J7, J8, J9: footprint HMTSW-102-X-X-S-X:SAMTEC_HMTSW-102-X-X-S-X -> HMTSW-102:SAMTEC_HMTSW-102-X-X-S-X
- J4: footprint ARJP11B-MASA-B-A-EMU2_ABR -> ARJP11B-MASA-B-A-EMU2_ABR:ARJP11B-MASA-B-A-EMU2_ABR
- J5: footprint 87520-0010BLF:AMPHENOL_87520-0010BLF -> 87520-0010BLF:CONN4_87520-0010_FCI
- SW1: footprint SW4_PTS815 SJM 250 SMTR LFS_CNK -> PTS815 SJM 250 SMTR LFS:SW4_PTS815 SJM 250 SMTR LFS_CNK
- U1: Untitled Field (none) -> https://www.amazon.com/crazydiodes-Original-Communication-C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
- U2: footprint OLIMEX_IC-FP:TSSOP-8_Pitch-0.65mm_Dimensions-4.40x3.00x1.20mm -> TPS2376PW(TSSOP-8):PW8
- U4: footprint OLIMEX_IC-FP:QFN32_EP(33)_5.00x5.00x0.90mm_Pitch_0.50mm -> LAN8710A-EZC(QFN32):QFN32_5X5MC_MCH-L
- U5: footprint OLIMEX_Regulators-FP:ESOIC-8 -> TX4138(ESOIC-8):ESOIC8_XDS
- U6: footprint OLIMEX_Cases-FP:ESP32-WROVER(WROOM)-UNIVERSAL_MODULE -> ESP32-WROOM-32E-N8:ESP32­WROOM­32E_EXP
Connections:
- net GND: now also Y1.2 (GND), Y1.4 (GND__1); no longer J5.SH1 (SHIELD), J5.SH2 (SHIELD__1)
- net at C5.1, U1.10 (XO): now also Y1.3 (OUT/IN)
- net at C4.1, U1.9 (XI): now also Y1.1 (IN/OUT)
- no-connect marks 18 -> 25
Other:
- moved on the sheet: SW1

Commit message: wait for testing result
Parts:
- removed BAT1: DW02S, OLIMEX_Connectors-FP:LIPO_BAT_VERTICAL_DW02S, symbol ESP32-PoE-ISO_Rev_K:BAT_CON
- removed C1, C6: 22uF/6.3V/20%/X5R/C0603, OLIMEX_RLC-FP:C_0603_5MIL_DWS, symbol ESP32-PoE-ISO_Rev_K:C
- removed C22: 22uF/6.3V/20%/X5R/C0603, Capacitor_SMD:C_0603_1608Metric, symbol ESP32-PoE-ISO_Rev_K:C
- removed C28: 1nF/50V/10%/X7R/C0402, Capacitor_SMD:C_0402_1005Metric, symbol ESP32-PoE-ISO_Rev_K:C
- removed CHRG1: LED/YELLOW/0603, LED_SMD:LED_0603_1608Metric, symbol ESP32-PoE-ISO_Rev_K:LED
- removed D1, D3: 1N5819S4/SOD123, Diode_SMD:D_SOD-123, symbol ESP32-PoE-ISO_Rev_K:D_Schottky
- removed FET1, FET2: WPM2015-3/TR, Package_TO_SOT_SMD:SOT-23, symbol ESP32-PoE-ISO_Rev_K:P-MOS+DIOD
- removed FID1, FID2, FID3, FID4, FID5, FID6: Fiducial, OLIMEX_Other-FP:Fiducial1x3, symbol ESP32-PoE-ISO_Rev_K:Fiducial
- removed L2: 2.2uH/1.5A/DCR=72mR/20%/3.00x3.00x1.50mm/CD32(NR3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, OLIMEX_RLC-FP:CD32, symbol ESP32-PoE-ISO_Rev_K:L
- removed MH1, MH2, MH3: Mounting_Hole_NPTH, OLIMEX_Other-FP:NPTH_2.2mm, symbol ESP32-PoE-ISO_Rev_K:Mounting_Hole_NPTH
- removed PWR1: LED/RED/0603, LED_SMD:LED_0603_1608Metric, symbol ESP32-PoE-ISO_Rev_K:LED
- removed R1, R6: 10k/R0402, Resistor_SMD:R_0402_1005Metric, symbol ESP32-PoE-ISO_Rev_K:R
- removed R16, R7: 470k/R0402, Resistor_SMD:R_0402_1005Metric, symbol ESP32-PoE-ISO_Rev_K:R
- removed R29: 220k/R0402, Resistor_SMD:R_0402_1005Metric, symbol ESP32-PoE-ISO_Rev_K:R
- removed R30: 49.9k/1%/R0402, Resistor_SMD:R_0402_1005Metric, symbol ESP32-PoE-ISO_Rev_K:R
- removed R4: 47k/R0402, Resistor_SMD:R_0402_1005Metric, symbol ESP32-PoE-ISO_Rev_K:R
- removed R5, R8: 2.2k/R0402, Resistor_SMD:R_0402_1005Metric, symbol ESP32-PoE-ISO_Rev_K:R
- removed R9: 100k/R0402, Resistor_SMD:R_0402_1005Metric, symbol ESP32-PoE-ISO_Rev_K:R
- removed RM1, RM2: RA1206_(4X0603)_4B8_2.2k, Resistor_SMD:R_Array_Concave_4x0603, symbol ESP32-PoE-ISO_Rev_K:RA1206_(4x0603)_4B8_Smashed
- removed U3: BL4054B-42TPRN(SOT23-5), Package_TO_SOT_SMD:SOT-23-5, symbol ESP32-PoE-ISO_Rev_K:BL4054B-42TPRN(SOT23-5)
- removed U7: SY8089AAAC(SOT23-5), Package_TO_SOT_SMD:SOT-23-5, symbol ESP32-PoE-ISO_Rev_K:SY8009AAAC(SOT23-5)
- added R31, R35: TC164-JR-072K2L, TC164_JR_072K2L:YAG_TC164_YAG, symbol TC164_JR_072K2L:TC164-JR-072K2L
Connections:
- net +3.3VLAN: now also R31.8, R35.5, R35.6, R35.7, R35.8
- net GND: now also R31.5, R31.6, R31.7
- net GPIO18/MDIO(RMII): now also R35.3
- net GPIO25/EMAC_RXD0(RMII): now also R35.2
- net GPIO26/EMAC_RXD1(RMII): now also R35.1
- net GPIO27/EMAC_RX_CRS_DV: now also R35.4
- net at U4.13 (RXER/RXD4/PHYAD0): now also R31.4
- net at U4.7 (RXCLK/PHYAD1): now also R31.3
- net at U4.8 (RXD3/PHYAD2): now also R31.2
- net at U4.9 (RXD2/RMIISEL): now also R31.1
Other:
- note removed: "Battery Measurement"
- note removed: "CHARGING"
- note removed: "External Power Sense"
- note removed: "Fiducials"
- note removed: "IBAT = 1000/Rprog = 100mA"
- note removed: "LiPo Charger"
- note removed: "Mounting Holes"
- note removed: "Power Supply"
- note removed: "Rprog"
- note removed: "Vout=0.6*(1+Ra/Rb)"
- moved on the sheet: C31, C4, C5, C7, C8, D2, D6, D7, D9, J11, J12, J13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
