File: Hardware/Gen3/OuterBoard/3.1/OuterBoard_rev3.1.kicad_sch (KiCad schematic)
At the start: 103 parts, among them J1 6130XX11121_61300611121, J3 F32R-1A7H1-11024, J42 UJ31-CH-G2-SMT-TR, J7 530470210, J8 530470210, SW1 PTS815 SJM 250 SMTR LFS, SW2 PTS815 SJM 250 SMTR LFS, U11 GD25Q64CSIGR, U2 BNO055, U2 MCP73812T-420I-OT, U3 MCP73812T-420I-OT, U3 MIC5504-3.3YM5, U5 MIC5504-1.8YM5, U6 MCP1700x-280xxTT, U7 ESP32-S3, Y1 ABM8G-40.000MHZ-18-D2Y-T

Commit message: stuff
Parts:
- removed D3: PMEG6010CEJ, Diode_SMD:D_SOD-323F, symbol Diode:PMEG6010CEJ
- removed J7, J8: 530470210, CON_530470210_MOL, symbol 53047-0210:530470210
- removed SW2: PTS815 SJM 250 SMTR LFS, SW4_PTS815 SJM 250 SMTR LFS_CNK, symbol PTS815:PTS815_SJM_250_SMTR_LFS
- removed TP10, TP7: TestPoint, TestPoint:TestPoint_Pad_D2.0mm, symbol Connector:TestPoint
- removed U11: GD25Q64CSIGR, SOP8_208MIL_GDV, symbol GD25Q64CSIGR:GD25Q64CSIGR
- removed XTAL1: ABS07-32.768KHZ-7-T, XTAL_ABS07-32.768KHZ-7-T_ABR, symbol ABS07-32.768KHZ-7-T:ABS07-32.768KHZ-7-T
- removed Y1: ABM8G-40.000MHZ-18-D2Y-T, CRYSTAL_ABM8G_ABR, symbol ABM8G_40_000MHZ_18_D2Y_T:ABM8G-40.000MHZ-18-D2Y-T
- added D10, D11: PMEG6010CEJ, Diode_SMD:D_SOD-323F, symbol Diode:PMEG6010CEJ
- added D8: LED, LED_SMD:LED_0603_1608Metric, symbol Device:LED
- added F1: NANOSMDC110F-2, FUS_NANO_TYCO_TYC, symbol NANOSMDC110F-2:NANOSMDC110F-2
- added J2: 6130XX11121_61300611121, 61300611121:61300611121, symbol 61300611121:6130XX11121_61300611121
- added J3, J4: 530470210, CON_530470210_MOL, symbol 53047-0210:530470210
- added R22: 0, Resistor_SMD:R_0402_1005Metric, symbol Device:R_US
- added R23: 1k, Resistor_SMD:R_0402_1005Metric, symbol Device:R_US
- added SW3: PTS815 SJM 250 SMTR LFS, SW4_PTS815 SJM 250 SMTR LFS_CNK, symbol PTS815:PTS815_SJM_250_SMTR_LFS
- added U2: GD25Q64CSIGR, SOP8_208MIL_GDV, symbol GD25Q64CSIGR:GD25Q64CSIGR
- added Y1: ABS07-32.768KHZ-7-T, ABS07-32.768KHZ-7-T:XTAL_ABS07-32.768KHZ-7-T, symbol ABS07-32.768KHZ-7-T:ABS07-32.768KHZ-7-T
- added Y2: ABM8G-40.000MHZ-18-D2Y-T, CRYSTAL_ABM8G_ABR, symbol ABM8G_40_000MHZ_18_D2Y_T:ABM8G-40.000MHZ-18-D2Y-T
- C10, C17, C9: footprint Capacitor_SMD:C_0805_2012Metric -> Capacitor_SMD:C_0603_1608Metric
- C10, C17, C9: footprint Capacitor_SMD:C_0805_2012Metric -> Capacitor_SMD:C_0402_1005Metric
- R11: value 0k -> 0; footprint Resistor_SMD:R_0805_2012Metric -> Resistor_SMD:R_0402_1005Metric
- R11: BOM NOSTUFF -> (none); now not fitted
- R14, R17, R19, R2, R20, R21, R3: footprint Resistor_SMD:R_0805_2012Metric -> Resistor_SMD:R_0402_1005Metric
- R15: footprint Resistor_SMD:R_0805_2012Metric -> Capacitor_SMD:C_0402_1005Metric
- R16: value 100 -> 1k; footprint Resistor_SMD:R_0805_2012Metric -> Resistor_SMD:R_0402_1005Metric
- SW1: Mfr C&K -> (none); Mfr P/N PTS815SJG250SMTRLFS -> (none); Price 0.085 -> (none); Purchase-URL https://www.lcsc.com/product-detail/Tactile-Switches_C-K-PT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 -> (none); Supplier 1 LCSC -> (none); Supplier 1 P/N C411883 -> (none)
- U7: footprint QFN56_7X7_EXP -> Package_DFN_QFN:QFN-56-1EP_7x7mm_P0.4mm_EP3.2x3.2mm
Connections:
- net +3.3V: now also R22.1; no longer U2.4 (NBOOT_LOAD_PIN)
- net +5V: now also D5.2 (A)
- net CHIP_EN: now also R15.2, SW3.1, SW3.2; no longer SW1.1
- net D0/A0: now also J1.6; no longer J1.5
- net D10/A10/MOSI: now also J2.4
- net D1/A1: now also J1.3; no longer J1.2
- net D2/A2: now also R19.1
- net D3/A3: now also R3.1
- net D4/I2C_SDA: now also R2.1
- net D5/I2C_SCL: now also R20.1
- net D8/A8/SCK: now also J2.6
- net D9/A9/MISO: now also J2.5
- net GND: now also SW1.3, D8.1 (K), SW3.3, SW3.4, U2.4 (VSS), Y2.2 (GND), Y2.4 (GND); no longer C10.2, C10.2, C9.2, C9.2, D11.2 (A), D12.2 (A), J1.1, J1.4, R21.2, R21.2, U2.2 (V_{SS}), U3.2 (V_{SS})
- net GPIO0: now also R15.2, SW1.1, SW1.2
- net GPIO33: no longer R19.1
- net GPIO34: no longer R3.1
- net GPIO35: no longer R2.1
- net GPIO36: no longer R20.1
- net IO21/USER_LED: now also J2.3
- net SPICLK: now also U2.6 (SCLK)
- net SPICS0: now also U2.1 (CS#)
- net SPID: now also U2.5 (SI(IO0))
- net SPIHD: now also U2.7 (HOLD#(IO3))
- net SPIQ: now also U2.2 (SO(IO1))
- net SPIWP: now also U2.3 (WP#(IO2))
- net VCC: no longer C10.1, C10.1, U2.1 (CE), U2.4 (V_{DD}), U3.1 (CE), U3.4 (V_{DD})
- net VDC: now also C10.1, C10.1, J1.2, J1.5, U2.1 (CE), U2.4 (V_{DD}), U3.1 (CE), U3.4 (V_{DD}), F1.1, R23.2
- net VDD_SPI: now also U2.8 (VCC)
- net GPIO45: now reaches U7.51 (GPIO45)
- net GPIO45: now also J2.1
- net GPIO46: now reaches U7.52 (GPIO46)
- net GPIO46: now also J2.2
- net at C14.1, U7.53 (XTAL_N): now also Y2.1
- net at C14.1, U7.54 (XTAL_P): now also Y2.3
- net at C14.1, U2.26 (XOUT32): now also Y1.1
- net at C15.1, U2.27 (XIN32): now also Y1.2
- removed net +BATT: C10.1, C10.1, D5.2 (A), J1.3, J1.6, U2.3 (V_{BAT}), U3.3 (V_{BAT})
- new net: R22.2, U2.4 (NBOOT_LOAD_PIN)
- new net: D10.1 (K), D11.1 (K), F1.2
- new net: D8.2 (A), R23.1
- new net +BATT1: C10.1, D10.2 (A), J3.1, U2.3 (V_{BAT})
- new net +BATT2: C10.1, D11.2 (A), J4.1, U3.3 (V_{BAT})
- new net GNDPWR: C10.2, C10.2, C9.2, C9.2, D11.2 (A), D12.2 (A), J1.1, J1.4, J3.2, J4.2, R21.2, R21.2, U2.2 (V_{SS}), U3.2 (V_{SS})
- no-connect marks 3 -> 4
Other:
- moved on the sheet: C10, C14, C9, D5, D6, J42, R14, R16, R17, R19, R2, R20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
