File: Hardware/Gen3/OuterBoard/3.1/OuterBoard_rev3.1.kicad_pcb (KiCad board)
At the start: 4 copper layers, 60.4 x 31.8 mm, 104 parts, among them J1 6130XX11121_61300611121, J10 F32R-1A7H1-11024, J42 UJ31-CH-G2-SMT-TR, J7 530470210, J8 530470210, SW1 PTS815 SJM 250 SMTR LFS, SW2 PTS815 SJM 250 SMTR LFS, U1 MCP73812T-420I-OT, U11 GD25Q64CSIGR, U3 MCP73812T-420I-OT, U4 MIC5504-3.3YM5, U5 MIC5504-1.8YM5, U6 MCP1700x-280xxTT, U8 BNO055, U9 ESP32-S3, Y1 ABM8G-40.000MHZ-18-D2Y-T

Commit message: stuff
Parts:
- removed J7, J8: 530470210, 53047-0210:CON_530470210_MOL
- removed SW2: PTS815 SJM 250 SMTR LFS, PTS815:SW4_PTS815 SJM 250 SMTR LFS_CNK
- removed TP10, TP7: TestPoint, TestPoint:TestPoint_Pad_D2.0mm
- removed U11: GD25Q64CSIGR, GD25Q64CSIGR:SOP8_208MIL_GDV
- removed XTAL1: ABS07-32.768KHZ-7-T, ABS07-32.768KHZ-7-T:XTAL_ABS07-32.768KHZ-7-T_ABR
- added D10: PMEG6010CEJ, Diode_SMD:D_SOD-323F, B.Cu at (114.0, 85.2)
- added D11: PMEG6010CEJ, Diode_SMD:D_SOD-323F, B.Cu at (117.6, 85.0)
- added F1: NANOSMDC110F-2, NANOSMDC110F-2:FUS_NANO_TYCO_TYC, B.Cu at (114.5, 100.2)
- added J2: 6130XX11121_61300611121, 61300611121:61300611121, F.Cu at (122.0, 104.0)
- added J3: 530470210, 53047-0210:CON_530470210_MOL, F.Cu at (119.8, 77.8)
- added J4: 530470210, 53047-0210:CON_530470210_MOL, F.Cu at (128.1, 77.7)
- added R22: 0, Resistor_SMD:R_0402_1005Metric, F.Cu at (113.4, 98.3)
- added R23: 1k, Resistor_SMD:R_0402_1005Metric, F.Cu at (119.6, 98.6)
- added SW3: PTS815 SJM 250 SMTR LFS, PTS815:SW4_PTS815 SJM 250 SMTR LFS_CNK, F.Cu at (144.7, 102.8)
- added U2: GD25Q64CSIGR, GD25Q64CSIGR:SOP8_208MIL_GDV, B.Cu at (131.8, 93.5)
- added Y2: ABM8G-40.000MHZ-18-D2Y-T, ABM8G_40_000MHZ_18_D2Y_T:CRYSTAL_ABM8G_ABR, F.Cu at (140.5, 89.3)
- C10, C11, C12, C13, C14, C16, C19, C20, C21, C22, C24, C25, C26, C27, C3, C38, C4, C44, C7, C8: footprint Capacitor_SMD:C_0805_2012Metric -> Capacitor_SMD:C_0603_1608Metric; moved to B.Cu
- C15, C17, C18, C32, C34, C36, C37, C39, C40, C42, C9: footprint Capacitor_SMD:C_0805_2012Metric -> Capacitor_SMD:C_0603_1608Metric
- C2: footprint Capacitor_SMD:C_0805_2012Metric -> Capacitor_SMD:C_0402_1005Metric; moved to B.Cu
- C28, C29, C41: footprint Capacitor_SMD:C_0805_2012Metric -> Capacitor_SMD:C_0402_1005Metric
- D13, D6, D7, FB1, L2, U1, U3, U4, U5, U6: moved to B.Cu
- D8: value PMEG6010CEJ -> LED; footprint Diode_SMD:D_SOD-323F -> LED_SMD:LED_0603_1608Metric
- R1, R4, R5: footprint Resistor_SMD:R_0805_2012Metric -> Resistor_SMD:R_0402_1005Metric; moved to B.Cu
- R11, R12, R16, R17, R18, R19, R2, R20, R21, R26, R3, R31, R7, R9: footprint Resistor_SMD:R_0805_2012Metric -> Resistor_SMD:R_0402_1005Metric
- R13, R14: footprint Resistor_SMD:R_0805_2012Metric -> Capacitor_SMD:C_0402_1005Metric
- R15: value 100 -> 1k; footprint Resistor_SMD:R_0805_2012Metric -> Resistor_SMD:R_0402_1005Metric
- R25: value 100 -> 1k; footprint Resistor_SMD:R_0805_2012Metric -> Resistor_SMD:R_0402_1005Metric; moved to B.Cu
- R6: value 0k -> 0; footprint Resistor_SMD:R_0805_2012Metric -> Resistor_SMD:R_0402_1005Metric
- U9: footprint ESP32S3:QFN56_7X7_EXP -> Package_DFN_QFN:QFN-56-1EP_7x7mm_P0.4mm_EP3.2x3.2mm
- Y1: value ABM8G-40.000MHZ-18-D2Y-T -> ABS07-32.768KHZ-7-T; footprint ABM8G_40_000MHZ_18_D2Y_T:CRYSTAL_ABM8G_ABR -> ABS07-32.768KHZ-7-T:XTAL_ABS07-32.768KHZ-7-T
- moved SW1 100.6 mm to (148.7, 78.4), turned to 90 degrees
- moved R26 98.3 mm to (129.2, 98.0)
- moved R21 95.6 mm to (129.2, 99.3), turned to 180 degrees
- moved U9 91.0 mm to (131.4, 88.2)
- moved J42 89.1 mm to (133.2, 98.4)
- moved J1 88.2 mm to (109.5, 89.8)
- moved H2 88.2 mm to (157.1, 78.3)
- moved H1 87.1 mm to (110.7, 102.5)
- moved J10 86.3 mm to (148.8, 94.7)
- moved U8 74.5 mm to (116.2, 90.2)
- moved R20 69.8 mm to (125.7, 82.5), turned to 90 degrees
- moved G*** 57.0 mm to (120.3, 99.4)
- moved C27 53.1 mm to (122.3, 91.5)
- moved C16 52.3 mm to (122.5, 87.9)
- moved C26 52.0 mm to (122.3, 95.2)
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Connections:
- C1 pad 2: GND -> GNDPWR
- C2 pad 2: GND -> GNDPWR
- C3 pad 1: VCC -> VDC
- C4 pad 1: +BATT -> +BATT1
- C4 pad 2: GND -> GNDPWR
- C7 pad 1: VCC -> VDC
- C8 pad 1: +BATT -> +BATT2
- C8 pad 2: GND -> GNDPWR
- D1 pad 2: GND -> GNDPWR
- D2 pad 2: GND -> GNDPWR
- D5 pad 2: +BATT -> +5V
- D8 pad 1: VDC -> GND
- D8 pad 2: +5V -> Net-(D8-A)
- J1 pad 1: GND -> GNDPWR
- J1 pad 2: D1/A1 -> VDC
- J1 pad 3: +BATT -> D1/A1
- J1 pad 4: GND -> GNDPWR
- J1 pad 5: D0/A0 -> VDC
- J1 pad 6: +BATT -> D0/A0
- R1 pad 2: GND -> GNDPWR
- R13 pad 2: Net-(R13-Pad2) -> CHIP_EN
- R14 pad 2: Net-(R14-Pad2) -> GPIO0
- R19 pad 1: GPIO33 -> D2/A2
- R2 pad 1: GPIO35 -> D4/I2C_SDA
- R20 pad 1: GPIO36 -> D5/I2C_SCL
- R3 pad 1: GPIO34 -> D3/A3
- R4 pad 2: GND -> GNDPWR
- SW1 pad 1: CHIP_EN -> GPIO0
- SW1 pad 2: Net-(R13-Pad2) -> GPIO0
- SW1 pad 3: unconnected-(SW1-Pad3) -> GND
- U1 pad 1: VCC -> VDC
- U1 pad 2: GND -> GNDPWR
- U1 pad 3: +BATT -> +BATT1
- U1 pad 4: VCC -> VDC
- U3 pad 1: VCC -> VDC
- U3 pad 2: GND -> GNDPWR
- U3 pad 3: +BATT -> +BATT2
- U3 pad 4: VCC -> VDC
- U8 pad 4: +3.3V -> Net-(U8-NBOOT_LOAD_PIN)
- U9 pad 2: Net-(J32-Pad02) -> Net-(C38-Pad1)
- U9 pad 3: Net-(J32-Pad02) -> Net-(C38-Pad1)
- U9 pad 51: unconnected-(U9-GPIO45-Pad51) -> GPIO45
- U9 pad 52: unconnected-(U9-GPIO46-Pad52) -> GPIO46
- U9 pad 55: Net-(J33-Pad01) -> +3.3V
- U9 pad 56: Net-(J33-Pad01) -> +3.3V
- Y1 pad 1: Net-(U9-XTAL_N) -> Net-(U8-XOUT32)
- Y1 pad 2: GND -> Net-(U8-XIN32)
Routing:
- net (no net): track 619.6 -> 0.00 mm, vias 7 -> 0
- net BNO_SDA: track 223.5 -> 19.1 mm, vias 3 -> 0
- net IO14/DVP_Y6: track 228.0 -> 48.8 mm, vias 5 -> 2
- net VCC: track 182.7 -> 14.7 mm, vias 0 -> 1
- net +BATT: track 135.6 -> 0.00 mm, vias 1 -> 0
- net BNO_SCL: track 137.5 -> 18.5 mm, vias 2 -> 0
- net MTCK/IO39/CAM_SCL: track 139.6 -> 23.2 mm, vias 4 -> 2
- net GND: track 202.0 -> 105.9 mm, vias 70 -> 35
- net MTDO/IO40/CAM_SDA: track 112.9 -> 21.9 mm, vias 5 -> 0
- net Net-(R6-Pad1): track 100.7 -> 13.9 mm, vias 2 -> 0
- net CHIP_EN: track 142.1 -> 61.8 mm
- net VDD_SPI: track 84.3 -> 6.12 mm, vias 6 -> 1
- net MTDI/IO41/PDM_DATA: track 77.2 -> 0.00 mm, vias 2 -> 0
- net MTMS/IO42/PDM_CLK: track 74.0 -> 0.00 mm, vias 2 -> 0
- net IO10/XMCLK: track 111.8 -> 39.4 mm, vias 4 -> 2
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- added copper zone on In1.Cu, net GNDPWR
Other:
- board size 60.4 x 31.8 mm -> 53.8 x 31.8 mm
- copper layers 4 -> 6
- board text added: "Sense Board Version 3.1 Designed in Stanford, CA"
- board text removed: "1v8 LDO"
- board text removed: "2v8 LDO"
- board text removed: "3v3 LDO"
- board text removed: "BATT/VCC -> VDC"
- board text removed: "CC Resistors"
- board text removed: "Camera Connector"
- board text removed: "Coil"
- board text removed: "ESP32"
- board text removed: "FTDI"
- board text removed: "IMU"
- board text removed: "JTAG"
- board text removed: "Motor Driver"
- board text removed: "SPI Flash"
- board text removed: "SenseDev Board Version 2.1 Designed in Stanford, CA"
- board text removed: "USB"
