File: Hardware/Gen3/OuterBoard/3.1b/OuterBoard_rev3.1.kicad_pcb (KiCad board)
At the start: 6 copper layers, 53.8 x 31.8 mm, 108 parts, among them J1 6130XX11121_61300611121, J10 F32R-1A7H1-11024, J2 6130XX11121_61300611121, J3 530470210, J4 530470210, J42 UJ31-CH-G2-SMT-TR, SW1 PTS815 SJM 250 SMTR LFS, SW3 PTS815 SJM 250 SMTR LFS, U1 MCP73812T-420I-OT, U2 GD25Q64CSIGR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

Commit message: stuff
Routing:
- net GND: track 98.1 -> 104.8 mm, vias 37 -> 35
Changed lines of the file:
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@@
 	)
 	(segment
+		(start 135.485 78.335)
+		(end 137.935 78.335)
+		(width 0.254)
+		(layer "F.Cu")
+		(net 1)
+	)
+	(segment
 		(start 111.749 84.0376)
 		(end 111.749 84.0628)
@@
 	)
 	(segment
-		(start 135.485 78.335)
-		(end 134 76.85)
-		(width 0.254)
-		(layer "F.Cu")
-		(net 1)
-	)
-	(segment
 		(start 134.9756 80.9956)
 		(end 134.97 80.99)
@@
 	)
 	(segment
+		(start 134.9756 83.5152)
+		(end 134.9756 81)
+		(width 0.254)
+		(layer "F.Cu")
+		(net 1)
+	)
+	(segment
 		(start 142.091512 93.0272)
 		(end 142.111489 93.007223)
@@
 	)
 	(segment
+		(start 132.535 78.335)
+		(end 135.485 78.335)
+		(width 0.254)
+		(layer "F.Cu")
+		(net 1)
+	)
+	(segment
 		(start 128.652394 99.384806)
 		(end 128.7232 99.314)
@@
 	)
 	(segment
+		(start 137.935 78.335)
+		(end 137.98 78.38)
+		(width 0.254)
+		(layer "F.Cu")
+		(net 1)
+	)
+	(segment
 		(start 121.1072 99.5681)
 		(end 121.8183 99.5681)
@@
 	)
 	(segment
+		(start 135.49 80.4856)
+		(end 135.49 78.34)
+		(width 0.254)
+		(layer "F.Cu")
+		(net 1)
+	)
+	(segment
 		(start 150.32 100.3364)
 		(end 150.6898 99.9666)
@@
 	)
 	(segment
+		(start 135.49 78.34)
+		(end 135.485 78.335)
+		(width 0.254)
+		(layer "F.Cu")
+		(net 1)
+	)
+	(segment
 		(start 142.1384 83.5914)
 		(end 142.1892 83.5406)
@@
 	)
 	(segment
+		(start 134.9756 81)
+		(end 135.49 80.4856)
+		(width 0.254)
+		(layer "F.Cu")
+		(net 1)
+	)
+	(segment
 		(start 133.1784 97.933)
 		(end 133.18 97.9346)
@@
 	)
 	(segment
-		(start 132.535 78.315)
-		(end 134 76.85)
-		(width 0.254)
-		(layer "F.Cu")
-		(net 1)
-	)
-	(segment
 		(start 139.0526 83.553)
 		(end 139.065 83.5406)
@@
 	)
 	(via
+		(at 137.98 78.38)
+		(size 0.6096)
+		(drill 0.3302)
+		(layers "F.Cu" "B.Cu")
+		(net 1)
+	)
+	(via
 		(at 117.889684 89.981291)
 		(size 0.6)
@@
 	)
 	(via
-		(at 134.97 83.51)
-		(size 0.6)
-		(drill 0.3)
-		(layers "F.Cu" "B.Cu")
-		(net 1)
-	)
-	(via
 		(at 117.201071 93.477539)
 		(size 0.6)
@@
 	)
 	(via
-		(at 134.97 80.99)
-		(size 0.6)
-		(drill 0.3)
-		(layers "F.Cu" "B.Cu")
-		(net 1)
-	)
-	(via
-		(at 134 76.85)
-		(size 0.6)
-		(drill 0.3)
-		(layers "F.Cu" "B.Cu")
-		(net 1)
-	)
-	(via
 		(at 145.7706 102.743)
 		(size 0.6)
@@
 		(polygon
 			(pts
-				(xy 112.5474 85.2678) (xy 131.3942 85.4202) (xy 131.3942 85.725) (xy 131.79 85.71) (xy 131.92 73.56)
+				(xy 112.5474 85.2678) (xy 131.3942 85.4202) (xy 131.3942 85.725) (xy 137.31 85.73) (xy 137.33 73.57)
 				(xy 162.7632 74.0664) (xy 163.1188 108.3818) (xy 112.8014 107.8992)
 			)

Commit message: stuff
Routing:
- net GND: track 104.8 -> 93.9 mm, vias 35 -> 38
Changed lines of the file:
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@@
 			(solder_mask_margin 0.102)
 		)
+		(model "${KIPRJMOD}/3D Models/6130XX11121_61300611121.step"
+			(offset
+				(xyz 0 0 0)
+			)
+			(scale
+				(xyz 1 1 1)
+			)
+			(rotate
+				(xyz 90 180 0)
+			)
+		)
 	)
 	(footprint "Capacitor_SMD:C_0201_0603Metric"
@@
 			(solder_mask_margin 0.102)
 		)
+		(model "${KIPRJMOD}/3D Models/6130XX11121_61300611121.step"
+			(offset
+				(xyz 0 0 0)
+			)
+			(scale
+				(xyz 1 1 1)
+			)
+			(rotate
+				(xyz 90 180 0)
+			)
+		)
 	)
 	(footprint "Package_DFN_QFN:QFN-56-1EP_7x7mm_P0.4mm_EP3.2x3.2mm"
@@
 	)
 	(segment
-		(start 135.485 78.335)
-		(end 137.935 78.335)
-		(width 0.254)
-		(layer "F.Cu")
-		(net 1)
-	)
-	(segment
 		(start 111.749 84.0376)
 		(end 111.749 84.0628)
@@
 	)
 	(segment
-		(start 134.9756 81)
-		(end 134.9756 80.9956)
-		(width 0.254)
+		(start 123.8146 88.6946)
+		(end 123.91 88.79)
+		(width 0.2)
 		(layer "F.Cu")
 		(net 1)
 	)
 	(segment
-		(start 123.8146 88.6946)
-		(end 123.91 88.79)
-		(width 0.2)
+		(start 134.9756 83.5152)
+		(end 134.9752 83.5152)
+		(width 0.254)
 		(layer "F.Cu")
 		(net 1)
@@
 	)
 	(segment
-		(start 134.9756 83.5152)
-		(end 134.9756 81)
-		(width 0.254)
-		(layer "F.Cu")
-		(net 1)
-	)
-	(segment
 		(start 142.091512 93.0272)
 		(end 142.111489 93.007223)
@@
 	)
 	(segment
-		(start 134.9756 83.5152)
-		(end 134.9752 83.5152)
-		(width 0.254)
-		(layer "F.Cu")
-		(net 1)
-	)
-	(segment
-		(start 132.535 78.335)
-		(end 135.485 78.335)
+		(start 134.9756 81)
+		(end 134.9756 80.9956)
 		(width 0.254)
 		(layer "F.Cu")
@@
 	)
 	(segment
-		(start 137.935 78.335)
-		(end 137.98 78.38)
-		(width 0.254)
-		(layer "F.Cu")
-		(net 1)
-	)
-	(segment
 		(start 121.1072 99.5681)
 		(end 121.8183 99.5681)
@@
 	)
 	(segment
-		(start 135.49 80.4856)
-		(end 135.49 78.34)
-		(width 0.254)
-		(layer "F.Cu")
-		(net 1)
-	)
-	(segment
 		(start 150.32 100.3364)
 		(end 150.6898 99.9666)
@@
 	)
 	(segment
-		(start 134.9756 81)
-		(end 135.49 80.4856)
-		(width 0.254)
-		(layer "F.Cu")
-		(net 1)
-	)
-	(segment
 		(start 133.1784 97.933)
 		(end 133.18 97.9346)
@@
 	)
 	(via
-		(at 137.98 78.38)
-		(size 0.6096)
-		(drill 0.3302)
-		(layers "F.Cu" "B.Cu")
-		(net 1)
-	)
-	(via
 		(at 117.889684 89.981291)
 		(size 0.6)
@@
 	)
 	(via
+		(at 135.485 78.335)
+		(size 0.6)
+		(drill 0.3)
+		(layers "F.Cu" "B.Cu")
+		(net 1)
+	)
+	(via
+		(at 132.535 78.335)
+		(size 0.6)
+		(drill 0.3)
+		(layers "F.Cu" "B.Cu")
+		(net 1)
+	)
+	(via
+		(at 134.97 80.99)
+		(size 0.6)
+		(drill 0.3)
+		(layers "F.Cu" "B.Cu")
+		(net 1)
+	)
+	(via
+		(at 134.97 83.51)
+		(size 0.6)
+		(drill 0.3)
+		(layers "F.Cu" "B.Cu")
+		(net 1)
+	)
+	(via
 		(at 114.681 96.9264)
 		(size 0.6)
@@
 		(start 134.0156 83.5152)
 		(end 134.0156 82.5856)
-		(width 0.2)
+		(width 0.254)
 		(layer "F.Cu")
 		(net 13)
@@
 		(start 133.9875 84.8113)
 		(end 133.9875 83.5433)
-		(width 0.2)
+		(width 0.254)
 		(layer "F.Cu")
 		(net 13)
@@
 		(polygon
 			(pts
-				(xy 112.5474 85.2678) (xy 131.3942 85.4202) (xy 131.3942 85.725) (xy 137.31 85.73) (xy 137.33 73.57)
-				(xy 162.7632 74.0664) (xy 163.1188 108.3818) (xy 112.8014 107.8992)
+				(xy 112.5474 85.2678) (xy 131.95 85.33) (xy 131.98 73.76) (xy 133.12 73.74) (xy 133.13 79.26) (xy 134.95 79.26)
+				(xy 134.91 73.77) (xy 162.7632 74.0664) (xy 163.1188 108.3818) (xy 112.8014 107.8992)
 			)
 		)
