File: Hardware/Gen3/OuterBoard/3.1b/OuterBoard_rev3.1.kicad_pcb (KiCad board)
At the start: 6 copper layers, 53.8 x 31.8 mm, 108 parts, among them J1 6130XX11121_61300611121, J10 F32R-1A7H1-11024, J2 6130XX11121_61300611121, J3 530470210, J4 530470210, J42 UJ31-CH-G2-SMT-TR, SW1 PTS815 SJM 250 SMTR LFS, SW3 PTS815 SJM 250 SMTR LFS, U1 MCP73812T-420I-OT, U2 GD25Q64CSIGR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

Commit message: stuff
Parts:
- removed J42: UJ31-CH-G2-SMT-TR, UJ31-CH-G2-SMT-TR:CUI_UJ31-CH-G2-SMT-TR
- added J5: 1054500101, 1054500101:CONN_105450-0101_MOL, F.Cu at (135.8, 102.7)
- moved C45 0.47 mm to (144.1, 89.3)
- moved C43 0.37 mm to (137.3, 89.3)
Routing:
- net GND: track 93.9 -> 105.8 mm, vias 38 -> 40
- net USB_DP: track 21.7 -> 24.7 mm, vias 2 -> 4
- net Net-(J5-PadB5): track 8.03 -> 10.6 mm
- net +5V: track 89.8 -> 92.2 mm
- net GPIO46: track 48.3 -> 46.8 mm
- net USB_DN: track 23.6 -> 24.6 mm
- net IO14/DVP_Y6: track 48.8 -> 49.8 mm
- net Net-(J5-PadA5): track 7.87 -> 8.71 mm
- net GPIO45: track 52.4 -> 51.7 mm
