File: Hardware/Gen3/OuterBoard/3.1b/OuterBoard_rev3.1.kicad_sch (KiCad schematic)
At the start: 107 parts, among them J1 6130XX11121_61300611121, J2 6130XX11121_61300611121, J3 530470210, J3 F32R-1A7H1-11024, J4 530470210, J42 UJ31-CH-G2-SMT-TR, SW1 PTS815 SJM 250 SMTR LFS, SW3 PTS815 SJM 250 SMTR LFS, U2 BNO055, U2 GD25Q64CSIGR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

Commit message: stuff
Parts:
- removed D6: LED, LED_SMD:LED_0603_1608Metric, symbol Device:LED
- removed J42: UJ31-CH-G2-SMT-TR, UJ31-CH-G2-SMT-TR:CUI_UJ31-CH-G2-SMT-TR, symbol UJ31_CH_G2_SMT_TR:UJ31-CH-G2-SMT-TR
- removed R16: 1k, Resistor_SMD:R_0402_1005Metric, symbol Device:R_US
- removed R17: 5.1K, Resistor_SMD:R_0402_1005Metric, symbol Device:R_US
- added D13: LED, LED_SMD:LED_0603_1608Metric, symbol Device:LED
- added J5: 1054500101, CONN_105450-0101_MOL, symbol 1054500101:1054500101
- added R25: 1k, Resistor_SMD:R_0402_1005Metric, symbol Device:R_US
- added R26: 5.1K, Resistor_SMD:R_0402_1005Metric, symbol Device:R_US
Connections:
- net +5V: now also J5.A4, J5.A9, J5.B4, J5.B9, R25.2
- net GND: now also D13.1 (K), J5.A1, J5.A12, J5.B1, J5.B12, R26.2
- net USB_DN: now also J5.A7, J5.B7
- net USB_DP: now also J5.A6, J5.B6
- net at R21.1: now also J5.B5
- new net: D13.2 (A), R25.1
- new net: J5.A5, R26.1
Other:
- moved on the sheet: ANT1, C14, C17, C9, D6, J2, L1, L2, R14, R15, R16, SW1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
