File: Hardware/Gen4/OuterBoard_4.1/OuterBoard_4.1.kicad_pcb (KiCad board)
At the start: 6 copper layers, 53.8 x 31.8 mm, 108 parts, among them J1 6130XX11121_61300611121, J10 F32R-1A7H1-11024, J2 6130XX11121_61300611121, J3 530470210, J4 530470210, J5 1054500101, SW1 PTS815 SJM 250 SMTR LFS, SW3 PTS815 SJM 250 SMTR LFS, U1 MCP73812T-420I-OT, U2 GD25Q64CSIGR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

Commit message: stuff
Parts:
- removed H1, H2: MountingHole, MountingHole:MountingHole_2.1mm
- removed J5: 1054500101, 1054500101:CONN_105450-0101_MOL
- removed R21, R26: 5.1K, Resistor_SMD:R_0402_1005Metric
- removed U6: MCP1700x-280xxTT, Package_TO_SOT_SMD:SOT-23
- added J6: 10118194-0001LF, 10118194-0001LF:AMPHENOL_10118194-0001LF, F.Cu at (134.7, 103.1)
- added U7: TLV75528PDBVR, TLV75528PDBVR:DBV0005A_N, B.Cu at (145.1, 78.5)
- ANT1, C33, C35, L1, R13, U9: moved to B.Cu
- U2: moved to F.Cu
- U4: value MIC5504-3.3YM5 -> AZ1117CH-3.3TRG1; footprint Package_TO_SOT_SMD:SOT-23-5 -> AZ1117CH_3_3TRG1:SOT-223_DIO
- moved C21 45.1 mm to (147.3, 63.8), turned to 0 degrees
- moved U5 41.6 mm to (147.9, 66.4)
- moved C19 40.8 mm to (146.0, 70.9)
- moved C26 40.3 mm to (154.7, 71.2)
- moved C24 40.0 mm to (152.7, 71.1)
- moved C25 32.8 mm to (150.8, 78.6), turned to 90 degrees
- moved C20 31.1 mm to (141.6, 78.5), turned to 90 degrees
- moved C27 29.3 mm to (148.6, 78.6), turned to 90 degrees
- moved C22 27.3 mm to (139.0, 78.5), turned to 90 degrees
- moved C43 27.0 mm to (164.3, 90.6), turned to 0 degrees
- moved SW1 24.2 mm to (149.4, 102.6), turned to 0 degrees
- moved Y2 24.2 mm to (164.3, 93.8), turned to 180 degrees
- moved C45 21.7 mm to (164.3, 97.3), turned to 180 degrees
- moved R14 21.1 mm to (153.4, 101.5), turned to -90 degrees
- moved D7 19.6 mm to (166.0, 79.8)
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Connections:
- C1 pad 2: GNDPWR -> GND
- C2 pad 2: GNDPWR -> GND
- C4 pad 2: GNDPWR -> GND
- C8 pad 2: GNDPWR -> GND
- D1 pad 2: GNDPWR -> GND
- D10 pad 1: Net-(D10-K) -> VAA
- D11 pad 1: Net-(D10-K) -> VAA
- D2 pad 2: GNDPWR -> GND
- F1 pad 2: Net-(D10-K) -> VAA
- J1 pad 1: GNDPWR -> GND
- J1 pad 4: GNDPWR -> GND
- J2 pad 1: GPIO45 -> GND
- J2 pad 3: IO21/USER_LED -> GND
- J2 pad 6: D8/A8/SCK -> VAA
- J3 pad 2: GNDPWR -> GND
- J4 pad 2: GNDPWR -> GND
- R1 pad 2: GNDPWR -> GND
- R4 pad 2: GNDPWR -> GND
- U1 pad 2: GNDPWR -> GND
- U3 pad 2: GNDPWR -> GND
- U4 pad 1: VDC -> GND
- U4 pad 2: GND -> +3.3V
- U4 pad 4: unconnected-(U4-NC-Pad4) -> GND
Routing:
- net VDC: track 115.4 -> 0.00 mm, vias 4 -> 0
- net GND: track 105.8 -> 0.00 mm, vias 40 -> 0
- net +5V: track 92.2 -> 0.00 mm, vias 1 -> 0
- net +2V8: track 89.0 -> 0.00 mm, vias 2 -> 0
- net CHIP_EN: track 61.8 -> 0.00 mm, vias 2 -> 0
- net +3.3V: track 59.2 -> 0.00 mm, vias 13 -> 0
- net +1V8: track 55.4 -> 0.00 mm, vias 2 -> 0
- net GPIO45: track 51.7 -> 0.00 mm, vias 1 -> 0
- net D1/A1: track 47.1 -> 0.00 mm, vias 1 -> 0
- net IO21/USER_LED: track 47.0 -> 0.00 mm, vias 1 -> 0
- net GPIO46: track 46.8 -> 0.00 mm, vias 1 -> 0
- net IO14/DVP_Y6: track 49.8 -> 3.01 mm, vias 2 -> 1
- net IO11/DVP_Y8: track 47.1 -> 3.28 mm, vias 2 -> 1
- net D8/A8/SCK: track 38.8 -> 0.00 mm, vias 1 -> 0
- net D9/A9/MISO: track 36.5 -> 0.00 mm, vias 1 -> 0
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- removed copper zone on In1.Cu, net GNDPWR
Other:
- board size 53.8 x 31.8 mm -> 47.9 x 31.8 mm

Commit message: stuff
Parts:
- C12, C14, C2, C44, D13, D6, FB1, R13, R25: moved to F.Cu
- C34, C36, C37, C39, C40, C41, C43, C45, C9, D9, R11, R12, R15, R19, R2, R20, R3, Y2: moved to B.Cu
- moved J2 34.1 mm to (143.0, 77.1)
- moved TP2 32.1 mm to (128.0, 104.5)
- moved C45 31.2 mm to (133.1, 99.2), turned to 0 degrees
- moved C43 31.1 mm to (133.3, 92.8), turned to 180 degrees
- moved Y2 31.1 mm to (133.3, 95.9), turned to 0 degrees
- moved TP1 28.6 mm to (124.6, 104.5)
- moved D7 28.2 mm to (147.6, 101.1), turned to 0 degrees
- moved U5 27.9 mm to (151.3, 94.1)
- moved C21 27.4 mm to (148.5, 91.2), turned to 180 degrees
- moved C24 26.6 mm to (150.6, 97.6)
- moved C26 26.6 mm to (152.6, 97.6)
- moved R15 24.0 mm to (148.7, 97.8)
- moved C32 23.9 mm to (135.8, 91.0), turned to 90 degrees
- moved D13 23.4 mm to (128.8, 97.3)
- moved R25 22.8 mm to (128.8, 99.5), turned to 0 degrees
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Routing:
- net GND: track 0.00 -> 1.43 mm, vias 0 -> 1
Other:
- board size 47.9 x 31.8 mm -> 38.5 x 31.8 mm

Commit message: stuff
Parts:
- C15, C17, C18, FB1, R10: moved to B.Cu
- C38, L2: moved to F.Cu
- moved C42 15.3 mm to (123.2, 94.3)
- moved C15 11.8 mm to (152.4, 86.2), turned to 90 degrees
- moved C36 8.93 mm to (125.2, 89.2), turned to 180 degrees
- moved C39 8.53 mm to (134.3, 83.2), turned to 90 degrees
- moved C38 8.48 mm to (136.7, 94.5), turned to -90 degrees
- moved C10 7.27 mm to (121.2, 98.9), turned to -90 degrees
- moved C43 7.27 mm to (131.3, 85.8)
- moved R10 7.12 mm to (148.0, 84.2)
- moved Y2 7.04 mm to (131.3, 89.1)
- moved C45 6.94 mm to (131.2, 92.5)
- moved FB1 6.76 mm to (150.3, 86.3), turned to -90 degrees
- moved C34 6.66 mm to (125.2, 87.6)
- moved R17 6.05 mm to (128.3, 91.6), turned to 180 degrees
- moved L2 5.69 mm to (139.8, 88.5)
- moved C41 5.59 mm to (127.3, 87.4), turned to 90 degrees
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Connections:
- J1 pad 2: VDC -> VAA
- J1 pad 3: D1/A1 -> GPIO45
- J1 pad 5: VDC -> VAA
- J1 pad 6: D0/A0 -> GPIO46
- J2 pad 2: GPIO46 -> D8/A8/SCK
- J2 pad 4: D10/A10/MOSI -> D9/A9/MISO
- J2 pad 5: D9/A9/MISO -> D10/A10/MOSI
Routing:
- net BNO_RST: track 0.00 -> 34.2 mm, vias 0 -> 2
- net GPIO0: track 0.00 -> 30.9 mm, vias 0 -> 2
- net BNO_INT: track 0.00 -> 29.9 mm, vias 0 -> 2
- net GPIO46: track 0.00 -> 26.3 mm
- net CHIP_EN: track 0.00 -> 21.8 mm, vias 0 -> 2
- net BNO_SCL: track 0.00 -> 19.9 mm, vias 0 -> 2
- net GPIO45: track 0.00 -> 19.0 mm
- net MTDO/IO40/CAM_SDA: track 0.00 -> 17.5 mm, vias 0 -> 1
- net D8/A8/SCK: track 0.00 -> 17.0 mm
- net BNO_SDA: track 0.00 -> 16.2 mm, vias 0 -> 2
- net USB_DN: track 0.00 -> 16.2 mm, vias 0 -> 1
- net USB_DP: track 0.00 -> 15.1 mm, vias 0 -> 1
- net MTCK/IO39/CAM_SCL: track 0.00 -> 15.0 mm, vias 0 -> 1
- net IO38/DVP_VSYNC: track 0.00 -> 14.6 mm, vias 0 -> 1
- net D10/A10/MOSI: track 0.00 -> 14.4 mm
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
Commit message: stuff
Parts:
- moved C39 0.72 mm to (134.3, 83.9)
- moved J2 0.46 mm to (143.1, 77.5)
- moved J1 0.29 mm to (118.9, 93.5)
- turned D4 to -90 degrees
Routing:
- net VDC: track 0.00 -> 123.4 mm, vias 0 -> 5
- net VAA: track 0.00 -> 70.9 mm
- net +3.3V: track 2.36 -> 47.3 mm, vias 0 -> 17
- net +2V8: track 0.00 -> 43.0 mm, vias 0 -> 2
- net GND: track 15.5 -> 48.7 mm, vias 6 -> 58
- net Net-(D1-K): track 0.00 -> 26.1 mm
- net Net-(D2-K): track 0.00 -> 22.0 mm
- net +1V8: track 0.00 -> 17.5 mm, vias 0 -> 1
- net +BATT2: track 0.00 -> 12.8 mm
- net VCC: track 0.00 -> 12.4 mm
- net MTCK/IO39/CAM_SCL: track 15.0 -> 25.5 mm, vias 1 -> 3
- net +BATT1: track 0.00 -> 8.53 mm
- net +5V: track 0.00 -> 8.18 mm
- net BNO_SDA: track 16.2 -> 20.6 mm
- net CAM_RESET: track 3.67 -> 8.02 mm
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- added copper zone on In1.Cu, net +3.3V
- added copper zone on In4.Cu, net GND
- removed copper zone on In2.Cu, net +3.3V
- removed copper zone on In1.Cu, net GND

Commit message: stuff
Parts:
- added TP3: TestPoint, Connector_PinHeader_1.00mm:PinHeader_1x01_P1.00mm_Vertical, F.Cu at (118.2, 84.2)
- added TP5: TestPoint, Connector_PinHeader_1.00mm:PinHeader_1x01_P1.00mm_Vertical, F.Cu at (118.2, 81.9)
- moved D4 3.34 mm to (126.2, 95.7)
Connections:
- C1 pad 2: GND -> GNDPWR
- C2 pad 2: GND -> GNDPWR
- C4 pad 2: GND -> GNDPWR
- C8 pad 2: GND -> GNDPWR
- D1 pad 2: GND -> GNDPWR
- D2 pad 2: GND -> GNDPWR
- J1 pad 1: GND -> GNDPWR
- J1 pad 4: GND -> GNDPWR
- J3 pad 2: GND -> GNDPWR
- J4 pad 2: GND -> GNDPWR
- R1 pad 2: GND -> GNDPWR
- R4 pad 2: GND -> GNDPWR
- U1 pad 2: GND -> GNDPWR
- U3 pad 2: GND -> GNDPWR
Routing:
- net GNDPWR: track 0.00 -> 55.4 mm, vias 0 -> 7
- net D0/A0: track 0.00 -> 35.7 mm, vias 0 -> 1
- net D1/A1: track 0.00 -> 34.2 mm, vias 0 -> 1
- net VDC: track 123.4 -> 128.8 mm
- net +3.3V: track 47.3 -> 52.5 mm, vias 17 -> 16
- net Net-(D2-K): track 22.0 -> 18.0 mm
- net VCC: track 12.4 -> 15.0 mm, vias 0 -> 2
- net Net-(U9-LNA_IN): track 0.00 -> 2.19 mm
- net Net-(ANT1-PadSIG): track 0.00 -> 2.08 mm
- net +2V8: track 43.0 -> 44.8 mm
- net MTDO/IO40/CAM_SDA: track 18.0 -> 16.4 mm
- net GND: track 48.7 -> 50.0 mm, vias 58 -> 54
- net Net-(D1-K): track 26.1 -> 25.8 mm, vias 0 -> 2
