File: Hardware/Gen4/OuterBoard_4.1/OuterBoard_4.1.kicad_sch (KiCad schematic)
At the start: 107 parts, among them J1 6130XX11121_61300611121, J2 6130XX11121_61300611121, J3 530470210, J3 F32R-1A7H1-11024, J4 530470210, J5 1054500101, SW1 PTS815 SJM 250 SMTR LFS, SW3 PTS815 SJM 250 SMTR LFS, U2 BNO055, U2 GD25Q64CSIGR, U2 MCP73812T-420I-OT, U3 MCP73812T-420I-OT, U3 MIC5504-3.3YM5, U5 MIC5504-1.8YM5, U6 MCP1700x-280xxTT, U7 ESP32-S3, Y1 ABS07-32.768KHZ-7-T, Y2 ABM8G-40.000MHZ-18-D2Y-T

Commit message: stuff
Parts:
- removed H1, H3: MountingHole, MountingHole:MountingHole_2.1mm, symbol Mechanical:MountingHole
- removed J5: 1054500101, CONN_105450-0101_MOL, symbol 1054500101:1054500101
- removed R21, R26: 5.1K, Resistor_SMD:R_0402_1005Metric, symbol Device:R_US
- removed U3: MIC5504-3.3YM5, Package_TO_SOT_SMD:SOT-23-5, symbol Regulator_Linear:MIC5504-3.3YM5
- removed U6: MCP1700x-280xxTT, Package_TO_SOT_SMD:SOT-23, symbol Regulator_Linear:MCP1700x-280xxTT
- added J6: 10118194-0001LF, 10118194-0001LF:AMPHENOL_10118194-0001LF, symbol 10118194-0001LF:10118194-0001LF
- added JP1: SolderJumper_2_Open, symbol Jumper:SolderJumper_2_Open
- added U4: AZ1117CH-3.3TRG1, SOT-223_DIO, symbol AZ1117CH_3_3TRG1:AZ1117CH-3.3TRG1
- added U7: TLV75528PDBVR, DBV0005A_N, symbol TLV75528PDBVR:TLV75528PDBVR
Connections:
- net GNDPWR is gone; now on net GND: C10.2, C10.2, C9.2, C9.2, D11.2 (A), D12.2 (A), J1.1, J1.4, J3.2, J4.2, R21.2, R21.2, U2.2 (V_{SS}), U3.2 (V_{SS})
- net +2V8: now also U7.5 (OUT)
- net +3.3V: now also U4.2 (OUTPUT)
- net +5V: now also J6.1 (VCC)
- net D8/A8/SCK: no longer J2.6
- net GND: now also J2.1, J2.3, J6.5 (GND), U4.1 (ADJ/GND), U4.4 (EPAD), U7.2 (GND)
- net GPIO45: no longer J2.1
- net IO21/USER_LED: no longer J2.3
- net USB_DN: now also J6.2 (D-)
- net USB_DP: now also J6.3 (D+)
- net VDC: now also JP1.2 (B), U4.3 (INPUT), U7.1 (IN), U7.3 (EN); no longer J1.2, J1.5
- net VAA: now reaches D10.1 (K), D11.1 (K), F1.2
- net VAA: now also J1.2, J1.5, J2.6, JP1.1 (A)
- no-connect marks 15 -> 6
Other:
- note added: "How to make it so that currents sum by batteries being in Parallel, I think it is just ORed right now"
- note added: "USB RECPT"
- note removed: "Mounting Holes"
- note removed: "USB-C RECPT"
- moved on the sheet: C10, C14, C15, C17, C9, D13, D4, FB1, J3, R11, R14, R15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

Commit message: stuff
Parts:
- added JP2: SolderJumper_2_Open, symbol Jumper:SolderJumper_2_Open
Connections:
- net D0/A0: no longer J1.6
- net D10/A10/MOSI: now also J2.5; no longer J2.4
- net D1/A1: no longer J1.3
- net D8/A8/SCK: now also J2.2
- net D9/A9/MISO: now also J2.4; no longer J2.5
- net GND: now also JP2.1 (A); no longer C10.2, C10.2, C9.2, C9.2, D11.2 (A), D12.2 (A), J1.1, J1.4, J3.2, J4.2, R21.2, R21.2, U2.2 (V_{SS}), U3.2 (V_{SS})
- net GPIO45: now also J1.3
- net GPIO46: now also J1.6; no longer J2.2
- new net GNDPWR: C10.2, C10.2, C9.2, C9.2, D11.2 (A), D12.2 (A), J1.1, J1.4, J3.2, J4.2, JP2.2 (B), R21.2, R21.2, U2.2 (V_{SS}), U3.2 (V_{SS})

Commit message: stuff
Parts:
- added TP3, TP5: TestPoint, Connector_PinHeader_1.00mm:PinHeader_1x01_P1.00mm_Vertical, symbol Connector:TestPoint
Connections:
- net D0/A0: now also TP5.1
- net D1/A1: now also TP3.1
Other:
- note removed: "How to make it so that currents sum by batteries being in Parallel, I think it is just ORed right now"
- moved on the sheet: D13, J6, JP2, R25

Commit message: stufff
Parts:
- added TP4, TP6: TestPoint, Connector_PinHeader_1.00mm:PinHeader_1x01_P1.00mm_Vertical, symbol Connector:TestPoint
Connections:
- net +3.3V: now also TP4.1
- net GND: now also TP6.1

Commit message: stuff
Parts:
- JP1, JP2: footprint (none) -> Jumper:SolderJumper-2_P1.3mm_Open_Pad1.0x1.5mm
Connections:
- no-connect marks 6 -> 13
Changed lines of the file:
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@@
 	)
 	(no_connect
+		(at 43.688 219.202)
+	)
+	(no_connect
+		(at 43.688 209.042)
+	)
+	(no_connect
 		(at 367.792 252.73)
 	)
@@
 	)
 	(no_connect
+		(at 43.688 216.662)
+	)
+	(no_connect
+		(at 43.688 201.422)
+	)
+	(no_connect
+		(at 43.688 211.582)
+	)
+	(no_connect
+		(at 43.688 221.742)
+	)
+	(no_connect
 		(at 478.536 113.538)
 	)
@@
 	)
 	(no_connect
+		(at 43.688 214.122)
+	)
+	(no_connect
 		(at 311.912 116.078)
 	)
@@
 	(wire
 		(pts
-			(xy 436.372 38.862) (xy 436.372 42.418)
+			(xy 436.372 36.576) (xy 436.372 42.418)
 		)
 		(stroke
@@
 	)
 	(symbol
-		(lib_id "Jumper:SolderJumper_2_Open")
-		(at 74.168 146.558 0)
-		(unit 1)
-		(exclude_from_sim yes)
-		(in_bom no)
-		(on_board yes)
-		(dnp no)
-		(property "Reference" "JP1"
-			(at 74.168 150.114 0)
-			(effects
-				(font
-					(size 1.27 1.27)
-				)
-			)
-		)
-		(property "Value" "SolderJumper_2_Open"
-			(at 74.168 152.654 0)
-			(effects
-				(font
-					(size 1.27 1.27)
-				)
-			)
-		)
-		(property "Footprint" ""
-			(at 74.168 146.558 0)
-			(effects
-				(font
-					(size 1.27 1.27)
-				)
-				(hide yes)
-			)
-		)
-		(property "Datasheet" "~"
-			(at 74.168 146.558 0)
-			(effects
-				(font
-					(size 1.27 1.27)
-				)
-				(hide yes)
-			)
-		)
-		(property "Description" "Solder Jumper, 2-pole, open"
-			(at 74.168 146.558 0)
-			(effects
-				(font
-					(size 1.27 1.27)
-				)
-				(hide yes)
-			)
-		)
-		(pin "2"
-		)
-		(pin "1"
-		)
-		(instances
-			(project ""
-				(path "/e0487af4-02df-420a-a23b-b16cb445dead"
-					(reference "JP1")
-					(unit 1)
-				)
-			)
-		)
-	)
-	(symbol
 		(lib_id "Device:C")
 		(at 354.584 172.974 0)
@@
 	(symbol
 		(lib_id "power:VAA")
-		(at 436.372 38.862 0)
+		(at 436.372 36.576 0)
 		(unit 1)
 		(exclude_from_sim no)
@@
 		(fields_autoplaced yes)
 		(property "Reference" "#PWR01"
-			(at 436.372 42.672 0)
+			(at 436.372 40.386 0)
 			(effects
 				(font
@@
 		)
 		(property "Value" "VAA"
-			(at 436.372 34.036 0)
+			(at 436.372 31.75 0)
 			(effects
 				(font
@@
 		)
 		(property "Footprint" ""
-			(at 436.372 38.862 0)
+			(at 436.372 36.576 0)
 			(effects
 				(font
@@
 		)
 		(property "Datasheet" ""
-			(at 436.372 38.862 0)
+			(at 436.372 36.576 0)
 			(effects
 				(font
@@
 		)
 		(property "Description" "Power symbol creates a global label with name \"VAA\""
-			(at 436.372 38.862 0)
+			(at 436.372 36.576 0)
 			(effects
 				(font
@@
 			)
 		)
-		(property "Footprint" ""
+		(property "Footprint" "Jumper:SolderJumper-2_P1.3mm_Open_Pad1.0x1.5mm"
 			(at 62.23 203.962 0)
 			(effects
@@
 					(unit 1)
 				)
+			)
+		)
+	)
+	(symbol
+		(lib_id "Jumper:SolderJumper_2_Open")
+		(at 74.168 146.558 0)
+		(unit 1)
+		(exclude_from_sim yes)
+		(in_bom no)
+		(on_board yes)
+		(dnp no)
+		(property "Reference" "JP1"
+			(at 74.168 150.114 0)
+			(effects
+				(font
+					(size 1.27 1.27)
+				)
+			)
+		)
+		(property "Value" "SolderJumper_2_Open"
+			(at 74.168 152.654 0)
+			(effects
+				(font
+					(size 1.27 1.27)
+				)
+			)
+		)
+		(property "Footprint" "Jumper:SolderJumper-2_P1.3mm_Open_Pad1.0x1.5mm"
+			(at 74.168 146.558 0)
+			(effects
+				(font
+					(size 1.27 1.27)
+				)
+				(hide yes)
+			)
+		)
+		(property "Datasheet" "~"
+			(at 74.168 146.558 0)
+			(effects
+				(font
+					(size 1.27 1.27)
+				)
+				(hide yes)
+			)
+		)
+		(property "Description" "Solder Jumper, 2-pole, open"
+			(at 74.168 146.558 0)
+			(effects
+				(font
+					(size 1.27 1.27)
+				)
+				(hide yes)
+			)
+		)
+		(pin "2"
+		)
+		(pin "1"
+		)
+		(instances
+			(project "OuterBoard_4.1"
+				(path "/e0487af4-02df-420a-a23b-b16cb445dead"
+					(reference "JP1")
+					(unit 1)
+				)
