File: Hardware/Gen4/OuterBoard_4.1/OuterBoard_4.1.kicad_sch (KiCad schematic)
At the start: 107 parts, among them J1 6130XX11121_61300611121, J2 6130XX11121_61300611121, J3 530470210, J3 F32R-1A7H1-11024, J4 530470210, J6 10118194-0001LF, SW1 PTS815 SJM 250 SMTR LFS, SW3 PTS815 SJM 250 SMTR LFS, U2 BNO055, U2 GD25Q64CSIGR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

Commit message: u
Parts:
- renumbered C9 to C1, C9 to C10, C10 to C11, C9 to C12, C9 to C13, C17 to C14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
