File: Hardware/Gen5/EthernetBoard/EthernetBoardv1.1/EthernetBoardv1.1.kicad_sch (KiCad schematic)
At the start: 0 parts

Commit message: stuff
Parts:
- added C1, C2: 0.1uF, symbol Device:C
- added C3, C4: 22uF, symbol Device:C
- added D1, D3, D4, D5, D6, D7: ESD5Zxx, Diode_SMD:D_SOD-523, symbol Diode:ESD5Zxx
- added D2: B130-E3, Diode_SMD:D_SMA, symbol Diode:B130-E3
- added D8: LED, symbol Device:LED
- added J1: RJ45_Wuerth_7499010211A, Connector_RJ:RJ45_Wuerth_7499010211A_Horizontal, symbol Connector:RJ45_Wuerth_7499010211A
- added J2, J3: Conn_01x19_Pin, symbol Connector:Conn_01x19_Pin
- added L1: L, symbol Device:L
- added P1: USB_C_Plug_USB2.0, symbol Connector:USB_C_Plug_USB2.0
- added Q1, Q2: SS8050, Package_TO_SOT_SMD:SOT-23, symbol Transistor_BJT:SS8050
- added R1, R2, R3, R4: 10R, symbol Device:R_US
- added R10, R6, R7, R8, R9: 49.9R, symbol Device:R_US
- added R11, R5: 332R, symbol Device:R_US
- added R12, R16, R17: 0R, symbol Device:R_US
- added R13, R14, R15: 10K, symbol Device:R_US
- added R18: 2K, symbol Device:R_US
- added R19: 1.5K, symbol Device:R_US
- added SW1, SW2: SW_Push, symbol Switch:SW_Push
- added U1: LAN8720A, Package_DFN_QFN:VQFN-24-1EP_4x4mm_P0.5mm_EP2.5x2.5mm_ThermalVias, symbol Interface_Ethernet:LAN8720A
- added U2: ESP32-S2-WROVER, RF_Module:ESP32-S2-WROVER, symbol RF_Module:ESP32-S2-WROVER
- added U3: AMS1117-3.3, Package_TO_SOT_SMD:SOT-223-3_TabPin2, symbol Regulator_Linear:AMS1117-3.3
- added U4: CP2102N-Axx-xQFN28, Package_DFN_QFN:QFN-28-1EP_5x5mm_P0.5mm_EP3.35x3.35mm, symbol Interface_USB:CP2102N-Axx-xQFN28
Connections:
- new net: J1.1 (TD+), R9.2, U1.21 (TXP)
- new net: R4.1, U1.11 (CRS_DV/MODE2)
- new net: R19.1, U1.12 (MDIO)
- new net: J1.10, R11.2
- new net: J1.11, R5.2
- new net: J1.2 (TD-), R8.2, U1.20 (TXN)
- new net: J1.3 (RD+), R7.2, U1.23 (RXP)
- new net: J1.6 (RD-), R6.2, U1.22 (RXN)
- new net: J1.8, J1.SH, R12.1
- new net: D6.1 (K), D7.1 (K)
- new net: Q1.1 (B), R14.2
- new net: R1.2, U1.8 (RXD0/MODE0)
- new net: D4.1 (K), D5.1 (K)
- new net: D1.1 (K), D3.1 (K)
- new net: R13.1, U4.11 (~{SUSPEND})
- new net: L1.1, U1.1 (VDD2A), U1.19 (VDD1A)
- new net: R3.1, U1.10 (RXER/PHYAD0)
- new net: R10.1, U1.24 (RBIAS)
- new net: R2.1, U1.7 (RXD1/MODE1)
- new net: Q2.1 (B), R15.2
- new net: D8.2 (A), R18.2
- new net: U2.1 (GND), U2.26 (GND), U2.42 (GND), U2.43 (GND)
- new net +3.3V: C4.1, J2.1 (Pin_1), U3.2 (VO)
- new net +5V: C3.1, D2.1 (K), R18.1, U3.3 (VI)
- new net CLK: J3.19 (Pin_19)
- new net CMD: J2.18 (Pin_18)
- new net CRS_DV: R4.2
- new net CTS: U4.23 (~{CTS})
- new net DCD: U4.1 (~{DCD})
- new net DSR: U4.27 (~{DSR})
- new net DTR: Q2.3 (C), R14.1, U4.28 (~{DTR})
- new net EN: C2.2, J2.2 (Pin_2), Q1.3 (C), SW2.2
- new net EXT_5V: J2.19 (Pin_19)
- new net GND: C1.1, C2.1, C3.2, C4.2, D3.2 (A), D5.2 (A), D7.2 (A), D8.1 (K), J1.12, J1.4 (CTD), J1.5 (CRD), J1.9, J2.14 (Pin_14), J3.1 (Pin_1), J3.7 (Pin_7), P1.A1 (GND), P1.A12 (GND), P1.B1 (GND), P1.B12 (GND), P1.S1 (SHIELD), R10.2, R12.2, R13.2, R6.1, R7.1, R8.1, R9.1, SW1.1, SW2.1, U3.1 (GND), U4.29 (GND), U4.3 (GND)
- new net IO0: C1.2, J3.14 (Pin_14), Q2.2 (E), SW1.2
- new net IO12: J2.13 (Pin_13)
- new net IO13: J2.15 (Pin_15)
- new net IO14: J2.12 (Pin_12)
- new net IO15: J3.16 (Pin_16)
- new net IO16: J3.12 (Pin_12)
- new net IO17: J3.11 (Pin_11)
- new net IO18: J3.9 (Pin_9)
- new net IO19: J3.8 (Pin_8)
- new net IO2: J3.15 (Pin_15)
- new net IO21: J3.6 (Pin_6)
- new net IO22: J3.3 (Pin_3)
- new net IO23: J3.2 (Pin_2)
- new net IO25: J2.9 (Pin_9)
- new net IO26: J2.10 (Pin_10)
- new net IO27: J2.11 (Pin_11)
- new net IO32: J2.7 (Pin_7)
- new net IO33: J2.8 (Pin_8)
- new net IO34: J2.5 (Pin_5)
- new net IO35: J2.6 (Pin_6)
- new net IO4: J3.13 (Pin_13)
- new net IO5: J3.10 (Pin_10)
- new net LED1: R5.1, U1.3 (LED1/REGOFF)
- new net LED2: R11.1, U1.2 (LED2/~{INTSEL})
- new net RI: U4.2 (~{RI}/CLK)
- new net RTS: Q1.2 (E), R15.1, U4.24 (~{RTS})
- new net RXD: R16.2, U4.25 (RXD)
- new net RXD0: J3.5 (Pin_5), R17.1, R2.2
- new net RXD1: R1.1
- new net SD0: J3.18 (Pin_18)
- new net SD1: J3.17 (Pin_17)
- new net SD2: J2.16 (Pin_16)
- new net SD3: J2.17 (Pin_17)
- new net SENSOR_VN: J2.4 (Pin_4)
- new net SENSOR_VP: J2.3 (Pin_3), U2.4 (IO01)
- new net TXD: R17.2, U4.26 (TXD)
- new net TXD0: J3.4 (Pin_4), R16.1, U1.17 (TXD0)
- new net TXD1: U1.18 (TXD1)
- new net TX_EN: U1.16 (TXEN)
- new net USB_DN: D4.2 (A), P1.A7 (D-), U4.5 (D-)
- new net USB_DP: D6.2 (A), P1.A6 (D+), U4.4 (D+)
- new net VBUS: D1.2 (A), D2.2 (A), P1.A4 (VBUS), P1.A9 (VBUS), P1.B4 (VBUS), P1.B9 (VBUS)
- new net VCC: L1.2, R19.2, R3.2, U1.9 (VDDIO)
- new net nRST: U1.15 (~{RST})
- no-connect marks 0 -> 13

Commit message: stuff
Parts:
- added C10, C7, C8, C9: 104, symbol Device:C
- added C11: 0.022uF, symbol Device:C
- added C5: 470pF, symbol Device:C
- added C6: 105, symbol Device:C
- added J4: Conn_02x07_Odd_Even, symbol Connector_Generic:Conn_02x07_Odd_Even
- added R20: 4.7K, symbol Device:R_US
- added R21, R22, R23: 33R, symbol Device:R_US
- added Y1: ASCO, Oscillator:Oscillator_SMD_Abracon_ASCO-4Pin_1.6x1.2mm, symbol Oscillator:ASCO
- R10: value 49.9R -> 12.5K
Connections:
- net CRS_DV: now also J4.7 (Pin_7)
- net GND: now also U1.25 (VSS), C10.2, C11.2, C5.2, C6.2, C7.2, C8.2, C9.2, J4.3 (Pin_3), J4.4 (Pin_4), Y1.2 (GND); no longer J1.12, J1.4 (CTD), J1.5 (CRD), J1.9, R6.1, R7.1, R8.1, R9.1
- net RXD0: now also J4.10 (Pin_10)
- net RXD1: now also J4.9 (Pin_9)
- net TXD0: now also J4.11 (Pin_11)
- net TXD1: now also J4.14 (Pin_14)
- net TX_EN: now also J4.12 (Pin_12)
- net VCC: now also C7.1, J4.1 (Pin_1), J4.2 (Pin_2), R20.2, Y1.4 (VDD)
- net nRST: now also C8.1, R20.1
- net at U1.14 (~{INT}/REFCLKO): now also R22.1
- net at U1.5 (XTAL1/CLKIN): now also R21.1
- net VDDCR: now reaches U1.6 (VDDCR)
- net VDDCR: now also C5.1, C6.1
- new net: R21.2, R23.1, Y1.3 (OUT)
- new net MDC: J4.5 (Pin_5)
- new net MDIO: J4.6 (Pin_6)
- new net R_RX_CLK: J4.8 (Pin_8), R22.2, R23.2
- new net VDDA: C10.1, C11.1, C9.1, J1.12, J1.4 (CTD), J1.5 (CRD), J1.9, R6.1, R7.1, R8.1, R9.1
- no-connect marks 13 -> 15
Other:
- note added: "Ethernet"
- note added: "Headers/Switches"
- note added: "Power"
- note added: "USB/Interface"
- moved on the sheet: C1, C2, J1, J2, J3, L1, Q1, Q2, R1, R10, R11, R12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
