File: Hardware/Gen5/EthernetBoard/EthernetBoardv1.1/EthernetBoardv1.1.kicad_sch (KiCad schematic)
At the start: 76 parts, among them J1 RJ45_Wuerth_7499010211A, J2 Conn_01x19_Pin, J3 Conn_01x19_Pin, J4 Conn_02x07_Odd_Even, J5 USB_C_Receptacle_USB2.0_16P, J6 Conn_01x02_Pin, Q1 SS8050, Q2 SS8050, SW1 SW_Push, SW2 SW_Push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

Commit message: stuff
Parts:
- added J7, J9: Conn_01x02_Pin, Connector_PinHeader_2.54mm:PinHeader_1x02_P2.54mm_Vertical, symbol Connector:Conn_01x02_Pin
- L1: footprint (none) -> Inductor_SMD:L_0603_1608Metric
Connections:
- net +3.3V: now also J7.2 (Pin_2), J9.2 (Pin_2)
- net GND: now also U5.1 (GND), U5.15 (GND), U5.38 (GND); no longer J5.S1 (SHIELD)
- net VDDA: now also J9.1 (Pin_1)
- net VDDCR: now also J7.1 (Pin_1)
- new net Earth: J5.S1 (SHIELD)
Other:
- note added: "Notes: Inductor Value 1% Resistors D120 Stackup - JLC Pcb Ethernet Port 1.6mm make with JLC components"
- note removed: "Notes: Inductor Value 1% Resistors D120 Stackup - JLC Pcb Ethernet Port Add test points"
- note removed: "Notes: Push Buttons"

Commit message: final
Connections:
- net EN: now also U5.3 (EN)
- net GND: now also U5.39_1 (EXP), U5.39_2 (EXP), U5.39_3 (EXP), U5.39_4 (EXP), U5.39_5 (EXP), U5.39_6 (EXP), U5.39_7 (EXP), U5.39_8 (EXP), U5.39_9 (EXP)
Other:
- note added: "Notes: Inductor Value 1% Resistors make with JLC components"
- note removed: "Notes: Inductor Value 1% Resistors D120 Stackup - JLC Pcb Ethernet Port 1.6mm make with JLC components"
Changed lines of the file:
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@@
 		)
 	)
-	(text "Notes:\nInductor Value\n1% Resistors\nD120 Stackup - JLC Pcb\nEthernet Port\n\n1.6mm\nmake with JLC components"
+	(text "Notes:\nInductor Value\n1% Resistors\n\nmake with JLC components"
 		(exclude_from_sim no)
 		(at 36.322 36.576 0)
@@
 	)
 	(junction
+		(at 356.87 95.25)
+		(diameter 0)
+		(color 0 0 0 0)
+	)
+	(junction
 		(at 388.62 189.23)
 		(diameter 0)
@@
 	(wire
 		(pts
+			(xy 356.87 92.71) (xy 356.87 95.25)
+		)
+		(stroke
+			(width 0)
+			(type default)
+		)
+	)
+	(wire
+		(pts
 			(xy 166.37 50.8) (xy 166.37 55.88)
 		)
@@
 	(wire
 		(pts
+			(xy 300.99 44.45) (xy 316.23 44.45)
+		)
+		(stroke
+			(width 0)
+			(type default)
+		)
+	)
+	(wire
+		(pts
 			(xy 127 182.88) (xy 140.97 182.88)
 		)
@@
 	(wire
 		(pts
+			(xy 351.79 92.71) (xy 356.87 92.71)
+		)
+		(stroke
+			(width 0)
+			(type default)
+		)
+	)
+	(wire
+		(pts
 			(xy 62.23 78.74) (xy 82.55 78.74)
 		)
@@
 		(effects
 			(font
+				(size 1.27 1.27)
+			)
+			(justify left bottom)
+		)
+	)
+	(label "EN"
+		(at 300.99 44.45 0)
+		(effects
+			(font
