File: Hardware/Gen5/EthernetBoard/EthernetBoardv1.1/EthernetBoardv1.1.kicad_pcb (KiCad board)
At the start: 4 copper layers, 100 x 100 mm, 75 parts, among them J1 RJ45_Wuerth_7499010211A, J2 Conn_01x19_Pin, J3 Conn_01x19_Pin, J4 Conn_02x07_Odd_Even, J5 USB_C_Receptacle_USB2.0_16P, J6 Conn_01x02_Pin, Q1 SS8050, Q2 SS8050, SW1 SW_Push, SW2 SW_Push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

Commit message: stuff
Other:
- board text added: "BOOT"
- board text added: "EN"
- board text added: "ESP32"
- board text added: "Ethernet"
- board text added: "Power"
- board text added: "USB"
Changed lines of the file:
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@@
 		(layer "Edge.Cuts")
+	)
+	(gr_text "USB\n"
+		(at 123 107.9 0)
+		(layer "F.SilkS")
+		(effects
+			(font
+				(size 1 1)
+				(thickness 0.1)
+			)
+			(justify left bottom)
+		)
+	)
+	(gr_text "ESP32"
+		(at 122.5 66.4 0)
+		(layer "F.SilkS")
+		(effects
+			(font
+				(size 1 1)
+				(thickness 0.1)
+			)
+			(justify left bottom)
+		)
+	)
+	(gr_text "Ethernet"
+		(at 61.5 67.7 0)
+		(layer "F.SilkS")
+		(effects
+			(font
+				(size 1 1)
+				(thickness 0.1)
+			)
+			(justify left bottom)
+		)
+	)
+	(gr_text "Power"
+		(at 81 124.3 0)
+		(layer "F.SilkS")
+		(effects
+			(font
+				(size 1 1)
+				(thickness 0.1)
+			)
+			(justify left bottom)
+		)
+	)
+	(gr_text "BOOT"
+		(at 117.7 73.7 0)
+		(layer "F.SilkS")
+		(effects
+			(font
+				(size 1 1)
+				(thickness 0.1)
+			)
+			(justify left bottom)
+		)
+	)
+	(gr_text "EN"
+		(at 150 55.5 0)
+		(layer "F.SilkS")
+		(effects
+			(font
+				(size 1 1)
+				(thickness 0.1)
+			)
+			(justify left bottom)
+		)
 	)
 	(gr_text "Ethernet Dev Board - Vine Internal rev 1.1\nCharm Lab, Stanford\nOctober 19 2025"

Commit message: stuff
Parts:
- added J7: Conn_01x02_Pin, Connector_PinHeader_2.54mm:PinHeader_1x02_P2.54mm_Vertical, F.Cu at (87.6, 84.8)
- added J9: Conn_01x02_Pin, Connector_PinHeader_2.54mm:PinHeader_1x02_P2.54mm_Vertical, F.Cu at (64.4, 107.6)
- added L1: L, Inductor_SMD:L_0603_1608Metric, F.Cu at (29.0, 137.5)
- moved C2 81.4 mm to (119.5, 127.5)
- moved SW2 81.4 mm to (123.5, 127.6)
- moved J1 5.65 mm to (75.8, 89.0)
- moved D3 3.58 mm to (147.2, 130.1)
- moved R2 3.28 mm to (92.8, 77.0)
- moved R13 2.83 mm to (129.6, 107.9)
- moved R19 2.52 mm to (91.0, 66.2)
- moved Q1 2.50 mm to (129.5, 126.2)
- moved R15 2.28 mm to (136.0, 126.4)
- moved J2 2.22 mm to (149.7, 47.3)
- moved D1 2.22 mm to (147.2, 125.5)
- moved R35 2.20 mm to (132.2, 108.0)
- moved R14 1.97 mm to (134.6, 129.6)
- moved R4 1.66 mm to (91.0, 68.4)
- moved R11 1.50 mm to (79.2, 76.7)
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Connections:
- J5 pad S1: GND -> Earth
- U5 pad 1: Net-(U5-GND-Pad1) -> GND
- U5 pad 15: Net-(U5-GND-Pad1) -> GND
- U5 pad 38: Net-(U5-GND-Pad1) -> GND
Routing:
- net Net-(U5-GND-Pad1): track 37.0 -> 0.00 mm
- net VDDA: track 43.4 -> 20.3 mm
- net GND: track 42.2 -> 51.7 mm, vias 25 -> 27
- net Net-(J1-Pad8): track 26.3 -> 32.5 mm
- net VDDCR: track 6.85 -> 12.3 mm
- net /DTR: track 11.5 -> 16.5 mm
- net /EN: track 115.0 -> 110.6 mm
- net /TXD: track 15.1 -> 19.3 mm
- net /TXD0: track 121.2 -> 117.0 mm
- net Net-(U1-RXD1/MODE1): track 4.39 -> 8.27 mm
- net /RTS: track 10.1 -> 13.8 mm
- net Net-(U4-~{SUSPEND}): track 2.66 -> 5.91 mm
- net Net-(Q1-B): track 2.12 -> 5.31 mm
- net VBUS: track 48.0 -> 44.9 mm
- net Net-(U1-MDIO): track 4.03 -> 6.88 mm
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- added copper zone on B.Cu, net Earth
- added copper zone on F.Cu, net Earth
- added copper zone on B.Cu, net GND
- added copper zone on F.Cu, net GND

Commit message: final
Parts:
- moved L1 83.7 mm to (75.0, 67.5), turned to 90 degrees
- moved R10 6.23 mm to (75.2, 76.8)
- moved R8 0.67 mm to (77.5, 68.0), turned to 0 degrees
- moved R21 0.15 mm to (84.0, 76.2)
- moved R9 0.10 mm to (77.5, 69.2)
Connections:
- U5 pad 3: unconnected-(U5-EN-Pad3) -> /EN
- U5 pad 39_1: Net-(U5-EXP-Pad39_1) -> GND
- U5 pad 39_2: Net-(U5-EXP-Pad39_1) -> GND
- U5 pad 39_3: Net-(U5-EXP-Pad39_1) -> GND
- U5 pad 39_4: Net-(U5-EXP-Pad39_1) -> GND
- U5 pad 39_5: Net-(U5-EXP-Pad39_1) -> GND
- U5 pad 39_6: Net-(U5-EXP-Pad39_1) -> GND
- U5 pad 39_7: Net-(U5-EXP-Pad39_1) -> GND
- U5 pad 39_8: Net-(U5-EXP-Pad39_1) -> GND
- U5 pad 39_9: Net-(U5-EXP-Pad39_1) -> GND
Routing:
- net VDDA: track 20.3 -> 70.0 mm, vias 0 -> 1
- net /RD_P: track 0.00 -> 32.0 mm, vias 0 -> 1
- net /RD_N: track 0.00 -> 30.1 mm, vias 0 -> 1
- net /TD_P: track 0.00 -> 28.6 mm, vias 0 -> 1
- net /TD_N: track 0.00 -> 27.9 mm, vias 0 -> 1
- net /EN: track 110.6 -> 131.3 mm
- net /TXD0: track 117.0 -> 136.6 mm
- net /USB_DN: track 0.00 -> 17.5 mm
- net /USB_DP: track 0.00 -> 17.5 mm
- net Earth: track 0.00 -> 13.5 mm
- net GND: track 51.7 -> 64.2 mm, vias 27 -> 31
- net Net-(U1-VDD1A): track 6.85 -> 15.8 mm, vias 2 -> 3
- net VCC: track 109.0 -> 116.9 mm, vias 4 -> 5
- net Net-(U1-RBIAS): track 1.53 -> 8.17 mm
- net /TXD1: track 19.8 -> 14.6 mm, vias 0 -> 1
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
Commit message: stuff
Routing:
- net /TD_P: track 28.6 -> 26.7 mm
- net Earth: track 13.5 -> 15.0 mm
- net /RD_P: track 32.0 -> 32.6 mm
- net /RD_N: track 30.1 -> 29.5 mm
