File: Hardware/Gen5/EthernetBoard/EthernetBoardv2.1_formfactor/EthernetBoardv1.2_formfactor/EthernetBoardv1.2_formfactor.kicad_sch (KiCad schematic)
At the start: 79 parts, among them J1 RJ45_Wuerth_7499010211A, J2 Conn_01x19_Pin, J3 Conn_01x19_Pin, J4 Conn_02x07_Odd_Even, J5 USB_C_Receptacle_USB2.0_16P, J6 Conn_01x02_Pin, J7 Conn_01x02_Pin, J9 Conn_01x02_Pin, Q1 SS8050, Q2 SS8050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

Commit message: update
Parts:
- removed J2, J3: Conn_01x19_Pin, Connector_PinHeader_2.54mm:PinHeader_1x19_P2.54mm_Vertical, symbol Connector:Conn_01x19_Pin
- removed J4: Conn_02x07_Odd_Even, Connector_PinHeader_2.54mm:PinHeader_2x07_P2.54mm_Vertical, symbol Connector_Generic:Conn_02x07_Odd_Even
- removed J6, J7, J9: Conn_01x02_Pin, Connector_PinHeader_2.54mm:PinHeader_1x02_P2.54mm_Vertical, symbol Connector:Conn_01x02_Pin
- removed TP1, TP2: TestPoint, TestPoint:TestPoint_Pad_2.0x2.0mm, symbol Connector:TestPoint
- added R37, R38, R39: 0R, Resistor_SMD:R_0201_0603Metric, symbol Device:R_US
- R12, R16, R17, R24, R25, R26, R27, R28, R29, R30, R31, R32: footprint Jumper:SolderJumper-2_P1.3mm_Bridged2Bar_RoundedPad1.0x1.5mm -> Resistor_SMD:R_0201_0603Metric
Connections:
- net +3.3V: now also R37.2, R38.2, R39.2
- net VCC: now also R37.1
- net VDDA: now also R39.1
- net VDDCR: now also R38.1
- no-connect marks 18 -> 17
Other:
- note removed: "Headers"

Commit message: done
Parts:
- C7: footprint Capacitor_SMD:C_0603_1608Metric -> Capacitor_SMD:C_0402_1005Metric
Changed lines of the file:
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@@
 			)
 		)
-		(property "Footprint" "Capacitor_SMD:C_0603_1608Metric"
+		(property "Footprint" "Capacitor_SMD:C_0402_1005Metric"
 			(at 111.4552 45.72 0)
 			(effects

Commit message: stuff
Parts:
- added R40, R41: 5.1k, Resistor_SMD:R_0603_1608Metric, symbol Device:R_US
- added R42: 10K, Resistor_SMD:R_0402_1005Metric, symbol Device:R_US
Connections:
- net +3.3V: now also R42.2
- net GND: now also R40.1, R41.1
- net IO0: now also R42.1
- net MDIO: now also R19.1, U1.12 (MDIO)
- net at J5.A5 (CC1): now also R40.2
- net at J5.B5 (CC2): now also R41.2
- no-connect marks 17 -> 15
Other:
- note added: "Notes: Added Enable Pullup (10K) for ESP Added BOOT Pullup (10K) Connected MDIO on PHY so ESP Routed out MDC Added 5.1K CC resistors to USB"
- note removed: "Notes: Added Enable Pullup (10K) for ESP"
- moved on the sheet: C1, C2, R36, SW1, SW2

Commit message: stuff
Changed lines of the file:
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@@
 		(dnp no)
 		(property "Reference" "R42"
-			(at 291.084 162.814 90)
+			(at 286.258 163.068 90)
 			(effects
 				(font
@@
 		)
 		(property "Value" "10K"
-			(at 291.338 171.704 90)
+			(at 286.258 171.704 90)
 			(effects
 				(font
@@
 		(dnp no)
 		(property "Reference" "R36"
-			(at 291.084 193.294 90)
+			(at 286.258 193.548 90)
 			(effects
 				(font
@@
 		)
 		(property "Value" "10K"
-			(at 291.338 202.184 90)
+			(at 286.258 202.184 90)
 			(effects
 				(font
